File: hardware/printer-board/FAN.sch (KiCad schematic (older format))
At the start: 7 parts

Commit message: update,
Parts:
- removed J?: FAN_OUTPUT, symbol Connector:Screw_Terminal_01x02
- removed Q?: STP55NF06, symbol Device:Q_NMOS_GDS
- removed R?: R100,0805, Resistor_SMD:R_0805_2012Metric_Pad1.15x1.40mm_HandSolder, symbol taobao-r:R100,0805
- removed R?: R104,0805, Resistor_SMD:R_0805_2012Metric_Pad1.15x1.40mm_HandSolder, symbol taobao-r:R104,0805
- removed R?: R182,0603, Resistor_SMD:R_0603_1608Metric_Pad1.05x0.95mm_HandSolder, symbol taobao-r:R182,0603
- added J24: FAN_OUTPUT, symbol Connector:Screw_Terminal_01x02
- added Q2: STP55NF06, symbol Device:Q_NMOS_GDS
- added R27: R100,0805, Resistor_SMD:R_0805_2012Metric_Pad1.15x1.40mm_HandSolder, symbol taobao-r:R100,0805
- added R28: R104,0805, Resistor_SMD:R_0805_2012Metric_Pad1.15x1.40mm_HandSolder, symbol taobao-r:R104,0805
- added R29: R182,0603, Resistor_SMD:R_0603_1608Metric_Pad1.05x0.95mm_HandSolder, symbol taobao-r:R182,0603
- gave numbers to parts that had none: 2
Connections:
- net +12V: now also J24.1 (Pin_1), R29.2
- net FAN_EN: now also R27.2, R28.2
- net GND: now also Q2.3 (S), R28.1
- net at D4.1 (K): now also J24.2 (Pin_2), Q2.2 (D)
- net at D4.2 (A): now also R29.1
- new net: Q2.1 (G), R27.1
Changed lines of the file:
@@
 EESchema Schematic File Version 4
+LIBS:printer-board-cache
 EELAYER 26 0
 EELAYER END
@@
 $Comp
 L Connector:Screw_Terminal_01x02 J?
-U 1 1 5CC0B91A
+U 1 1 5CC04D5E
 P 7600 3050
-AR Path="/5CC0B758/5CC0B91A" Ref="J?"  Part="1"
-AR Path="/5CC12903/5CC0B91A" Ref="J?"  Part="1"
-AR Path="/5CC130A8/5CC0B91A" Ref="J?"  Part="1"
-F 0 "J?" H 7519 2725 50  0000 C CNN
+AR Path="/5CC0B758/5CC04D5E" Ref="J?"  Part="1"
+AR Path="/5CC12903/5CC04D5E" Ref="J24"  Part="1"
+AR Path="/5CC130A8/5CC04D5E" Ref="J?"  Part="1"
+F 0 "J24" H 7519 2725 50  0000 C CNN
 F 1 "FAN_OUTPUT" H 7519 2816 50  0000 C CNN
 F 2 "" H 7600 3050 50  0001 C CNN
@@
 $Comp
 L Device:Q_NMOS_GDS Q?
-U 1 1 5CC0BC7B
+U 1 1 5CC04D5F
 P 5450 3250
-AR Path="/5CC0B758/5CC0BC7B" Ref="Q?"  Part="1"
-AR Path="/5CC12903/5CC0BC7B" Ref="Q?"  Part="1"
-AR Path="/5CC130A8/5CC0BC7B" Ref="Q?"  Part="1"
-F 0 "Q?" H 5656 3296 50  0000 L CNN
+AR Path="/5CC0B758/5CC04D5F" Ref="Q?"  Part="1"
+AR Path="/5CC12903/5CC04D5F" Ref="Q2"  Part="1"
+AR Path="/5CC130A8/5CC04D5F" Ref="Q?"  Part="1"
+F 0 "Q2" H 5656 3296 50  0000 L CNN
 F 1 "STP55NF06" H 5656 3205 50  0000 L CNN
 F 2 "" H 5650 3350 50  0001 C CNN
@@
 $Comp
 L taobao-r:R100,0805 R?
-U 1 1 5CC0BDB8
+U 1 1 5CC04D60
 P 4800 3250
-AR Path="/5CC0B758/5CC0BDB8" Ref="R?"  Part="1"
-AR Path="/5CC12903/5CC0BDB8" Ref="R?"  Part="1"
-AR Path="/5CC130A8/5CC0BDB8" Ref="R?"  Part="1"
-F 0 "R?" V 4604 3250 50  0000 C CNN
+AR Path="/5CC0B758/5CC04D60" Ref="R?"  Part="1"
+AR Path="/5CC12903/5CC04D60" Ref="R27"  Part="1"
+AR Path="/5CC130A8/5CC04D60" Ref="R?"  Part="1"
+F 0 "R27" V 4604 3250 50  0000 C CNN
 F 1 "R100,0805" V 4695 3250 50  0000 C CNN
 F 2 "Resistor_SMD:R_0805_2012Metric_Pad1.15x1.40mm_HandSolder" H 4800 3250 50  0001 C CNN
@@
 $Comp
 L taobao-r:R104,0805 R?
-U 1 1 5CC0BF5E
+U 1 1 5CC04D61
 P 4800 3650
-AR Path="/5CC0B758/5CC0BF5E" Ref="R?"  Part="1"
-AR Path="/5CC12903/5CC0BF5E" Ref="R?"  Part="1"
-AR Path="/5CC130A8/5CC0BF5E" Ref="R?"  Part="1"
-F 0 "R?" V 4604 3650 50  0000 C CNN
+AR Path="/5CC0B758/5CC04D61" Ref="R?"  Part="1"
+AR Path="/5CC12903/5CC04D61" Ref="R28"  Part="1"
+AR Path="/5CC130A8/5CC04D61" Ref="R?"  Part="1"
+F 0 "R28" V 4604 3650 50  0000 C CNN
 F 1 "R104,0805" V 4695 3650 50  0000 C CNN
 F 2 "Resistor_SMD:R_0805_2012Metric_Pad1.15x1.40mm_HandSolder" H 4800 3650 50  0001 C CNN
@@
 P 5550 3850
 AR Path="/5CC0B758/5CC0C00C" Ref="#PWR?"  Part="1"
-AR Path="/5CC12903/5CC0C00C" Ref="#PWR?"  Part="1"
+AR Path="/5CC12903/5CC0C00C" Ref="#PWR0229"  Part="1"
 AR Path="/5CC130A8/5CC0C00C" Ref="#PWR?"  Part="1"
-F 0 "#PWR?" H 5550 3600 50  0001 C CNN
+F 0 "#PWR0229" H 5550 3600 50  0001 C CNN
 F 1 "GND" H 5555 3677 50  0000 C CNN
 F 2 "" H 5550 3850 50  0001 C CNN
@@
 $Comp
 L taobao-r:R182,0603 R?
-U 1 1 5CC0C120
+U 1 1 5CC04D63
 P 6400 3500
-AR Path="/5CC0B758/5CC0C120" Ref="R?"  Part="1"
-AR Path="/5CC12903/5CC0C120" Ref="R?"  Part="1"
-AR Path="/5CC130A8/5CC0C120" Ref="R?"  Part="1"
-F 0 "R?" H 6459 3546 50  0000 L CNN
+AR Path="/5CC0B758/5CC04D63" Ref="R?"  Part="1"
+AR Path="/5CC12903/5CC04D63" Ref="R29"  Part="1"
+AR Path="/5CC130A8/5CC04D63" Ref="R?"  Part="1"
+F 0 "R29" H 6459 3546 50  0000 L CNN
 F 1 "R182,0603" H 6459 3455 50  0000 L CNN
 F 2 "Resistor_SMD:R_0603_1608Metric_Pad1.05x0.95mm_HandSolder" H 6400 3500 50  0001 C CNN
@@
 	4300 3250 4700 3250
 $Comp
-L power:+12V #PWR?
+L power:+12V #PWR0230
 U 1 1 5CC12C79
 P 7000 2750
-AR Path="/5CC12903/5CC12C79" Ref="#PWR?"  Part="1"
+AR Path="/5CC12903/5CC12C79" Ref="#PWR0230"  Part="1"
 AR Path="/5CC130A8/5CC12C79" Ref="#PWR?"  Part="1"
-F 0 "#PWR?" H 7000 2600 50  0001 C CNN
+F 0 "#PWR0230" H 7000 2600 50  0001 C CNN
 F 1 "+12V" H 7015 2923 50  0000 C CNN
 F 2 "" H 7000 2750 50  0001 C CNN
@@
 	7000 3050 7250 3050
 $Comp
-L taobao-led:LED_BLUE,0603 D?
+L taobao-led:LED_BLUE,0603 D4
 U 1 1 5CC12FAA
 P 6400 3200
-AR Path="/5CC12903/5CC12FAA" Ref="D?"  Part="1"
+AR Path="/5CC12903/5CC12FAA" Ref="D4"  Part="1"
 AR Path="/5CC130A8/5CC12FAA" Ref="D?"  Part="1"
-F 0 "D?" V 6354 3298 50  0000 L CNN
+F 0 "D4" V 6354 3298 50  0000 L CNN
 F 1 "LED_BLUE,0603" V 6445 3298 50  0000 L CNN
 F 2 "LED_SMD:LED_0603_1608Metric_Pad1.05x0.95mm_HandSolder" V 6400 3200 50  0001 C CNN
@@
 $EndComp
 $Comp
-L power:+12V #PWR?
+L power:+12V #PWR0231
 U 1 1 5CC14EFC
 P 4900 4350
-AR Path="/5CC12903/5CC14EFC" Ref="#PWR?"  Part="1"
+AR Path="/5CC12903/5CC14EFC" Ref="#PWR0231"  Part="1"
 AR Path="/5CC130A8/5CC14EFC" Ref="#PWR?"  Part="1"
-F 0 "#PWR?" H 4900 4200 50  0001 C CNN
+F 0 "#PWR0231" H 4900 4200 50  0001 C CNN
 F 1 "+12V" V 4915 4478 50  0000 L CNN
 F 2 "" H 4900 4350 50  0001 C CNN
@@
 P 5400 4350
 AR Path="/5CC0B758/5CC14F25" Ref="#PWR?"  Part="1"
-AR Path="/5CC12903/5CC14F25" Ref="#PWR?"  Part="1"
+AR Path="/5CC12903/5CC14F25" Ref="#PWR0232"  Part="1"
 AR Path="/5CC130A8/5CC14F25" Ref="#PWR?"  Part="1"
-F 0 "#PWR?" H 5400 4100 50  0001 C CNN
+F 0 "#PWR0232" H 5400 4100 50  0001 C CNN
 F 1 "GND" H 5405 4177 50  0000 C CNN
 F 2 "" H 5400 4350 50  0001 C CNN
@@
 $EndComp
 $Comp
-L taobao-cp:CP100uf,16V C?
+L taobao-cp:CP100uf,16V C27
 U 1 1 5CC14FB8
 P 5150 4350
-F 0 "C?" V 5375 4350 50  0000 C CNN
+F 0 "C27" V 5375 4350 50  0000 C CNN
 F 1 "CP100uf,16V" V 5284 4350 50  0000 C CNN
 F 2 "Capacitor_SMD:CP_Elec_6.3x5.3" H 5150 4350 50  0001 C CNN

Commit message: update,
Changed lines of the file:
@@
 $Descr A4 11693 8268
 encoding utf-8
-Sheet 15 20
+Sheet 15 21
 Title ""
 Date ""
@@
 AR Path="/5CC12903/5CC04D5E" Ref="J24"  Part="1"
 AR Path="/5CC130A8/5CC04D5E" Ref="J?"  Part="1"
-F 0 "J24" H 7519 2725 50  0000 C CNN
+AR Path="/5CC19D48/5CC04D5E" Ref="J?"  Part="1"
+F 0 "J?" H 7519 2725 50  0000 C CNN
 F 1 "FAN_OUTPUT" H 7519 2816 50  0000 C CNN
 F 2 "" H 7600 3050 50  0001 C CNN
@@
 AR Path="/5CC12903/5CC04D5F" Ref="Q2"  Part="1"
 AR Path="/5CC130A8/5CC04D5F" Ref="Q?"  Part="1"
-F 0 "Q2" H 5656 3296 50  0000 L CNN
+AR Path="/5CC19D48/5CC04D5F" Ref="Q?"  Part="1"
+F 0 "Q?" H 5656 3296 50  0000 L CNN
 F 1 "STP55NF06" H 5656 3205 50  0000 L CNN
 F 2 "" H 5650 3350 50  0001 C CNN
@@
 AR Path="/5CC12903/5CC04D60" Ref="R27"  Part="1"
 AR Path="/5CC130A8/5CC04D60" Ref="R?"  Part="1"
-F 0 "R27" V 4604 3250 50  0000 C CNN
+AR Path="/5CC19D48/5CC04D60" Ref="R?"  Part="1"
+F 0 "R?" V 4604 3250 50  0000 C CNN
 F 1 "R100,0805" V 4695 3250 50  0000 C CNN
 F 2 "Resistor_SMD:R_0805_2012Metric_Pad1.15x1.40mm_HandSolder" H 4800 3250 50  0001 C CNN
@@
 AR Path="/5CC12903/5CC04D61" Ref="R28"  Part="1"
 AR Path="/5CC130A8/5CC04D61" Ref="R?"  Part="1"
-F 0 "R28" V 4604 3650 50  0000 C CNN
+AR Path="/5CC19D48/5CC04D61" Ref="R?"  Part="1"
+F 0 "R?" V 4604 3650 50  0000 C CNN
 F 1 "R104,0805" V 4695 3650 50  0000 C CNN
 F 2 "Resistor_SMD:R_0805_2012Metric_Pad1.15x1.40mm_HandSolder" H 4800 3650 50  0001 C CNN
@@
 AR Path="/5CC12903/5CC0C00C" Ref="#PWR0229"  Part="1"
 AR Path="/5CC130A8/5CC0C00C" Ref="#PWR?"  Part="1"
-F 0 "#PWR0229" H 5550 3600 50  0001 C CNN
+AR Path="/5CC19D48/5CC0C00C" Ref="#PWR?"  Part="1"
+F 0 "#PWR?" H 5550 3600 50  0001 C CNN
 F 1 "GND" H 5555 3677 50  0000 C CNN
 F 2 "" H 5550 3850 50  0001 C CNN
@@
 AR Path="/5CC12903/5CC04D63" Ref="R29"  Part="1"
 AR Path="/5CC130A8/5CC04D63" Ref="R?"  Part="1"
-F 0 "R29" H 6459 3546 50  0000 L CNN
+AR Path="/5CC19D48/5CC04D63" Ref="R?"  Part="1"
+F 0 "R?" H 6459 3546 50  0000 L CNN
 F 1 "R182,0603" H 6459 3455 50  0000 L CNN
 F 2 "Resistor_SMD:R_0603_1608Metric_Pad1.05x0.95mm_HandSolder" H 6400 3500 50  0001 C CNN
@@
 AR Path="/5CC12903/5CC12C79" Ref="#PWR0230"  Part="1"
 AR Path="/5CC130A8/5CC12C79" Ref="#PWR?"  Part="1"
-F 0 "#PWR0230" H 7000 2600 50  0001 C CNN
+AR Path="/5CC19D48/5CC12C79" Ref="#PWR?"  Part="1"
+F 0 "#PWR?" H 7000 2600 50  0001 C CNN
 F 1 "+12V" H 7015 2923 50  0000 C CNN
 F 2 "" H 7000 2750 50  0001 C CNN
@@
 AR Path="/5CC12903/5CC12FAA" Ref="D4"  Part="1"
 AR Path="/5CC130A8/5CC12FAA" Ref="D?"  Part="1"
-F 0 "D4" V 6354 3298 50  0000 L CNN
+AR Path="/5CC19D48/5CC12FAA" Ref="D?"  Part="1"
+F 0 "D?" V 6354 3298 50  0000 L CNN
 F 1 "LED_BLUE,0603" V 6445 3298 50  0000 L CNN
 F 2 "LED_SMD:LED_0603_1608Metric_Pad1.05x0.95mm_HandSolder" V 6400 3200 50  0001 C CNN
@@
 AR Path="/5CC12903/5CC14EFC" Ref="#PWR0231"  Part="1"
 AR Path="/5CC130A8/5CC14EFC" Ref="#PWR?"  Part="1"
-F 0 "#PWR0231" H 4900 4200 50  0001 C CNN
+AR Path="/5CC19D48/5CC14EFC" Ref="#PWR?"  Part="1"
+F 0 "#PWR?" H 4900 4200 50  0001 C CNN
 F 1 "+12V" V 4915 4478 50  0000 L CNN
 F 2 "" H 4900 4350 50  0001 C CNN
@@
 AR Path="/5CC12903/5CC14F25" Ref="#PWR0232"  Part="1"
 AR Path="/5CC130A8/5CC14F25" Ref="#PWR?"  Part="1"
-F 0 "#PWR0232" H 5400 4100 50  0001 C CNN
+AR Path="/5CC19D48/5CC14F25" Ref="#PWR?"  Part="1"
+F 0 "#PWR?" H 5400 4100 50  0001 C CNN
 F 1 "GND" H 5405 4177 50  0000 C CNN
 F 2 "" H 5400 4350 50  0001 C CNN
@@
 U 1 1 5CC14FB8
 P 5150 4350
-F 0 "C27" V 5375 4350 50  0000 C CNN
+AR Path="/5CC12903/5CC14FB8" Ref="C27"  Part="1"
+AR Path="/5CC19D48/5CC14FB8" Ref="C?"  Part="1"
+F 0 "C?" V 5375 4350 50  0000 C CNN
 F 1 "CP100uf,16V" V 5284 4350 50  0000 C CNN
 F 2 "Capacitor_SMD:CP_Elec_6.3x5.3" H 5150 4350 50  0001 C CNN
