File: hardware/printer-board/HOT-END.sch (KiCad schematic (older format))
At the start: 7 parts

Commit message: update,
Parts:
- Q3: renamed from Q?; footprint (none) -> Package_TO_SOT_SMD:TO-263-2
- gave numbers to parts that had none: 6
Changed lines of the file:
@@
 EESchema Schematic File Version 4
+LIBS:printer-board-cache
 EELAYER 26 0
 EELAYER END
@@
 AR Path="/5CC0B758/5CC19EB5" Ref="J?"  Part="1"
 AR Path="/5CC12903/5CC19EB5" Ref="J?"  Part="1"
-AR Path="/5CC130A8/5CC19EB5" Ref="J?"  Part="1"
-F 0 "J?" H 7769 2725 50  0000 C CNN
+AR Path="/5CC130A8/5CC19EB5" Ref="J25"  Part="1"
+F 0 "J25" H 7769 2725 50  0000 C CNN
 F 1 "HOT_END" H 7769 2816 50  0000 C CNN
 F 2 "" H 7850 3050 50  0001 C CNN
@@
 AR Path="/5CC0B758/5CC19EBC" Ref="Q?"  Part="1"
 AR Path="/5CC12903/5CC19EBC" Ref="Q?"  Part="1"
-F 0 "Q?" H 5906 3296 50  0000 L CNN
+AR Path="/5CC130A8/5CC19EBC" Ref="Q3"  Part="1"
+F 0 "Q3" H 5906 3296 50  0000 L CNN
 F 1 "WSK220N04" H 5906 3205 50  0000 L CNN
-F 2 "" H 5900 3350 50  0001 C CNN
+F 2 "Package_TO_SOT_SMD:TO-263-2" H 5900 3350 50  0001 C CNN
 F 3 "~" H 5700 3250 50  0001 C CNN
 	1    5700 3250
@@
 AR Path="/5CC0B758/5CC19EC3" Ref="R?"  Part="1"
 AR Path="/5CC12903/5CC19EC3" Ref="R?"  Part="1"
-F 0 "R?" V 4854 3250 50  0000 C CNN
+AR Path="/5CC130A8/5CC19EC3" Ref="R30"  Part="1"
+F 0 "R30" V 4854 3250 50  0000 C CNN
 F 1 "R100,0805" V 4945 3250 50  0000 C CNN
 F 2 "Resistor_SMD:R_0805_2012Metric_Pad1.15x1.40mm_HandSolder" H 5050 3250 50  0001 C CNN
@@
 AR Path="/5CC0B758/5CC19ECA" Ref="R?"  Part="1"
 AR Path="/5CC12903/5CC19ECA" Ref="R?"  Part="1"
-F 0 "R?" V 4854 3650 50  0000 C CNN
+AR Path="/5CC130A8/5CC19ECA" Ref="R31"  Part="1"
+F 0 "R31" V 4854 3650 50  0000 C CNN
 F 1 "R104,0805" V 4945 3650 50  0000 C CNN
 F 2 "Resistor_SMD:R_0805_2012Metric_Pad1.15x1.40mm_HandSolder" H 5050 3650 50  0001 C CNN
@@
 AR Path="/5CC0B758/5CC19ED1" Ref="#PWR?"  Part="1"
 AR Path="/5CC12903/5CC19ED1" Ref="#PWR?"  Part="1"
-F 0 "#PWR?" H 5800 3600 50  0001 C CNN
+AR Path="/5CC130A8/5CC19ED1" Ref="#PWR0233"  Part="1"
+F 0 "#PWR0233" H 5800 3600 50  0001 C CNN
 F 1 "GND" H 5805 3677 50  0000 C CNN
 F 2 "" H 5800 3850 50  0001 C CNN
@@
 AR Path="/5CC0B758/5CC19EDC" Ref="R?"  Part="1"
 AR Path="/5CC12903/5CC19EDC" Ref="R?"  Part="1"
-F 0 "R?" H 6709 3546 50  0000 L CNN
+AR Path="/5CC130A8/5CC19EDC" Ref="R32"  Part="1"
+F 0 "R32" H 6709 3546 50  0000 L CNN
 F 1 "R182,0603" H 6709 3455 50  0000 L CNN
 F 2 "Resistor_SMD:R_0603_1608Metric_Pad1.05x0.95mm_HandSolder" H 6650 3500 50  0001 C CNN
@@
 AR Path="/5CC0B758/5CC19EE3" Ref="D?"  Part="1"
 AR Path="/5CC12903/5CC19EE3" Ref="D?"  Part="1"
-F 0 "D?" V 6604 3298 50  0000 L CNN
+AR Path="/5CC130A8/5CC19EE3" Ref="D5"  Part="1"
+F 0 "D5" V 6604 3298 50  0000 L CNN
 F 1 "LED_RED,0603" V 6695 3298 50  0000 L CNN
 F 2 "LED_SMD:LED_0603_1608Metric_Pad1.05x0.95mm_HandSolder" V 6650 3200 50  0001 C CNN
@@
 AR Path="/5CC0B758/5CC19EF0" Ref="#PWR?"  Part="1"
 AR Path="/5CC12903/5CC19EF0" Ref="#PWR?"  Part="1"
-F 0 "#PWR?" H 7350 2900 50  0001 C CNN
+AR Path="/5CC130A8/5CC19EF0" Ref="#PWR0234"  Part="1"
+F 0 "#PWR0234" H 7350 2900 50  0001 C CNN
 F 1 "+12V2" V 7365 3178 50  0000 L CNN
 F 2 "" H 7350 3050 50  0001 C CNN
@@
 AR Path="/5CC0B758/5CC19F05" Ref="#PWR?"  Part="1"
 AR Path="/5CC12903/5CC19F05" Ref="#PWR?"  Part="1"
-F 0 "#PWR?" H 5150 4200 50  0001 C CNN
+AR Path="/5CC130A8/5CC19F05" Ref="#PWR0235"  Part="1"
+F 0 "#PWR0235" H 5150 4200 50  0001 C CNN
 F 1 "+12V2" V 5165 4478 50  0000 L CNN
 F 2 "" H 5150 4350 50  0001 C CNN
@@
 AR Path="/5CC0B758/5CC19F0B" Ref="#PWR?"  Part="1"
 AR Path="/5CC12903/5CC19F0B" Ref="#PWR?"  Part="1"
-F 0 "#PWR?" H 5800 4100 50  0001 C CNN
+AR Path="/5CC130A8/5CC19F0B" Ref="#PWR0236"  Part="1"
+F 0 "#PWR0236" H 5800 4100 50  0001 C CNN
 F 1 "GND" V 5805 4222 50  0000 R CNN
 F 2 "" H 5800 4350 50  0001 C CNN
@@
 $EndComp
 $Comp
-L taobao-cp:CP100uf,16V C?
+L taobao-cp:CP100uf,16V C28
 U 1 1 5CC19F11
 P 5450 4350
-F 0 "C?" V 5675 4350 50  0000 C CNN
+F 0 "C28" V 5675 4350 50  0000 C CNN
 F 1 "CP100uf,16V" V 5584 4350 50  0000 C CNN
 F 2 "Capacitor_SMD:CP_Elec_6.3x5.3" H 5450 4350 50  0001 C CNN
