File: hardware/printer-board/HOTEND_2.sch (KiCad schematic (older format))
At the start: 7 parts, among them J25 HOT_END, Q4 WSK220N04

Commit message: update,
Parts:
- J25: footprint footprint-lib:s2b-ph-kl,hotend_output -> footprint-lib:mpt_0,5%2f2-2,54,heatbed
Changed lines of the file:
@@
 $Descr A4 11693 8268
 encoding utf-8
-Sheet 29 34
+Sheet 29 33
 Title ""
 Date ""
@@
 F 0 "J25" H 5219 2825 50  0000 C CNN
 F 1 "HOT_END" H 5219 2916 50  0000 C CNN
-F 2 "footprint-lib:s2b-ph-kl,hotend_output" H 5300 3150 50  0001 C CNN
+F 2 "footprint-lib:mpt_0,5%2f2-2,54,heatbed" H 5300 3150 50  0001 C CNN
 F 3 "~" H 5300 3150 50  0001 C CNN
 	1    5300 3150

Commit message: update hotend,
Parts:
- removed C32: CP100uf,16V, Capacitor_SMD:CP_Elec_6.3x5.3, symbol taobao-cp:CP100uf,16V
- Q4: footprint Package_TO_SOT_SMD:TO-263-2 -> footprint-lib:TO-263-2,drill_array
Connections:
- net -12V: now reaches D9.1 (K), J25.2 (Pin_2), Q4.2 (D)
Other:
- moved on the sheet: D9, J25, R40
Changed lines of the file:
@@
 EESchema Schematic File Version 4
-LIBS:printer-board-cache
 EELAYER 26 0
 EELAYER END
 $Descr A4 11693 8268
 encoding utf-8
-Sheet 29 33
+Sheet 1 1
 Title ""
 Date ""
@@
 L Connector:Screw_Terminal_01x02 J?
 U 1 1 5CC2240E
-P 5300 3150
+P 5300 2950
 AR Path="/5CC0B758/5CC2240E" Ref="J?"  Part="1"
 AR Path="/5CC12903/5CC2240E" Ref="J?"  Part="1"
 AR Path="/5CC130A8/5CC2240E" Ref="J?"  Part="1"
 AR Path="/5CC22025/5CC222D5/5CC2240E" Ref="J25"  Part="1"
-F 0 "J25" H 5219 2825 50  0000 C CNN
-F 1 "HOT_END" H 5219 2916 50  0000 C CNN
-F 2 "footprint-lib:mpt_0,5%2f2-2,54,heatbed" H 5300 3150 50  0001 C CNN
-F 3 "~" H 5300 3150 50  0001 C CNN
-	1    5300 3150
-	1    0    0    1
+AR Path="/5CC2240E" Ref="J25"  Part="1"
+F 0 "J25" H 5219 2625 50  0000 C CNN
+F 1 "HOT_END" H 5219 2716 50  0000 C CNN
+F 2 "footprint-lib:mpt_0,5%2f2-2,54,heatbed" H 5300 2950 50  0001 C CNN
+F 3 "~" H 5300 2950 50  0001 C CNN
+	1    5300 2950
+	1    0    0    -1
 $EndComp
 $Comp
@@
 AR Path="/5CC130A8/5CC19EBC" Ref="Q?"  Part="1"
 AR Path="/5CC22025/5CC222D5/5CC19EBC" Ref="Q4"  Part="1"
+AR Path="/5CC19EBC" Ref="Q4"  Part="1"
 F 0 "Q4" H 3356 3396 50  0000 L CNN
 F 1 "WSK220N04" H 3356 3305 50  0000 L CNN
-F 2 "Package_TO_SOT_SMD:TO-263-2" H 3350 3450 50  0001 C CNN
+F 2 "footprint-lib:TO-263-2,drill_array" H 3350 3450 50  0001 C CNN
 F 3 "~" H 3150 3350 50  0001 C CNN
 	1    3150 3350
@@
 AR Path="/5CC130A8/5CC22410" Ref="R?"  Part="1"
 AR Path="/5CC22025/5CC222D5/5CC22410" Ref="R39"  Part="1"
+AR Path="/5CC22410" Ref="R39"  Part="1"
 F 0 "R39" V 2304 3350 50  0000 C CNN
 F 1 "R100,0805" V 2395 3350 50  0000 C CNN
@@
 AR Path="/5CC130A8/5CC19ECA" Ref="R?"  Part="1"
 AR Path="/5CC22025/5CC222D5/5CC19ECA" Ref="R41"  Part="1"
+AR Path="/5CC19ECA" Ref="R41"  Part="1"
 F 0 "R41" V 2304 3750 50  0000 C CNN
 F 1 "R104,0805" V 2395 3750 50  0000 C CNN
@@
 AR Path="/5CC130A8/5CC19ED1" Ref="#PWR?"  Part="1"
 AR Path="/5CC22025/5CC222D5/5CC19ED1" Ref="#PWR0254"  Part="1"
+AR Path="/5CC19ED1" Ref="#PWR0254"  Part="1"
 F 0 "#PWR0254" H 3250 3700 50  0001 C CNN
 F 1 "GND" H 3255 3777 50  0000 C CNN
@@
 L taobao-r:R182,0603 R?
 U 1 1 5CC22413
-P 4100 3600
+P 4100 2500
 AR Path="/5CC0B758/5CC22413" Ref="R?"  Part="1"
 AR Path="/5CC12903/5CC22413" Ref="R?"  Part="1"
 AR Path="/5CC130A8/5CC22413" Ref="R?"  Part="1"
 AR Path="/5CC22025/5CC222D5/5CC22413" Ref="R40"  Part="1"
-F 0 "R40" H 4159 3646 50  0000 L CNN
-F 1 "R182,0603" H 4159 3555 50  0000 L CNN
-F 2 "Resistor_SMD:R_0603_1608Metric_Pad1.05x0.95mm_HandSolder" H 4100 3600 50  0001 C CNN
-F 3 "~" H 4100 3600 50  0001 C CNN
-	1    4100 3600
-	1    0    0    -1
+AR Path="/5CC22413" Ref="R40"  Part="1"
+F 0 "R40" H 4159 2546 50  0000 L CNN
+F 1 "R182,0603" H 4159 2455 50  0000 L CNN
+F 2 "Resistor_SMD:R_0603_1608Metric_Pad1.05x0.95mm_HandSolder" H 4100 2500 50  0001 C CNN
+F 3 "~" H 4100 2500 50  0001 C CNN
+	1    4100 2500
+	1    0    0    1
 $EndComp
 $Comp
 L taobao-led:LED_RED,0603 D?
 U 1 1 5CC19EE3
-P 4100 3300
+P 4100 2800
 AR Path="/5CC0B758/5CC19EE3" Ref="D?"  Part="1"
 AR Path="/5CC12903/5CC19EE3" Ref="D?"  Part="1"
 AR Path="/5CC130A8/5CC19EE3" Ref="D?"  Part="1"
 AR Path="/5CC22025/5CC222D5/5CC19EE3" Ref="D9"  Part="1"
-F 0 "D9" V 4054 3398 50  0000 L CNN
-F 1 "LED_RED,0603" V 4145 3398 50  0000 L CNN
-F 2 "LED_SMD:LED_0603_1608Metric_Pad1.05x0.95mm_HandSolder" V 4100 3300 50  0001 C CNN
-F 3 "" V 4100 3300 50  0001 C CNN
-	1    4100 3300
-	0    1    1    0
+AR Path="/5CC19EE3" Ref="D9"  Part="1"
+F 0 "D9" V 4054 2898 50  0000 L CNN
+F 1 "LED_RED,0603" V 4145 2898 50  0000 L CNN
+F 2 "LED_SMD:LED_0603_1608Metric_Pad1.05x0.95mm_HandSolder" V 4100 2800 50  0001 C CNN
+F 3 "" V 4100 2800 50  0001 C CNN
+	1    4100 2800
+	0    1    -1   0
 $EndComp
 Wire Wire Line
@@
 	3250 3050 3250 3150
 Wire Wire Line
-	4100 3200 4100 3050
+	4100 2900 4100 3050
 Connection ~ 4100 3050
 Wire Wire Line
 	4100 3050 3250 3050
 Wire Wire Line
-	4100 3400 4100 3500
+	4100 2700 4100 2600
 Wire Wire Line
-	5100 3150 4950 3150
+	5100 2950 4950 2950
 Wire Wire Line
-	4950 3150 4950 3800
+	4950 2950 4950 2300
 Wire Wire Line
-	4950 3800 4100 3800
+	4950 2300 4700 2300
 Wire Wire Line
-	4100 3800 4100 3700
-Connection ~ 4950 3150
+	4100 2300 4100 2400
 Text HLabel 1500 900  0    50   Input ~ 0
 HOTEND_EN
@@
 Wire Wire Line
 	2000 3350 2400 3350
-$Comp
-L taobao-components:+12V2 #PWR?
-U 1 1 5CC22415
-P 2600 4450
-AR Path="/5CC0B758/5CC22415" Ref="#PWR?"  Part="1"
-AR Path="/5CC12903/5CC22415" Ref="#PWR?"  Part="1"
-AR Path="/5CC130A8/5CC22415" Ref="#PWR?"  Part="1"
-AR Path="/5CC22025/5CC222D5/5CC22415" Ref="#PWR0255"  Part="1"
-F 0 "#PWR0255" H 2600 4300 50  0001 C CNN
-F 1 "+12V2" V 2615 4578 50  0000 L CNN
-F 2 "" H 2600 4450 50  0001 C CNN
-F 3 "" H 2600 4450 50  0001 C CNN
-	1    2600 4450
-	0    -1   -1   0
-$EndComp
-$Comp
-L power:GND #PWR?
-U 1 1 5CC22416
-P 3250 4450
-AR Path="/5CC0B758/5CC22416" Ref="#PWR?"  Part="1"
-AR Path="/5CC12903/5CC22416" Ref="#PWR?"  Part="1"
-AR Path="/5CC130A8/5CC22416" Ref="#PWR?"  Part="1"
-AR Path="/5CC22025/5CC222D5/5CC22416" Ref="#PWR0256"  Part="1"
-F 0 "#PWR0256" H 3250 4200 50  0001 C CNN
-F 1 "GND" V 3255 4322 50  0000 R CNN
-F 2 "" H 3250 4450 50  0001 C CNN
-F 3 "" H 3250 4450 50  0001 C CNN
-	1    3250 4450
-	0    -1   -1   0
-$EndComp
-$Comp
-L taobao-cp:CP100uf,16V C32
-U 1 1 5CC22417
-P 2900 4450
-F 0 "C32" V 3125 4450 50  0000 C CNN
-F 1 "CP100uf,16V" V 3034 4450 50  0000 C CNN
-F 2 "Capacitor_SMD:CP_Elec_6.3x5.3" H 2900 4450 50  0001 C CNN
-F 3 "~" H 2900 4450 50  0001 C CNN
-	1    2900 4450
-	0    -1   -1   0
-$EndComp
-Wire Wire Line
-	2600 4450 2800 4450
-Wire Wire Line
-	3000 4450 3250 4450
 $Bitmap
 Pos 9550 5000
@@
 L power:+12V #PWR0257
 U 1 1 5CC3323B
-P 4750 2850
-F 0 "#PWR0257" H 4750 2700 50  0001 C CNN
-F 1 "+12V" H 4765 3023 50  0000 C CNN
-F 2 "" H 4750 2850 50  0001 C CNN
-F 3 "" H 4750 2850 50  0001 C CNN
-	1    4750 2850
-	1    0    0    -1
+P 4700 2000
+F 0 "#PWR0257" H 4700 1850 50  0001 C CNN
+F 1 "+12V" H 4715 2173 50  0000 C CNN
+F 2 "" H 4700 2000 50  0001 C CNN
+F 3 "" H 4700 2000 50  0001 C CNN
+	1    4700 2000
+	-1   0    0    -1
 $EndComp
 Wire Wire Line
-	4750 2850 4750 3150
-Wire Wire Line
-	4750 3150 4950 3150
+	4700 2000 4700 2300
+Text Label 4600 3050 2    50   ~ 0
+-12V
+Connection ~ 4700 2300
+Wire Wire Line
+	4700 2300 4100 2300
+Text Label 4450 2300 2    50   ~ 0
+12V_led
 $EndSCHEMATC
