File: hardware/printer-board/SSD1306.sch (KiCad schematic (older format))
At the start: 1 part

Commit message: update,
Parts:
- added JP? (x2): Jumper_NO_Small, symbol Device:Jumper_NO_Small
Connections:
- net SCL: now also JP?.2
- net SDA: now also JP?.2
- new net SSD1309_SCL: JP?.1
- new net SSD1309_SDA: JP?.1
Other:
- moved on the sheet: J?
Changed lines of the file:
@@
 L Connector:Conn_01x08_Male J?
 U 1 1 5CC2EC35
-P 10150 1600
-F 0 "J?" H 10256 2078 50  0000 C CNN
-F 1 "Conn_01x08_Male" H 10256 1987 50  0000 C CNN
-F 2 "" H 10150 1600 50  0001 C CNN
-F 3 "~" H 10150 1600 50  0001 C CNN
-	1    10150 1600
+P 5900 4200
+F 0 "J?" H 6006 4678 50  0000 C CNN
+F 1 "Conn_01x08_Male" H 6006 4587 50  0000 C CNN
+F 2 "" H 5900 4200 50  0001 C CNN
+F 3 "~" H 5900 4200 50  0001 C CNN
+	1    5900 4200
 	1    0    0    -1
 $EndComp
@@
 L power:+5V #PWR?
 U 1 1 5CC2ED67
-P 10650 1250
-F 0 "#PWR?" H 10650 1100 50  0001 C CNN
-F 1 "+5V" H 10665 1423 50  0000 C CNN
-F 2 "" H 10650 1250 50  0001 C CNN
-F 3 "" H 10650 1250 50  0001 C CNN
-	1    10650 1250
+P 6400 3850
+F 0 "#PWR?" H 6400 3700 50  0001 C CNN
+F 1 "+5V" H 6415 4023 50  0000 C CNN
+F 2 "" H 6400 3850 50  0001 C CNN
+F 3 "" H 6400 3850 50  0001 C CNN
+	1    6400 3850
 	1    0    0    -1
 $EndComp
 Wire Wire Line
-	10350 1300 10650 1300
+	6100 3900 6400 3900
 Wire Wire Line
-	10650 1300 10650 1250
+	6400 3900 6400 3850
 $Comp
 L power:GND #PWR?
 U 1 1 5CC2EDEA
-P 10800 1450
-F 0 "#PWR?" H 10800 1200 50  0001 C CNN
-F 1 "GND" H 10805 1277 50  0000 C CNN
-F 2 "" H 10800 1450 50  0001 C CNN
-F 3 "" H 10800 1450 50  0001 C CNN
-	1    10800 1450
+P 6550 3850
+F 0 "#PWR?" H 6550 3600 50  0001 C CNN
+F 1 "GND" H 6555 3677 50  0000 C CNN
+F 2 "" H 6550 3850 50  0001 C CNN
+F 3 "" H 6550 3850 50  0001 C CNN
+	1    6550 3850
+	-1   0    0    1
+$EndComp
+Wire Wire Line
+	6100 4000 6550 4000
+Text Label 6400 4100 2    50   ~ 0
+SDA
+Wire Wire Line
+	6400 4100 6100 4100
+Wire Wire Line
+	6400 4200 6100 4200
+Wire Wire Line
+	6400 4300 6100 4300
+Wire Wire Line
+	6400 4400 6100 4400
+Wire Wire Line
+	6400 4500 6100 4500
+Wire Wire Line
+	6400 4600 6100 4600
+Text Label 6400 4200 2    50   ~ 0
+SCL
+Text Label 6400 4300 2    50   ~ 0
+D31
+Text Label 6400 4400 2    50   ~ 0
+D33
+Text Label 6400 4500 2    50   ~ 0
+D35
+Text Label 6400 4600 2    50   ~ 0
+D37
+Wire Wire Line
+	6550 3850 6550 4000
+Text HLabel 1300 700  0    50   Input ~ 0
+SSD1309_SDA
+Text HLabel 1300 800  0    50   Input ~ 0
+SSD1309_SCL
+Text Label 1800 700  2    50   ~ 0
+SDA
+Text Label 1800 800  2    50   ~ 0
+SCL
+$Comp
+L Device:Jumper_NO_Small JP?
+U 1 1 5CE587AA
+P 1550 700
+F 0 "JP?" H 1550 900 50  0000 C CNN
+F 1 "Jumper_NO_Small" H 1550 800 50  0000 C CNN
+F 2 "" H 1550 700 50  0001 C CNN
+F 3 "~" H 1550 700 50  0001 C CNN
+	1    1550 700
+	1    0    0    -1
+$EndComp
+$Comp
+L Device:Jumper_NO_Small JP?
+U 1 1 5CE587EA
+P 1550 800
+F 0 "JP?" H 1550 700 50  0000 C CNN
+F 1 "Jumper_NO_Small" H 1550 600 50  0000 C CNN
+F 2 "" H 1550 800 50  0001 C CNN
+F 3 "~" H 1550 800 50  0001 C CNN
+	1    1550 800
 	1    0    0    -1
 $EndComp
 Wire Wire Line
-	10350 1400 10800 1400
+	1300 700  1450 700
 Wire Wire Line
-	10800 1400 10800 1450
-Text Label 10650 1500 2    50   ~ 0
-SDA
+	1300 800  1450 800
 Wire Wire Line
-	10650 1500 10350 1500
+	1650 700  1800 700
 Wire Wire Line
-	10650 1600 10350 1600
-Wire Wire Line
-	10650 1700 10350 1700
-Wire Wire Line
-	10650 1800 10350 1800
-Wire Wire Line
-	10650 1900 10350 1900
-Wire Wire Line
-	10650 2000 10350 2000
-Text Label 10650 1600 2    50   ~ 0
-SCL
-Text Label 10650 1700 2    50   ~ 0
-D31
-Text Label 10650 1800 2    50   ~ 0
-D33
-Text Label 10650 1900 2    50   ~ 0
-D35
-Text Label 10650 2000 2    50   ~ 0
-D37
+	1650 800  1800 800
 $EndSCHEMATC

Commit message: update annotations,
Parts:
- gave numbers to parts that had none: 3
Changed lines of the file:
@@
 $EndBitmap
 $Comp
-L Connector:Conn_01x08_Male J?
+L Connector:Conn_01x08_Male J20
 U 1 1 5CC2EC35
 P 5900 4200
-F 0 "J?" H 6006 4678 50  0000 C CNN
+F 0 "J20" H 6006 4678 50  0000 C CNN
 F 1 "Conn_01x08_Male" H 6006 4587 50  0000 C CNN
 F 2 "" H 5900 4200 50  0001 C CNN
@@
 $EndComp
 $Comp
-L power:+5V #PWR?
+L power:+5V #PWR044
 U 1 1 5CC2ED67
 P 6400 3850
-F 0 "#PWR?" H 6400 3700 50  0001 C CNN
+F 0 "#PWR044" H 6400 3700 50  0001 C CNN
 F 1 "+5V" H 6415 4023 50  0000 C CNN
 F 2 "" H 6400 3850 50  0001 C CNN
@@
 	6400 3900 6400 3850
 $Comp
-L power:GND #PWR?
+L power:GND #PWR045
 U 1 1 5CC2EDEA
 P 6550 3850
-F 0 "#PWR?" H 6550 3600 50  0001 C CNN
+F 0 "#PWR045" H 6550 3600 50  0001 C CNN
 F 1 "GND" H 6555 3677 50  0000 C CNN
 F 2 "" H 6550 3850 50  0001 C CNN
@@
 SCL
 $Comp
-L Device:Jumper_NO_Small JP?
+L Device:Jumper_NO_Small JP7
 U 1 1 5CE587AA
 P 1550 700
-F 0 "JP?" H 1550 900 50  0000 C CNN
+F 0 "JP7" H 1550 900 50  0000 C CNN
 F 1 "Jumper_NO_Small" H 1550 800 50  0000 C CNN
 F 2 "" H 1550 700 50  0001 C CNN
@@
 $EndComp
 $Comp
-L Device:Jumper_NO_Small JP?
+L Device:Jumper_NO_Small JP8
 U 1 1 5CE587EA
 P 1550 800
-F 0 "JP?" H 1550 700 50  0000 C CNN
+F 0 "JP8" H 1550 700 50  0000 C CNN
 F 1 "Jumper_NO_Small" H 1550 600 50  0000 C CNN
 F 2 "" H 1550 800 50  0001 C CNN
