File: hardware/printer-board/MP1584EN_power.sch (KiCad schematic (older format))
At the start: 8 parts, among them U14 AMS1117-3.3

Commit message: update,
Parts:
- removed C37, C38: C104,0603, Capacitor_SMD:C_0603_1608Metric_Pad1.05x0.95mm_HandSolder, symbol taobao-c:C104,0603
- removed C39: CP47uf,50V, w_smd_cap:c_elec_6.3x7.7, symbol taobao-cp:CP47uf,50V
- removed D21: 3v3 HEALTHY, LED_SMD:LED_0603_1608Metric_Pad1.05x0.95mm_HandSolder, symbol taobao-led:LED_GREEN,0603
- removed JP1, JP2: Jumper_NO_Small, Jumper:SolderJumper-2_P1.3mm_Bridged2Bar_RoundedPad1.0x1.5mm, symbol Device:Jumper_NO_Small
- removed R65: R102,0603, Resistor_SMD:R_0603_1608Metric_Pad1.05x0.95mm_HandSolder, symbol taobao-r:R102,0603
- removed U14: AMS1117-3.3, Package_TO_SOT_SMD:SOT-223-3_TabPin2, symbol Regulator_Linear:AMS1117-3.3
- added C?: CP10uf,50V, Capacitor_SMD:CP_Elec_5x5.3, symbol taobao-cp:CP10uf,50V
- added C?: C104,0603, Capacitor_SMD:C_0603_1608Metric_Pad1.05x0.95mm_HandSolder, symbol taobao-c:C104,0603
- added C?: C226,6.3v, symbol taobao-c:C226,6.3v
- added C?: C221,0603, Capacitor_SMD:C_0603_1608Metric_Pad1.05x0.95mm_HandSolder, symbol taobao-c:C221,0603
- added D?: SD_1N5822_SS34, symbol taobao-sd:SD_1N5822_SS34
- added L?: L_10uH,CD43, w_smd_inductors:inductor_smd_4.8x2.8mm, symbol taobao-l:L_10uH,CD43
- added R? (x2): R104,0603, Resistor_SMD:R_0603_1608Metric_Pad1.05x0.95mm_HandSolder, symbol taobao-r:R104,0603
- added R?: R204,0603, Resistor_SMD:R_0603_1608Metric_Pad1.05x0.95mm_HandSolder, symbol taobao-r:R204,0603
- added R?: R203,0603, Resistor_SMD:R_0603_1608Metric_Pad1.05x0.95mm_HandSolder, symbol taobao-r:R203,0603
- added R?: R473,0603, Resistor_SMD:R_0603_1608Metric_Pad1.05x0.95mm_HandSolder, symbol taobao-r:R473,0603
- added R?: R124,0603, Resistor_SMD:R_0603_1608Metric_Pad1.05x0.95mm_HandSolder, symbol taobao-r:R124,0603
- added U?: MP1584, symbol taobao-components:MP1584
Connections:
- net GND: now also C?.2, C?.2, D?.2 (A), R?.2, R?.2, R?.2, R?.2, U?.1 (SW), U?.5 (GND)
- new net: C?.1, U?.3 (COMP)
- new net: R?.1, R?.2, U?.4 (FB)
- new net: R?.1, U?.6 (FREQ)
- new net: C?.2, U?.8 (BST)
- new net: C?.1, D?.1 (K), L?.1
- new net: C?.2, R?.1
- new net +12V: C?.1, R?.1, U?.7 (VIN)
- new net +3V3_STM32: C?.1, L?.2, R?.1
- new net EN: R?.1, R?.2, U?.2 (EN)

Commit message: update,
Parts:
- gave numbers to parts that had none: 13
Changed lines of the file:
@@
 $Descr A4 11693 8268
 encoding utf-8
-Sheet 20 34
+Sheet 20 35
 Title ""
 Date ""
@@
 $EndDescr
 $Comp
-L taobao-components:MP1584 U?
+L taobao-components:MP1584 U11
 U 1 1 5CC88A9B
 P 5800 4750
-F 0 "U?" H 5800 5428 50  0000 C CNN
+F 0 "U11" H 5800 5428 50  0000 C CNN
 F 1 "MP1584" H 5800 5337 50  0000 C CNN
 F 2 "" H 5800 4750 50  0001 C CNN
@@
 $EndComp
 $Comp
-L power:+12V #PWR?
+L power:+12V #PWR099
 U 1 1 5CC88B56
 P 3450 3950
-F 0 "#PWR?" H 3450 3800 50  0001 C CNN
+F 0 "#PWR099" H 3450 3800 50  0001 C CNN
 F 1 "+12V" H 3465 4123 50  0000 C CNN
 F 2 "" H 3450 3950 50  0001 C CNN
@@
 $EndComp
 $Comp
-L taobao-components:+3V3_STM32 #PWR?
+L taobao-components:+3V3_STM32 #PWR0100
 U 1 1 5CC88C4D
 P 8150 4050
-F 0 "#PWR?" H 8150 3900 50  0001 C CNN
+F 0 "#PWR0100" H 8150 3900 50  0001 C CNN
 F 1 "+3V3_STM32" H 8165 4223 50  0000 C CNN
 F 2 "" H 8150 4050 50  0001 C CNN
@@
 $EndComp
 $Comp
-L taobao-cp:CP10uf,50V C?
+L taobao-cp:CP10uf,50V C46
 U 1 1 5CC88D54
 P 4050 4200
-F 0 "C?" H 3963 4246 50  0000 R CNN
+F 0 "C46" H 3963 4246 50  0000 R CNN
 F 1 "CP10uf,50V" H 3963 4155 50  0000 R CNN
 F 2 "Capacitor_SMD:CP_Elec_5x5.3" H 4050 4200 50  0001 C CNN
@@
 $EndComp
 $Comp
-L taobao-r:R104,0603 R?
+L taobao-r:R104,0603 R83
 U 1 1 5CC88E57
 P 4400 4350
-F 0 "R?" H 4459 4396 50  0000 L CNN
+F 0 "R83" H 4459 4396 50  0000 L CNN
 F 1 "R104,0603" H 4459 4305 50  0000 L CNN
 F 2 "Resistor_SMD:R_0603_1608Metric_Pad1.05x0.95mm_HandSolder" H 4400 4350 50  0001 C CNN
@@
 $EndComp
 $Comp
-L power:GND #PWR?
+L power:GND #PWR0121
 U 1 1 5CC8922E
 P 4850 5550
-F 0 "#PWR?" H 4850 5300 50  0001 C CNN
+F 0 "#PWR0121" H 4850 5300 50  0001 C CNN
 F 1 "GND" H 4855 5377 50  0000 C CNN
 F 2 "" H 4850 5550 50  0001 C CNN
@@
 $EndComp
 $Comp
-L power:GND #PWR?
+L power:GND #PWR0125
 U 1 1 5CC89248
 P 5800 5550
-F 0 "#PWR?" H 5800 5300 50  0001 C CNN
+F 0 "#PWR0125" H 5800 5300 50  0001 C CNN
 F 1 "GND" H 5805 5377 50  0000 C CNN
 F 2 "" H 5800 5550 50  0001 C CNN
@@
 	5250 4600 5000 4600
 $Comp
-L taobao-c:C104,0603 C?
+L taobao-c:C104,0603 C4
 U 1 1 5CC89A9F
 P 6150 4150
-F 0 "C?" V 5921 4150 50  0000 C CNN
+F 0 "C4" V 5921 4150 50  0000 C CNN
 F 1 "C104,0603" V 6012 4150 50  0000 C CNN
 F 2 "Capacitor_SMD:C_0603_1608Metric_Pad1.05x0.95mm_HandSolder" H 6150 4150 50  0001 C CNN
@@
 $EndComp
 $Comp
-L taobao-sd:SD_1N5822_SS34 D?
+L taobao-sd:SD_1N5822_SS34 D30
 U 1 1 5CC89BF2
 P 6550 4400
-F 0 "D?" V 6504 4468 50  0000 L CNN
+F 0 "D30" V 6504 4468 50  0000 L CNN
 F 1 "SD_1N5822_SS34" V 6595 4468 50  0000 L CNN
 F 2 "" V 6550 4400 50  0001 C CNN
@@
 $EndBitmap
 $Comp
-L taobao-r:R204,0603 R?
+L taobao-r:R204,0603 R87
 U 1 1 5CC8A2C0
 P 4850 5250
-F 0 "R?" H 4909 5296 50  0000 L CNN
+F 0 "R87" H 4909 5296 50  0000 L CNN
 F 1 "R204,0603" H 4909 5205 50  0000 L CNN
 F 2 "Resistor_SMD:R_0603_1608Metric_Pad1.05x0.95mm_HandSolder" H 4850 5250 50  0001 C CNN
@@
 Connection ~ 4050 4050
 $Comp
-L power:GND #PWR?
+L power:GND #PWR0105
 U 1 1 5CC8AA85
 P 4050 4400
-F 0 "#PWR?" H 4050 4150 50  0001 C CNN
+F 0 "#PWR0105" H 4050 4150 50  0001 C CNN
 F 1 "GND" H 4055 4227 50  0000 C CNN
 F 2 "" H 4050 4400 50  0001 C CNN
@@
 Connection ~ 4400 4750
 $Comp
-L taobao-r:R203,0603 R?
+L taobao-r:R203,0603 R86
 U 1 1 5CC8B239
 P 3650 5000
-F 0 "R?" H 3709 5046 50  0000 L CNN
+F 0 "R86" H 3709 5046 50  0000 L CNN
 F 1 "R203,0603" H 3709 4955 50  0000 L CNN
 F 2 "Resistor_SMD:R_0603_1608Metric_Pad1.05x0.95mm_HandSolder" H 3650 5000 50  0001 C CNN
@@
 	3650 4750 3050 4750
 $Comp
-L power:GND #PWR?
+L power:GND #PWR0120
 U 1 1 5CC8B462
 P 3650 5250
-F 0 "#PWR?" H 3650 5000 50  0001 C CNN
+F 0 "#PWR0120" H 3650 5000 50  0001 C CNN
 F 1 "GND" H 3655 5077 50  0000 C CNN
 F 2 "" H 3650 5250 50  0001 C CNN
@@
 	3650 5250 3650 5100
 $Comp
-L taobao-l:L_10uH,CD43 L?
+L taobao-l:L_10uH,CD43 L3
 U 1 1 5CC8B7D8
 P 7000 4150
-F 0 "L?" V 7185 4150 50  0000 C CNN
+F 0 "L3" V 7185 4150 50  0000 C CNN
 F 1 "L_10uH,CD43" V 7094 4150 50  0000 C CNN
 F 2 "w_smd_inductors:inductor_smd_4.8x2.8mm" H 7000 4150 50  0001 C CNN
@@
 	6550 4150 6550 4300
 $Comp
-L power:GND #PWR?
+L power:GND #PWR0111
 U 1 1 5CC8BD24
 P 6750 4600
-F 0 "#PWR?" H 6750 4350 50  0001 C CNN
+F 0 "#PWR0111" H 6750 4350 50  0001 C CNN
 F 1 "GND" V 6755 4472 50  0000 R CNN
 F 2 "" H 6750 4600 50  0001 C CNN
@@
 Connection ~ 6550 4150
 $Comp
-L taobao-c:C226,6.3v C?
+L taobao-c:C226,6.3v C47
 U 1 1 5CC8CA95
 P 7400 4350
-F 0 "C?" H 7492 4396 50  0000 L CNN
+F 0 "C47" H 7492 4396 50  0000 L CNN
 F 1 "C226,6.3v" H 7492 4305 50  0000 L CNN
 F 2 "" H 7400 4350 50  0001 C CNN
@@
 	7400 4150 7100 4150
 $Comp
-L power:GND #PWR?
+L power:GND #PWR0110
 U 1 1 5CC8D71C
 P 7400 4500
-F 0 "#PWR?" H 7400 4250 50  0001 C CNN
+F 0 "#PWR0110" H 7400 4250 50  0001 C CNN
 F 1 "GND" H 7405 4327 50  0000 C CNN
 F 2 "" H 7400 4500 50  0001 C CNN
@@
 Connection ~ 7400 4150
 $Comp
-L taobao-r:R473,0603 R?
+L taobao-r:R473,0603 R85
 U 1 1 5CC8E0D0
 P 6850 4900
-F 0 "R?" H 6909 4946 50  0000 L CNN
+F 0 "R85" H 6909 4946 50  0000 L CNN
 F 1 "R473,0603" H 6909 4855 50  0000 L CNN
 F 2 "Resistor_SMD:R_0603_1608Metric_Pad1.05x0.95mm_HandSolder" H 6850 4900 50  0001 C CNN
@@
 Connection ~ 6850 4750
 $Comp
-L taobao-r:R124,0603 R?
+L taobao-r:R124,0603 R84
 U 1 1 5CC8F64C
 P 7450 4750
-F 0 "R?" V 7254 4750 50  0000 C CNN
+F 0 "R84" V 7254 4750 50  0000 C CNN
 F 1 "R124,0603" V 7345 4750 50  0000 C CNN
 F 2 "Resistor_SMD:R_0603_1608Metric_Pad1.05x0.95mm_HandSolder" H 7450 4750 50  0001 C CNN
@@
 Connection ~ 8150 4150
 $Comp
-L power:GND #PWR?
+L power:GND #PWR0119
 U 1 1 5CC901DA
 P 6850 5050
-F 0 "#PWR?" H 6850 4800 50  0001 C CNN
+F 0 "#PWR0119" H 6850 4800 50  0001 C CNN
 F 1 "GND" H 6855 4877 50  0000 C CNN
 F 2 "" H 6850 5050 50  0001 C CNN
@@
 	6850 5050 6850 5000
 $Comp
-L taobao-c:C221,0603 C?
+L taobao-c:C221,0603 C48
 U 1 1 5CC907CE
 P 6400 5100
-F 0 "C?" H 6492 5146 50  0000 L CNN
+F 0 "C48" H 6492 5146 50  0000 L CNN
 F 1 "C221,0603" H 6492 5055 50  0000 L CNN
 F 2 "Capacitor_SMD:C_0603_1608Metric_Pad1.05x0.95mm_HandSolder" H 6400 5100 50  0001 C CNN
@@
 $EndComp
 $Comp
-L taobao-r:R104,0603 R?
+L taobao-r:R104,0603 R88
 U 1 1 5CC90923
 P 6400 5400
-F 0 "R?" H 6459 5446 50  0000 L CNN
+F 0 "R88" H 6459 5446 50  0000 L CNN
 F 1 "R104,0603" H 6459 5355 50  0000 L CNN
 F 2 "Resistor_SMD:R_0603_1608Metric_Pad1.05x0.95mm_HandSolder" H 6400 5400 50  0001 C CNN
@@
 	6400 4900 6400 5000
 $Comp
-L power:GND #PWR?
+L power:GND #PWR0130
 U 1 1 5CC91000
 P 6400 5550
-F 0 "#PWR?" H 6400 5300 50  0001 C CNN
+F 0 "#PWR0130" H 6400 5300 50  0001 C CNN
 F 1 "GND" H 6405 5377 50  0000 C CNN
 F 2 "" H 6400 5550 50  0001 C CNN
