File: hardware/printer-board/STM32_CORE.sch (KiCad schematic (older format))
At the start: 0 parts

Commit message: update,
Changed lines of the file:
@@
 STM32F407VET6(F103VET6/F103VCT6)
 $Sheet
-S 900  800  800  650
+S 3200 4250 800  650
 U 5CC2989A
 F0 "STM32_CORE_MCU" 50
 F1 "STM32_CORE_MCU.sch" 50
+F2 "D-" B R 4000 4500 50
+F3 "D+" B R 4000 4600 50
+F4 "SDA1" B R 4000 4700 50
+F5 "SCL1" B R 4000 4800 50
 $EndSheet
 $Sheet
-S 900  1800 800  650
-U 5CC2A1CB
-F0 "STM32_CORE_USB" 50
-F1 "STM32_CORE_USB.sch" 50
-$EndSheet
-$Sheet
-S 900  2800 800  650
+S 6750 4250 800  650
 U 5CC2B423
 F0 "STM32_CORE_POWER" 50
@@
 $EndSheet
 $Sheet
-S 900  3700 800  650
+S 5700 4250 800  650
 U 5CC2BD61
 F0 "STM32_CORE_IO" 50
 F1 "STM32_CORE_IO.sch" 50
 $EndSheet
+$Sheet
+S 4700 4250 800  650
+U 5CC2A1CB
+F0 "STM32_CORE_USB" 50
+F1 "STM32_CORE_USB.sch" 50
+F2 "D-" B L 4700 4500 50
+F3 "D+" B L 4700 4600 50
+$EndSheet
+Text HLabel 1200 900  0    50   Input ~ 0
+STM32_D-
+Text HLabel 1200 1000 0    50   Input ~ 0
+STM32_D+
+Wire Wire Line
+	4000 4500 4700 4500
+Wire Wire Line
+	4000 4600 4700 4600
+Text Label 4550 4500 2    50   ~ 0
+STM32_D-
+Text Label 4550 4600 2    50   ~ 0
+STM32_D+
+Wire Wire Line
+	1200 900  1900 900
+Wire Wire Line
+	1200 1000 1900 1000
+Text Label 1900 900  2    50   ~ 0
+STM32_D-
+Text Label 1900 1000 2    50   ~ 0
+STM32_D+
+Text HLabel 1200 1150 0    50   Input ~ 0
+STM32_SDA1
+Text HLabel 1200 1250 0    50   Input ~ 0
+STM32_SCL1
+Wire Wire Line
+	1200 1150 1900 1150
+Wire Wire Line
+	1200 1250 1900 1250
+Text Label 1900 1150 2    50   ~ 0
+STM32_SDA1
+Text Label 1900 1250 2    50   ~ 0
+STM32_SCL1
+Wire Wire Line
+	4000 4700 4600 4700
+Wire Wire Line
+	4000 4800 4600 4800
+Text Label 4600 4700 2    50   ~ 0
+STM32_SDA1
+Text Label 4600 4800 2    50   ~ 0
+STM32_SCL1
 $EndSCHEMATC

Commit message: update,
Other:
- note added: "When using serial, the UART used for communication with the host\n is fixed to pins PA9 (TX) and PA10 (RX). When using USB, the PA11\n (D-) and PA12 (D+) pins are reserved. The USB code assumes that\n PA12 (D+) has a fixed pullup resistor attached to it."
Changed lines of the file:
@@
 $Descr A4 11693 8268
 encoding utf-8
-Sheet 16 32
+Sheet 16 33
 Title ""
 Date ""
@@
 Text Label 4600 4800 2    50   ~ 0
 STM32_SCL1
+Text Notes 3200 3950 0    50   ~ 0
+When using serial, the UART used for communication with the host\n is fixed to pins PA9 (TX) and PA10 (RX). When using USB, the PA11\n (D-) and PA12 (D+) pins are reserved. The USB code assumes that\n PA12 (D+) has a fixed pullup resistor attached to it.
 $EndSCHEMATC

Commit message: update,
Changed lines of the file:
@@
 $Descr A4 11693 8268
 encoding utf-8
-Sheet 16 33
+Sheet 15 34
 Title ""
 Date ""
@@
 Text Notes 3200 3950 0    50   ~ 0
 When using serial, the UART used for communication with the host\n is fixed to pins PA9 (TX) and PA10 (RX). When using USB, the PA11\n (D-) and PA12 (D+) pins are reserved. The USB code assumes that\n PA12 (D+) has a fixed pullup resistor attached to it.
+$Sheet
+S 6750 5350 800  650
+U 5CC86673
+F0 "MP1584EN_power" 50
+F1 "MP1584EN_power.sch" 50
+$EndSheet
 $EndSCHEMATC
