File: hardware/printer-board/MP2303A_power_supply.sch (KiCad schematic (older format))
At the start: 11 parts, among them U12 MP2303A_ALT

Commit message: update,
Parts:
- removed C50: CP10uf,25V, Capacitor_SMD:CP_Elec_4x5.3, symbol taobao-cp:CP10uf,25V
- removed C52, C53: CP22uf,16V, Capacitor_SMD:CP_Elec_4x5.3, symbol taobao-cp:CP22uf,16V
- added C50: C106,0603, Capacitor_SMD:C_0603_1608Metric_Pad1.05x0.95mm_HandSolder, symbol taobao-c:C106,0603
- added C53: C226,6.3v,0603, Capacitor_SMD:C_0603_1608Metric_Pad1.05x0.95mm_HandSolder, symbol taobao-c:C226,6.3v,0603
Connections:
- net +12V: now also C50.1
- net +3V3_STM32: now also C53.1
- net GND: now also C50.2, C53.2
Changed lines of the file:
@@
-$EndComp
-$Comp
-L taobao-cp:CP10uf,25V C50
-U 1 1 5CC8BC46
-P 3100 3350
-F 0 "C50" H 3200 3400 50  0000 L CNN
-F 1 "CP10uf,25V" H 3200 3350 50  0000 L CNN
-F 2 "Capacitor_SMD:CP_Elec_4x5.3" H 3100 3350 50  0001 C CNN
-F 3 "~" H 3100 3350 50  0001 C CNN
-	1    3100 3350
-	1    0    0    -1
 $EndComp
 $Comp
@@
 EndData
 $EndBitmap
-$Comp
-L taobao-cp:CP22uf,16V C52
-U 1 1 5CC8D98B
-P 6800 4150
-F 0 "C52" H 6900 4200 50  0000 L CNN
-F 1 "CP22uf,16V" H 6900 4150 50  0000 L CNN
-F 2 "Capacitor_SMD:CP_Elec_4x5.3" H 6800 4150 50  0001 C CNN
-F 3 "~" H 6800 4150 50  0001 C CNN
-	1    6800 4150
-	1    0    0    -1
-$EndComp
-$Comp
-L taobao-cp:CP22uf,16V C53
-U 1 1 5CC8D9EF
-P 7050 4150
-F 0 "C53" H 7150 4200 50  0000 L CNN
-F 1 "CP22uf,16V" H 7150 4150 50  0000 L CNN
-F 2 "Capacitor_SMD:CP_Elec_4x5.3" H 7050 4150 50  0001 C CNN
-F 3 "~" H 7050 4150 50  0001 C CNN
-	1    7050 4150
-	1    0    0    -1
-$EndComp
-Wire Wire Line
-	6500 3750 6800 3750
-Wire Wire Line
-	6800 3750 6800 4050
-Wire Wire Line
-	6800 3750 7050 3750
 Wire Wire Line
 	7050 3750 7050 4050
-Connection ~ 6800 3750
-Wire Wire Line
-	6800 4250 6800 4850
-Wire Wire Line
-	6800 4850 6200 4850
 Connection ~ 6200 4850
 Wire Wire Line
 	7050 4250 7050 4850
-Wire Wire Line
-	7050 4850 6800 4850
-Connection ~ 6800 4850
 Wire Wire Line
 	6550 3450 7050 3450
@@
 	7050 3250 7050 3450
 Connection ~ 7050 3450
+Wire Wire Line
+	6500 3750 7050 3750
+Wire Wire Line
+	6200 4850 7050 4850
+$Comp
+L taobao-c:C226,6.3v,0603 C53
+U 1 1 5CC95BA7
+P 7050 4150
+F 0 "C53" H 7150 4200 50  0000 L CNN
+F 1 "C226,6.3v,0603" H 7150 4150 50  0000 L CNN
+F 2 "Capacitor_SMD:C_0603_1608Metric_Pad1.05x0.95mm_HandSolder" H 7050 4150 50  0001 C CNN
+F 3 "~" H 7050 4150 50  0001 C CNN
+	1    7050 4150
+	1    0    0    -1
+$EndComp
+$Comp
+L taobao-c:C106,0603 C50
+U 1 1 5CC95CF5
+P 3100 3350
+F 0 "C50" H 3200 3400 50  0000 L CNN
+F 1 "C106,0603" H 3200 3350 50  0000 L CNN
+F 2 "Capacitor_SMD:C_0603_1608Metric_Pad1.05x0.95mm_HandSolder" H 3100 3350 50  0001 C CNN
+F 3 "~" H 3100 3350 50  0001 C CNN
+	1    3100 3350
+	1    0    0    -1
+$EndComp
 $EndSCHEMATC
