File: hardware/printer-board/Z3_STEPPER_DRIVER.sch (KiCad schematic (older format))
At the start: 7 parts, among them J13 MS_SELECT, J14 TO_MOTOR, U8 A4988_MODULE

Commit message: update,
Parts:
- removed R15: R103,0603, Resistor_SMD:R_0603_1608Metric_Pad1.05x0.95mm_HandSolder, symbol taobao-r:R103,0603
- added D?: LED_BLUE,0603, LED_SMD:LED_0603_1608Metric_Pad1.05x0.95mm_HandSolder, symbol taobao-led:LED_BLUE,0603
- added R?: R103,0603, Resistor_SMD:R_0603_1608Metric_Pad1.05x0.95mm_HandSolder, symbol taobao-r:R103,0603
- added R?: R102,0603, Resistor_SMD:R_0603_1608Metric_Pad1.05x0.95mm_HandSolder, symbol taobao-r:R102,0603
- J14: footprint footprint-lib:s4b-ph-kl,stepper_motor_terminal -> Connector_PinHeader_2.54mm:PinHeader_1x04_P2.54mm_Vertical
Connections:
- net +3V3_STM32: now also R?.1, R?.1
- net ~EN~: now also D?.1 (K), R?.2
- new net: D?.2 (A), R?.2
Changed lines of the file:
@@
 $Descr A4 11693 8268
 encoding utf-8
-Sheet 1 34
+Sheet 9 33
 Title ""
 Date ""
@@
 F 3 "" H 5650 3200 50  0001 C CNN
 	1    5650 3150
-	1    0    0    -1
-$EndComp
-$Comp
-L taobao-r:R103,0603 R?
-U 1 1 5CC04CC5
-P 4650 2200
-AR Path="/5CC02AB8/5CC04CC5" Ref="R?"  Part="1"
-AR Path="/5CC049BB/5CC04CC5" Ref="R?"  Part="1"
-AR Path="/5CC0A4B9/5CC04CC5" Ref="R?"  Part="1"
-AR Path="/5CC0A53C/5CC04CC5" Ref="R?"  Part="1"
-AR Path="/5CC0A8C5/5CC04CC5" Ref="R?"  Part="1"
-AR Path="/5CC0A8CA/5CC04CC5" Ref="R?"  Part="1"
-AR Path="/5CC0A8CF/5CC04CC5" Ref="R15"  Part="1"
-AR Path="/5CC0AED8/5CC04CC5" Ref="R?"  Part="1"
-AR Path="/5CC04CC5" Ref="R15"  Part="1"
-F 0 "R15" H 4709 2246 50  0000 L CNN
-F 1 "R103,0603" H 4709 2155 50  0000 L CNN
-F 2 "Resistor_SMD:R_0603_1608Metric_Pad1.05x0.95mm_HandSolder" H 4650 2200 50  0001 C CNN
-F 3 "~" H 4650 2200 50  0001 C CNN
-	1    4650 2200
 	1    0    0    -1
 $EndComp
@@
 F 0 "J14" H 6980 3092 50  0000 L CNN
 F 1 "TO_MOTOR" H 6980 3001 50  0000 L CNN
-F 2 "footprint-lib:s4b-ph-kl,stepper_motor_terminal" H 6900 3100 50  0001 C CNN
+F 2 "Connector_PinHeader_2.54mm:PinHeader_1x04_P2.54mm_Vertical" H 6900 3100 50  0001 C CNN
 F 3 "~" H 6900 3100 50  0001 C CNN
 	1    6900 3100
@@
 Text Label 4600 2800 0    50   ~ 0
 ~EN~
-Wire Wire Line
-	4600 2800 4900 2800
-Wire Wire Line
-	4650 1950 4650 2100
-Wire Wire Line
-	4650 2300 4650 2400
-Wire Wire Line
-	4650 2400 4900 2400
-Wire Wire Line
-	4900 2400 4900 2800
-Connection ~ 4900 2800
-Wire Wire Line
-	4900 2800 5150 2800
 Wire Wire Line
 	3500 2900 3700 2900
@@
 $Comp
 L taobao-components:+3V3_STM32 #PWR?
-U 1 1 5CC40A9D
-P 4650 1950
-F 0 "#PWR?" H 4650 1800 50  0001 C CNN
-F 1 "+3V3_STM32" H 4665 2123 50  0000 C CNN
-F 2 "" H 4650 1950 50  0001 C CNN
-F 3 "" H 4650 1950 50  0001 C CNN
-	1    4650 1950
-	1    0    0    -1
-$EndComp
-$Comp
-L taobao-components:+3V3_STM32 #PWR?
 U 1 1 5CC40ABB
 P 3500 2700
@@
 	0    1    1    0
 $EndComp
+Wire Wire Line
+	4600 2800 4850 2800
+$Comp
+L taobao-r:R103,0603 R?
+U 1 1 5CC5CA27
+P 5000 2200
+AR Path="/5CC02AB8/5CC5CA27" Ref="R?"  Part="1"
+AR Path="/5CC049BB/5CC5CA27" Ref="R?"  Part="1"
+AR Path="/5CC0A4B9/5CC5CA27" Ref="R?"  Part="1"
+AR Path="/5CC0A53C/5CC5CA27" Ref="R?"  Part="1"
+AR Path="/5CC0A8C5/5CC5CA27" Ref="R?"  Part="1"
+AR Path="/5CC0A8CA/5CC5CA27" Ref="R?"  Part="1"
+AR Path="/5CC0A8CF/5CC5CA27" Ref="R?"  Part="1"
+AR Path="/5CC0AEC9/5CC5CA27" Ref="R?"  Part="1"
+F 0 "R?" H 5059 2246 50  0000 L CNN
+F 1 "R103,0603" H 5059 2155 50  0000 L CNN
+F 2 "Resistor_SMD:R_0603_1608Metric_Pad1.05x0.95mm_HandSolder" H 5000 2200 50  0001 C CNN
+F 3 "~" H 5000 2200 50  0001 C CNN
+	1    5000 2200
+	1    0    0    -1
+$EndComp
+Wire Wire Line
+	5000 1950 5000 2000
+$Comp
+L taobao-components:+3V3_STM32 #PWR?
+U 1 1 5CC5CA2F
+P 5000 1950
+F 0 "#PWR?" H 5000 1800 50  0001 C CNN
+F 1 "+3V3_STM32" H 5015 2123 50  0000 C CNN
+F 2 "" H 5000 1950 50  0001 C CNN
+F 3 "" H 5000 1950 50  0001 C CNN
+	1    5000 1950
+	1    0    0    -1
+$EndComp
+$Comp
+L taobao-r:R102,0603 R?
+U 1 1 5CC5CA35
+P 4850 2200
+AR Path="/5CC15C35/5CC5CA35" Ref="R?"  Part="1"
+AR Path="/5CC0AEC9/5CC5CA35" Ref="R?"  Part="1"
+F 0 "R?" H 4950 2250 50  0000 L CNN
+F 1 "R102,0603" H 4950 2200 50  0000 L CNN
+F 2 "Resistor_SMD:R_0603_1608Metric_Pad1.05x0.95mm_HandSolder" H 4850 2200 50  0001 C CNN
+F 3 "~" H 4850 2200 50  0001 C CNN
+	1    4850 2200
+	1    0    0    -1
+$EndComp
+$Comp
+L taobao-led:LED_BLUE,0603 D?
+U 1 1 5CC5CA3C
+P 4850 2450
+AR Path="/5CC15C35/5CC5CA3C" Ref="D?"  Part="1"
+AR Path="/5CC0AEC9/5CC5CA3C" Ref="D?"  Part="1"
+F 0 "D?" V 4900 2350 50  0000 R CNN
+F 1 "LED_BLUE,0603" V 4850 2350 50  0000 R CNN
+F 2 "LED_SMD:LED_0603_1608Metric_Pad1.05x0.95mm_HandSolder" V 4850 2450 50  0001 C CNN
+F 3 "" V 4850 2450 50  0001 C CNN
+	1    4850 2450
+	0    -1   -1   0
+$EndComp
+Wire Wire Line
+	4850 2300 4850 2350
+Wire Wire Line
+	4850 2100 4850 2000
+Wire Wire Line
+	5000 2300 5000 2800
+Wire Wire Line
+	4850 2550 4850 2800
+Connection ~ 5000 2000
+Wire Wire Line
+	5000 2000 5000 2100
+Wire Wire Line
+	4850 2000 5000 2000
+Connection ~ 4850 2800
+Wire Wire Line
+	4850 2800 5000 2800
+Connection ~ 5000 2800
+Wire Wire Line
+	5000 2800 5150 2800
 $EndSCHEMATC

Commit message: update label,
Parts:
- J14: value TO_MOTOR -> Z3
Connections:
- net DIR renamed Z3_DIR
- net STEP renamed Z3_STEP
- net ~EN~ renamed ~Z3_EN~
Changed lines of the file:
@@
 $EndComp
 Text Label 4400 3400 0    50   ~ 0
-STEP
+Z3_STEP
 Text Label 4400 3500 0    50   ~ 0
-DIR
+Z3_DIR
 Wire Wire Line
 	4400 3400 5150 3400
@@
 AR Path="/5CC04CFC" Ref="J14"  Part="1"
 F 0 "J14" H 6980 3092 50  0000 L CNN
-F 1 "TO_MOTOR" H 6980 3001 50  0000 L CNN
+F 1 "Z3" H 6980 3001 50  0000 L CNN
 F 2 "Connector_PinHeader_2.54mm:PinHeader_1x04_P2.54mm_Vertical" H 6900 3100 50  0001 C CNN
 F 3 "~" H 6900 3100 50  0001 C CNN
@@
 	4900 3300 5150 3300
 Text Label 4600 2800 0    50   ~ 0
-~EN~
+~Z3_EN~
 Wire Wire Line
 	3500 2900 3700 2900
@@
 	5750 4250 5950 4250
 Text HLabel 1000 800  0    50   Input ~ 0
-~EN~
+~Z3_EN~
 Text Label 1300 800  0    50   ~ 0
-~EN~
+~Z3_EN~
 Wire Wire Line
 	1000 800  1300 800
@@
 	1000 1000 1300 1000
 Text HLabel 1000 900  0    50   Input ~ 0
-STEP
+Z3_STEP
 Text HLabel 1000 1000 0    50   Input ~ 0
-DIR
+Z3_DIR
 Text Label 1300 900  0    50   ~ 0
-STEP
+Z3_STEP
 Text Label 1300 1000 0    50   ~ 0
-DIR
+Z3_DIR
 $Bitmap
 Pos 9350 5200
@@
 U 1 1 5CC5CA2F
 P 5000 1950
+AR Path="/5CC0AEC9/5CC5CA2F" Ref="#PWR?"  Part="1"
+AR Path="/5CC0A8CF/5CC5CA2F" Ref="#PWR?"  Part="1"
 F 0 "#PWR?" H 5000 1800 50  0001 C CNN
 F 1 "+3V3_STM32" H 5015 2123 50  0000 C CNN
@@
 AR Path="/5CC15C35/5CC5CA35" Ref="R?"  Part="1"
 AR Path="/5CC0AEC9/5CC5CA35" Ref="R?"  Part="1"
+AR Path="/5CC0A8CF/5CC5CA35" Ref="R?"  Part="1"
 F 0 "R?" H 4950 2250 50  0000 L CNN
 F 1 "R102,0603" H 4950 2200 50  0000 L CNN
@@
 AR Path="/5CC15C35/5CC5CA3C" Ref="D?"  Part="1"
 AR Path="/5CC0AEC9/5CC5CA3C" Ref="D?"  Part="1"
+AR Path="/5CC0A8CF/5CC5CA3C" Ref="D?"  Part="1"
 F 0 "D?" V 4900 2350 50  0000 R CNN
 F 1 "LED_BLUE,0603" V 4850 2350 50  0000 R CNN

Commit message: update annotations,
Parts:
- gave numbers to parts that had none: 4
Changed lines of the file:
@@
 $EndBitmap
 $Comp
-L taobao-components:+3V3_STM32 #PWR?
+L taobao-components:+3V3_STM32 #PWR023
 U 1 1 5CC40ABB
 P 3500 2700
-F 0 "#PWR?" H 3500 2550 50  0001 C CNN
+F 0 "#PWR023" H 3500 2550 50  0001 C CNN
 F 1 "+3V3_STM32" H 3515 2873 50  0000 C CNN
 F 2 "" H 3500 2700 50  0001 C CNN
@@
 $EndComp
 $Comp
-L taobao-components:+3V3_STM32 #PWR?
+L taobao-components:+3V3_STM32 #PWR025
 U 1 1 5CC40AD2
 P 5400 4250
-F 0 "#PWR?" H 5400 4100 50  0001 C CNN
+F 0 "#PWR025" H 5400 4100 50  0001 C CNN
 F 1 "+3V3_STM32" V 5415 4378 50  0000 L CNN
 F 2 "" H 5400 4250 50  0001 C CNN
@@
 $EndComp
 $Comp
-L taobao-components:+3V3_STM32 #PWR?
+L taobao-components:+3V3_STM32 #PWR024
 U 1 1 5CC40AFB
 P 6600 3400
-F 0 "#PWR?" H 6600 3250 50  0001 C CNN
+F 0 "#PWR024" H 6600 3250 50  0001 C CNN
 F 1 "+3V3_STM32" V 6615 3528 50  0000 L CNN
 F 2 "" H 6600 3400 50  0001 C CNN
@@
 $EndComp
 $Comp
-L taobao-c:C104,0603 C?
+L taobao-c:C104,0603 C13
 U 1 1 5CC40BF1
 P 5650 4250
-F 0 "C?" V 5421 4250 50  0000 C CNN
+F 0 "C13" V 5421 4250 50  0000 C CNN
 F 1 "C104,0603" V 5512 4250 50  0000 C CNN
 F 2 "Capacitor_SMD:C_0603_1608Metric_Pad1.05x0.95mm_HandSolder" H 5650 4250 50  0001 C CNN
@@
 AR Path="/5CC0A8C5/5CC5CA27" Ref="R?"  Part="1"
 AR Path="/5CC0A8CA/5CC5CA27" Ref="R?"  Part="1"
-AR Path="/5CC0A8CF/5CC5CA27" Ref="R?"  Part="1"
+AR Path="/5CC0A8CF/5CC5CA27" Ref="R23"  Part="1"
 AR Path="/5CC0AEC9/5CC5CA27" Ref="R?"  Part="1"
-F 0 "R?" H 5059 2246 50  0000 L CNN
+F 0 "R23" H 5059 2246 50  0000 L CNN
 F 1 "R103,0603" H 5059 2155 50  0000 L CNN
 F 2 "Resistor_SMD:R_0603_1608Metric_Pad1.05x0.95mm_HandSolder" H 5000 2200 50  0001 C CNN
@@
 P 5000 1950
 AR Path="/5CC0AEC9/5CC5CA2F" Ref="#PWR?"  Part="1"
-AR Path="/5CC0A8CF/5CC5CA2F" Ref="#PWR?"  Part="1"
-F 0 "#PWR?" H 5000 1800 50  0001 C CNN
+AR Path="/5CC0A8CF/5CC5CA2F" Ref="#PWR022"  Part="1"
+F 0 "#PWR022" H 5000 1800 50  0001 C CNN
 F 1 "+3V3_STM32" H 5015 2123 50  0000 C CNN
 F 2 "" H 5000 1950 50  0001 C CNN
@@
 AR Path="/5CC15C35/5CC5CA35" Ref="R?"  Part="1"
 AR Path="/5CC0AEC9/5CC5CA35" Ref="R?"  Part="1"
-AR Path="/5CC0A8CF/5CC5CA35" Ref="R?"  Part="1"
-F 0 "R?" H 4950 2250 50  0000 L CNN
+AR Path="/5CC0A8CF/5CC5CA35" Ref="R22"  Part="1"
+F 0 "R22" H 4950 2250 50  0000 L CNN
 F 1 "R102,0603" H 4950 2200 50  0000 L CNN
 F 2 "Resistor_SMD:R_0603_1608Metric_Pad1.05x0.95mm_HandSolder" H 4850 2200 50  0001 C CNN
@@
 AR Path="/5CC15C35/5CC5CA3C" Ref="D?"  Part="1"
 AR Path="/5CC0AEC9/5CC5CA3C" Ref="D?"  Part="1"
-AR Path="/5CC0A8CF/5CC5CA3C" Ref="D?"  Part="1"
-F 0 "D?" V 4900 2350 50  0000 R CNN
+AR Path="/5CC0A8CF/5CC5CA3C" Ref="D24"  Part="1"
+F 0 "D24" V 4900 2350 50  0000 R CNN
 F 1 "LED_BLUE,0603" V 4850 2350 50  0000 R CNN
 F 2 "LED_SMD:LED_0603_1608Metric_Pad1.05x0.95mm_HandSolder" V 4850 2450 50  0001 C CNN
