File: hardware/printer-board/Z_STEPPER_DRIVER.sch (KiCad schematic (older format))
At the start: 7 parts, among them J7 MS_SELECT, J8 TO_MOTOR, U5 A4988_MODULE

Commit message: update,
Parts:
- removed R9: R103,0603, Resistor_SMD:R_0603_1608Metric_Pad1.05x0.95mm_HandSolder, symbol taobao-r:R103,0603
- added D?: LED_BLUE,0603, LED_SMD:LED_0603_1608Metric_Pad1.05x0.95mm_HandSolder, symbol taobao-led:LED_BLUE,0603
- added R?: R103,0603, Resistor_SMD:R_0603_1608Metric_Pad1.05x0.95mm_HandSolder, symbol taobao-r:R103,0603
- added R?: R102,0603, Resistor_SMD:R_0603_1608Metric_Pad1.05x0.95mm_HandSolder, symbol taobao-r:R102,0603
- J8: footprint footprint-lib:s4b-ph-kl,stepper_motor_terminal -> Connector_PinHeader_2.54mm:PinHeader_1x04_P2.54mm_Vertical
Connections:
- net +3V3_STM32: now also R?.1, R?.1
- net ~EN~: now also D?.1 (K), R?.2
- new net: D?.2 (A), R?.2
Changed lines of the file:
@@
 $Descr A4 11693 8268
 encoding utf-8
-Sheet 1 34
+Sheet 6 33
 Title ""
 Date ""
@@
 F 3 "" H 5650 3200 50  0001 C CNN
 	1    5650 3150
-	1    0    0    -1
-$EndComp
-$Comp
-L taobao-r:R103,0603 R?
-U 1 1 5CC04CCA
-P 4650 2200
-AR Path="/5CC02AB8/5CC04CCA" Ref="R?"  Part="1"
-AR Path="/5CC049BB/5CC04CCA" Ref="R?"  Part="1"
-AR Path="/5CC0A4B9/5CC04CCA" Ref="R?"  Part="1"
-AR Path="/5CC0A53C/5CC04CCA" Ref="R9"  Part="1"
-AR Path="/5CC0A8C5/5CC04CCA" Ref="R?"  Part="1"
-AR Path="/5CC0A8CA/5CC04CCA" Ref="R?"  Part="1"
-AR Path="/5CC0A8CF/5CC04CCA" Ref="R?"  Part="1"
-AR Path="/5CC0AEC9/5CC04CCA" Ref="R?"  Part="1"
-AR Path="/5CC04CCA" Ref="R9"  Part="1"
-F 0 "R9" H 4709 2246 50  0000 L CNN
-F 1 "R103,0603" H 4709 2155 50  0000 L CNN
-F 2 "Resistor_SMD:R_0603_1608Metric_Pad1.05x0.95mm_HandSolder" H 4650 2200 50  0001 C CNN
-F 3 "~" H 4650 2200 50  0001 C CNN
-	1    4650 2200
 	1    0    0    -1
 $EndComp
@@
 F 0 "J8" H 6980 3092 50  0000 L CNN
 F 1 "TO_MOTOR" H 6980 3001 50  0000 L CNN
-F 2 "footprint-lib:s4b-ph-kl,stepper_motor_terminal" H 6900 3100 50  0001 C CNN
+F 2 "Connector_PinHeader_2.54mm:PinHeader_1x04_P2.54mm_Vertical" H 6900 3100 50  0001 C CNN
 F 3 "~" H 6900 3100 50  0001 C CNN
 	1    6900 3100
@@
 Text Label 4600 2800 0    50   ~ 0
 ~EN~
-Wire Wire Line
-	4600 2800 4900 2800
-Wire Wire Line
-	4650 1950 4650 2100
-Wire Wire Line
-	4650 2300 4650 2400
-Wire Wire Line
-	4650 2400 4900 2400
-Wire Wire Line
-	4900 2400 4900 2800
-Connection ~ 4900 2800
-Wire Wire Line
-	4900 2800 5150 2800
 Wire Wire Line
 	3500 2900 3700 2900
@@
 $Comp
 L taobao-components:+3V3_STM32 #PWR?
-U 1 1 5CC40B18
-P 4650 1950
-F 0 "#PWR?" H 4650 1800 50  0001 C CNN
-F 1 "+3V3_STM32" H 4665 2123 50  0000 C CNN
-F 2 "" H 4650 1950 50  0001 C CNN
-F 3 "" H 4650 1950 50  0001 C CNN
-	1    4650 1950
-	1    0    0    -1
-$EndComp
-$Comp
-L taobao-components:+3V3_STM32 #PWR?
 U 1 1 5CC40B36
 P 3500 2700
@@
 	0    1    1    0
 $EndComp
+Wire Wire Line
+	4600 2800 4900 2800
+$Comp
+L taobao-r:R103,0603 R?
+U 1 1 5CC57FC6
+P 5050 2200
+AR Path="/5CC02AB8/5CC57FC6" Ref="R?"  Part="1"
+AR Path="/5CC049BB/5CC57FC6" Ref="R?"  Part="1"
+AR Path="/5CC0A4B9/5CC57FC6" Ref="R?"  Part="1"
+AR Path="/5CC0A53C/5CC57FC6" Ref="R?"  Part="1"
+AR Path="/5CC0A8C5/5CC57FC6" Ref="R?"  Part="1"
+AR Path="/5CC0A8CA/5CC57FC6" Ref="R?"  Part="1"
+AR Path="/5CC0A8CF/5CC57FC6" Ref="R?"  Part="1"
+AR Path="/5CC0AEC9/5CC57FC6" Ref="R?"  Part="1"
+F 0 "R?" H 5109 2246 50  0000 L CNN
+F 1 "R103,0603" H 5109 2155 50  0000 L CNN
+F 2 "Resistor_SMD:R_0603_1608Metric_Pad1.05x0.95mm_HandSolder" H 5050 2200 50  0001 C CNN
+F 3 "~" H 5050 2200 50  0001 C CNN
+	1    5050 2200
+	1    0    0    -1
+$EndComp
+Wire Wire Line
+	5050 1950 5050 2000
+$Comp
+L taobao-components:+3V3_STM32 #PWR?
+U 1 1 5CC57FCE
+P 5050 1950
+AR Path="/5CC0AEC9/5CC57FCE" Ref="#PWR?"  Part="1"
+AR Path="/5CC0A53C/5CC57FCE" Ref="#PWR?"  Part="1"
+F 0 "#PWR?" H 5050 1800 50  0001 C CNN
+F 1 "+3V3_STM32" H 5065 2123 50  0000 C CNN
+F 2 "" H 5050 1950 50  0001 C CNN
+F 3 "" H 5050 1950 50  0001 C CNN
+	1    5050 1950
+	1    0    0    -1
+$EndComp
+$Comp
+L taobao-r:R102,0603 R?
+U 1 1 5CC57FD4
+P 4900 2200
+AR Path="/5CC15C35/5CC57FD4" Ref="R?"  Part="1"
+AR Path="/5CC0AEC9/5CC57FD4" Ref="R?"  Part="1"
+AR Path="/5CC0A53C/5CC57FD4" Ref="R?"  Part="1"
+F 0 "R?" H 5000 2250 50  0000 L CNN
+F 1 "R102,0603" H 5000 2200 50  0000 L CNN
+F 2 "Resistor_SMD:R_0603_1608Metric_Pad1.05x0.95mm_HandSolder" H 4900 2200 50  0001 C CNN
+F 3 "~" H 4900 2200 50  0001 C CNN
+	1    4900 2200
+	1    0    0    -1
+$EndComp
+$Comp
+L taobao-led:LED_BLUE,0603 D?
+U 1 1 5CC57FDB
+P 4900 2450
+AR Path="/5CC15C35/5CC57FDB" Ref="D?"  Part="1"
+AR Path="/5CC0AEC9/5CC57FDB" Ref="D?"  Part="1"
+AR Path="/5CC0A53C/5CC57FDB" Ref="D?"  Part="1"
+F 0 "D?" V 4950 2350 50  0000 R CNN
+F 1 "LED_BLUE,0603" V 4900 2350 50  0000 R CNN
+F 2 "LED_SMD:LED_0603_1608Metric_Pad1.05x0.95mm_HandSolder" V 4900 2450 50  0001 C CNN
+F 3 "" V 4900 2450 50  0001 C CNN
+	1    4900 2450
+	0    -1   -1   0
+$EndComp
+Wire Wire Line
+	4900 2300 4900 2350
+Wire Wire Line
+	4900 2100 4900 2000
+Wire Wire Line
+	5050 2300 5050 2800
+Wire Wire Line
+	4900 2550 4900 2800
+Connection ~ 5050 2000
+Wire Wire Line
+	5050 2000 5050 2100
+Wire Wire Line
+	4900 2000 5050 2000
+Connection ~ 4900 2800
+Wire Wire Line
+	4900 2800 5050 2800
+Connection ~ 5050 2800
+Wire Wire Line
+	5050 2800 5150 2800
 $EndSCHEMATC

Commit message: update label,
Parts:
- J8: value TO_MOTOR -> Z
Connections:
- net DIR renamed Z_DIR
- net STEP renamed Z_STEP
- net ~EN~ renamed ~Z_EN~
Changed lines of the file:
@@
 $EndComp
 Text Label 4400 3400 0    50   ~ 0
-STEP
+Z_STEP
 Text Label 4400 3500 0    50   ~ 0
-DIR
+Z_DIR
 Wire Wire Line
 	4400 3400 5150 3400
@@
 AR Path="/5CC04D02" Ref="J8"  Part="1"
 F 0 "J8" H 6980 3092 50  0000 L CNN
-F 1 "TO_MOTOR" H 6980 3001 50  0000 L CNN
+F 1 "Z" H 6980 3001 50  0000 L CNN
 F 2 "Connector_PinHeader_2.54mm:PinHeader_1x04_P2.54mm_Vertical" H 6900 3100 50  0001 C CNN
 F 3 "~" H 6900 3100 50  0001 C CNN
@@
 	4900 3300 5150 3300
 Text Label 4600 2800 0    50   ~ 0
-~EN~
+~Z_EN~
 Wire Wire Line
 	3500 2900 3700 2900
@@
 	5750 4250 5950 4250
 Text HLabel 1000 800  0    50   Input ~ 0
-~EN~
+~Z_EN~
 Text Label 1300 800  0    50   ~ 0
-~EN~
+~Z_EN~
 Wire Wire Line
 	1000 800  1300 800
@@
 	1000 1000 1300 1000
 Text HLabel 1000 900  0    50   Input ~ 0
-STEP
+Z_STEP
 Text HLabel 1000 1000 0    50   Input ~ 0
-DIR
+Z_DIR
 Text Label 1300 900  0    50   ~ 0
-STEP
+Z_STEP
 Text Label 1300 1000 0    50   ~ 0
-DIR
+Z_DIR
 $Bitmap
 Pos 9350 5200

Commit message: update annotations,
Parts:
- gave numbers to parts that had none: 4
Changed lines of the file:
@@
 $EndBitmap
 $Comp
-L taobao-components:+3V3_STM32 #PWR?
+L taobao-components:+3V3_STM32 #PWR015
 U 1 1 5CC40B36
 P 3500 2700
-F 0 "#PWR?" H 3500 2550 50  0001 C CNN
+F 0 "#PWR015" H 3500 2550 50  0001 C CNN
 F 1 "+3V3_STM32" H 3515 2873 50  0000 C CNN
 F 2 "" H 3500 2700 50  0001 C CNN
@@
 $EndComp
 $Comp
-L taobao-components:+3V3_STM32 #PWR?
+L taobao-components:+3V3_STM32 #PWR017
 U 1 1 5CC40B4D
 P 5400 4250
-F 0 "#PWR?" H 5400 4100 50  0001 C CNN
+F 0 "#PWR017" H 5400 4100 50  0001 C CNN
 F 1 "+3V3_STM32" V 5415 4378 50  0000 L CNN
 F 2 "" H 5400 4250 50  0001 C CNN
@@
 $EndComp
 $Comp
-L taobao-c:C104,0603 C?
+L taobao-c:C104,0603 C9
 U 1 1 5CC40BE7
 P 5650 4250
-F 0 "C?" V 5421 4250 50  0000 C CNN
+F 0 "C9" V 5421 4250 50  0000 C CNN
 F 1 "C104,0603" V 5512 4250 50  0000 C CNN
 F 2 "Capacitor_SMD:C_0603_1608Metric_Pad1.05x0.95mm_HandSolder" H 5650 4250 50  0001 C CNN
@@
 $EndComp
 $Comp
-L taobao-components:+3V3_STM32 #PWR?
+L taobao-components:+3V3_STM32 #PWR016
 U 1 1 5CC40CCA
 P 6600 3400
-F 0 "#PWR?" H 6600 3250 50  0001 C CNN
+F 0 "#PWR016" H 6600 3250 50  0001 C CNN
 F 1 "+3V3_STM32" V 6615 3528 50  0000 L CNN
 F 2 "" H 6600 3400 50  0001 C CNN
@@
 AR Path="/5CC049BB/5CC57FC6" Ref="R?"  Part="1"
 AR Path="/5CC0A4B9/5CC57FC6" Ref="R?"  Part="1"
-AR Path="/5CC0A53C/5CC57FC6" Ref="R?"  Part="1"
+AR Path="/5CC0A53C/5CC57FC6" Ref="R19"  Part="1"
 AR Path="/5CC0A8C5/5CC57FC6" Ref="R?"  Part="1"
 AR Path="/5CC0A8CA/5CC57FC6" Ref="R?"  Part="1"
 AR Path="/5CC0A8CF/5CC57FC6" Ref="R?"  Part="1"
 AR Path="/5CC0AEC9/5CC57FC6" Ref="R?"  Part="1"
-F 0 "R?" H 5109 2246 50  0000 L CNN
+F 0 "R19" H 5109 2246 50  0000 L CNN
 F 1 "R103,0603" H 5109 2155 50  0000 L CNN
 F 2 "Resistor_SMD:R_0603_1608Metric_Pad1.05x0.95mm_HandSolder" H 5050 2200 50  0001 C CNN
@@
 P 5050 1950
 AR Path="/5CC0AEC9/5CC57FCE" Ref="#PWR?"  Part="1"
-AR Path="/5CC0A53C/5CC57FCE" Ref="#PWR?"  Part="1"
-F 0 "#PWR?" H 5050 1800 50  0001 C CNN
+AR Path="/5CC0A53C/5CC57FCE" Ref="#PWR014"  Part="1"
+F 0 "#PWR014" H 5050 1800 50  0001 C CNN
 F 1 "+3V3_STM32" H 5065 2123 50  0000 C CNN
 F 2 "" H 5050 1950 50  0001 C CNN
@@
 AR Path="/5CC15C35/5CC57FD4" Ref="R?"  Part="1"
 AR Path="/5CC0AEC9/5CC57FD4" Ref="R?"  Part="1"
-AR Path="/5CC0A53C/5CC57FD4" Ref="R?"  Part="1"
-F 0 "R?" H 5000 2250 50  0000 L CNN
+AR Path="/5CC0A53C/5CC57FD4" Ref="R15"  Part="1"
+F 0 "R15" H 5000 2250 50  0000 L CNN
 F 1 "R102,0603" H 5000 2200 50  0000 L CNN
 F 2 "Resistor_SMD:R_0603_1608Metric_Pad1.05x0.95mm_HandSolder" H 4900 2200 50  0001 C CNN
@@
 AR Path="/5CC15C35/5CC57FDB" Ref="D?"  Part="1"
 AR Path="/5CC0AEC9/5CC57FDB" Ref="D?"  Part="1"
-AR Path="/5CC0A53C/5CC57FDB" Ref="D?"  Part="1"
-F 0 "D?" V 4950 2350 50  0000 R CNN
+AR Path="/5CC0A53C/5CC57FDB" Ref="D22"  Part="1"
+F 0 "D22" V 4950 2350 50  0000 R CNN
 F 1 "LED_BLUE,0603" V 4900 2350 50  0000 R CNN
 F 2 "LED_SMD:LED_0603_1608Metric_Pad1.05x0.95mm_HandSolder" V 4900 2450 50  0001 C CNN
