File: hardware/printer-board/E0_STEPPER_DRIVER.sch (KiCad schematic (older format))
At the start: 7 parts, among them J15 MS_SELECT, J16 E0, U9 A4988_MODULE

Commit message: update,
Parts:
- added D?: LED_BLUE,0603, LED_SMD:LED_0603_1608Metric_Pad1.05x0.95mm_HandSolder, symbol taobao-led:LED_BLUE,0603
- added R?: R102,0603, Resistor_SMD:R_0603_1608Metric_Pad1.05x0.95mm_HandSolder, symbol taobao-r:R102,0603
Connections:
- net +3V3_STM32: now also R?.1
- net ~EN~: now also D?.1 (K)
- new net: D?.2 (A), R?.2
Other:
- moved on the sheet: R17
Changed lines of the file:
@@
 $Descr A4 11693 8268
 encoding utf-8
-Sheet 10 34
+Sheet 10 33
 Title ""
 Date ""
@@
 L taobao-r:R103,0603 R?
 U 1 1 5CC04CC7
-P 4650 2200
+P 4900 2200
 AR Path="/5CC02AB8/5CC04CC7" Ref="R?"  Part="1"
 AR Path="/5CC049BB/5CC04CC7" Ref="R?"  Part="1"
@@
 AR Path="/5CC0A8CF/5CC04CC7" Ref="R?"  Part="1"
 AR Path="/5CC0AEC9/5CC04CC7" Ref="R17"  Part="1"
-F 0 "R17" H 4709 2246 50  0000 L CNN
-F 1 "R103,0603" H 4709 2155 50  0000 L CNN
-F 2 "Resistor_SMD:R_0603_1608Metric_Pad1.05x0.95mm_HandSolder" H 4650 2200 50  0001 C CNN
-F 3 "~" H 4650 2200 50  0001 C CNN
-	1    4650 2200
+F 0 "R17" H 4959 2246 50  0000 L CNN
+F 1 "R103,0603" H 4959 2155 50  0000 L CNN
+F 2 "Resistor_SMD:R_0603_1608Metric_Pad1.05x0.95mm_HandSolder" H 4900 2200 50  0001 C CNN
+F 3 "~" H 4900 2200 50  0001 C CNN
+	1    4900 2200
 	1    0    0    -1
 $EndComp
@@
 ~EN~
 Wire Wire Line
-	4600 2800 4900 2800
-Wire Wire Line
-	4650 1950 4650 2100
-Wire Wire Line
-	4650 2300 4650 2400
-Wire Wire Line
-	4650 2400 4900 2400
-Wire Wire Line
-	4900 2400 4900 2800
+	4600 2800 4750 2800
+Wire Wire Line
+	4900 1950 4900 2000
 Connection ~ 4900 2800
 Wire Wire Line
@@
 L taobao-components:+3V3_STM32 #PWR?
 U 1 1 5CC8CD5D
-P 4650 1950
-F 0 "#PWR?" H 4650 1800 50  0001 C CNN
-F 1 "+3V3_STM32" H 4665 2123 50  0000 C CNN
-F 2 "" H 4650 1950 50  0001 C CNN
-F 3 "" H 4650 1950 50  0001 C CNN
-	1    4650 1950
+P 4900 1950
+F 0 "#PWR?" H 4900 1800 50  0001 C CNN
+F 1 "+3V3_STM32" H 4915 2123 50  0000 C CNN
+F 2 "" H 4900 1950 50  0001 C CNN
+F 3 "" H 4900 1950 50  0001 C CNN
+	1    4900 1950
 	1    0    0    -1
 $EndComp
@@
 	0    1    1    0
 $EndComp
+$Comp
+L taobao-r:R102,0603 R?
+U 1 1 5CC4C25E
+P 4750 2200
+AR Path="/5CC15C35/5CC4C25E" Ref="R?"  Part="1"
+AR Path="/5CC0AEC9/5CC4C25E" Ref="R?"  Part="1"
+F 0 "R?" H 4850 2250 50  0000 L CNN
+F 1 "R102,0603" H 4850 2200 50  0000 L CNN
+F 2 "Resistor_SMD:R_0603_1608Metric_Pad1.05x0.95mm_HandSolder" H 4750 2200 50  0001 C CNN
+F 3 "~" H 4750 2200 50  0001 C CNN
+	1    4750 2200
+	1    0    0    -1
+$EndComp
+$Comp
+L taobao-led:LED_BLUE,0603 D?
+U 1 1 5CC4C265
+P 4750 2450
+AR Path="/5CC15C35/5CC4C265" Ref="D?"  Part="1"
+AR Path="/5CC0AEC9/5CC4C265" Ref="D?"  Part="1"
+F 0 "D?" V 4800 2350 50  0000 R CNN
+F 1 "LED_BLUE,0603" V 4750 2350 50  0000 R CNN
+F 2 "LED_SMD:LED_0603_1608Metric_Pad1.05x0.95mm_HandSolder" V 4750 2450 50  0001 C CNN
+F 3 "" V 4750 2450 50  0001 C CNN
+	1    4750 2450
+	0    -1   -1   0
+$EndComp
+Wire Wire Line
+	4750 2300 4750 2350
+Wire Wire Line
+	4750 2100 4750 2000
+Wire Wire Line
+	4900 2300 4900 2800
+Wire Wire Line
+	4750 2550 4750 2800
+Connection ~ 4750 2800
+Wire Wire Line
+	4750 2800 4900 2800
+Connection ~ 4900 2000
+Wire Wire Line
+	4900 2000 4900 2100
+Wire Wire Line
+	4750 2000 4900 2000
 $EndSCHEMATC

Commit message: update label,
Connections:
- net DIR renamed E0_DIR
- net STEP renamed E0_STEP
- net ~EN~ renamed ~E0_EN~
Changed lines of the file:
@@
 $EndComp
 Text Label 4400 3400 0    50   ~ 0
-STEP
+E0_STEP
 Text Label 4400 3500 0    50   ~ 0
-DIR
+E0_DIR
 Wire Wire Line
 	4400 3400 5150 3400
@@
 	4900 3300 5150 3300
 Text Label 4600 2800 0    50   ~ 0
-~EN~
+~E0_EN~
 Wire Wire Line
 	4600 2800 4750 2800
@@
 	5750 4250 5950 4250
 Text HLabel 1000 800  0    50   Input ~ 0
-~EN~
+~E0_EN~
 Text Label 1300 800  0    50   ~ 0
-~EN~
+~E0_EN~
 Wire Wire Line
 	1000 800  1300 800
@@
 	1000 1000 1300 1000
 Text HLabel 1000 900  0    50   Input ~ 0
-STEP
+E0_STEP
 Text HLabel 1000 1000 0    50   Input ~ 0
-DIR
+E0_DIR
 Text Label 1300 900  0    50   ~ 0
-STEP
+E0_STEP
 Text Label 1300 1000 0    50   ~ 0
-DIR
+E0_DIR
 $Bitmap
 Pos 9600 5200

Commit message: update annotations,
Parts:
- gave numbers to parts that had none: 3
Changed lines of the file:
@@
 $EndBitmap
 $Comp
-L taobao-components:+3V3_STM32 #PWR?
+L taobao-components:+3V3_STM32 #PWR026
 U 1 1 5CC8CD5D
 P 4900 1950
-F 0 "#PWR?" H 4900 1800 50  0001 C CNN
+F 0 "#PWR026" H 4900 1800 50  0001 C CNN
 F 1 "+3V3_STM32" H 4915 2123 50  0000 C CNN
 F 2 "" H 4900 1950 50  0001 C CNN
@@
 $EndComp
 $Comp
-L taobao-components:+3V3_STM32 #PWR?
+L taobao-components:+3V3_STM32 #PWR027
 U 1 1 5CC8CDB8
 P 3500 2700
-F 0 "#PWR?" H 3500 2550 50  0001 C CNN
+F 0 "#PWR027" H 3500 2550 50  0001 C CNN
 F 1 "+3V3_STM32" H 3515 2873 50  0000 C CNN
 F 2 "" H 3500 2700 50  0001 C CNN
@@
 $EndComp
 $Comp
-L taobao-components:+3V3_STM32 #PWR?
+L taobao-components:+3V3_STM32 #PWR028
 U 1 1 5CC8CEC9
 P 6600 3400
-F 0 "#PWR?" H 6600 3250 50  0001 C CNN
+F 0 "#PWR028" H 6600 3250 50  0001 C CNN
 F 1 "+3V3_STM32" V 6615 3528 50  0000 L CNN
 F 2 "" H 6600 3400 50  0001 C CNN
@@
 $EndComp
 $Comp
-L taobao-components:+3V3_STM32 #PWR?
+L taobao-components:+3V3_STM32 #PWR029
 U 1 1 5CC8DC63
 P 5400 4250
-F 0 "#PWR?" H 5400 4100 50  0001 C CNN
+F 0 "#PWR029" H 5400 4100 50  0001 C CNN
 F 1 "+3V3_STM32" V 5415 4378 50  0000 L CNN
 F 2 "" H 5400 4250 50  0001 C CNN
@@
 $EndComp
 $Comp
-L taobao-c:C104,0603 C?
+L taobao-c:C104,0603 C15
 U 1 1 5CC8EC71
 P 5650 4250
-F 0 "C?" V 5787 4250 50  0000 C CNN
+F 0 "C15" V 5787 4250 50  0000 C CNN
 F 1 "C104,0603" V 5878 4250 50  0000 C CNN
 F 2 "Capacitor_SMD:C_0603_1608Metric_Pad1.05x0.95mm_HandSolder" H 5650 4250 50  0001 C CNN
@@
 P 4750 2200
 AR Path="/5CC15C35/5CC4C25E" Ref="R?"  Part="1"
-AR Path="/5CC0AEC9/5CC4C25E" Ref="R?"  Part="1"
-F 0 "R?" H 4850 2250 50  0000 L CNN
+AR Path="/5CC0AEC9/5CC4C25E" Ref="R39"  Part="1"
+F 0 "R39" H 4850 2250 50  0000 L CNN
 F 1 "R102,0603" H 4850 2200 50  0000 L CNN
 F 2 "Resistor_SMD:R_0603_1608Metric_Pad1.05x0.95mm_HandSolder" H 4750 2200 50  0001 C CNN
@@
 P 4750 2450
 AR Path="/5CC15C35/5CC4C265" Ref="D?"  Part="1"
-AR Path="/5CC0AEC9/5CC4C265" Ref="D?"  Part="1"
-F 0 "D?" V 4800 2350 50  0000 R CNN
+AR Path="/5CC0AEC9/5CC4C265" Ref="D25"  Part="1"
+F 0 "D25" V 4800 2350 50  0000 R CNN
 F 1 "LED_BLUE,0603" V 4750 2350 50  0000 R CNN
 F 2 "LED_SMD:LED_0603_1608Metric_Pad1.05x0.95mm_HandSolder" V 4750 2450 50  0001 C CNN

Commit message: update,
Parts:
- J16: footprint footprint-lib:s4b-ph-kl,stepper_motor_terminal -> footprint-lib:b4b-ph-kl,stepper_terminal
- U9: footprint Module:Pololu_Breakout-16_15.2x20.3mm -> footprint-lib:Pololu_Breakout-16_15.2x20.3mm
Changed lines of the file:
@@
 $Descr A4 11693 8268
 encoding utf-8
-Sheet 10 33
+Sheet 7 33
 Title ""
 Date ""
@@
 F 0 "U9" H 5650 3765 50  0000 C CNN
 F 1 "A4988_MODULE" H 5650 3674 50  0000 C CNN
-F 2 "Module:Pololu_Breakout-16_15.2x20.3mm" H 5650 3200 50  0001 C CNN
+F 2 "footprint-lib:Pololu_Breakout-16_15.2x20.3mm" H 5650 3200 50  0001 C CNN
 F 3 "" H 5650 3200 50  0001 C CNN
 	1    5650 3150
@@
 F 0 "J16" H 6980 3092 50  0000 L CNN
 F 1 "E0" H 6980 3001 50  0000 L CNN
-F 2 "footprint-lib:s4b-ph-kl,stepper_motor_terminal" H 6900 3100 50  0001 C CNN
+F 2 "footprint-lib:b4b-ph-kl,stepper_terminal" H 6900 3100 50  0001 C CNN
 F 3 "~" H 6900 3100 50  0001 C CNN
 	1    6900 3100
