File: hardware/printer-board/st7920 type lcd.sch (KiCad schematic (older format))
At the start: 3 parts

Commit message: update,
Parts:
- gave numbers to parts that had none: 1
Changed lines of the file:
@@
 $Descr A4 11693 8268
 encoding utf-8
-Sheet 33 34
+Sheet 33 35
 Title ""
 Date ""
@@
 P 1550 950
 AR Path="/5CC19D48/5CE587EA" Ref="JP8"  Part="1"
-AR Path="/5CC8321E/5CE587EA" Ref="JP?"  Part="1"
-AR Path="/5CC86287/5CE587EA" Ref="JP?"  Part="1"
-F 0 "JP?" H 1550 1135 50  0000 C CNN
+AR Path="/5CC8321E/5CE587EA" Ref="JP8"  Part="1"
+AR Path="/5CC86287/5CE587EA" Ref="JP13"  Part="1"
+F 0 "JP13" H 1550 1135 50  0000 C CNN
 F 1 "Jumper_NO_Small" H 1550 1044 50  0000 C CNN
 F 2 "" H 1550 950 50  0001 C CNN
@@
 P 1550 700
 AR Path="/5CC19D48/5CE587AA" Ref="JP7"  Part="1"
-AR Path="/5CC8321E/5CE587AA" Ref="JP?"  Part="1"
-AR Path="/5CC86287/5CE587AA" Ref="JP?"  Part="1"
-F 0 "JP?" H 1550 885 50  0000 C CNN
+AR Path="/5CC8321E/5CE587AA" Ref="JP7"  Part="1"
+AR Path="/5CC86287/5CE587AA" Ref="JP12"  Part="1"
+F 0 "JP12" H 1550 885 50  0000 C CNN
 F 1 "Jumper_NO_Small" H 1550 794 50  0000 C CNN
 F 2 "" H 1550 700 50  0001 C CNN
@@
 P 1550 1150
 AR Path="/5CC19D48/5CC83513" Ref="JP?"  Part="1"
-AR Path="/5CC8321E/5CC83513" Ref="JP?"  Part="1"
-AR Path="/5CC86287/5CC83513" Ref="JP?"  Part="1"
-F 0 "JP?" H 1550 1057 50  0000 C CNN
+AR Path="/5CC8321E/5CC83513" Ref="JP11"  Part="1"
+AR Path="/5CC86287/5CC83513" Ref="JP14"  Part="1"
+F 0 "JP14" H 1550 1057 50  0000 C CNN
 F 1 "Jumper_NO_Small" H 1550 966 50  0000 C CNN
 F 2 "" H 1550 1150 50  0001 C CNN

Commit message: update,
Parts:
- added J20, J25: Conn_02x05_Odd_Even, Connector_PinHeader_2.54mm:PinHeader_2x05_P2.54mm_Vertical, symbol Connector_Generic:Conn_02x05_Odd_Even
Connections:
- new net +5V: J20.2 (Pin_2)
- new net GND: J20.1 (Pin_1)

Commit message: update,
Changed lines of the file:
@@
 AR Path="/5CC8321E/5CE587EA" Ref="JP8"  Part="1"
 AR Path="/5CC86287/5CE587EA" Ref="JP13"  Part="1"
-F 0 "JP13" H 1550 1135 50  0000 C CNN
+F 0 "JP8" H 1550 1135 50  0000 C CNN
 F 1 "Jumper_NO_Small" H 1550 1044 50  0000 C CNN
 F 2 "" H 1550 950 50  0001 C CNN
@@
 AR Path="/5CC8321E/5CE587AA" Ref="JP7"  Part="1"
 AR Path="/5CC86287/5CE587AA" Ref="JP12"  Part="1"
-F 0 "JP12" H 1550 885 50  0000 C CNN
+F 0 "JP7" H 1550 885 50  0000 C CNN
 F 1 "Jumper_NO_Small" H 1550 794 50  0000 C CNN
 F 2 "" H 1550 700 50  0001 C CNN
@@
 AR Path="/5CC8321E/5CC83513" Ref="JP11"  Part="1"
 AR Path="/5CC86287/5CC83513" Ref="JP14"  Part="1"
-F 0 "JP14" H 1550 1057 50  0000 C CNN
+F 0 "JP11" H 1550 1057 50  0000 C CNN
 F 1 "Jumper_NO_Small" H 1550 966 50  0000 C CNN
 F 2 "" H 1550 1150 50  0001 C CNN
@@
 AR Path="/5CC8321E/5CCAAC62" Ref="J20"  Part="1"
 AR Path="/5CC86287/5CCAAC62" Ref="J26"  Part="1"
-F 0 "J26" H 5900 4550 50  0000 C CNN
+F 0 "J20" H 5900 4550 50  0000 C CNN
 F 1 "Conn_02x05_Odd_Even" H 5900 4450 50  0000 C CNN
 F 2 "Connector_PinHeader_2.54mm:PinHeader_2x05_P2.54mm_Vertical" H 5850 4100 50  0001 C CNN
@@
 AR Path="/5CC8321E/5CCAACDC" Ref="J25"  Part="1"
 AR Path="/5CC86287/5CCAACDC" Ref="J36"  Part="1"
-F 0 "J36" H 5900 5750 50  0000 C CNN
+F 0 "J25" H 5900 5750 50  0000 C CNN
 F 1 "Conn_02x05_Odd_Even" H 5900 5650 50  0000 C CNN
 F 2 "Connector_PinHeader_2.54mm:PinHeader_2x05_P2.54mm_Vertical" H 5850 5300 50  0001 C CNN
@@
 AR Path="/5CC8321E/5CCAAF2A" Ref="#PWR0106"  Part="1"
 AR Path="/5CC86287/5CCAAF2A" Ref="#PWR0108"  Part="1"
-F 0 "#PWR0108" H 5250 3650 50  0001 C CNN
+F 0 "#PWR0106" H 5250 3650 50  0001 C CNN
 F 1 "GND" V 5250 3750 50  0000 R CNN
 F 2 "" H 5250 3900 50  0001 C CNN
@@
 AR Path="/5CC8321E/5CCAB01C" Ref="#PWR0107"  Part="1"
 AR Path="/5CC86287/5CCAB01C" Ref="#PWR0109"  Part="1"
-F 0 "#PWR0109" H 6650 3750 50  0001 C CNN
+F 0 "#PWR0107" H 6650 3750 50  0001 C CNN
 F 1 "+5V" V 6650 4050 50  0000 L CNN
 F 2 "" H 6650 3900 50  0001 C CNN

Commit message: update,
Parts:
- JP11, JP7, JP8: footprint (none) -> SolderJumper-2_P1.3mm_Open_TrianglePad1.0x1.5mm
Changed lines of the file:
@@
 F 0 "JP8" H 1550 1135 50  0000 C CNN
 F 1 "Jumper_NO_Small" H 1550 1044 50  0000 C CNN
-F 2 "" H 1550 950 50  0001 C CNN
+F 2 "SolderJumper-2_P1.3mm_Open_TrianglePad1.0x1.5mm" H 1550 950 50  0001 C CNN
 F 3 "~" H 1550 950 50  0001 C CNN
 	1    1550 950
@@
 F 0 "JP7" H 1550 885 50  0000 C CNN
 F 1 "Jumper_NO_Small" H 1550 794 50  0000 C CNN
-F 2 "" H 1550 700 50  0001 C CNN
+F 2 "SolderJumper-2_P1.3mm_Open_TrianglePad1.0x1.5mm" H 1550 700 50  0001 C CNN
 F 3 "~" H 1550 700 50  0001 C CNN
 	1    1550 700
@@
 F 0 "JP11" H 1550 1057 50  0000 C CNN
 F 1 "Jumper_NO_Small" H 1550 966 50  0000 C CNN
-F 2 "" H 1550 1150 50  0001 C CNN
+F 2 "SolderJumper-2_P1.3mm_Open_TrianglePad1.0x1.5mm" H 1550 1150 50  0001 C CNN
 F 3 "~" H 1550 1150 50  0001 C CNN
 	1    1550 1150
