File: hardware/printer-board/Y_STEPPER_DRIVER.kicad_pcb (KiCad board)
At the start: 2 copper layers, 9 parts, among them J5 MS_SELECT, J6 Y, U4 A4988_MODULE

Commit message: update for stepper Z,
Parts:
- removed D29: LED_BLUE,0603, LED_SMD:LED_0603_1608Metric_Pad1.05x0.95mm_HandSolder
- added C1: CP100uf,35V, Capacitor_SMD:C_0603_1608Metric_Pad1.05x0.95mm_HandSolder, F.Cu at (190.6, 45.3)
- added C10: CP100uf,25V, Capacitor_SMD:CP_Elec_6.3x7.7, F.Cu at (297.3, 53.2)
- added C11: C104,0603, Capacitor_SMD:C_0603_1608Metric_Pad1.05x0.95mm_HandSolder, F.Cu at (297.6, 59.1)
- added C12: CP100uf,25V, Capacitor_SMD:CP_Elec_6.3x7.7, F.Cu at (240.3, 109.1)
- added C13: C104,0603, Capacitor_SMD:C_0603_1608Metric_Pad1.05x0.95mm_HandSolder, F.Cu at (237.3, 115.0)
- added C14: C106,0603, Capacitor_SMD:C_0603_1608Metric_Pad1.05x0.95mm_HandSolder, F.Cu at (295.6, 127.7)
- added C15: C106,0603, Capacitor_SMD:C_0603_1608Metric_Pad1.05x0.95mm_HandSolder, F.Cu at (292.3, 136.8)
- added C16: C106,0603, Capacitor_SMD:C_0603_1608Metric_Pad1.05x0.95mm_HandSolder, F.Cu at (292.3, 127.7)
- added C17: C106,0603, Capacitor_SMD:C_0603_1608Metric_Pad1.05x0.95mm_HandSolder, F.Cu at (295.6, 129.2)
- added C18: C106,0603, Capacitor_SMD:C_0603_1608Metric_Pad1.05x0.95mm_HandSolder, F.Cu at (292.3, 132.3)
- added C19: C104,0603, Capacitor_SMD:C_0603_1608Metric_Pad1.05x0.95mm_HandSolder, F.Cu at (221.4, 140.3)
- added C2: CP100uf,25V, Capacitor_SMD:CP_Elec_6.3x7.7, F.Cu at (160.0, 109.1)
- added C20: CP100uf,35V, Capacitor_SMD:CP_Elec_6.3x7.7, F.Cu at (235.1, 137.6)
- added C21: C104,0603, Capacitor_SMD:C_0603_1608Metric_Pad1.05x0.95mm_HandSolder, F.Cu at (295.3, 86.0)
- added C22: C10pf,0603, Capacitor_SMD:C_0603_1608Metric_Pad1.05x0.95mm_HandSolder, F.Cu at (281.9, 85.8)
- added C23: C104,0603, Capacitor_SMD:C_0603_1608Metric_Pad1.05x0.95mm_HandSolder, F.Cu at (308.3, 76.8)
- added C24: C10pf,0603, Capacitor_SMD:C_0603_1608Metric_Pad1.05x0.95mm_HandSolder, F.Cu at (285.2, 85.8)
- added C25: C104,0603, Capacitor_SMD:C_0603_1608Metric_Pad1.05x0.95mm_HandSolder, F.Cu at (295.1, 82.0)
- added C26: C104,0603, Capacitor_SMD:C_0603_1608Metric_Pad1.05x0.95mm_HandSolder, F.Cu at (295.1, 80.4)
- added C27: C104,0603, Capacitor_SMD:C_0603_1608Metric_Pad1.05x0.95mm_HandSolder, F.Cu at (298.5, 80.4)
- added C28: C104,0603, Capacitor_SMD:C_0603_1608Metric_Pad1.05x0.95mm_HandSolder, F.Cu at (295.1, 83.5)
- added C29: C105,0603, Capacitor_SMD:C_0603_1608Metric_Pad1.05x0.95mm_HandSolder, F.Cu at (305.0, 75.3)
- added C3: C104,0603, Capacitor_SMD:C_0603_1608Metric_Pad1.05x0.95mm_HandSolder, F.Cu at (166.4, 109.9)
- added C30: C104,0603, Capacitor_SMD:C_0603_1608Metric_Pad1.05x0.95mm_HandSolder, F.Cu at (298.5, 78.9)
- added C31: C104,0603, Capacitor_SMD:C_0603_1608Metric_Pad1.05x0.95mm_HandSolder, F.Cu at (291.9, 85.8)
- added C32: C104,0603, Capacitor_SMD:C_0603_1608Metric_Pad1.05x0.95mm_HandSolder, F.Cu at (288.6, 85.8)
- added C33: CP220uf,16V, Capacitor_SMD:C_0603_1608Metric_Pad1.05x0.95mm_HandSolder, F.Cu at (147.7, 149.0)
- added C34: CP220uf,16V, Capacitor_SMD:C_0603_1608Metric_Pad1.05x0.95mm_HandSolder, F.Cu at (144.3, 149.0)
- added C35: CP220uf,25V, Capacitor_SMD:C_0603_1608Metric_Pad1.05x0.95mm_HandSolder, F.Cu at (144.3, 150.5)
- added C36: CP100uf,16V, Capacitor_SMD:CP_Elec_6.3x5.3, F.Cu at (259.2, 130.5)
- added C37: CP100uf,16V, Capacitor_SMD:CP_Elec_6.3x5.3, F.Cu at (321.8, 48.1)
- added C38: CP100uf,16V, Capacitor_SMD:CP_Elec_6.3x5.3, F.Cu at (259.2, 145.1)
- added C39: CP100uf,25V, Capacitor_SMD:CP_Elec_6.3x7.7, F.Cu at (257.2, 77.0)
- added C4: CP100uf,25V, Capacitor_SMD:CP_Elec_6.3x7.7, F.Cu at (200.2, 109.1)
- added C40: C104,0603, Capacitor_SMD:C_0603_1608Metric_Pad1.05x0.95mm_HandSolder, F.Cu at (254.2, 84.5)
- added C41: CP100uf,25V, Capacitor_SMD:CP_Elec_6.3x7.7, F.Cu at (257.2, 53.2)
- added C42: C104,0603, Capacitor_SMD:C_0603_1608Metric_Pad1.05x0.95mm_HandSolder, F.Cu at (263.6, 54.0)
- added C43: C104,0603, Capacitor_SMD:C_0603_1608Metric_Pad1.05x0.95mm_HandSolder, F.Cu at (274.0, 103.0)
- added C44: CP100uf,16V, Capacitor_SMD:CP_Elec_6.3x5.3, F.Cu at (280.3, 95.8)
- added C46: C104,0603, Capacitor_SMD:C_0603_1608Metric_Pad1.05x0.95mm_HandSolder, F.Cu at (325.3, 92.3)
- added C47: C332,0603, Capacitor_SMD:C_0603_1608Metric_Pad1.05x0.95mm_HandSolder, F.Cu at (322.0, 92.3)
- added C48: C103,0603, Capacitor_SMD:C_0603_1608Metric_Pad1.05x0.95mm_HandSolder, F.Cu at (318.6, 93.8)
- added C49: C226,6.3v,0603, Capacitor_SMD:C_0603_1608Metric_Pad1.05x0.95mm_HandSolder, F.Cu at (328.7, 93.8)
- added C5: C104,0603, Capacitor_SMD:C_0603_1608Metric_Pad1.05x0.95mm_HandSolder, F.Cu at (197.2, 116.6)
- added C50: C106,0603, Capacitor_SMD:C_0603_1608Metric_Pad1.05x0.95mm_HandSolder, F.Cu at (224.8, 152.9)
- added C51: C104,0603, Capacitor_SMD:C_0603_1608Metric_Pad1.05x0.95mm_HandSolder, F.Cu at (228.1, 151.4)
- added C52: C332,0603, Capacitor_SMD:C_0603_1608Metric_Pad1.05x0.95mm_HandSolder, F.Cu at (221.4, 152.9)
- added C53: C103,0603, Capacitor_SMD:C_0603_1608Metric_Pad1.05x0.95mm_HandSolder, F.Cu at (224.8, 151.4)
- added C54: C226,6.3v,0603, Capacitor_SMD:C_0603_1608Metric_Pad1.05x0.95mm_HandSolder, F.Cu at (221.4, 151.4)
- added C6: CP100uf,25V, Capacitor_SMD:CP_Elec_6.3x7.7, F.Cu at (160.0, 133.1)
- added C7: C104,0603, Capacitor_SMD:C_0603_1608Metric_Pad1.05x0.95mm_HandSolder, F.Cu at (160.3, 139.0)
- added C9: C104,0603, Capacitor_SMD:C_0603_1608Metric_Pad1.05x0.95mm_HandSolder, F.Cu at (197.1, 140.5)
- added D1: 5V HEALTHY, LED_SMD:LED_0603_1608Metric_Pad1.05x0.95mm_HandSolder, F.Cu at (141.2, 93.6)
- added D10: LED_BLUE,0603, LED_SMD:LED_0603_1608Metric_Pad1.05x0.95mm_HandSolder, F.Cu at (315.2, 79.3)
- added D11: LED_BLUE,0603, LED_SMD:LED_0603_1608Metric_Pad1.05x0.95mm_HandSolder, F.Cu at (318.6, 79.3)
- added D12: LED_BLUE,0603, LED_SMD:LED_0603_1608Metric_Pad1.05x0.95mm_HandSolder, F.Cu at (318.6, 80.9)
- added D13: LED_BLUE,0603, LED_SMD:LED_0603_1608Metric_Pad1.05x0.95mm_HandSolder, F.Cu at (325.4, 79.3)
- added D14: LED_BLUE,0603, LED_SMD:LED_0603_1608Metric_Pad1.05x0.95mm_HandSolder, F.Cu at (322.0, 79.3)
- added D15: SD_M4, Diode_SMD:D_SOD-323_HandSoldering, F.Cu at (221.8, 136.1)
- added D16: SD_M4, Diode_SMD:D_SOD-323_HandSoldering, F.Cu at (225.8, 136.1)
- added D17: PB9, LED_SMD:LED_0603_1608Metric_Pad1.05x0.95mm_HandSolder, F.Cu at (278.5, 85.8)
- added D18: LED_RED,0603, LED_SMD:LED_0603_1608Metric_Pad1.05x0.95mm_HandSolder, F.Cu at (295.3, 102.5)
- added D19: LED_RED,0603, LED_SMD:LED_0603_1608Metric_Pad1.05x0.95mm_HandSolder, F.Cu at (265.4, 122.5)
- added D2: LED_BLUE,0603, LED_SMD:LED_0603_1608Metric_Pad1.05x0.95mm_HandSolder, F.Cu at (157.0, 115.4)
- added D20: LED_BLUE,0603, LED_SMD:LED_0603_1608Metric_Pad1.05x0.95mm_HandSolder, F.Cu at (259.8, 134.9)
- added D21: LED_BLUE,0603, LED_SMD:LED_0603_1608Metric_Pad1.05x0.95mm_HandSolder, F.Cu at (322.4, 52.4)
- added D22: LED_BLUE,0603, LED_SMD:LED_0603_1608Metric_Pad1.05x0.95mm_HandSolder, F.Cu at (272.1, 142.3)
- added D23: LED_BLUE,0603, LED_SMD:LED_0603_1608Metric_Pad1.05x0.95mm_HandSolder, F.Cu at (254.2, 81.4)
- added D24: LED_BLUE,0603, LED_SMD:LED_0603_1608Metric_Pad1.05x0.95mm_HandSolder, F.Cu at (254.2, 57.5)
- added D3: LED_BLUE,0603, LED_SMD:LED_0603_1608Metric_Pad1.05x0.95mm_HandSolder, F.Cu at (197.2, 113.5)
- added D4: LED_BLUE,0603, LED_SMD:LED_0603_1608Metric_Pad1.05x0.95mm_HandSolder, F.Cu at (157.0, 137.4)
- added D5: LED_BLUE,0603, LED_SMD:LED_0603_1608Metric_Pad1.05x0.95mm_HandSolder, F.Cu at (197.1, 137.4)
- added D6: LED_BLUE,0603, LED_SMD:LED_0603_1608Metric_Pad1.05x0.95mm_HandSolder, F.Cu at (294.3, 57.5)
- added D7: LED_BLUE,0603, LED_SMD:LED_0603_1608Metric_Pad1.05x0.95mm_HandSolder, F.Cu at (237.3, 113.5)
- added D8: LED_RED,0603, LED_SMD:LED_0603_1608Metric_Pad1.05x0.95mm_HandSolder, F.Cu at (295.3, 119.1)
- added D9: LED_BLUE,0603, LED_SMD:LED_0603_1608Metric_Pad1.05x0.95mm_HandSolder, F.Cu at (315.2, 80.9)
- added F1: 16V/30A, w_misc_comp:fuse_smf, F.Cu at (225.0, 127.0)
- added F2: 30V/5A, w_misc_comp:fuse_smf, F.Cu at (225.0, 132.4)
- added H1: MOUNT_M3, MountingHole:MountingHole_2.7mm_M2.5, F.Cu at (3.00, 3.00)
- added H2: MOUNT_M3, MountingHole:MountingHole_2.7mm_M2.5, F.Cu at (97.0, 3.00)
- added H3: MOUNT_M3, MountingHole:MountingHole_2.7mm_M2.5, F.Cu at (3.00, 97.0)
- added H4: MOUNT_M3, MountingHole:MountingHole_2.7mm_M2.5, F.Cu at (97.0, 97.0)
- added J1: USB_DEBUG, Connector_PinHeader_1.27mm:PinHeader_1x05_P1.27mm_Vertical, F.Cu at (187.4, 45.7)
- added J10: MS_SELECT, Connector_PinHeader_2.54mm:PinHeader_2x03_P2.54mm_Vertical, F.Cu at (304.8, 46.3)
- added J11: E0, footprint-lib:b4b-ph-kl,stepper_terminal, F.Cu at (297.8, 46.6)
- added J12: MS_SELECT, Connector_PinHeader_2.54mm:PinHeader_2x03_P2.54mm_Vertical, F.Cu at (247.8, 102.3)
- added J13: E1, footprint-lib:b4b-ph-kl,stepper_terminal, F.Cu at (240.8, 102.6)
- added J14: HEATBED, footprint-lib:mpt_0,5%2f2-2,54,heatbed, F.Cu at (309.5, 113.4)
- added J15: X_MIN, footprint-lib:b3b-ph-kl,end_stop, F.Cu at (317.7, 70.5)
- added J16: X_MAX, footprint-lib:b3b-ph-kl,end_stop, F.Cu at (317.7, 75.6)
- added J17: Y_MIN, footprint-lib:b3b-ph-kl,end_stop, F.Cu at (326.1, 70.5)
- added J18: Y_MAX, footprint-lib:b3b-ph-kl,end_stop, F.Cu at (326.1, 75.6)
- added J19: Z_MIN, footprint-lib:b3b-ph-kl,end_stop, F.Cu at (334.5, 70.5)
- added J2: MS_SELECT, Connector_PinHeader_2.54mm:PinHeader_2x03_P2.54mm_Vertical, F.Cu at (167.5, 102.3)
- added J20: Z_MAX, footprint-lib:b3b-ph-kl,end_stop, F.Cu at (334.5, 75.6)
- added J21: HEATBED_TEMP, w_conn_jst-ph:b2b-ph-kl, F.Cu at (281.1, 134.1)
- added J22: HOTEND_TEMP0, w_conn_jst-ph:b2b-ph-kl, F.Cu at (281.1, 129.1)
- added J23: HOTEND_TEMP1, w_conn_jst-ph:b2b-ph-kl, F.Cu at (287.4, 129.1)
- added J24: AUX_TEMP, w_conn_jst-ph:b2b-ph-kl, F.Cu at (287.4, 134.1)
- added J25: 12V_INPUT_2, footprint-lib:mpt_0,5%2f2-2,54,12V_SRC, F.Cu at (245.3, 130.8)
- added J26: 12V_INPUT, footprint-lib:mpt_0,5%2f2-2,54,12V_SRC, F.Cu at (239.3, 130.8)
- added J27: 12V_OUT, footprint-lib:mpt_0,5%2f2-2,54,12V_SRC, F.Cu at (233.3, 130.8)
- added J28: SWD, Connector_PinHeader_1.27mm:PinHeader_1x04_P1.27mm_Vertical, F.Cu at (307.2, 69.6)
- added J29: USB_DEBUG, Connector_PinHeader_1.27mm:PinHeader_1x05_P1.27mm_Vertical, F.Cu at (157.4, 149.5)
- added J3: X, footprint-lib:b4b-ph-kl,stepper_terminal, F.Cu at (160.5, 102.6)
- added J30: PWR_DEBUG, Connector_PinHeader_1.27mm:PinHeader_1x05_P1.27mm_Vertical, F.Cu at (141.1, 149.5)
- added J31: HOT_END, footprint-lib:mpt_0,5%2f2-2,54,heatbed, F.Cu at (309.5, 96.8)
- added J32: HOT_END, footprint-lib:mpt_0,5%2f2-2,54,heatbed, F.Cu at (279.6, 116.8)
- added J33: TO FAN0, footprint-lib:b2b-ph-kl,fan_pwm_out, F.Cu at (267.2, 129.1)
- added J34: TO FAN1, footprint-lib:b2b-ph-kl,fan_pwm_out, F.Cu at (329.8, 46.6)
- added J35: TO FAN2, footprint-lib:b2b-ph-kl,fan_pwm_out, F.Cu at (267.2, 143.6)
- added J36: MS_SELECT, Connector_PinHeader_2.54mm:PinHeader_2x03_P2.54mm_Vertical, F.Cu at (264.7, 70.2)
- added J37: Z2, footprint-lib:b4b-ph-kl,stepper_terminal, F.Cu at (257.7, 70.5)
- added J38: MS_SELECT, Connector_PinHeader_2.54mm:PinHeader_2x03_P2.54mm_Vertical, F.Cu at (264.7, 46.3)
- added J39: Y, footprint-lib:b4b-ph-kl,stepper_terminal, F.Cu at (257.7, 46.6)
- added J4: MS_SELECT, Connector_PinHeader_2.54mm:PinHeader_2x03_P2.54mm_Vertical, F.Cu at (207.7, 102.3)
- added J40: Conn_01x07, Connector_PinHeader_1.27mm:PinHeader_1x07_P1.27mm_Vertical, F.Cu at (273.9, 93.4)
- added J41: EXP1, Connector_PinHeader_2.54mm:PinHeader_2x05_P2.54mm_Vertical, F.Cu at (261.8, 94.1)
- added J42: EXP2, Connector_PinHeader_2.54mm:PinHeader_2x05_P2.54mm_Vertical, F.Cu at (268.0, 94.1)
- added J7: Z1, footprint-lib:b4b-ph-kl,stepper_terminal, F.Cu at (160.5, 126.5)
- added J8: MS_SELECT, Connector_PinHeader_2.54mm:PinHeader_2x03_P2.54mm_Vertical, F.Cu at (207.6, 126.2)
- added J9: Z3, footprint-lib:b4b-ph-kl,stepper_terminal, F.Cu at (200.6, 126.5)
- added JP1: Jumper_NO_Small, Jumper:SolderJumper-2_P1.3mm_Open_TrianglePad1.0x1.5mm, F.Cu at (141.2, 95.7)
- added JP2: Jumper_NO_Small, Jumper:SolderJumper-2_P1.3mm_Open_TrianglePad1.0x1.5mm, F.Cu at (187.5, 54.7)
- added JP3: Jumper_NO_Small, Jumper:SolderJumper-2_P1.3mm_Open_TrianglePad1.0x1.5mm, F.Cu at (194.0, 45.8)
- added JP4: Jumper_NO_Small, Jumper:SolderJumper-2_P1.3mm_Open_TrianglePad1.0x1.5mm, F.Cu at (144.6, 94.1)
- added JP5: Jumper_NO_Small, SolderJumper-2_P1.3mm_Open_TrianglePad1.0x1.5mm, F.Cu at (221.4, 138.3)
- added JP6: Jumper_NO_Small, SolderJumper-2_P1.3mm_Open_TrianglePad1.0x1.5mm, F.Cu at (298.5, 84.0)
- added JP7: Jumper_NO_Small, SolderJumper-2_P1.3mm_Open_TrianglePad1.0x1.5mm, F.Cu at (305.2, 78.8)
- added L1: L_Small, w_smd_inductors:inductor_smd_0603, F.Cu at (301.3, 83.4)
- added L2: L_15uH, w_smd_inductors:inductor_smd_4.8x2.8mm, F.Cu at (327.2, 88.8)
- added L3: L_15uH, w_smd_inductors:inductor_smd_4.8x2.8mm, F.Cu at (229.9, 147.9)
- added Q1: WSK220N04, footprint-lib:TO-263-2,drill_array, F.Cu at (298.1, 112.6)
- added Q2: STP55NF06, footprint-lib:TO-263-2,drill_array, F.Cu at (298.1, 96.0)
- added Q3: STP55NF06, footprint-lib:TO-263-2,drill_array, F.Cu at (268.3, 116.0)
- added Q4: D882, footprint-lib:SOT-89-3,thermal_vias, F.Cu at (266.5, 134.6)
- added Q5: D882, footprint-lib:SOT-89-3,thermal_vias, F.Cu at (329.1, 52.2)
- added Q6: D882, footprint-lib:SOT-89-3,thermal_vias, F.Cu at (266.5, 149.2)
- added R1: R153,0603, Resistor_SMD:R_0603_1608Metric_Pad1.05x0.95mm_HandSolder, F.Cu at (238.4, 94.5)
- added R10: R103,0603, Resistor_SMD:R_0603_1608Metric_Pad1.05x0.95mm_HandSolder, F.Cu at (160.4, 115.4)
- added R11: R104,0603, Resistor_SMD:R_0603_1608Metric_Pad1.05x0.95mm_HandSolder, F.Cu at (197.2, 115.0)
- added R12: R102,0603, Resistor_SMD:R_0603_1608Metric_Pad1.05x0.95mm_HandSolder, F.Cu at (206.6, 109.9)
- added R13: R103,0603, Resistor_SMD:R_0603_1608Metric_Pad1.05x0.95mm_HandSolder, F.Cu at (200.5, 115.0)
- added R14: R104,0603, Resistor_SMD:R_0603_1608Metric_Pad1.05x0.95mm_HandSolder, F.Cu at (166.4, 133.9)
- added R15: R102,0603, Resistor_SMD:R_0603_1608Metric_Pad1.05x0.95mm_HandSolder, F.Cu at (157.0, 139.0)
- added R16: R103,0603, Resistor_SMD:R_0603_1608Metric_Pad1.05x0.95mm_HandSolder, F.Cu at (157.0, 140.5)
- added R17: R104,0603, Resistor_SMD:R_0603_1608Metric_Pad1.05x0.95mm_HandSolder, F.Cu at (197.1, 139.0)
- added R18: R102,0603, Resistor_SMD:R_0603_1608Metric_Pad1.05x0.95mm_HandSolder, F.Cu at (206.5, 133.9)
- added R19: R103,0603, Resistor_SMD:R_0603_1608Metric_Pad1.05x0.95mm_HandSolder, F.Cu at (200.4, 139.0)
- added R2: R153,0603, Resistor_SMD:R_0603_1608Metric_Pad1.05x0.95mm_HandSolder, F.Cu at (238.4, 93.0)
- added R20: R104,0603, Resistor_SMD:R_0603_1608Metric_Pad1.05x0.95mm_HandSolder, F.Cu at (303.7, 54.0)
- added R21: R102,0603, Resistor_SMD:R_0603_1608Metric_Pad1.05x0.95mm_HandSolder, F.Cu at (294.3, 60.6)
- added R22: R103,0603, Resistor_SMD:R_0603_1608Metric_Pad1.05x0.95mm_HandSolder, F.Cu at (294.3, 59.1)
- added R23: R104,0603, Resistor_SMD:R_0603_1608Metric_Pad1.05x0.95mm_HandSolder, F.Cu at (240.6, 115.0)
- added R24: R102,0603, Resistor_SMD:R_0603_1608Metric_Pad1.05x0.95mm_HandSolder, F.Cu at (246.7, 109.9)
- added R25: R103,0603, Resistor_SMD:R_0603_1608Metric_Pad1.05x0.95mm_HandSolder, F.Cu at (237.3, 116.6)
- added R26: R100,0805, Resistor_SMD:R_0805_2012Metric_Pad1.15x1.40mm_HandSolder, F.Cu at (308.3, 117.6)
- added R27: R104,0805, Resistor_SMD:R_0805_2012Metric_Pad1.15x1.40mm_HandSolder, F.Cu at (291.7, 119.3)
- added R28: R182,0603, Resistor_SMD:R_0603_1608Metric_Pad1.05x0.95mm_HandSolder, F.Cu at (298.6, 119.0)
- added R29: R102,0603, Resistor_SMD:R_0603_1608Metric_Pad1.05x0.95mm_HandSolder, F.Cu at (332.0, 82.3)
- added R3: R152,0603, Resistor_SMD:R_0603_1608Metric_Pad1.05x0.95mm_HandSolder, F.Cu at (241.7, 93.0)
- added R30: R102,0603, Resistor_SMD:R_0603_1608Metric_Pad1.05x0.95mm_HandSolder, F.Cu at (328.7, 79.3)
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Connections:
- net /Y_DIR renamed /Z1_~E1_STEP~PER_DRIVER/Z1_DIR
- net /Y_STEP renamed /Z1_~E1_STEP~PER_DRIVER/Z1_STEP
- C45 pad 1: GND -> +12V
- C45 pad 2: +3V3_STM32 -> GND
- J5 pad 2: +3V3_STM32 -> Net-(J5-Pad2)
- J5 pad 4: +3V3_STM32 -> Net-(J5-Pad4)
- J6 pad 2: Net-(J6-Pad2) -> +3V3
- J6 pad 4: Net-(J6-Pad4) -> +3V3
- R6 pad 1: GND -> /orange_pi/USB-DP2
- R6 pad 2: Net-(J5-Pad1) -> +3V3
- R78 pad 1: +3V3_STM32 -> Net-(R78-Pad1)
- R78 pad 2: Net-(D29-Pad2) -> GND
- R79 pad 1: +3V3_STM32 -> +3V3
- R79 pad 2: /~Y_EN~ -> Net-(R78-Pad1)
- U4 pad 1: /~Y_EN~ -> /Z1_~E1_STEP~PER_DRIVER/~Z1_EN~
- U4 pad 10: +3V3_STM32 -> +3V3
- U4 pad 11: Net-(J6-Pad4) -> Net-(J7-Pad4)
- U4 pad 12: Net-(J6-Pad3) -> Net-(J7-Pad3)
- U4 pad 13: Net-(J6-Pad2) -> Net-(J7-Pad2)
- U4 pad 14: Net-(J6-Pad1) -> Net-(J7-Pad1)
- U4 pad 2: Net-(J5-Pad1) -> Net-(J6-Pad1)
- U4 pad 3: Net-(J5-Pad3) -> Net-(J6-Pad3)
- U4 pad 4: Net-(J5-Pad5) -> Net-(J6-Pad5)
Other:
- board outline added: 100 x 100 mm

Commit message: update hotend footprint,
Parts:
- removed C1: CP100uf,35V, Capacitor_SMD:C_0603_1608Metric_Pad1.05x0.95mm_HandSolder
- removed C10, C12, C2, C39, C4, C6, C8: CP100uf,25V, Capacitor_SMD:CP_Elec_6.3x7.7
- removed C11, C13, C19, C21, C23, C25, C26, C27, C28, C3, C30, C31, C32, C40, C43, C46, C5, C51, C7, C9: C104,0603, Capacitor_SMD:C_0603_1608Metric_Pad1.05x0.95mm_HandSolder
- removed C14, C15, C16, C17, C18, C45, C50: C106,0603, Capacitor_SMD:C_0603_1608Metric_Pad1.05x0.95mm_HandSolder
- removed C20: CP100uf,35V, Capacitor_SMD:CP_Elec_6.3x7.7
- removed C22, C24: C10pf,0603, Capacitor_SMD:C_0603_1608Metric_Pad1.05x0.95mm_HandSolder
- removed C29: C105,0603, Capacitor_SMD:C_0603_1608Metric_Pad1.05x0.95mm_HandSolder
- removed C33, C34: CP220uf,16V, Capacitor_SMD:C_0603_1608Metric_Pad1.05x0.95mm_HandSolder
- removed C35: CP220uf,25V, Capacitor_SMD:C_0603_1608Metric_Pad1.05x0.95mm_HandSolder
- removed C36, C37, C38, C44: CP100uf,16V, Capacitor_SMD:CP_Elec_6.3x5.3
- removed C47, C52: C332,0603, Capacitor_SMD:C_0603_1608Metric_Pad1.05x0.95mm_HandSolder
- removed C48, C53: C103,0603, Capacitor_SMD:C_0603_1608Metric_Pad1.05x0.95mm_HandSolder
- removed C49, C54: C226,6.3v,0603, Capacitor_SMD:C_0603_1608Metric_Pad1.05x0.95mm_HandSolder
- removed D1: 5V HEALTHY, LED_SMD:LED_0603_1608Metric_Pad1.05x0.95mm_HandSolder
- removed D10, D11, D12, D13, D14, D2, D20, D21, D22, D23, D3, D4, D5, D6, D7, D9: LED_BLUE,0603, LED_SMD:LED_0603_1608Metric_Pad1.05x0.95mm_HandSolder
- removed D15, D16: SD_M4, Diode_SMD:D_SOD-323_HandSoldering
- removed D17: PB9, LED_SMD:LED_0603_1608Metric_Pad1.05x0.95mm_HandSolder
- removed D18, D19, D8: LED_RED,0603, LED_SMD:LED_0603_1608Metric_Pad1.05x0.95mm_HandSolder
- removed F1: 16V/30A, w_misc_comp:fuse_smf
- removed F2: 30V/5A, w_misc_comp:fuse_smf
- removed J1, J29: USB_DEBUG, Connector_PinHeader_1.27mm:PinHeader_1x05_P1.27mm_Vertical
- removed J10, J12, J2, J36, J4, J6, J8: MS_SELECT, Connector_PinHeader_2.54mm:PinHeader_2x03_P2.54mm_Vertical
- removed J11: E0, footprint-lib:b4b-ph-kl,stepper_terminal
- removed J13: E1, footprint-lib:b4b-ph-kl,stepper_terminal
- removed J14: HEATBED, footprint-lib:mpt_0,5%2f2-2,54,heatbed
- removed J15: X_MIN, footprint-lib:b3b-ph-kl,end_stop
- removed J16: X_MAX, footprint-lib:b3b-ph-kl,end_stop
- removed J17: Y_MIN, footprint-lib:b3b-ph-kl,end_stop
- removed J18: Y_MAX, footprint-lib:b3b-ph-kl,end_stop
- removed J19: Z_MIN, footprint-lib:b3b-ph-kl,end_stop
- removed J20: Z_MAX, footprint-lib:b3b-ph-kl,end_stop
- removed J21: HEATBED_TEMP, w_conn_jst-ph:b2b-ph-kl
- removed J22: HOTEND_TEMP0, w_conn_jst-ph:b2b-ph-kl
- removed J23: HOTEND_TEMP1, w_conn_jst-ph:b2b-ph-kl
- removed J24: AUX_TEMP, w_conn_jst-ph:b2b-ph-kl
- removed J25: 12V_INPUT_2, footprint-lib:mpt_0,5%2f2-2,54,12V_SRC
- removed J26: 12V_INPUT, footprint-lib:mpt_0,5%2f2-2,54,12V_SRC
- removed J27: 12V_OUT, footprint-lib:mpt_0,5%2f2-2,54,12V_SRC
- removed J28: SWD, Connector_PinHeader_1.27mm:PinHeader_1x04_P1.27mm_Vertical
- removed J3: X, footprint-lib:b4b-ph-kl,stepper_terminal
- removed J30: PWR_DEBUG, Connector_PinHeader_1.27mm:PinHeader_1x05_P1.27mm_Vertical
- removed J31, J32: HOT_END, footprint-lib:mpt_0,5%2f2-2,54,heatbed
- removed J33: TO FAN0, footprint-lib:b2b-ph-kl,fan_pwm_out
- removed J34: TO FAN1, footprint-lib:b2b-ph-kl,fan_pwm_out
- removed J35: TO FAN2, footprint-lib:b2b-ph-kl,fan_pwm_out
- removed J37: Z2, footprint-lib:b4b-ph-kl,stepper_terminal
- removed J40: Conn_01x07, Connector_PinHeader_1.27mm:PinHeader_1x07_P1.27mm_Vertical
- removed J41: EXP1, Connector_PinHeader_2.54mm:PinHeader_2x05_P2.54mm_Vertical
- removed J42: EXP2, Connector_PinHeader_2.54mm:PinHeader_2x05_P2.54mm_Vertical
- removed J5: Z, footprint-lib:b4b-ph-kl,stepper_terminal
- removed J7: Z1, footprint-lib:b4b-ph-kl,stepper_terminal
- removed J9: Z3, footprint-lib:b4b-ph-kl,stepper_terminal
- removed JP1, JP2, JP3, JP4: Jumper_NO_Small, Jumper:SolderJumper-2_P1.3mm_Open_TrianglePad1.0x1.5mm
- removed JP5, JP6, JP7: Jumper_NO_Small, SolderJumper-2_P1.3mm_Open_TrianglePad1.0x1.5mm
- removed L1: L_Small, w_smd_inductors:inductor_smd_0603
- removed L2, L3: L_15uH, w_smd_inductors:inductor_smd_4.8x2.8mm
- removed Q1: WSK220N04, footprint-lib:TO-263-2,drill_array
- removed Q2, Q3: STP55NF06, footprint-lib:TO-263-2,drill_array
- removed Q4, Q5, Q6: D882, footprint-lib:SOT-89-3,thermal_vias
- removed R1, R2: R153,0603, Resistor_SMD:R_0603_1608Metric_Pad1.05x0.95mm_HandSolder
- removed R10, R13, R16, R19, R22, R25, R45, R46, R70, R75, R78: R103,0603, Resistor_SMD:R_0603_1608Metric_Pad1.05x0.95mm_HandSolder
- removed R11, R14, R17, R20, R23, R68: R104,0603, Resistor_SMD:R_0603_1608Metric_Pad1.05x0.95mm_HandSolder
- removed R12, R15, R18, R21, R24, R29, R30, R31, R32, R33, R34, R44, R69, R7, R9: R102,0603, Resistor_SMD:R_0603_1608Metric_Pad1.05x0.95mm_HandSolder
- removed R26, R50, R53, R56, R60: R100,0805, Resistor_SMD:R_0805_2012Metric_Pad1.15x1.40mm_HandSolder
- removed R27, R51, R54, R57, R61, R65: R104,0805, Resistor_SMD:R_0805_2012Metric_Pad1.15x1.40mm_HandSolder
- removed R28, R52, R55, R59, R63, R67: R182,0603, Resistor_SMD:R_0603_1608Metric_Pad1.05x0.95mm_HandSolder
- removed R3, R49, R6: R152,0603, Resistor_SMD:R_0603_1608Metric_Pad1.05x0.95mm_HandSolder
- removed R35, R36, R37, R38, R39, R40, R41: R472,0603, Resistor_SMD:R_0603_1608Metric_Pad1.05x0.95mm_HandSolder
- removed R4, R47, R48, R5: R220,0603, Resistor_SMD:R_0603_1608Metric_Pad1.05x0.95mm_HandSolder
- removed R42, R43: R0,0603, Resistor_SMD:R_0603_1608Metric_Pad1.05x0.95mm_HandSolder
- removed R58, R62, R66: R100,0603, Resistor_SMD:R_0603_1608Metric_Pad1.05x0.95mm_HandSolder
- removed R64: R100,0805, Resistor_SMD:R_0603_1608Metric_Pad1.05x0.95mm_HandSolder
- removed R74, R77: R562,0603, Resistor_SMD:R_0603_1608Metric_Pad1.05x0.95mm_HandSolder
- removed R76, R79: R333,0603, Resistor_SMD:R_0603_1608Metric_Pad1.05x0.95mm_HandSolder
- removed R8: R104,0603, Resistor_SMD:R_0805_2012Metric_Pad1.15x1.40mm_HandSolder
- removed SW1: SW_Push, Button_Switch_SMD:SW_SPST_CK_RS282G05A3
- removed TH1: Thermistor_NTC, Resistor_SMD:R_0603_1608Metric_Pad1.05x0.95mm_HandSolder
- removed U1: orange_pi_zero, footprint-lib:orangepi-zero
- removed U11, U12: MP2303A_ALT, footprint-lib:SOIC-8_3.9x4.9mm_P1.27mm,thermal_via
- removed U2, U3, U4, U5, U6, U7, U9: A4988_MODULE, footprint-lib:Pololu_Breakout-16_15.2x20.3mm
- removed U8: STM32F407VET6, w_smd_lqfp:TQFP-100
- removed Y1: O_8M, Crystal:Crystal_HC49-4H_Vertical
- R72: moved to B.Cu
- moved J38 222.5 mm to (42.2, 53.0)
- moved C42 215.4 mm to (48.2, 52.2), turned to 90 degrees
- moved J39 214.2 mm to (45.0, 72.0)
- moved C41 212.6 mm to (45.0, 65.8)
- moved R71 209.3 mm to (48.2, 56.0), turned to 270 degrees
- moved R73 205.9 mm to (48.2, 59.8), turned to 270 degrees
- moved D24 203.5 mm to (51.2, 72.5), turned to 90 degrees
- moved R72 203.3 mm to (51.2, 72.5), turned to 90 degrees
- moved U10 199.6 mm to (38.7, 50.5)

Commit message: update,
Parts:
- removed H1, H2, H3, H4: MOUNT_M3, MountingHole:MountingHole_2.7mm_M2.5
- moved C41 59.6 mm to (9.00, 18.2)
- moved C42 59.6 mm to (12.2, 4.75)
- moved D24 59.6 mm to (15.2, 25.0)
- moved J38 59.6 mm to (6.25, 5.50)
- moved J39 59.6 mm to (9.00, 24.5)
- moved R71 59.6 mm to (12.2, 8.50)
- moved R72 59.6 mm to (15.2, 25.0)
- moved R73 59.6 mm to (12.2, 12.2)
- moved U10 59.6 mm to (2.75, 3.05)
Connections:
- net +3V3 renamed +3V3_STM32
- net /Y_~E1_STEP~PER_DRIVER/Y_DIR renamed /Y_DIR
- net /Y_~E1_STEP~PER_DRIVER/Y_STEP renamed /Y_STEP
- net /Y_~E1_STEP~PER_DRIVER/~Y_EN~ renamed /~Y_EN~
Other:
- board outline removed

Commit message: update,
Parts:
- added C1: CP100uf,10V, Capacitor_SMD:CP_Elec_6.3x5.3, F.Cu at (76.3, 33.4)
- added C10: CP100uf,25V, Capacitor_SMD:CP_Elec_6.3x7.7, F.Cu at (9.23, 64.2)
- added C11: C104,0603, Capacitor_SMD:C_0603_1608Metric_Pad1.05x0.95mm_HandSolder, F.Cu at (20.6, 67.2)
- added C12: CP100uf,25V, Capacitor_SMD:CP_Elec_6.3x7.7, F.Cu at (9.23, 48.3)
- added C13: C104,0603, Capacitor_SMD:C_0603_1608Metric_Pad1.05x0.95mm_HandSolder, F.Cu at (16.8, 51.3)
- added C14: C106,0603, Capacitor_SMD:C_0603_1608Metric_Pad1.05x0.95mm_HandSolder, B.Cu at (2.75, 31.8)
- added C15: C106,0603, Capacitor_SMD:C_0603_1608Metric_Pad1.05x0.95mm_HandSolder, B.Cu at (10.0, 31.8)
- added C16: C106,0603, Capacitor_SMD:C_0603_1608Metric_Pad1.05x0.95mm_HandSolder, B.Cu at (16.8, 31.8)
- added C17: C106,0603, Capacitor_SMD:C_0603_1608Metric_Pad1.05x0.95mm_HandSolder, B.Cu at (23.5, 31.8)
- added C18: C106,0603, Capacitor_SMD:C_0603_1608Metric_Pad1.05x0.95mm_HandSolder, B.Cu at (27.4, 20.1)
- added C19: C104,0603, Capacitor_SMD:C_0603_1608Metric_Pad1.05x0.95mm_HandSolder, F.Cu at (11.0, 1.75)
- added C2: CP100uf,25V, Capacitor_SMD:CP_Elec_6.3x7.7, F.Cu at (90.5, 90.2)
- added C20: CP100uf,35V, Capacitor_SMD:CP_Elec_6.3x7.7, F.Cu at (11.8, 9.35)
- added C21: C104,0603, Capacitor_SMD:C_0603_1608Metric_Pad1.05x0.95mm_HandSolder, B.Cu at (40.2, 69.8)
- added C22: C10pf,0603, Capacitor_SMD:C_0603_1608Metric_Pad1.05x0.95mm_HandSolder, B.Cu at (28.5, 62.2)
- added C23: C104,0603, Capacitor_SMD:C_0603_1608Metric_Pad1.05x0.95mm_HandSolder, B.Cu at (33.1, 60.3)
- added C24: C10pf,0603, Capacitor_SMD:C_0603_1608Metric_Pad1.05x0.95mm_HandSolder, B.Cu at (35.8, 69.2)
- added C25: C104,0603, Capacitor_SMD:C_0603_1608Metric_Pad1.05x0.95mm_HandSolder, B.Cu at (31.4, 56.1)
- added C26: C104,0603, Capacitor_SMD:C_0603_1608Metric_Pad1.05x0.95mm_HandSolder, B.Cu at (42.3, 47.9)
- added C27: C104,0603, Capacitor_SMD:C_0603_1608Metric_Pad1.05x0.95mm_HandSolder, B.Cu at (50.8, 58.5)
- added C28: C104,0603, Capacitor_SMD:C_0603_1608Metric_Pad1.05x0.95mm_HandSolder, B.Cu at (42.6, 66.6)
- added C29: C105,0603, Capacitor_SMD:C_0603_1608Metric_Pad1.05x0.95mm_HandSolder, B.Cu at (34.7, 61.9)
- added C3: C104,0603, Capacitor_SMD:C_0603_1608Metric_Pad1.05x0.95mm_HandSolder, F.Cu at (93.5, 74.8)
- added C30: C104,0603, Capacitor_SMD:C_0603_1608Metric_Pad1.05x0.95mm_HandSolder, B.Cu at (49.7, 59.6)
- added C31: C104,0603, Capacitor_SMD:C_0603_1608Metric_Pad1.05x0.95mm_HandSolder, B.Cu at (43.3, 49.0)
- added C32: C104,0603, Capacitor_SMD:C_0603_1608Metric_Pad1.05x0.95mm_HandSolder, B.Cu at (47.6, 68.0)
- added C36: CP1uf,50V, Capacitor_SMD:CP_Elec_4x5.3, F.Cu at (21.5, 13.8)
- added C37: CP1uf,50V, Capacitor_SMD:CP_Elec_4x5.3, F.Cu at (29.5, 13.8)
- added C38: CP1uf,50V, Capacitor_SMD:CP_Elec_4x5.3, F.Cu at (38.0, 13.8)
- added C39: CP100uf,25V, Capacitor_SMD:CP_Elec_6.3x7.7, F.Cu at (25.7, 90.2)
- added C4: CP100uf,25V, Capacitor_SMD:CP_Elec_6.3x7.7, F.Cu at (58.1, 90.2)
- added C40: C104,0603, Capacitor_SMD:C_0603_1608Metric_Pad1.05x0.95mm_HandSolder, F.Cu at (29.8, 78.6)
- added C43: C104,0603, Capacitor_SMD:C_0603_1608Metric_Pad1.05x0.95mm_HandSolder, F.Cu at (133.3, 61.4)
- added C44: CP100uf,16V, Capacitor_SMD:CP_Elec_6.3x5.3, F.Cu at (37.2, 21.0)
- added C45: C106,0603, Capacitor_SMD:C_0603_1608Metric_Pad1.05x0.95mm_HandSolder, F.Cu at (67.5, 33.5)
- added C46: C104,0603, Capacitor_SMD:C_0603_1608Metric_Pad1.05x0.95mm_HandSolder, F.Cu at (71.5, 40.0)
- added C47: C332,0603, Capacitor_SMD:C_0603_1608Metric_Pad1.05x0.95mm_HandSolder, F.Cu at (63.0, 41.0)
- added C48: C103,0603, Capacitor_SMD:C_0603_1608Metric_Pad1.05x0.95mm_HandSolder, F.Cu at (70.0, 32.5)
- added C49: C226,6.3v,0603, Capacitor_SMD:C_0603_1608Metric_Pad1.05x0.95mm_HandSolder, F.Cu at (63.0, 37.5)
- added C5: C104,0603, Capacitor_SMD:C_0603_1608Metric_Pad1.05x0.95mm_HandSolder, F.Cu at (61.5, 82.5)
- added C50: C106,0603, Capacitor_SMD:C_0603_1608Metric_Pad1.05x0.95mm_HandSolder, F.Cu at (48.2, 40.2)
- added C51: C104,0603, Capacitor_SMD:C_0603_1608Metric_Pad1.05x0.95mm_HandSolder, F.Cu at (43.5, 33.2)
- added C52: C332,0603, Capacitor_SMD:C_0603_1608Metric_Pad1.05x0.95mm_HandSolder, F.Cu at (49.2, 30.0)
- added C53: C103,0603, Capacitor_SMD:C_0603_1608Metric_Pad1.05x0.95mm_HandSolder, F.Cu at (45.5, 40.8)
- added C54: C226,6.3v,0603, Capacitor_SMD:C_0603_1608Metric_Pad1.05x0.95mm_HandSolder, F.Cu at (52.3, 35.5)
- added C55: C105,0603, Capacitor_SMD:C_0603_1608Metric_Pad1.05x0.95mm_HandSolder, B.Cu at (38.7, 65.9)
- added C6: CP100uf,25V, Capacitor_SMD:CP_Elec_6.3x7.7, F.Cu at (41.9, 90.2)
- added C7: C104,0603, Capacitor_SMD:C_0603_1608Metric_Pad1.05x0.95mm_HandSolder, F.Cu at (45.8, 78.6)
- added C8: CP100uf,25V, Capacitor_SMD:CP_Elec_6.3x7.7, F.Cu at (9.50, 90.2)
- added C9: C104,0603, Capacitor_SMD:C_0603_1608Metric_Pad1.05x0.95mm_HandSolder, F.Cu at (12.5, 82.5)
- added D1: 5V HEALTHY, LED_SMD:LED_0603_1608Metric_Pad1.05x0.95mm_HandSolder, F.Cu at (50.8, 70.8)
- added D10: LED_BLUE,0603, LED_SMD:LED_0603_1608Metric_Pad1.05x0.95mm_HandSolder, F.Cu at (91.9, 9.25)
- added D11: LED_BLUE,0603, LED_SMD:LED_0603_1608Metric_Pad1.05x0.95mm_HandSolder, F.Cu at (93.7, 9.30)
- added D12: LED_BLUE,0603, LED_SMD:LED_0603_1608Metric_Pad1.05x0.95mm_HandSolder, F.Cu at (95.4, 9.30)
- added D13: LED_BLUE,0603, LED_SMD:LED_0603_1608Metric_Pad1.05x0.95mm_HandSolder, F.Cu at (98.9, 9.30)
- added D14: LED_BLUE,0603, LED_SMD:LED_0603_1608Metric_Pad1.05x0.95mm_HandSolder, F.Cu at (97.2, 9.30)
- added D15: SD_M4, Diode_SMD:D_SOD-323_HandSoldering, F.Cu at (11.2, 3.75)
- added D16: SD_M4, Diode_SMD:D_SOD-323_HandSoldering, F.Cu at (21.4, 21.4)
- added D17: PB9, LED_SMD:LED_0603_1608Metric_Pad1.05x0.95mm_HandSolder, F.Cu at (30.3, 52.5)
- added D18: LED_RED,0603, LED_SMD:LED_0603_1608Metric_Pad1.05x0.95mm_HandSolder, F.Cu at (63.9, 5.50)
- added D19: LED_RED,0603, LED_SMD:LED_0603_1608Metric_Pad1.05x0.95mm_HandSolder, F.Cu at (75.8, 5.50)
- added D2: LED_BLUE,0603, LED_SMD:LED_0603_1608Metric_Pad1.05x0.95mm_HandSolder, F.Cu at (92.2, 97.7)
- added D20: LED_BLUE,0603, LED_SMD:LED_0603_1608Metric_Pad1.05x0.95mm_HandSolder, F.Cu at (25.1, 2.52)
- added D21: LED_BLUE,0603, LED_SMD:LED_0603_1608Metric_Pad1.05x0.95mm_HandSolder, F.Cu at (33.4, 2.52)
- added D22: LED_BLUE,0603, LED_SMD:LED_0603_1608Metric_Pad1.05x0.95mm_HandSolder, F.Cu at (41.8, 2.50)
- added D23: LED_BLUE,0603, LED_SMD:LED_0603_1608Metric_Pad1.05x0.95mm_HandSolder, F.Cu at (33.0, 97.7)
- added D3: LED_BLUE,0603, LED_SMD:LED_0603_1608Metric_Pad1.05x0.95mm_HandSolder, F.Cu at (63.1, 97.7)
- added D4: LED_BLUE,0603, LED_SMD:LED_0603_1608Metric_Pad1.05x0.95mm_HandSolder, F.Cu at (48.1, 97.7)
- added D5: LED_BLUE,0603, LED_SMD:LED_0603_1608Metric_Pad1.05x0.95mm_HandSolder, F.Cu at (17.8, 97.7)
- added D6: LED_BLUE,0603, LED_SMD:LED_0603_1608Metric_Pad1.05x0.95mm_HandSolder, F.Cu at (3.00, 70.5)
- added D7: LED_BLUE,0603, LED_SMD:LED_0603_1608Metric_Pad1.05x0.95mm_HandSolder, F.Cu at (3.00, 54.7)
- added D8: LED_RED,0603, LED_SMD:LED_0603_1608Metric_Pad1.05x0.95mm_HandSolder, F.Cu at (51.8, 5.50)
- added D9: LED_BLUE,0603, LED_SMD:LED_0603_1608Metric_Pad1.05x0.95mm_HandSolder, F.Cu at (90.2, 9.25)
- added F1: 16V/30A, w_misc_comp:fuse_smf, F.Cu at (11.8, 17.9)
- added F2: 30V/5A, w_misc_comp:fuse_smf, F.Cu at (11.8, 26.4)
- added H1: MOUNT_M3, MountingHole:MountingHole_2.7mm_M2.5, F.Cu at (3.00, 3.00)
- added H2: MOUNT_M3, MountingHole:MountingHole_2.7mm_M2.5, F.Cu at (97.0, 3.00)
- added H3: MOUNT_M3, MountingHole:MountingHole_2.7mm_M2.5, F.Cu at (3.00, 97.0)
- added H4: MOUNT_M3, MountingHole:MountingHole_2.7mm_M2.5, F.Cu at (97.0, 97.0)
- added J1: USB_DEBUG, Connector_PinHeader_1.27mm:PinHeader_1x05_P1.27mm_Vertical, F.Cu at (91.4, 65.4)
- added J10: MS_SELECT, Connector_PinHeader_2.54mm:PinHeader_2x03_P2.54mm_Vertical, F.Cu at (22.5, 61.2)
- added J11: E0, footprint-lib:b4b-ph-kl,stepper_terminal, F.Cu at (2.40, 64.2)
- added J12: MS_SELECT, Connector_PinHeader_2.54mm:PinHeader_2x03_P2.54mm_Vertical, F.Cu at (22.4, 45.3)
- added J13: E1, footprint-lib:b4b-ph-kl,stepper_terminal, F.Cu at (2.40, 48.2)
- added J14: HEATBED, footprint-lib:mpt_0,5%2f2-2,54,heatbed, F.Cu at (46.8, 3.00)
- added J15: X_MIN, footprint-lib:b3b-ph-kl,end_stop, F.Cu at (85.0, 2.25)
- added J16: X_MAX, footprint-lib:b3b-ph-kl,end_stop, F.Cu at (85.0, 8.00)
- added J17: Y_MIN, footprint-lib:b3b-ph-kl,end_stop, F.Cu at (85.0, 13.8)
- added J18: Y_MAX, footprint-lib:b3b-ph-kl,end_stop, F.Cu at (85.0, 19.5)
- added J19: Z_MIN, footprint-lib:b3b-ph-kl,end_stop, F.Cu at (94.5, 13.5)
- added J2: MS_SELECT, Connector_PinHeader_2.54mm:PinHeader_2x03_P2.54mm_Vertical, F.Cu at (87.5, 77.0)
- added J20: Z_MAX, footprint-lib:b3b-ph-kl,end_stop, F.Cu at (94.5, 19.5)
- added J21: HEATBED_TEMP, w_conn_jst-ph:b2b-ph-kl, F.Cu at (2.39, 36.2)
- added J22: HOTEND_TEMP0, w_conn_jst-ph:b2b-ph-kl, F.Cu at (9.26, 36.2)
- added J23: HOTEND_TEMP1, w_conn_jst-ph:b2b-ph-kl, F.Cu at (16.1, 36.2)
- added J24: AUX_TEMP, w_conn_jst-ph:b2b-ph-kl, F.Cu at (23.0, 36.2)
- added J25: 12V_INPUT_2, footprint-lib:mpt_0,5%2f2-2,54,12V_SRC, F.Cu at (3.25, 18.2)
- added J26: 12V_INPUT, footprint-lib:mpt_0,5%2f2-2,54,12V_SRC, F.Cu at (3.15, 26.4)
- added J27: 12V_OUT, footprint-lib:mpt_0,5%2f2-2,54,12V_SRC, F.Cu at (3.15, 10.2)
- added J28: SWD, Connector_PinHeader_1.27mm:PinHeader_1x04_P1.27mm_Vertical, F.Cu at (37.4, 42.6)
- added J29: USB_DEBUG, Connector_PinHeader_1.27mm:PinHeader_1x05_P1.27mm_Vertical, F.Cu at (33.4, 47.6)
- added J3: X, footprint-lib:b4b-ph-kl,stepper_terminal, F.Cu at (86.0, 97.3)
- added J30: PWR_DEBUG, Connector_PinHeader_1.27mm:PinHeader_1x05_P1.27mm_Vertical, F.Cu at (29.4, 42.8)
- added J31: HOT_END, footprint-lib:mpt_0,5%2f2-2,54,heatbed, F.Cu at (58.8, 3.00)
- added J32: HOT_END, footprint-lib:mpt_0,5%2f2-2,54,heatbed, F.Cu at (70.8, 3.00)
- added J33: TO FAN0, footprint-lib:b2b-ph-kl,fan_pwm_out, F.Cu at (21.0, 2.00)
- added J34: TO FAN1, footprint-lib:b2b-ph-kl,fan_pwm_out, F.Cu at (29.2, 2.00)
- added J35: TO FAN2, footprint-lib:b2b-ph-kl,fan_pwm_out, F.Cu at (37.5, 2.00)
- added J36: MS_SELECT, Connector_PinHeader_2.54mm:PinHeader_2x03_P2.54mm_Vertical, F.Cu at (22.7, 77.0)
- added J37: Z2, footprint-lib:b4b-ph-kl,stepper_terminal, F.Cu at (26.7, 97.3)
- added J4: MS_SELECT, Connector_PinHeader_2.54mm:PinHeader_2x03_P2.54mm_Vertical, F.Cu at (55.1, 77.0)
- added J40: Conn_01x07, Connector_PinHeader_1.27mm:PinHeader_1x07_P1.27mm_Vertical, F.Cu at (124.0, 61.8)
- added J41: EXP1, Connector_PinHeader_2.54mm:PinHeader_2x05_P2.54mm_Vertical, F.Cu at (39.0, 38.4)
- added J42: EXP2, Connector_PinHeader_2.54mm:PinHeader_2x05_P2.54mm_Vertical, F.Cu at (31.8, 38.4)
- added J5: Z, footprint-lib:b4b-ph-kl,stepper_terminal, F.Cu at (56.8, 97.3)
- added J6: MS_SELECT, Connector_PinHeader_2.54mm:PinHeader_2x03_P2.54mm_Vertical, F.Cu at (38.9, 77.0)
- added J7: Z1, footprint-lib:b4b-ph-kl,stepper_terminal, F.Cu at (41.8, 97.3)
- added J8: MS_SELECT, Connector_PinHeader_2.54mm:PinHeader_2x03_P2.54mm_Vertical, F.Cu at (6.50, 77.0)
- added J9: Z3, footprint-lib:b4b-ph-kl,stepper_terminal, F.Cu at (11.6, 97.3)
- added JP5: Jumper_NO_Small, SolderJumper-2_P1.3mm_Open_TrianglePad1.0x1.5mm, B.Cu at (8.55, 22.2)
- added JP6: Jumper_NO_Small, SolderJumper-2_P1.3mm_Open_TrianglePad1.0x1.5mm, B.Cu at (42.3, 58.2)
- added JP7: Jumper_NO_Small, SolderJumper-2_P1.3mm_Open_TrianglePad1.0x1.5mm, B.Cu at (44.2, 60.1)
- added JP8: SolderJumper_3_Open, Jumper:SolderJumper-3_P2.0mm_Open_TrianglePad1.0x1.5mm_NumberLabels, F.Cu at (128.6, 61.9)
- added L1: L_Small, w_smd_inductors:inductor_smd_0603, F.Cu at (40.2, 69.8)
- added L2: L_15uH, w_smd_inductors:inductor_smd_4.8x2.8mm, F.Cu at (61.8, 33.8)
- added L3: L_15uH, w_smd_inductors:inductor_smd_4.8x2.8mm, F.Cu at (53.5, 39.2)
- added Q1: WSK220N04, footprint-lib:TO-263-2,thermal_vias, F.Cu at (49.2, 15.0)
- added Q2: STP55NF06, footprint-lib:TO-263-2,thermal_vias, F.Cu at (61.2, 15.0)
- added Q3: STP55NF06, footprint-lib:TO-263-2,thermal_vias, F.Cu at (73.2, 15.0)
- added Q4: D882, footprint-lib:SOT-89-3,thermal_vias, F.Cu at (21.1, 8.00)
- added Q5: D882, footprint-lib:SOT-89-3,thermal_vias, F.Cu at (29.2, 8.00)
- added Q6: D882, footprint-lib:SOT-89-3,thermal_vias, F.Cu at (37.8, 8.00)
- added R1: R153,0603, Resistor_SMD:R_0603_1608Metric_Pad1.05x0.95mm_HandSolder, F.Cu at (76.2, 61.5)
- added R10: R103,0603, Resistor_SMD:R_0603_1608Metric_Pad1.05x0.95mm_HandSolder, F.Cu at (93.5, 82.5)
- added R11: R104,0603, Resistor_SMD:R_0603_1608Metric_Pad1.05x0.95mm_HandSolder, F.Cu at (61.5, 78.6)
- added R12: R102,0603, Resistor_SMD:R_0603_1608Metric_Pad1.05x0.95mm_HandSolder, B.Cu at (63.1, 97.7)
- added R13: R103,0603, Resistor_SMD:R_0603_1608Metric_Pad1.05x0.95mm_HandSolder, F.Cu at (61.5, 74.8)
- added R14: R104,0603, Resistor_SMD:R_0603_1608Metric_Pad1.05x0.95mm_HandSolder, F.Cu at (45.8, 74.8)
- added R15: R102,0603, Resistor_SMD:R_0603_1608Metric_Pad1.05x0.95mm_HandSolder, B.Cu at (48.0, 97.7)
- added R16: R103,0603, Resistor_SMD:R_0603_1608Metric_Pad1.05x0.95mm_HandSolder, F.Cu at (45.8, 82.5)
- added R17: R104,0603, Resistor_SMD:R_0603_1608Metric_Pad1.05x0.95mm_HandSolder, F.Cu at (12.5, 78.6)
- added R18: R102,0603, Resistor_SMD:R_0603_1608Metric_Pad1.05x0.95mm_HandSolder, B.Cu at (17.8, 97.7)
- added R19: R103,0603, Resistor_SMD:R_0603_1608Metric_Pad1.05x0.95mm_HandSolder, F.Cu at (12.5, 74.8)
- added R2: R153,0603, Resistor_SMD:R_0603_1608Metric_Pad1.05x0.95mm_HandSolder, F.Cu at (78.2, 61.5)
- added R20: R104,0603, Resistor_SMD:R_0603_1608Metric_Pad1.05x0.95mm_HandSolder, F.Cu at (24.4, 67.2)
- added R21: R102,0603, Resistor_SMD:R_0603_1608Metric_Pad1.05x0.95mm_HandSolder, B.Cu at (3.00, 70.5)
- added R22: R103,0603, Resistor_SMD:R_0603_1608Metric_Pad1.05x0.95mm_HandSolder, F.Cu at (16.8, 67.2)
- added R23: R104,0603, Resistor_SMD:R_0603_1608Metric_Pad1.05x0.95mm_HandSolder, F.Cu at (20.6, 51.3)
- added R24: R102,0603, Resistor_SMD:R_0603_1608Metric_Pad1.05x0.95mm_HandSolder, F.Cu at (24.4, 51.3)
- added R25: R103,0603, Resistor_SMD:R_0603_1608Metric_Pad1.05x0.95mm_HandSolder, B.Cu at (3.00, 54.7)
- added R26: R100,0805, Resistor_SMD:R_0805_2012Metric_Pad1.15x1.40mm_HandSolder, B.Cu at (46.8, 19.5)
- added R27: R104,0805, Resistor_SMD:R_0805_2012Metric_Pad1.15x1.40mm_HandSolder, B.Cu at (51.8, 19.5)
- added R28: R182,0603, Resistor_SMD:R_0603_1608Metric_Pad1.05x0.95mm_HandSolder, B.Cu at (51.8, 5.50)
- added R29: R102,0603, Resistor_SMD:R_0603_1608Metric_Pad1.05x0.95mm_HandSolder, B.Cu at (90.2, 9.25)
- added R30: R102,0603, Resistor_SMD:R_0603_1608Metric_Pad1.05x0.95mm_HandSolder, B.Cu at (91.9, 9.25)
- added R31: R102,0603, Resistor_SMD:R_0603_1608Metric_Pad1.05x0.95mm_HandSolder, B.Cu at (93.7, 9.30)
- added R32: R102,0603, Resistor_SMD:R_0603_1608Metric_Pad1.05x0.95mm_HandSolder, B.Cu at (95.4, 9.30)
- added R33: R102,0603, Resistor_SMD:R_0603_1608Metric_Pad1.05x0.95mm_HandSolder, B.Cu at (98.9, 9.30)
- added R34: R102,0603, Resistor_SMD:R_0603_1608Metric_Pad1.05x0.95mm_HandSolder, B.Cu at (97.2, 9.30)
- added R35: R472,0603, Resistor_SMD:R_0603_1608Metric_Pad1.05x0.95mm_HandSolder, F.Cu at (2.75, 31.8)
- added R36: R472,0603, Resistor_SMD:R_0603_1608Metric_Pad1.05x0.95mm_HandSolder, F.Cu at (10.0, 31.8)
- added R37: R472,0603, Resistor_SMD:R_0603_1608Metric_Pad1.05x0.95mm_HandSolder, F.Cu at (16.8, 31.8)
- added R38: R472,0603, Resistor_SMD:R_0603_1608Metric_Pad1.05x0.95mm_HandSolder, F.Cu at (23.5, 31.8)
- added R39: R472,0603, Resistor_SMD:R_0603_1608Metric_Pad1.05x0.95mm_HandSolder, F.Cu at (27.4, 20.1)
- added R4: R220,0603, Resistor_SMD:R_0603_1608Metric_Pad1.05x0.95mm_HandSolder, B.Cu at (86.1, 70.8)
- added R40: R472,0603, Resistor_SMD:R_0603_1608Metric_Pad1.05x0.95mm_HandSolder, B.Cu at (44.6, 55.9)
- added R41: R472,0603, Resistor_SMD:R_0603_1608Metric_Pad1.05x0.95mm_HandSolder, B.Cu at (46.5, 57.8)
- added R42: R0,0603, Resistor_SMD:R_0603_1608Metric_Pad1.05x0.95mm_HandSolder, B.Cu at (37.7, 64.9)
- added R43: R0,0603, Resistor_SMD:R_0603_1608Metric_Pad1.05x0.95mm_HandSolder, B.Cu at (36.6, 63.8)
- added R44: R102,0603, Resistor_SMD:R_0603_1608Metric_Pad1.05x0.95mm_HandSolder, B.Cu at (30.3, 52.5)
- added R45: R103,0603, Resistor_SMD:R_0603_1608Metric_Pad1.05x0.95mm_HandSolder, B.Cu at (40.2, 56.0)
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Connections:
- net +3V3_STM32 renamed +3V3
- net /Y_DIR renamed /Y_~E1_STEP~PER_DRIVER/Y_DIR
- net /Y_STEP renamed /Y_~E1_STEP~PER_DRIVER/Y_STEP
- net /~Y_EN~ renamed /Y_~E1_STEP~PER_DRIVER/~Y_EN~
- U10 pad 11: Net-(J39-Pad4) -> Net-(J39-Pad1)
- U10 pad 12: Net-(J39-Pad3) -> Net-(J39-Pad2)
- U10 pad 13: Net-(J39-Pad2) -> Net-(J39-Pad3)
- U10 pad 14: Net-(J39-Pad1) -> Net-(J39-Pad4)
Other:
- board outline added: 100 x 100 mm
