File: hardware/printer-board/Z3_STEPPER_DRIVER.kicad_pcb (KiCad board)
At the start: 2 copper layers, 100 x 100 mm, 13 parts, among them J8 MS_SELECT, J9 Z3, U5 A4988_MODULE

Commit message: update,
Parts:
- removed H1, H2, H3, H4: MOUNT_M3, MountingHole:MountingHole_2.7mm_M2.5
- moved C8 63.8 mm to (9.50, 18.0)
- moved C9 63.8 mm to (12.5, 11.0)
- moved D5 63.8 mm to (15.8, 25.0)
- moved J8 63.8 mm to (6.50, 5.50)
- moved J9 63.8 mm to (9.50, 24.5)
- moved R17 63.8 mm to (12.5, 7.50)
- moved R18 63.8 mm to (15.8, 25.0)
- moved R19 63.8 mm to (12.5, 3.87)
- moved U5 63.8 mm to (3.18, 2.95)
Other:
- board outline removed
Changed lines of the file:
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@@
   (general
     (thickness 1.6)
-    (drawings 8)
+    (drawings 0)
     (tracks 0)
     (zones 0)
-    (modules 13)
+    (modules 9)
     (nets 16)
   )
@@
   )
   (module Capacitor_SMD:CP_Elec_6.3x7.7 (layer F.Cu)
-    (at 45 71)
+    (at 9.5 18)
     (descr "SMD capacitor, aluminum electrolytic, Nichicon, 6.3x7.7mm")
     (tags "capacitor electrolytic")
@@
   )
   (module Capacitor_SMD:C_0603_1608Metric_Pad1.05x0.95mm_HandSolder (layer F.Cu)
-    (at 48 64 270)
+    (at 12.5 11 270)
     (descr "Capacitor SMD 0603 (1608 Metric), square (rectangular) end terminal, IPC_7351 nominal with elongated pad for handsoldering. (Body size source: http://www.tortai-tech.com/upload/download/2011102023233369053.pdf), generated with kicad-footprint-generator")
     (tags "capacitor handsolder")
@@
   )
   (module Connector_PinHeader_2.54mm:PinHeader_2x03_P2.54mm_Vertical (layer F.Cu)
-    (at 42 58.5)
+    (at 6.5 5.5)
     (descr "Through hole straight pin header, 2x03, 2.54mm pitch, double rows")
     (tags "Through hole pin header THT 2x03 2.54mm double row")
@@
   )
   (module LED_SMD:LED_0603_1608Metric_Pad1.05x0.95mm_HandSolder (layer F.Cu)
-    (at 51.25 78 90)
+    (at 15.75 25 90)
     (descr "LED SMD 0603 (1608 Metric), square (rectangular) end terminal, IPC_7351 nominal, (Body size source: http://www.tortai-tech.com/upload/download/2011102023233369053.pdf), generated with kicad-footprint-generator")
     (tags "LED handsolder")
@@
   )
   (module Resistor_SMD:R_0603_1608Metric_Pad1.05x0.95mm_HandSolder (layer F.Cu)
-    (at 48 56.874999 90)
+    (at 12.5 3.874999 90)
     (descr "Resistor SMD 0603 (1608 Metric), square (rectangular) end terminal, IPC_7351 nominal with elongated pad for handsoldering. (Body size source: http://www.tortai-tech.com/upload/download/2011102023233369053.pdf), generated with kicad-footprint-generator")
     (tags "resistor handsolder")
@@
   )
   (module Resistor_SMD:R_0603_1608Metric_Pad1.05x0.95mm_HandSolder (layer B.Cu)
-    (at 51.25 78 90)
+    (at 15.75 25 90)
     (descr "Resistor SMD 0603 (1608 Metric), square (rectangular) end terminal, IPC_7351 nominal with elongated pad for handsoldering. (Body size source: http://www.tortai-tech.com/upload/download/2011102023233369053.pdf), generated with kicad-footprint-generator")
     (tags "resistor handsolder")
@@
   )
   (module Resistor_SMD:R_0603_1608Metric_Pad1.05x0.95mm_HandSolder (layer F.Cu)
-    (at 48 60.5 90)
+    (at 12.5 7.5 90)
     (descr "Resistor SMD 0603 (1608 Metric), square (rectangular) end terminal, IPC_7351 nominal with elongated pad for handsoldering. (Body size source: http://www.tortai-tech.com/upload/download/2011102023233369053.pdf), generated with kicad-footprint-generator")
     (tags "resistor handsolder")
@@
   )
   (module footprint-lib:Pololu_Breakout-16_15.2x20.3mm (layer F.Cu)
-    (at 38.675001 55.945001)
+    (at 3.175001 2.945001)
     (descr "Pololu Breakout 16-pin 15.2x20.3mm 0.6x0.8\\")
     (tags "Pololu Breakout")
@@
   )
   (module footprint-lib:b4b-ph-kl,stepper_terminal (layer F.Cu)
-    (at 45 77.5)
+    (at 9.5 24.5)
     (descr "JST PH series connector, B4B-PH-KL")
     (fp_text reference J9 (at 0 -2.99974) (layer F.SilkS)
@@
     )
   )
-  (module MountingHole:MountingHole_2.7mm_M2.5 locked (layer F.Cu)
-    (at 3 97)
-    (descr "Mounting Hole 2.7mm, no annular, M2.5")
-    (tags "mounting hole 2.7mm no annular m2.5")
-    (attr virtual)
-    (fp_text reference H3 (at 0 -3.7) (layer F.SilkS)
-      (effects (font (size 1 1) (thickness 0.15)))
-    )
-    (fp_text value MOUNT_M3 (at 0 3.7) (layer F.Fab)
-      (effects (font (size 1 1) (thickness 0.15)))
-    )
-    (fp_text user %R (at 0.3 0) (layer F.Fab)
-      (effects (font (size 1 1) (thickness 0.15)))
-    )
-    (fp_circle (center 0 0) (end 2.7 0) (layer Cmts.User) (width 0.15))
-    (fp_circle (center 0 0) (end 2.95 0) (layer F.CrtYd) (width 0.05))
-    (pad 1 np_thru_hole circle (at 0 0) (size 2.7 2.7) (drill 2.7) (layers *.Cu *.Mask))
-  )
-  (module MountingHole:MountingHole_2.7mm_M2.5 locked (layer F.Cu)
-    (at 97 97)
-    (descr "Mounting Hole 2.7mm, no annular, M2.5")
-    (tags "mounting hole 2.7mm no annular m2.5")
-    (attr virtual)
-    (fp_text reference H4 (at 0 -3.7) (layer F.SilkS)
-      (effects (font (size 1 1) (thickness 0.15)))
-    )
-    (fp_text value MOUNT_M3 (at 0 3.7) (layer F.Fab)
-      (effects (font (size 1 1) (thickness 0.15)))
-    )
-    (fp_text user %R (at 0.3 0) (layer F.Fab)
-      (effects (font (size 1 1) (thickness 0.15)))
-    )
-    (fp_circle (center 0 0) (end 2.7 0) (layer Cmts.User) (width 0.15))
-    (fp_circle (center 0 0) (end 2.95 0) (layer F.CrtYd) (width 0.05))
-    (pad 1 np_thru_hole circle (at 0 0) (size 2.7 2.7) (drill 2.7) (layers *.Cu *.Mask))
-  )
-  (module MountingHole:MountingHole_2.7mm_M2.5 locked (layer F.Cu)
-    (at 3 3)
-    (descr "Mounting Hole 2.7mm, no annular, M2.5")
-    (tags "mounting hole 2.7mm no annular m2.5")
-    (attr virtual)
-    (fp_text reference H1 (at 0 -3.7) (layer F.SilkS)
-      (effects (font (size 1 1) (thickness 0.15)))
-    )
-    (fp_text value MOUNT_M3 (at 0 3.7) (layer F.Fab)
-      (effects (font (size 1 1) (thickness 0.15)))
-    )
-    (fp_text user %R (at 0.3 0) (layer F.Fab)
-      (effects (font (size 1 1) (thickness 0.15)))
-    )
-    (fp_circle (center 0 0) (end 2.7 0) (layer Cmts.User) (width 0.15))
-    (fp_circle (center 0 0) (end 2.95 0) (layer F.CrtYd) (width 0.05))
-    (pad 1 np_thru_hole circle (at 0 0) (size 2.7 2.7) (drill 2.7) (layers *.Cu *.Mask))
-  )
-  (module MountingHole:MountingHole_2.7mm_M2.5 locked (layer F.Cu)
-    (at 97 3)
-    (descr "Mounting Hole 2.7mm, no annular, M2.5")
-    (tags "mounting hole 2.7mm no annular m2.5")
-    (attr virtual)
-    (fp_text reference H2 (at 0 -3.7) (layer F.SilkS)
-      (effects (font (size 1 1) (thickness 0.15)))
-    )
-    (fp_text value MOUNT_M3 (at 0 3.7) (layer F.Fab)
-      (effects (font (size 1 1) (thickness 0.15)))
-    )
-    (fp_circle (center 0 0) (end 2.95 0) (layer F.CrtYd) (width 0.05))
-    (fp_circle (center 0 0) (end 2.7 0) (layer Cmts.User) (width 0.15))
-    (fp_text user %R (at 0.3 0) (layer F.Fab)
-      (effects (font (size 1 1) (thickness 0.15)))
-    )
-    (pad 1 np_thru_hole circle (at 0 0) (size 2.7 2.7) (drill 2.7) (layers *.Cu *.Mask))
-  )
-  (gr_arc (start 2.5 97.5) (end 0 97.5) (angle -90) (layer Edge.Cuts) (width 0.15))
-  (gr_arc (start 97.5 97.5) (end 97.5 100) (angle -90) (layer Edge.Cuts) (width 0.15))
-  (gr_arc (start 97.5 2.5) (end 100 2.5) (angle -90) (layer Edge.Cuts) (width 0.15))
-  (gr_arc (start 2.5 2.5) (end 2.5 0) (angle -90) (layer Edge.Cuts) (width 0.15))
-  (gr_line (start 97.5 0) (end 2.5 0) (layer Edge.Cuts) (width 0.15))
-  (gr_line (start 100 97.5) (end 100 2.5) (layer Edge.Cuts) (width 0.15))
-  (gr_line (start 2.5 100) (end 97.5 100) (layer Edge.Cuts) (width 0.15))
-  (gr_line (start 0 2.5) (end 0 97.5) (layer Edge.Cuts) (width 0.15))
 )

Commit message: update,
Parts:
- added C1: CP100uf,10V, Capacitor_SMD:CP_Elec_6.3x5.3, F.Cu at (76.3, 33.4)
- added C10: CP100uf,25V, Capacitor_SMD:CP_Elec_6.3x7.7, F.Cu at (9.23, 64.2)
- added C11: C104,0603, Capacitor_SMD:C_0603_1608Metric_Pad1.05x0.95mm_HandSolder, F.Cu at (20.6, 67.2)
- added C12: CP100uf,25V, Capacitor_SMD:CP_Elec_6.3x7.7, F.Cu at (9.23, 48.3)
- added C13: C104,0603, Capacitor_SMD:C_0603_1608Metric_Pad1.05x0.95mm_HandSolder, F.Cu at (16.8, 51.3)
- added C14: C106,0603, Capacitor_SMD:C_0603_1608Metric_Pad1.05x0.95mm_HandSolder, B.Cu at (2.75, 31.8)
- added C15: C106,0603, Capacitor_SMD:C_0603_1608Metric_Pad1.05x0.95mm_HandSolder, B.Cu at (10.0, 31.8)
- added C16: C106,0603, Capacitor_SMD:C_0603_1608Metric_Pad1.05x0.95mm_HandSolder, B.Cu at (16.8, 31.8)
- added C17: C106,0603, Capacitor_SMD:C_0603_1608Metric_Pad1.05x0.95mm_HandSolder, B.Cu at (23.5, 31.8)
- added C18: C106,0603, Capacitor_SMD:C_0603_1608Metric_Pad1.05x0.95mm_HandSolder, B.Cu at (27.4, 20.1)
- added C19: C104,0603, Capacitor_SMD:C_0603_1608Metric_Pad1.05x0.95mm_HandSolder, F.Cu at (11.0, 1.75)
- added C2: CP100uf,25V, Capacitor_SMD:CP_Elec_6.3x7.7, F.Cu at (90.5, 90.2)
- added C20: CP100uf,35V, Capacitor_SMD:CP_Elec_6.3x7.7, F.Cu at (11.8, 9.35)
- added C21: C104,0603, Capacitor_SMD:C_0603_1608Metric_Pad1.05x0.95mm_HandSolder, B.Cu at (40.2, 69.8)
- added C22: C10pf,0603, Capacitor_SMD:C_0603_1608Metric_Pad1.05x0.95mm_HandSolder, B.Cu at (28.5, 62.2)
- added C23: C104,0603, Capacitor_SMD:C_0603_1608Metric_Pad1.05x0.95mm_HandSolder, B.Cu at (33.1, 60.3)
- added C24: C10pf,0603, Capacitor_SMD:C_0603_1608Metric_Pad1.05x0.95mm_HandSolder, B.Cu at (35.8, 69.2)
- added C25: C104,0603, Capacitor_SMD:C_0603_1608Metric_Pad1.05x0.95mm_HandSolder, B.Cu at (31.4, 56.1)
- added C26: C104,0603, Capacitor_SMD:C_0603_1608Metric_Pad1.05x0.95mm_HandSolder, B.Cu at (42.3, 47.9)
- added C27: C104,0603, Capacitor_SMD:C_0603_1608Metric_Pad1.05x0.95mm_HandSolder, B.Cu at (50.8, 58.5)
- added C28: C104,0603, Capacitor_SMD:C_0603_1608Metric_Pad1.05x0.95mm_HandSolder, B.Cu at (42.6, 66.6)
- added C29: C105,0603, Capacitor_SMD:C_0603_1608Metric_Pad1.05x0.95mm_HandSolder, B.Cu at (34.7, 61.9)
- added C3: C104,0603, Capacitor_SMD:C_0603_1608Metric_Pad1.05x0.95mm_HandSolder, F.Cu at (93.5, 74.8)
- added C30: C104,0603, Capacitor_SMD:C_0603_1608Metric_Pad1.05x0.95mm_HandSolder, B.Cu at (49.7, 59.6)
- added C31: C104,0603, Capacitor_SMD:C_0603_1608Metric_Pad1.05x0.95mm_HandSolder, B.Cu at (43.3, 49.0)
- added C32: C104,0603, Capacitor_SMD:C_0603_1608Metric_Pad1.05x0.95mm_HandSolder, B.Cu at (47.6, 68.0)
- added C36: CP1uf,50V, Capacitor_SMD:CP_Elec_4x5.3, F.Cu at (21.5, 13.8)
- added C37: CP1uf,50V, Capacitor_SMD:CP_Elec_4x5.3, F.Cu at (29.5, 13.8)
- added C38: CP1uf,50V, Capacitor_SMD:CP_Elec_4x5.3, F.Cu at (38.0, 13.8)
- added C39: CP100uf,25V, Capacitor_SMD:CP_Elec_6.3x7.7, F.Cu at (25.7, 90.2)
- added C4: CP100uf,25V, Capacitor_SMD:CP_Elec_6.3x7.7, F.Cu at (58.1, 90.2)
- added C40: C104,0603, Capacitor_SMD:C_0603_1608Metric_Pad1.05x0.95mm_HandSolder, F.Cu at (29.8, 78.6)
- added C41: CP100uf,25V, Capacitor_SMD:CP_Elec_6.3x7.7, F.Cu at (74.3, 90.2)
- added C42: C104,0603, Capacitor_SMD:C_0603_1608Metric_Pad1.05x0.95mm_HandSolder, F.Cu at (77.8, 74.8)
- added C43: C104,0603, Capacitor_SMD:C_0603_1608Metric_Pad1.05x0.95mm_HandSolder, F.Cu at (133.3, 61.4)
- added C44: CP100uf,16V, Capacitor_SMD:CP_Elec_6.3x5.3, F.Cu at (37.2, 21.0)
- added C45: C106,0603, Capacitor_SMD:C_0603_1608Metric_Pad1.05x0.95mm_HandSolder, F.Cu at (67.5, 33.5)
- added C46: C104,0603, Capacitor_SMD:C_0603_1608Metric_Pad1.05x0.95mm_HandSolder, F.Cu at (71.5, 40.0)
- added C47: C332,0603, Capacitor_SMD:C_0603_1608Metric_Pad1.05x0.95mm_HandSolder, F.Cu at (63.0, 41.0)
- added C48: C103,0603, Capacitor_SMD:C_0603_1608Metric_Pad1.05x0.95mm_HandSolder, F.Cu at (70.0, 32.5)
- added C49: C226,6.3v,0603, Capacitor_SMD:C_0603_1608Metric_Pad1.05x0.95mm_HandSolder, F.Cu at (63.0, 37.5)
- added C5: C104,0603, Capacitor_SMD:C_0603_1608Metric_Pad1.05x0.95mm_HandSolder, F.Cu at (61.5, 82.5)
- added C50: C106,0603, Capacitor_SMD:C_0603_1608Metric_Pad1.05x0.95mm_HandSolder, F.Cu at (48.2, 40.2)
- added C51: C104,0603, Capacitor_SMD:C_0603_1608Metric_Pad1.05x0.95mm_HandSolder, F.Cu at (43.5, 33.2)
- added C52: C332,0603, Capacitor_SMD:C_0603_1608Metric_Pad1.05x0.95mm_HandSolder, F.Cu at (49.2, 30.0)
- added C53: C103,0603, Capacitor_SMD:C_0603_1608Metric_Pad1.05x0.95mm_HandSolder, F.Cu at (45.5, 40.8)
- added C54: C226,6.3v,0603, Capacitor_SMD:C_0603_1608Metric_Pad1.05x0.95mm_HandSolder, F.Cu at (52.3, 35.5)
- added C55: C105,0603, Capacitor_SMD:C_0603_1608Metric_Pad1.05x0.95mm_HandSolder, B.Cu at (38.7, 65.9)
- added C6: CP100uf,25V, Capacitor_SMD:CP_Elec_6.3x7.7, F.Cu at (41.9, 90.2)
- added C7: C104,0603, Capacitor_SMD:C_0603_1608Metric_Pad1.05x0.95mm_HandSolder, F.Cu at (45.8, 78.6)
- added D1: 5V HEALTHY, LED_SMD:LED_0603_1608Metric_Pad1.05x0.95mm_HandSolder, F.Cu at (50.8, 70.8)
- added D10: LED_BLUE,0603, LED_SMD:LED_0603_1608Metric_Pad1.05x0.95mm_HandSolder, F.Cu at (91.9, 9.25)
- added D11: LED_BLUE,0603, LED_SMD:LED_0603_1608Metric_Pad1.05x0.95mm_HandSolder, F.Cu at (93.7, 9.30)
- added D12: LED_BLUE,0603, LED_SMD:LED_0603_1608Metric_Pad1.05x0.95mm_HandSolder, F.Cu at (95.4, 9.30)
- added D13: LED_BLUE,0603, LED_SMD:LED_0603_1608Metric_Pad1.05x0.95mm_HandSolder, F.Cu at (98.9, 9.30)
- added D14: LED_BLUE,0603, LED_SMD:LED_0603_1608Metric_Pad1.05x0.95mm_HandSolder, F.Cu at (97.2, 9.30)
- added D15: SD_M4, Diode_SMD:D_SOD-323_HandSoldering, F.Cu at (11.2, 3.75)
- added D16: SD_M4, Diode_SMD:D_SOD-323_HandSoldering, F.Cu at (21.4, 21.4)
- added D17: PB9, LED_SMD:LED_0603_1608Metric_Pad1.05x0.95mm_HandSolder, F.Cu at (30.3, 52.5)
- added D18: LED_RED,0603, LED_SMD:LED_0603_1608Metric_Pad1.05x0.95mm_HandSolder, F.Cu at (63.9, 5.50)
- added D19: LED_RED,0603, LED_SMD:LED_0603_1608Metric_Pad1.05x0.95mm_HandSolder, F.Cu at (75.8, 5.50)
- added D2: LED_BLUE,0603, LED_SMD:LED_0603_1608Metric_Pad1.05x0.95mm_HandSolder, F.Cu at (92.2, 97.7)
- added D20: LED_BLUE,0603, LED_SMD:LED_0603_1608Metric_Pad1.05x0.95mm_HandSolder, F.Cu at (25.1, 2.52)
- added D21: LED_BLUE,0603, LED_SMD:LED_0603_1608Metric_Pad1.05x0.95mm_HandSolder, F.Cu at (33.4, 2.52)
- added D22: LED_BLUE,0603, LED_SMD:LED_0603_1608Metric_Pad1.05x0.95mm_HandSolder, F.Cu at (41.8, 2.50)
- added D23: LED_BLUE,0603, LED_SMD:LED_0603_1608Metric_Pad1.05x0.95mm_HandSolder, F.Cu at (33.0, 97.7)
- added D24: LED_BLUE,0603, LED_SMD:LED_0603_1608Metric_Pad1.05x0.95mm_HandSolder, F.Cu at (78.2, 97.7)
- added D3: LED_BLUE,0603, LED_SMD:LED_0603_1608Metric_Pad1.05x0.95mm_HandSolder, F.Cu at (63.1, 97.7)
- added D4: LED_BLUE,0603, LED_SMD:LED_0603_1608Metric_Pad1.05x0.95mm_HandSolder, F.Cu at (48.1, 97.7)
- added D6: LED_BLUE,0603, LED_SMD:LED_0603_1608Metric_Pad1.05x0.95mm_HandSolder, F.Cu at (3.00, 70.5)
- added D7: LED_BLUE,0603, LED_SMD:LED_0603_1608Metric_Pad1.05x0.95mm_HandSolder, F.Cu at (3.00, 54.7)
- added D8: LED_RED,0603, LED_SMD:LED_0603_1608Metric_Pad1.05x0.95mm_HandSolder, F.Cu at (51.8, 5.50)
- added D9: LED_BLUE,0603, LED_SMD:LED_0603_1608Metric_Pad1.05x0.95mm_HandSolder, F.Cu at (90.2, 9.25)
- added F1: 16V/30A, w_misc_comp:fuse_smf, F.Cu at (11.8, 17.9)
- added F2: 30V/5A, w_misc_comp:fuse_smf, F.Cu at (11.8, 26.4)
- added H1: MOUNT_M3, MountingHole:MountingHole_2.7mm_M2.5, F.Cu at (3.00, 3.00)
- added H2: MOUNT_M3, MountingHole:MountingHole_2.7mm_M2.5, F.Cu at (97.0, 3.00)
- added H3: MOUNT_M3, MountingHole:MountingHole_2.7mm_M2.5, F.Cu at (3.00, 97.0)
- added H4: MOUNT_M3, MountingHole:MountingHole_2.7mm_M2.5, F.Cu at (97.0, 97.0)
- added J1: USB_DEBUG, Connector_PinHeader_1.27mm:PinHeader_1x05_P1.27mm_Vertical, F.Cu at (91.4, 65.4)
- added J10: MS_SELECT, Connector_PinHeader_2.54mm:PinHeader_2x03_P2.54mm_Vertical, F.Cu at (22.5, 61.2)
- added J11: E0, footprint-lib:b4b-ph-kl,stepper_terminal, F.Cu at (2.40, 64.2)
- added J12: MS_SELECT, Connector_PinHeader_2.54mm:PinHeader_2x03_P2.54mm_Vertical, F.Cu at (22.4, 45.3)
- added J13: E1, footprint-lib:b4b-ph-kl,stepper_terminal, F.Cu at (2.40, 48.2)
- added J14: HEATBED, footprint-lib:mpt_0,5%2f2-2,54,heatbed, F.Cu at (46.8, 3.00)
- added J15: X_MIN, footprint-lib:b3b-ph-kl,end_stop, F.Cu at (85.0, 2.25)
- added J16: X_MAX, footprint-lib:b3b-ph-kl,end_stop, F.Cu at (85.0, 8.00)
- added J17: Y_MIN, footprint-lib:b3b-ph-kl,end_stop, F.Cu at (85.0, 13.8)
- added J18: Y_MAX, footprint-lib:b3b-ph-kl,end_stop, F.Cu at (85.0, 19.5)
- added J19: Z_MIN, footprint-lib:b3b-ph-kl,end_stop, F.Cu at (94.5, 13.5)
- added J2: MS_SELECT, Connector_PinHeader_2.54mm:PinHeader_2x03_P2.54mm_Vertical, F.Cu at (87.5, 77.0)
- added J20: Z_MAX, footprint-lib:b3b-ph-kl,end_stop, F.Cu at (94.5, 19.5)
- added J21: HEATBED_TEMP, w_conn_jst-ph:b2b-ph-kl, F.Cu at (2.39, 36.2)
- added J22: HOTEND_TEMP0, w_conn_jst-ph:b2b-ph-kl, F.Cu at (9.26, 36.2)
- added J23: HOTEND_TEMP1, w_conn_jst-ph:b2b-ph-kl, F.Cu at (16.1, 36.2)
- added J24: AUX_TEMP, w_conn_jst-ph:b2b-ph-kl, F.Cu at (23.0, 36.2)
- added J25: 12V_INPUT_2, footprint-lib:mpt_0,5%2f2-2,54,12V_SRC, F.Cu at (3.25, 18.2)
- added J26: 12V_INPUT, footprint-lib:mpt_0,5%2f2-2,54,12V_SRC, F.Cu at (3.15, 26.4)
- added J27: 12V_OUT, footprint-lib:mpt_0,5%2f2-2,54,12V_SRC, F.Cu at (3.15, 10.2)
- added J28: SWD, Connector_PinHeader_1.27mm:PinHeader_1x04_P1.27mm_Vertical, F.Cu at (37.4, 42.6)
- added J29: USB_DEBUG, Connector_PinHeader_1.27mm:PinHeader_1x05_P1.27mm_Vertical, F.Cu at (33.4, 47.6)
- added J3: X, footprint-lib:b4b-ph-kl,stepper_terminal, F.Cu at (86.0, 97.3)
- added J30: PWR_DEBUG, Connector_PinHeader_1.27mm:PinHeader_1x05_P1.27mm_Vertical, F.Cu at (29.4, 42.8)
- added J31: HOT_END, footprint-lib:mpt_0,5%2f2-2,54,heatbed, F.Cu at (58.8, 3.00)
- added J32: HOT_END, footprint-lib:mpt_0,5%2f2-2,54,heatbed, F.Cu at (70.8, 3.00)
- added J33: TO FAN0, footprint-lib:b2b-ph-kl,fan_pwm_out, F.Cu at (21.0, 2.00)
- added J34: TO FAN1, footprint-lib:b2b-ph-kl,fan_pwm_out, F.Cu at (29.2, 2.00)
- added J35: TO FAN2, footprint-lib:b2b-ph-kl,fan_pwm_out, F.Cu at (37.5, 2.00)
- added J36: MS_SELECT, Connector_PinHeader_2.54mm:PinHeader_2x03_P2.54mm_Vertical, F.Cu at (22.7, 77.0)
- added J37: Z2, footprint-lib:b4b-ph-kl,stepper_terminal, F.Cu at (26.7, 97.3)
- added J38: MS_SELECT, Connector_PinHeader_2.54mm:PinHeader_2x03_P2.54mm_Vertical, F.Cu at (71.3, 77.0)
- added J39: Y, footprint-lib:b4b-ph-kl,stepper_terminal, F.Cu at (71.9, 97.3)
- added J4: MS_SELECT, Connector_PinHeader_2.54mm:PinHeader_2x03_P2.54mm_Vertical, F.Cu at (55.1, 77.0)
- added J40: Conn_01x07, Connector_PinHeader_1.27mm:PinHeader_1x07_P1.27mm_Vertical, F.Cu at (124.0, 61.8)
- added J41: EXP1, Connector_PinHeader_2.54mm:PinHeader_2x05_P2.54mm_Vertical, F.Cu at (39.0, 38.4)
- added J42: EXP2, Connector_PinHeader_2.54mm:PinHeader_2x05_P2.54mm_Vertical, F.Cu at (31.8, 38.4)
- added J5: Z, footprint-lib:b4b-ph-kl,stepper_terminal, F.Cu at (56.8, 97.3)
- added J6: MS_SELECT, Connector_PinHeader_2.54mm:PinHeader_2x03_P2.54mm_Vertical, F.Cu at (38.9, 77.0)
- added J7: Z1, footprint-lib:b4b-ph-kl,stepper_terminal, F.Cu at (41.8, 97.3)
- added JP5: Jumper_NO_Small, SolderJumper-2_P1.3mm_Open_TrianglePad1.0x1.5mm, B.Cu at (8.55, 22.2)
- added JP6: Jumper_NO_Small, SolderJumper-2_P1.3mm_Open_TrianglePad1.0x1.5mm, B.Cu at (42.3, 58.2)
- added JP7: Jumper_NO_Small, SolderJumper-2_P1.3mm_Open_TrianglePad1.0x1.5mm, B.Cu at (44.2, 60.1)
- added JP8: SolderJumper_3_Open, Jumper:SolderJumper-3_P2.0mm_Open_TrianglePad1.0x1.5mm_NumberLabels, F.Cu at (128.6, 61.9)
- added L1: L_Small, w_smd_inductors:inductor_smd_0603, F.Cu at (40.2, 69.8)
- added L2: L_15uH, w_smd_inductors:inductor_smd_4.8x2.8mm, F.Cu at (61.8, 33.8)
- added L3: L_15uH, w_smd_inductors:inductor_smd_4.8x2.8mm, F.Cu at (53.5, 39.2)
- added Q1: WSK220N04, footprint-lib:TO-263-2,thermal_vias, F.Cu at (49.2, 15.0)
- added Q2: STP55NF06, footprint-lib:TO-263-2,thermal_vias, F.Cu at (61.2, 15.0)
- added Q3: STP55NF06, footprint-lib:TO-263-2,thermal_vias, F.Cu at (73.2, 15.0)
- added Q4: D882, footprint-lib:SOT-89-3,thermal_vias, F.Cu at (21.1, 8.00)
- added Q5: D882, footprint-lib:SOT-89-3,thermal_vias, F.Cu at (29.2, 8.00)
- added Q6: D882, footprint-lib:SOT-89-3,thermal_vias, F.Cu at (37.8, 8.00)
- added R1: R153,0603, Resistor_SMD:R_0603_1608Metric_Pad1.05x0.95mm_HandSolder, F.Cu at (76.2, 61.5)
- added R10: R103,0603, Resistor_SMD:R_0603_1608Metric_Pad1.05x0.95mm_HandSolder, F.Cu at (93.5, 82.5)
- added R11: R104,0603, Resistor_SMD:R_0603_1608Metric_Pad1.05x0.95mm_HandSolder, F.Cu at (61.5, 78.6)
- added R12: R102,0603, Resistor_SMD:R_0603_1608Metric_Pad1.05x0.95mm_HandSolder, B.Cu at (63.1, 97.7)
- added R13: R103,0603, Resistor_SMD:R_0603_1608Metric_Pad1.05x0.95mm_HandSolder, F.Cu at (61.5, 74.8)
- added R14: R104,0603, Resistor_SMD:R_0603_1608Metric_Pad1.05x0.95mm_HandSolder, F.Cu at (45.8, 74.8)
- added R15: R102,0603, Resistor_SMD:R_0603_1608Metric_Pad1.05x0.95mm_HandSolder, B.Cu at (48.0, 97.7)
- added R16: R103,0603, Resistor_SMD:R_0603_1608Metric_Pad1.05x0.95mm_HandSolder, F.Cu at (45.8, 82.5)
- added R2: R153,0603, Resistor_SMD:R_0603_1608Metric_Pad1.05x0.95mm_HandSolder, F.Cu at (78.2, 61.5)
- added R20: R104,0603, Resistor_SMD:R_0603_1608Metric_Pad1.05x0.95mm_HandSolder, F.Cu at (24.4, 67.2)
- added R21: R102,0603, Resistor_SMD:R_0603_1608Metric_Pad1.05x0.95mm_HandSolder, B.Cu at (3.00, 70.5)
- added R22: R103,0603, Resistor_SMD:R_0603_1608Metric_Pad1.05x0.95mm_HandSolder, F.Cu at (16.8, 67.2)
- added R23: R104,0603, Resistor_SMD:R_0603_1608Metric_Pad1.05x0.95mm_HandSolder, F.Cu at (20.6, 51.3)
- added R24: R102,0603, Resistor_SMD:R_0603_1608Metric_Pad1.05x0.95mm_HandSolder, F.Cu at (24.4, 51.3)
- added R25: R103,0603, Resistor_SMD:R_0603_1608Metric_Pad1.05x0.95mm_HandSolder, B.Cu at (3.00, 54.7)
- added R26: R100,0805, Resistor_SMD:R_0805_2012Metric_Pad1.15x1.40mm_HandSolder, B.Cu at (46.8, 19.5)
- added R27: R104,0805, Resistor_SMD:R_0805_2012Metric_Pad1.15x1.40mm_HandSolder, B.Cu at (51.8, 19.5)
- added R28: R182,0603, Resistor_SMD:R_0603_1608Metric_Pad1.05x0.95mm_HandSolder, B.Cu at (51.8, 5.50)
- added R29: R102,0603, Resistor_SMD:R_0603_1608Metric_Pad1.05x0.95mm_HandSolder, B.Cu at (90.2, 9.25)
- added R30: R102,0603, Resistor_SMD:R_0603_1608Metric_Pad1.05x0.95mm_HandSolder, B.Cu at (91.9, 9.25)
- added R31: R102,0603, Resistor_SMD:R_0603_1608Metric_Pad1.05x0.95mm_HandSolder, B.Cu at (93.7, 9.30)
- added R32: R102,0603, Resistor_SMD:R_0603_1608Metric_Pad1.05x0.95mm_HandSolder, B.Cu at (95.4, 9.30)
- added R33: R102,0603, Resistor_SMD:R_0603_1608Metric_Pad1.05x0.95mm_HandSolder, B.Cu at (98.9, 9.30)
- added R34: R102,0603, Resistor_SMD:R_0603_1608Metric_Pad1.05x0.95mm_HandSolder, B.Cu at (97.2, 9.30)
- added R35: R472,0603, Resistor_SMD:R_0603_1608Metric_Pad1.05x0.95mm_HandSolder, F.Cu at (2.75, 31.8)
- added R36: R472,0603, Resistor_SMD:R_0603_1608Metric_Pad1.05x0.95mm_HandSolder, F.Cu at (10.0, 31.8)
- added R37: R472,0603, Resistor_SMD:R_0603_1608Metric_Pad1.05x0.95mm_HandSolder, F.Cu at (16.8, 31.8)
- added R38: R472,0603, Resistor_SMD:R_0603_1608Metric_Pad1.05x0.95mm_HandSolder, F.Cu at (23.5, 31.8)
- added R39: R472,0603, Resistor_SMD:R_0603_1608Metric_Pad1.05x0.95mm_HandSolder, F.Cu at (27.4, 20.1)
- added R4: R220,0603, Resistor_SMD:R_0603_1608Metric_Pad1.05x0.95mm_HandSolder, B.Cu at (86.1, 70.8)
- added R40: R472,0603, Resistor_SMD:R_0603_1608Metric_Pad1.05x0.95mm_HandSolder, B.Cu at (44.6, 55.9)
- added R41: R472,0603, Resistor_SMD:R_0603_1608Metric_Pad1.05x0.95mm_HandSolder, B.Cu at (46.5, 57.8)
- added R42: R0,0603, Resistor_SMD:R_0603_1608Metric_Pad1.05x0.95mm_HandSolder, B.Cu at (37.7, 64.9)
- added R43: R0,0603, Resistor_SMD:R_0603_1608Metric_Pad1.05x0.95mm_HandSolder, B.Cu at (36.6, 63.8)
- added R44: R102,0603, Resistor_SMD:R_0603_1608Metric_Pad1.05x0.95mm_HandSolder, B.Cu at (30.3, 52.5)
- added R45: R103,0603, Resistor_SMD:R_0603_1608Metric_Pad1.05x0.95mm_HandSolder, B.Cu at (40.2, 56.0)
- added R46: R103,0603, Resistor_SMD:R_0603_1608Metric_Pad1.05x0.95mm_HandSolder, B.Cu at (39.1, 55.0)
- added R47: R220,0603, Resistor_SMD:R_0603_1608Metric_Pad1.05x0.95mm_HandSolder, F.Cu at (51.5, 50.2)
- added R48: R220,0603, Resistor_SMD:R_0603_1608Metric_Pad1.05x0.95mm_HandSolder, F.Cu at (51.5, 51.8)
- added R49: R152,0603, Resistor_SMD:R_0603_1608Metric_Pad1.05x0.95mm_HandSolder, B.Cu at (51.6, 51.0)
- added R5: R220,0603, Resistor_SMD:R_0603_1608Metric_Pad1.05x0.95mm_HandSolder, B.Cu at (84.5, 70.8)
- added R50: R100,0805, Resistor_SMD:R_0805_2012Metric_Pad1.15x1.40mm_HandSolder, B.Cu at (58.8, 19.5)
- added R51: R104,0805, Resistor_SMD:R_0805_2012Metric_Pad1.15x1.40mm_HandSolder, B.Cu at (63.8, 19.5)
- added R52: R182,0603, Resistor_SMD:R_0603_1608Metric_Pad1.05x0.95mm_HandSolder, B.Cu at (63.8, 5.50)
- added R53: R100,0805, Resistor_SMD:R_0805_2012Metric_Pad1.15x1.40mm_HandSolder, B.Cu at (70.8, 20.0)
- added R54: R104,0805, Resistor_SMD:R_0805_2012Metric_Pad1.15x1.40mm_HandSolder, B.Cu at (75.8, 20.0)
- added R55: R182,0603, Resistor_SMD:R_0603_1608Metric_Pad1.05x0.95mm_HandSolder, B.Cu at (75.8, 5.50)
- added R56: R100,0805, Resistor_SMD:R_0805_2012Metric_Pad1.15x1.40mm_HandSolder, B.Cu at (22.9, 5.10)
- added R57: R104,0805, Resistor_SMD:R_0805_2012Metric_Pad1.15x1.40mm_HandSolder, B.Cu at (19.4, 5.10)
- added R58: R100,0603, Resistor_SMD:R_0603_1608Metric_Pad1.05x0.95mm_HandSolder, B.Cu at (25.1, 2.50)
- added R59: R182,0603, Resistor_SMD:R_0603_1608Metric_Pad1.05x0.95mm_HandSolder, B.Cu at (21.1, 5.10)
- added R6: R152,0603, Resistor_SMD:R_0603_1608Metric_Pad1.05x0.95mm_HandSolder, B.Cu at (82.9, 70.8)
- added R60: R100,0805, Resistor_SMD:R_0805_2012Metric_Pad1.15x1.40mm_HandSolder, B.Cu at (31.0, 5.25)
- added R61: R104,0805, Resistor_SMD:R_0805_2012Metric_Pad1.15x1.40mm_HandSolder, B.Cu at (27.5, 5.25)
- added R62: R100,0603, Resistor_SMD:R_0603_1608Metric_Pad1.05x0.95mm_HandSolder, B.Cu at (29.2, 5.38)
- added R63: R182,0603, Resistor_SMD:R_0603_1608Metric_Pad1.05x0.95mm_HandSolder, B.Cu at (33.4, 2.50)
- added R64: R100,0805, Resistor_SMD:R_0603_1608Metric_Pad1.05x0.95mm_HandSolder, B.Cu at (39.2, 5.25)
- added R65: R104,0805, Resistor_SMD:R_0805_2012Metric_Pad1.15x1.40mm_HandSolder, B.Cu at (36.0, 5.25)
- added R66: R100,0603, Resistor_SMD:R_0603_1608Metric_Pad1.05x0.95mm_HandSolder, B.Cu at (37.8, 5.25)
- added R67: R182,0603, Resistor_SMD:R_0603_1608Metric_Pad1.05x0.95mm_HandSolder, B.Cu at (41.8, 2.50)
- added R68: R104,0603, Resistor_SMD:R_0603_1608Metric_Pad1.05x0.95mm_HandSolder, F.Cu at (29.8, 74.8)
- added R69: R102,0603, Resistor_SMD:R_0603_1608Metric_Pad1.05x0.95mm_HandSolder, B.Cu at (33.0, 97.7)
- added R7: R102,0603, Resistor_SMD:R_0603_1608Metric_Pad1.05x0.95mm_HandSolder, B.Cu at (50.8, 70.8)
- added R70: R103,0603, Resistor_SMD:R_0603_1608Metric_Pad1.05x0.95mm_HandSolder, F.Cu at (29.8, 82.5)
- added R71: R104,0603, Resistor_SMD:R_0603_1608Metric_Pad1.05x0.95mm_HandSolder, F.Cu at (77.8, 78.6)
- added R72: R102,0603, Resistor_SMD:R_0603_1608Metric_Pad1.05x0.95mm_HandSolder, B.Cu at (78.2, 97.7)
- added R73: R103,0603, Resistor_SMD:R_0603_1608Metric_Pad1.05x0.95mm_HandSolder, F.Cu at (77.8, 82.5)
- added R74: R562,0603, Resistor_SMD:R_0603_1608Metric_Pad1.05x0.95mm_HandSolder, F.Cu at (59.5, 41.0)
- added R75: R103,0603, Resistor_SMD:R_0603_1608Metric_Pad1.05x0.95mm_HandSolder, F.Cu at (59.5, 37.5)
- added R76: R333,0603, Resistor_SMD:R_0603_1608Metric_Pad1.05x0.95mm_HandSolder, F.Cu at (59.5, 39.2)
- added R77: R562,0603, Resistor_SMD:R_0603_1608Metric_Pad1.05x0.95mm_HandSolder, F.Cu at (52.8, 30.0)
- added R78: R103,0603, Resistor_SMD:R_0603_1608Metric_Pad1.05x0.95mm_HandSolder, F.Cu at (52.2, 32.0)
- added R79: R333,0603, Resistor_SMD:R_0603_1608Metric_Pad1.05x0.95mm_HandSolder, F.Cu at (52.2, 33.8)
- added R8: R104,0603, Resistor_SMD:R_0603_1608Metric_Pad1.05x0.95mm_HandSolder, F.Cu at (93.5, 78.6)
- added R9: R102,0603, Resistor_SMD:R_0603_1608Metric_Pad1.05x0.95mm_HandSolder, B.Cu at (92.2, 97.7)
- added SW1: SW_Push, Button_Switch_SMD:SW_SPST_CK_RS282G05A3, F.Cu at (47.6, 68.0)
- added TH1: Thermistor_NTC, Resistor_SMD:R_0603_1608Metric_Pad1.05x0.95mm_HandSolder, F.Cu at (27.4, 21.6)
- added U1: orange_pi_zero, footprint-lib:orangepi-zero, B.Cu at (52.0, 69.5)
- added U10: A4988_MODULE, footprint-lib:Pololu_Breakout-16_15.2x20.3mm, F.Cu at (68.1, 74.4)
- added U11: MP2303A_ALT, footprint-lib:SOIC-8_3.9x4.9mm_P1.27mm,thermal_via, F.Cu at (68.0, 38.1)
- added U12: MP2303A_ALT, footprint-lib:SOIC-8_3.9x4.9mm_P1.27mm,thermal_via, F.Cu at (47.5, 35.1)
- added U2: A4988_MODULE, footprint-lib:Pololu_Breakout-16_15.2x20.3mm, F.Cu at (84.3, 74.4)
- added U3: A4988_MODULE, footprint-lib:Pololu_Breakout-16_15.2x20.3mm, F.Cu at (51.9, 74.4)
- added U4: A4988_MODULE, footprint-lib:Pololu_Breakout-16_15.2x20.3mm, F.Cu at (35.6, 74.4)
- added U6: A4988_MODULE, footprint-lib:Pololu_Breakout-16_15.2x20.3mm, F.Cu at (25.0, 57.9)
- added U7: A4988_MODULE, footprint-lib:Pololu_Breakout-16_15.2x20.3mm, F.Cu at (25.0, 41.9)
- added U8: STM32F407VET6, w_smd_lqfp:TQFP-100, F.Cu at (40.9, 57.5)
- added U9: A4988_MODULE, footprint-lib:Pololu_Breakout-16_15.2x20.3mm, F.Cu at (19.4, 74.4)
- added Y1: O_8M, Crystal:Crystal_HC49-4H_Vertical, F.Cu at (30.6, 64.0)
- moved J9 72.8 mm to (11.6, 97.3), turned to 180 degrees
- moved R18 72.7 mm to (17.8, 97.7)
- moved D5 72.7 mm to (17.8, 97.7)
- moved C8 72.2 mm to (9.50, 90.2)
- moved C9 71.5 mm to (12.5, 82.5)
- moved J8 71.5 mm to (6.50, 77.0)
- moved U5 71.5 mm to (3.18, 74.4)
- moved R17 71.1 mm to (12.5, 78.6)
- moved R19 70.9 mm to (12.5, 74.8)
Connections:
- U5 pad 11: Net-(J9-Pad4) -> Net-(J9-Pad1)
- U5 pad 12: Net-(J9-Pad3) -> Net-(J9-Pad2)
- U5 pad 13: Net-(J9-Pad2) -> Net-(J9-Pad3)
- U5 pad 14: Net-(J9-Pad1) -> Net-(J9-Pad4)
Other:
- board outline added: 100 x 100 mm
