File: hardware/printer-board/orange_pi.sch (KiCad schematic (older format))
At the start: 12 parts, among them J40 USB_DEBUG, U1 orange_pi_zero

Commit message: update to re-annotation,
Parts:
- renumbered D4 to D1, J40 to J1, JP3 to JP1, JP4 to JP2, JP5 to JP3, JP6 to JP4, R5 to R4, R7 to R5, R9 to R6, R27 to R7
Changed lines of the file:
@@
 AR Path="/5CC01E08/5CC01846" Ref="U?"  Part="1"
 AR Path="/5CC02AB6/5CC01846" Ref="U?"  Part="1"
-AR Path="/5CC01846" Ref="U1"  Part="1"
+AR Path="/5CC01846" Ref="U?"  Part="1"
 F 0 "U1" H 9000 5537 60  0000 C CNN
 F 1 "orange_pi_zero" H 9000 5431 60  0000 C CNN
@@
 $EndComp
 $Comp
-L power:GND #PWR0102
+L power:GND #PWR08
 U 1 1 5CC01A30
 P 6400 2350
-AR Path="/5CC0166A/5CC01A30" Ref="#PWR0102"  Part="1"
+AR Path="/5CC0166A/5CC01A30" Ref="#PWR08"  Part="1"
 AR Path="/5CC01E08/5CC01A30" Ref="#PWR?"  Part="1"
 AR Path="/5CC02AB6/5CC01A30" Ref="#PWR?"  Part="1"
-AR Path="/5CC01A30" Ref="#PWR0102"  Part="1"
-F 0 "#PWR0102" H 6400 2100 50  0001 C CNN
+AR Path="/5CC01A30" Ref="#PWR?"  Part="1"
+F 0 "#PWR08" H 6400 2100 50  0001 C CNN
 F 1 "GND" H 6405 2177 50  0000 C CNN
 F 2 "" H 6400 2350 50  0001 C CNN
@@
 	6400 2250 6400 2350
 $Comp
-L power:GND #PWR0104
+L power:GND #PWR011
 U 1 1 5CC01AC2
 P 9350 1200
-AR Path="/5CC0166A/5CC01AC2" Ref="#PWR0104"  Part="1"
+AR Path="/5CC0166A/5CC01AC2" Ref="#PWR011"  Part="1"
 AR Path="/5CC01E08/5CC01AC2" Ref="#PWR?"  Part="1"
 AR Path="/5CC02AB6/5CC01AC2" Ref="#PWR?"  Part="1"
-AR Path="/5CC01AC2" Ref="#PWR0104"  Part="1"
-F 0 "#PWR0104" H 9350 950 50  0001 C CNN
+AR Path="/5CC01AC2" Ref="#PWR?"  Part="1"
+F 0 "#PWR011" H 9350 950 50  0001 C CNN
 F 1 "GND" V 9355 1072 50  0000 R CNN
 F 2 "" H 9350 1200 50  0001 C CNN
@@
 $EndBitmap
 $Comp
-L taobao-components:+5V_PI_SRC #PWR0101
+L taobao-components:+5V_PI_SRC #PWR07
 U 1 1 5CC325A1
 P 6400 2000
-F 0 "#PWR0101" H 6400 1850 50  0001 C CNN
+F 0 "#PWR07" H 6400 1850 50  0001 C CNN
 F 1 "+5V_PI_SRC" H 6450 2200 50  0000 C CNN
 F 2 "" H 6400 2000 50  0001 C CNN
@@
 $EndComp
 $Comp
-L taobao-components:+5V_PI_SRC #PWR0103
+L taobao-components:+5V_PI_SRC #PWR010
 U 1 1 5CC325F8
 P 8700 1200
-F 0 "#PWR0103" H 8700 1050 50  0001 C CNN
+F 0 "#PWR010" H 8700 1050 50  0001 C CNN
 F 1 "+5V_PI_SRC" V 8750 1350 50  0000 L CNN
 F 2 "" H 8700 1200 50  0001 C CNN
@@
 $EndComp
 $Comp
-L power:GND #PWR0112
+L power:GND #PWR012
 U 1 1 5CC326F9
 P 9350 1650
-AR Path="/5CC0166A/5CC326F9" Ref="#PWR0112"  Part="1"
+AR Path="/5CC0166A/5CC326F9" Ref="#PWR012"  Part="1"
 AR Path="/5CC01E08/5CC326F9" Ref="#PWR?"  Part="1"
 AR Path="/5CC02AB6/5CC326F9" Ref="#PWR?"  Part="1"
-AR Path="/5CC326F9" Ref="#PWR0112"  Part="1"
-F 0 "#PWR0112" H 9350 1400 50  0001 C CNN
+AR Path="/5CC326F9" Ref="#PWR?"  Part="1"
+F 0 "#PWR012" H 9350 1400 50  0001 C CNN
 F 1 "GND" V 9355 1522 50  0000 R CNN
 F 2 "" H 9350 1650 50  0001 C CNN
@@
 	9100 1650 9350 1650
 $Comp
-L taobao-components:+5V_PI_SRC #PWR0113
+L taobao-components:+5V_PI_SRC #PWR09
 U 1 1 5CC32707
 P 8200 1650
-F 0 "#PWR0113" H 8200 1500 50  0001 C CNN
+F 0 "#PWR09" H 8200 1500 50  0001 C CNN
 F 1 "+5V_PI_SRC" V 8250 1800 50  0000 L CNN
 F 2 "" H 8200 1650 50  0001 C CNN
@@
 $EndComp
 $Comp
-L taobao-r:R102,0603 R27
+L taobao-r:R102,0603 R7
 U 1 1 5CC327C3
 P 8650 1650
-F 0 "R27" V 8400 1650 50  0000 C CNN
+F 0 "R7" V 8400 1650 50  0000 C CNN
 F 1 "R102,0603" V 8500 1650 50  0000 C CNN
 F 2 "Resistor_SMD:R_0603_1608Metric_Pad1.05x0.95mm_HandSolder" H 8650 1650 50  0001 C CNN
@@
 $EndComp
 $Comp
-L taobao-components:LED_GREEN D4
+L taobao-components:LED_GREEN D1
 U 1 1 5CC32901
 P 9000 1650
-F 0 "D4" H 9000 1400 50  0000 C CNN
+F 0 "D1" H 9000 1400 50  0000 C CNN
 F 1 "5V HEALTHY" H 9000 1500 50  0000 C CNN
 F 2 "LED_SMD:LED_0603_1608Metric_Pad1.05x0.95mm_HandSolder" V 9000 1650 50  0001 C CNN
@@
 P 4000 5000
 AR Path="/5CC29851/5CC2A1CB/5CE44033" Ref="J?"  Part="1"
-AR Path="/5CC0166A/5CE44033" Ref="J40"  Part="1"
-AR Path="/5CE44033" Ref="J1"  Part="1"
-F 0 "J40" H 3900 5450 50  0000 C CNN
+AR Path="/5CC0166A/5CE44033" Ref="J1"  Part="1"
+AR Path="/5CE44033" Ref="J?"  Part="1"
+F 0 "J1" H 3900 5450 50  0000 C CNN
 F 1 "USB_DEBUG" H 3900 5350 50  0000 C CNN
 F 2 "Connector_PinHeader_1.27mm:PinHeader_1x05_P1.27mm_Vertical" H 4000 5000 50  0001 C CNN
@@
 P 4550 4700
 AR Path="/5CC29851/5CC2A1CB/5CE4403A" Ref="#PWR?"  Part="1"
-AR Path="/5CC0166A/5CE4403A" Ref="#PWR05"  Part="1"
-AR Path="/5CE4403A" Ref="#PWR05"  Part="1"
-F 0 "#PWR05" H 4550 4550 50  0001 C CNN
+AR Path="/5CC0166A/5CE4403A" Ref="#PWR04"  Part="1"
+AR Path="/5CE4403A" Ref="#PWR?"  Part="1"
+F 0 "#PWR04" H 4550 4550 50  0001 C CNN
 F 1 "+5V" H 4600 4900 50  0000 C CNN
 F 2 "" H 4550 4700 50  0001 C CNN
@@
 P 4550 5350
 AR Path="/5CC29851/5CC2A1CB/5CE44042" Ref="#PWR?"  Part="1"
-AR Path="/5CC0166A/5CE44042" Ref="#PWR06"  Part="1"
-AR Path="/5CE44042" Ref="#PWR06"  Part="1"
-F 0 "#PWR06" H 4550 5100 50  0001 C CNN
+AR Path="/5CC0166A/5CE44042" Ref="#PWR05"  Part="1"
+AR Path="/5CE44042" Ref="#PWR?"  Part="1"
+F 0 "#PWR05" H 4550 5100 50  0001 C CNN
 F 1 "GND" H 4600 5150 50  0000 C CNN
 F 2 "" H 4550 5350 50  0001 C CNN
@@
 P 4550 4900
 AR Path="/5CC29851/5CC2A1CB/5CE4404D" Ref="R?"  Part="1"
-AR Path="/5CC0166A/5CE4404D" Ref="R5"  Part="1"
-AR Path="/5CE4404D" Ref="R5"  Part="1"
-F 0 "R5" V 4300 4900 50  0000 C CNN
+AR Path="/5CC0166A/5CE4404D" Ref="R4"  Part="1"
+AR Path="/5CE4404D" Ref="R?"  Part="1"
+F 0 "R4" V 4300 4900 50  0000 C CNN
 F 1 "R220,0603" V 4400 4900 50  0000 C CNN
 F 2 "Resistor_SMD:R_0603_1608Metric_Pad1.05x0.95mm_HandSolder" H 4550 4900 50  0001 C CNN
@@
 P 4550 5000
 AR Path="/5CC29851/5CC2A1CB/5CE44054" Ref="R?"  Part="1"
-AR Path="/5CC0166A/5CE44054" Ref="R7"  Part="1"
-AR Path="/5CE44054" Ref="R7"  Part="1"
-F 0 "R7" V 4300 5000 50  0000 C CNN
+AR Path="/5CC0166A/5CE44054" Ref="R5"  Part="1"
+AR Path="/5CE44054" Ref="R?"  Part="1"
+F 0 "R5" V 4300 5000 50  0000 C CNN
 F 1 "R220,0603" V 4400 5000 50  0000 C CNN
 F 2 "Resistor_SMD:R_0603_1608Metric_Pad1.05x0.95mm_HandSolder" H 4550 5000 50  0001 C CNN
@@
 P 4750 5250
 AR Path="/5CC29851/5CC2A1CB/5CE4405F" Ref="R?"  Part="1"
-AR Path="/5CC0166A/5CE4405F" Ref="R9"  Part="1"
-AR Path="/5CE4405F" Ref="R9"  Part="1"
-F 0 "R9" H 4850 5300 50  0000 L CNN
+AR Path="/5CC0166A/5CE4405F" Ref="R6"  Part="1"
+AR Path="/5CE4405F" Ref="R?"  Part="1"
+F 0 "R6" H 4850 5300 50  0000 L CNN
 F 1 "R152,0603" H 4850 5250 50  0000 L CNN
 F 2 "Resistor_SMD:R_0603_1608Metric_Pad1.05x0.95mm_HandSolder" H 4750 5250 50  0001 C CNN
@@
 P 4750 5450
 AR Path="/5CC29851/5CC2A1CB/5CE44066" Ref="#PWR?"  Part="1"
-AR Path="/5CC0166A/5CE44066" Ref="#PWR07"  Part="1"
-AR Path="/5CE44066" Ref="#PWR07"  Part="1"
-F 0 "#PWR07" H 4750 5300 50  0001 C CNN
+AR Path="/5CC0166A/5CE44066" Ref="#PWR06"  Part="1"
+AR Path="/5CE44066" Ref="#PWR?"  Part="1"
+F 0 "#PWR06" H 4750 5300 50  0001 C CNN
 F 1 "+3V3_STM32" H 4750 5650 50  0000 C CNN
 F 2 "" H 4750 5450 50  0001 C CNN
@@
 	4750 5000 5700 5000
 $Comp
-L Device:Jumper_NO_Small JP3
+L Device:Jumper_NO_Small JP1
 U 1 1 5CE47FCE
 P 1450 800
-F 0 "JP3" H 1450 1000 50  0000 C CNN
+F 0 "JP1" H 1450 1000 50  0000 C CNN
 F 1 "Jumper_NO_Small" H 1450 900 50  0000 C CNN
 F 2 "Jumper:SolderJumper-2_P1.3mm_Open_TrianglePad1.0x1.5mm" H 1450 800 50  0001 C CNN
@@
 $EndComp
 $Comp
-L Device:Jumper_NO_Small JP4
+L Device:Jumper_NO_Small JP2
 U 1 1 5CE4801F
 P 1450 900
-F 0 "JP4" H 1450 1100 50  0000 C CNN
+F 0 "JP2" H 1450 1100 50  0000 C CNN
 F 1 "Jumper_NO_Small" H 1450 1000 50  0000 C CNN
 F 2 "Jumper:SolderJumper-2_P1.3mm_Open_TrianglePad1.0x1.5mm" H 1450 900 50  0001 C CNN
@@
 $EndComp
 $Comp
-L Device:Jumper_NO_Small JP5
+L Device:Jumper_NO_Small JP3
 U 1 1 5CE48043
 P 1450 1000
-F 0 "JP5" H 1450 1200 50  0000 C CNN
+F 0 "JP3" H 1450 1200 50  0000 C CNN
 F 1 "Jumper_NO_Small" H 1450 1100 50  0000 C CNN
 F 2 "Jumper:SolderJumper-2_P1.3mm_Open_TrianglePad1.0x1.5mm" H 1450 1000 50  0001 C CNN
@@
 $EndComp
 $Comp
-L Device:Jumper_NO_Small JP6
+L Device:Jumper_NO_Small JP4
 U 1 1 5CE48098
 P 1450 1100
-F 0 "JP6" H 1450 1300 50  0000 C CNN
+F 0 "JP4" H 1450 1300 50  0000 C CNN
 F 1 "Jumper_NO_Small" H 1450 1200 50  0000 C CNN
 F 2 "Jumper:SolderJumper-2_P1.3mm_Open_TrianglePad1.0x1.5mm" H 1450 1100 50  0001 C CNN

Commit message: update,
Connections:
- net +5V: now also J1.5 (Pin_5); no longer J1.1 (Pin_1)
- net GND: now also J1.1 (Pin_1); no longer J1.4 (Pin_4), J1.5 (Pin_5)
Other:
- moved on the sheet: JP1, JP2, JP3, JP4
Changed lines of the file:
@@
 EESchema Schematic File Version 4
-LIBS:printer-board-cache
+LIBS:orange_pi-cache
 EELAYER 26 0
 EELAYER END
 $Descr A4 11693 8268
 encoding utf-8
-Sheet 1 29
+Sheet 1 1
 Title ""
 Date ""
@@
 AR Path="/5CC01E08/5CC01846" Ref="U?"  Part="1"
 AR Path="/5CC02AB6/5CC01846" Ref="U?"  Part="1"
-AR Path="/5CC01846" Ref="U?"  Part="1"
+AR Path="/5CC01846" Ref="U1"  Part="1"
 F 0 "U1" H 9000 5537 60  0000 C CNN
 F 1 "orange_pi_zero" H 9000 5431 60  0000 C CNN
@@
 AR Path="/5CC01E08/5CC01A30" Ref="#PWR?"  Part="1"
 AR Path="/5CC02AB6/5CC01A30" Ref="#PWR?"  Part="1"
-AR Path="/5CC01A30" Ref="#PWR?"  Part="1"
+AR Path="/5CC01A30" Ref="#PWR08"  Part="1"
 F 0 "#PWR08" H 6400 2100 50  0001 C CNN
 F 1 "GND" H 6405 2177 50  0000 C CNN
@@
 AR Path="/5CC01E08/5CC01AC2" Ref="#PWR?"  Part="1"
 AR Path="/5CC02AB6/5CC01AC2" Ref="#PWR?"  Part="1"
-AR Path="/5CC01AC2" Ref="#PWR?"  Part="1"
+AR Path="/5CC01AC2" Ref="#PWR011"  Part="1"
 F 0 "#PWR011" H 9350 950 50  0001 C CNN
 F 1 "GND" V 9355 1072 50  0000 R CNN
@@
 AR Path="/5CC01E08/5CC326F9" Ref="#PWR?"  Part="1"
 AR Path="/5CC02AB6/5CC326F9" Ref="#PWR?"  Part="1"
-AR Path="/5CC326F9" Ref="#PWR?"  Part="1"
+AR Path="/5CC326F9" Ref="#PWR012"  Part="1"
 F 0 "#PWR012" H 9350 1400 50  0001 C CNN
 F 1 "GND" V 9355 1522 50  0000 R CNN
@@
 Wire Wire Line
 	7250 2650 7950 2650
-Text Label 2600 800  2    50   ~ 0
+Text Label 2600 700  2    50   ~ 0
 USB-DM2
-Text Label 2600 900  2    50   ~ 0
+Text Label 2600 800  2    50   ~ 0
 USB-DP2
-Text Label 2600 1000 2    50   ~ 0
+Text Label 2600 1150 2    50   ~ 0
 USB-DM3
-Text Label 2600 1100 2    50   ~ 0
+Text Label 2600 1250 2    50   ~ 0
 USB-DP3
-Text HLabel 1100 800  0    50   Input ~ 0
+Text HLabel 1100 700  0    50   Input ~ 0
 OPI_USB-DM2
-Text HLabel 1100 900  0    50   Input ~ 0
+Text HLabel 1100 800  0    50   Input ~ 0
 OPI_USB-DP2
-Text HLabel 1100 1000 0    50   Input ~ 0
+Text HLabel 1100 1150 0    50   Input ~ 0
 OPI_USB-DM3
-Text HLabel 1100 1100 0    50   Input ~ 0
+Text HLabel 1100 1250 0    50   Input ~ 0
 OPI_USB-DP3
 $Comp
@@
 AR Path="/5CC29851/5CC2A1CB/5CE44033" Ref="J?"  Part="1"
 AR Path="/5CC0166A/5CE44033" Ref="J1"  Part="1"
-AR Path="/5CE44033" Ref="J?"  Part="1"
+AR Path="/5CE44033" Ref="J1"  Part="1"
 F 0 "J1" H 3900 5450 50  0000 C CNN
 F 1 "USB_DEBUG" H 3900 5350 50  0000 C CNN
@@
 L power:+5V #PWR?
 U 1 1 5CE4403A
-P 4550 4700
+P 4550 5300
 AR Path="/5CC29851/5CC2A1CB/5CE4403A" Ref="#PWR?"  Part="1"
 AR Path="/5CC0166A/5CE4403A" Ref="#PWR04"  Part="1"
-AR Path="/5CE4403A" Ref="#PWR?"  Part="1"
-F 0 "#PWR04" H 4550 4550 50  0001 C CNN
-F 1 "+5V" H 4600 4900 50  0000 C CNN
-F 2 "" H 4550 4700 50  0001 C CNN
-F 3 "" H 4550 4700 50  0001 C CNN
-	1    4550 4700
-	1    0    0    -1
+AR Path="/5CE4403A" Ref="#PWR04"  Part="1"
+F 0 "#PWR04" H 4550 5150 50  0001 C CNN
+F 1 "+5V" H 4600 5500 50  0000 C CNN
+F 2 "" H 4550 5300 50  0001 C CNN
+F 3 "" H 4550 5300 50  0001 C CNN
+	1    4550 5300
+	1    0    0    1
 $EndComp
 Wire Wire Line
-	4550 4700 4550 4800
+	4550 5300 4550 5200
 Wire Wire Line
-	4550 4800 4200 4800
+	4550 5200 4200 5200
 $Comp
 L power:GND #PWR?
 U 1 1 5CE44042
-P 4550 5350
+P 4550 4650
 AR Path="/5CC29851/5CC2A1CB/5CE44042" Ref="#PWR?"  Part="1"
 AR Path="/5CC0166A/5CE44042" Ref="#PWR05"  Part="1"
-AR Path="/5CE44042" Ref="#PWR?"  Part="1"
-F 0 "#PWR05" H 4550 5100 50  0001 C CNN
-F 1 "GND" H 4600 5150 50  0000 C CNN
-F 2 "" H 4550 5350 50  0001 C CNN
-F 3 "" H 4550 5350 50  0001 C CNN
-	1    4550 5350
-	1    0    0    -1
+AR Path="/5CE44042" Ref="#PWR05"  Part="1"
+F 0 "#PWR05" H 4550 4400 50  0001 C CNN
+F 1 "GND" H 4600 4450 50  0000 C CNN
+F 2 "" H 4550 4650 50  0001 C CNN
+F 3 "" H 4550 4650 50  0001 C CNN
+	1    4550 4650
+	1    0    0    1
 $EndComp
 Wire Wire Line
-	4200 5200 4550 5200
+	4200 4800 4550 4800
 Wire Wire Line
-	4550 5200 4550 5350
+	4550 4800 4550 4650
 Wire Wire Line
 	4200 5100 4550 5100
-Wire Wire Line
-	4550 5100 4550 5200
-Connection ~ 4550 5200
 $Comp
 L taobao-r:R220,0603 R?
@@
 AR Path="/5CC29851/5CC2A1CB/5CE4404D" Ref="R?"  Part="1"
 AR Path="/5CC0166A/5CE4404D" Ref="R4"  Part="1"
-AR Path="/5CE4404D" Ref="R?"  Part="1"
+AR Path="/5CE4404D" Ref="R4"  Part="1"
 F 0 "R4" V 4300 4900 50  0000 C CNN
 F 1 "R220,0603" V 4400 4900 50  0000 C CNN
@@
 AR Path="/5CC29851/5CC2A1CB/5CE44054" Ref="R?"  Part="1"
 AR Path="/5CC0166A/5CE44054" Ref="R5"  Part="1"
-AR Path="/5CE44054" Ref="R?"  Part="1"
+AR Path="/5CE44054" Ref="R5"  Part="1"
 F 0 "R5" V 4300 5000 50  0000 C CNN
 F 1 "R220,0603" V 4400 5000 50  0000 C CNN
@@
 AR Path="/5CC29851/5CC2A1CB/5CE4405F" Ref="R?"  Part="1"
 AR Path="/5CC0166A/5CE4405F" Ref="R6"  Part="1"
-AR Path="/5CE4405F" Ref="R?"  Part="1"
+AR Path="/5CE4405F" Ref="R6"  Part="1"
 F 0 "R6" H 4850 5300 50  0000 L CNN
 F 1 "R152,0603" H 4850 5250 50  0000 L CNN
@@
 AR Path="/5CC29851/5CC2A1CB/5CE44066" Ref="#PWR?"  Part="1"
 AR Path="/5CC0166A/5CE44066" Ref="#PWR06"  Part="1"
-AR Path="/5CE44066" Ref="#PWR?"  Part="1"
+AR Path="/5CE44066" Ref="#PWR06"  Part="1"
 F 0 "#PWR06" H 4750 5300 50  0001 C CNN
 F 1 "+3V3_STM32" H 4750 5650 50  0000 C CNN
@@
 L Device:Jumper_NO_Small JP1
 U 1 1 5CE47FCE
-P 1450 800
-F 0 "JP1" H 1450 1000 50  0000 C CNN
-F 1 "Jumper_NO_Small" H 1450 900 50  0000 C CNN
-F 2 "Jumper:SolderJumper-2_P1.3mm_Open_TrianglePad1.0x1.5mm" H 1450 800 50  0001 C CNN
-F 3 "~" H 1450 800 50  0001 C CNN
-	1    1450 800
+P 1450 700
+F 0 "JP1" H 1450 900 50  0000 C CNN
+F 1 "Jumper_NO_Small" H 1450 800 50  0000 C CNN
+F 2 "Jumper:SolderJumper-2_P1.3mm_Open_TrianglePad1.0x1.5mm" H 1450 700 50  0001 C CNN
+F 3 "~" H 1450 700 50  0001 C CNN
+	1    1450 700
 	1    0    0    -1
 $EndComp
@@
 L Device:Jumper_NO_Small JP2
 U 1 1 5CE4801F
-P 1450 900
-F 0 "JP2" H 1450 1100 50  0000 C CNN
-F 1 "Jumper_NO_Small" H 1450 1000 50  0000 C CNN
-F 2 "Jumper:SolderJumper-2_P1.3mm_Open_TrianglePad1.0x1.5mm" H 1450 900 50  0001 C CNN
-F 3 "~" H 1450 900 50  0001 C CNN
-	1    1450 900
+P 1450 800
+F 0 "JP2" H 1450 1000 50  0000 C CNN
+F 1 "Jumper_NO_Small" H 1450 900 50  0000 C CNN
+F 2 "Jumper:SolderJumper-2_P1.3mm_Open_TrianglePad1.0x1.5mm" H 1450 800 50  0001 C CNN
+F 3 "~" H 1450 800 50  0001 C CNN
+	1    1450 800
 	1    0    0    -1
 $EndComp
@@
 L Device:Jumper_NO_Small JP3
 U 1 1 5CE48043
-P 1450 1000
-F 0 "JP3" H 1450 1200 50  0000 C CNN
-F 1 "Jumper_NO_Small" H 1450 1100 50  0000 C CNN
-F 2 "Jumper:SolderJumper-2_P1.3mm_Open_TrianglePad1.0x1.5mm" H 1450 1000 50  0001 C CNN
-F 3 "~" H 1450 1000 50  0001 C CNN
-	1    1450 1000
+P 1450 1150
+F 0 "JP3" H 1450 1350 50  0000 C CNN
+F 1 "Jumper_NO_Small" H 1450 1250 50  0000 C CNN
+F 2 "Jumper:SolderJumper-2_P1.3mm_Open_TrianglePad1.0x1.5mm" H 1450 1150 50  0001 C CNN
+F 3 "~" H 1450 1150 50  0001 C CNN
+	1    1450 1150
 	1    0    0    -1
 $EndComp
@@
 L Device:Jumper_NO_Small JP4
 U 1 1 5CE48098
-P 1450 1100
-F 0 "JP4" H 1450 1300 50  0000 C CNN
-F 1 "Jumper_NO_Small" H 1450 1200 50  0000 C CNN
-F 2 "Jumper:SolderJumper-2_P1.3mm_Open_TrianglePad1.0x1.5mm" H 1450 1100 50  0001 C CNN
-F 3 "~" H 1450 1100 50  0001 C CNN
-	1    1450 1100
+P 1450 1250
+F 0 "JP4" H 1450 1450 50  0000 C CNN
+F 1 "Jumper_NO_Small" H 1450 1350 50  0000 C CNN
+F 2 "Jumper:SolderJumper-2_P1.3mm_Open_TrianglePad1.0x1.5mm" H 1450 1250 50  0001 C CNN
+F 3 "~" H 1450 1250 50  0001 C CNN
+	1    1450 1250
 	1    0    0    -1
 $EndComp
 Wire Wire Line
+	1100 700  1350 700
+Wire Wire Line
 	1100 800  1350 800
 Wire Wire Line
-	1100 900  1350 900
+	1100 1150 1350 1150
 Wire Wire Line
-	1100 1000 1350 1000
+	1100 1250 1350 1250
 Wire Wire Line
-	1100 1100 1350 1100
+	1550 700  2600 700
 Wire Wire Line
 	1550 800  2600 800
 Wire Wire Line
-	1550 900  2600 900
-Wire Wire Line
-	1550 1000 2600 1000
+	1550 1150 2600 1150
 Wire Wire Line
-	1550 1100 2600 1100
+	1550 1250 2600 1250
 $EndSCHEMATC

Commit message: update driver positin,
Parts:
- removed C1: CP100uf,35V, Capacitor_SMD:C_0603_1608Metric_Pad1.05x0.95mm_HandSolder, symbol taobao-cp:CP100uf,35V
- removed JP1, JP2, JP3, JP4: Jumper_NO_Small, Jumper:SolderJumper-2_P1.3mm_Open_TrianglePad1.0x1.5mm, symbol Device:Jumper_NO_Small
- added C1: CP100uf,10V, Capacitor_SMD:CP_Elec_6.3x5.3, symbol taobao-cp:CP100uf,10V
Connections:
- net USB-DM2 is gone; now on net OPI_USB-DM2: R4.1, U1.3 (USB-DM2)
- net USB-DM3 is gone; now on net OPI_USB-DM3: U1.5 (USB-DM3)
- net USB-DP2 is gone; now on net OPI_USB-DP2: R5.1, R6.1, U1.4 (USB-DP2)
- net USB-DP3 is gone; now on net OPI_USB-DP3: U1.6 (USB-DP3)
- net +5V_PI_SRC: now also C1.1
- net GND: now also C1.2
Changed lines of the file:
@@
 Text HLabel 1100 1250 0    50   Input ~ 0
 OPI_USB-DP3
-$Comp
-L taobao-cp:CP100uf,35V C1
-U 1 1 5CE43439
-P 9000 1200
-F 0 "C1" V 9250 1200 50  0000 C CNN
-F 1 "CP100uf,35V" V 9150 1200 50  0000 C CNN
-F 2 "Capacitor_SMD:C_0603_1608Metric_Pad1.05x0.95mm_HandSolder" H 9000 1200 50  0001 C CNN
-F 3 "~" H 9000 1200 50  0001 C CNN
-	1    9000 1200
-	0    -1   -1   0
-$EndComp
 Wire Wire Line
 	6400 2150 7950 2150
@@
 Wire Wire Line
 	4750 5000 5700 5000
+Wire Wire Line
+	1100 700  2600 700
+Wire Wire Line
+	1100 800  2600 800
+Wire Wire Line
+	1100 1150 2600 1150
+Wire Wire Line
+	1100 1250 2600 1250
 $Comp
-L Device:Jumper_NO_Small JP1
-U 1 1 5CE47FCE
-P 1450 700
-F 0 "JP1" H 1450 900 50  0000 C CNN
-F 1 "Jumper_NO_Small" H 1450 800 50  0000 C CNN
-F 2 "Jumper:SolderJumper-2_P1.3mm_Open_TrianglePad1.0x1.5mm" H 1450 700 50  0001 C CNN
-F 3 "~" H 1450 700 50  0001 C CNN
-	1    1450 700
-	1    0    0    -1
+L taobao-cp:CP100uf,10V C1
+U 1 1 5CCCEC7F
+P 9000 1200
+F 0 "C1" V 9225 1200 50  0000 C CNN
+F 1 "CP100uf,10V" V 9134 1200 50  0000 C CNN
+F 2 "Capacitor_SMD:CP_Elec_6.3x5.3" H 9000 1200 50  0001 C CNN
+F 3 "~" H 9000 1200 50  0001 C CNN
+	1    9000 1200
+	0    -1   -1   0
 $EndComp
-$Comp
-L Device:Jumper_NO_Small JP2
-U 1 1 5CE4801F
-P 1450 800
-F 0 "JP2" H 1450 1000 50  0000 C CNN
-F 1 "Jumper_NO_Small" H 1450 900 50  0000 C CNN
-F 2 "Jumper:SolderJumper-2_P1.3mm_Open_TrianglePad1.0x1.5mm" H 1450 800 50  0001 C CNN
-F 3 "~" H 1450 800 50  0001 C CNN
-	1    1450 800
-	1    0    0    -1
-$EndComp
-$Comp
-L Device:Jumper_NO_Small JP3
-U 1 1 5CE48043
-P 1450 1150
-F 0 "JP3" H 1450 1350 50  0000 C CNN
-F 1 "Jumper_NO_Small" H 1450 1250 50  0000 C CNN
-F 2 "Jumper:SolderJumper-2_P1.3mm_Open_TrianglePad1.0x1.5mm" H 1450 1150 50  0001 C CNN
-F 3 "~" H 1450 1150 50  0001 C CNN
-	1    1450 1150
-	1    0    0    -1
-$EndComp
-$Comp
-L Device:Jumper_NO_Small JP4
-U 1 1 5CE48098
-P 1450 1250
-F 0 "JP4" H 1450 1450 50  0000 C CNN
-F 1 "Jumper_NO_Small" H 1450 1350 50  0000 C CNN
-F 2 "Jumper:SolderJumper-2_P1.3mm_Open_TrianglePad1.0x1.5mm" H 1450 1250 50  0001 C CNN
-F 3 "~" H 1450 1250 50  0001 C CNN
-	1    1450 1250
-	1    0    0    -1
-$EndComp
-Wire Wire Line
-	1100 700  1350 700
-Wire Wire Line
-	1100 800  1350 800
-Wire Wire Line
-	1100 1150 1350 1150
-Wire Wire Line
-	1100 1250 1350 1250
-Wire Wire Line
-	1550 700  2600 700
-Wire Wire Line
-	1550 800  2600 800
-Wire Wire Line
-	1550 1150 2600 1150
-Wire Wire Line
-	1550 1250 2600 1250
 $EndSCHEMATC

Commit message: update,
Other:
- note added: "THIS IS OPTIONAL\nREFER TO STM32 SIDE"
- moved on the sheet: R6
Changed lines of the file:
@@
 L taobao-r:R152,0603 R?
 U 1 1 5CE4405F
-P 4750 5250
+P 5100 5250
 AR Path="/5CC29851/5CC2A1CB/5CE4405F" Ref="R?"  Part="1"
 AR Path="/5CC0166A/5CE4405F" Ref="R6"  Part="1"
 AR Path="/5CE4405F" Ref="R6"  Part="1"
-F 0 "R6" H 4850 5300 50  0000 L CNN
-F 1 "R152,0603" H 4850 5250 50  0000 L CNN
-F 2 "Resistor_SMD:R_0603_1608Metric_Pad1.05x0.95mm_HandSolder" H 4750 5250 50  0001 C CNN
-F 3 "~" H 4750 5250 50  0001 C CNN
-	1    4750 5250
+F 0 "R6" H 5200 5300 50  0000 L CNN
+F 1 "R152,0603" H 5200 5250 50  0000 L CNN
+F 2 "Resistor_SMD:R_0603_1608Metric_Pad1.05x0.95mm_HandSolder" H 5100 5250 50  0001 C CNN
+F 3 "~" H 5100 5250 50  0001 C CNN
+	1    5100 5250
 	1    0    0    -1
 $EndComp
@@
 L taobao-components:+3V3_STM32 #PWR?
 U 1 1 5CE44066
-P 4750 5450
+P 5100 5650
 AR Path="/5CC29851/5CC2A1CB/5CE44066" Ref="#PWR?"  Part="1"
 AR Path="/5CC0166A/5CE44066" Ref="#PWR06"  Part="1"
 AR Path="/5CE44066" Ref="#PWR06"  Part="1"
-F 0 "#PWR06" H 4750 5300 50  0001 C CNN
-F 1 "+3V3_STM32" H 4750 5650 50  0000 C CNN
-F 2 "" H 4750 5450 50  0001 C CNN
-F 3 "" H 4750 5450 50  0001 C CNN
-	1    4750 5450
+F 0 "#PWR06" H 5100 5500 50  0001 C CNN
+F 1 "+3V3_STM32" H 5100 5850 50  0000 C CNN
+F 2 "" H 5100 5650 50  0001 C CNN
+F 3 "" H 5100 5650 50  0001 C CNN
+	1    5100 5650
 	-1   0    0    1
 $EndComp
 Wire Wire Line
-	4750 5350 4750 5450
-Wire Wire Line
-	4750 5000 4750 5150
-Connection ~ 4750 5000
-Wire Wire Line
-	4750 5000 4650 5000
+	5100 5350 5100 5650
 Text Label 5700 4900 2    50   ~ 0
 USB-DM2
@@
 Wire Wire Line
 	4650 4900 5700 4900
-Wire Wire Line
-	4750 5000 5700 5000
 Wire Wire Line
 	1100 700  2600 700
@@
 	0    -1   -1   0
 $EndComp
+Wire Wire Line
+	4650 5000 5100 5000
+Wire Wire Line
+	5100 5000 5100 5150
+Connection ~ 5100 5000
+Wire Wire Line
+	5100 5000 5700 5000
+Wire Notes Line
+	4950 5100 4950 5450
+Wire Notes Line
+	4950 5450 6100 5450
+Wire Notes Line
+	6100 5450 6100 5100
+Wire Notes Line
+	6100 5100 4950 5100
+Text Notes 5250 5450 0    50   ~ 0
+THIS IS OPTIONAL\nREFER TO STM32 SIDE
 $EndSCHEMATC
