File: hardware/printer-board/orange_pi.sch (KiCad schematic (older format))
At the start: 8 parts, among them J1 USB_DEBUG, U1 orange_pi_zero

Commit message: update,
Parts:
- J1: footprint Connector_PinHeader_1.27mm:PinHeader_1x05_P1.27mm_Vertical -> Connector_PinHeader_1.27mm:PinHeader_1x04_P1.27mm_Vertical; symbol Connector_Generic:Conn_01x05 -> Connector_Generic:Conn_01x04
Connections:
- net +5V: now also J1.4 (Pin_4); no longer J1.5 (Pin_5)
- net OPI_USB-DM2: now also J1.2 (Pin_2), R4.2; no longer R4.1, U1.3 (USB-DM2)
- net OPI_USB-DP2: now also J1.3 (Pin_3), R5.2; no longer R5.1, R6.1, U1.4 (USB-DP2)
- net OPI_USB-DM3 renamed USB-DM3
- net OPI_USB-DP3 renamed USB-DP3
- new net USB-DM2: R4.1, U1.3 (USB-DM2)
- new net USB-DP2: R5.1, R6.1, U1.4 (USB-DP2)
Other:
- moved on the sheet: R4, R5
Changed lines of the file:
@@
 	7250 2650 7950 2650
 Text Label 2600 700  2    50   ~ 0
-USB-DM2
+OPI_USB-DM2
 Text Label 2600 800  2    50   ~ 0
-USB-DP2
-Text Label 2600 1150 2    50   ~ 0
-USB-DM3
-Text Label 2600 1250 2    50   ~ 0
-USB-DP3
+OPI_USB-DP2
 Text HLabel 1100 700  0    50   Input ~ 0
 OPI_USB-DM2
 Text HLabel 1100 800  0    50   Input ~ 0
 OPI_USB-DP2
-Text HLabel 1100 1150 0    50   Input ~ 0
-OPI_USB-DM3
-Text HLabel 1100 1250 0    50   Input ~ 0
-OPI_USB-DP3
 Wire Wire Line
 	6400 2150 7950 2150
@@
 	6400 2250 7950 2250
 $Comp
-L Connector_Generic:Conn_01x05 J?
+L Connector_Generic:Conn_01x04 J?
 U 1 1 5CE44033
-P 4000 5000
+P 4000 4900
 AR Path="/5CC29851/5CC2A1CB/5CE44033" Ref="J?"  Part="1"
 AR Path="/5CC0166A/5CE44033" Ref="J1"  Part="1"
 AR Path="/5CE44033" Ref="J1"  Part="1"
-F 0 "J1" H 3900 5450 50  0000 C CNN
-F 1 "USB_DEBUG" H 3900 5350 50  0000 C CNN
-F 2 "Connector_PinHeader_1.27mm:PinHeader_1x05_P1.27mm_Vertical" H 4000 5000 50  0001 C CNN
-F 3 "~" H 4000 5000 50  0001 C CNN
-	1    4000 5000
+F 0 "J1" H 3900 5350 50  0000 C CNN
+F 1 "USB_DEBUG" H 3900 5250 50  0000 C CNN
+F 2 "Connector_PinHeader_1.27mm:PinHeader_1x04_P1.27mm_Vertical" H 4000 4900 50  0001 C CNN
+F 3 "~" H 4000 4900 50  0001 C CNN
+	1    4000 4900
 	-1   0    0    -1
 $EndComp
@@
 L power:+5V #PWR?
 U 1 1 5CE4403A
-P 4550 5300
+P 4550 5200
 AR Path="/5CC29851/5CC2A1CB/5CE4403A" Ref="#PWR?"  Part="1"
 AR Path="/5CC0166A/5CE4403A" Ref="#PWR04"  Part="1"
 AR Path="/5CE4403A" Ref="#PWR04"  Part="1"
-F 0 "#PWR04" H 4550 5150 50  0001 C CNN
-F 1 "+5V" H 4600 5500 50  0000 C CNN
-F 2 "" H 4550 5300 50  0001 C CNN
-F 3 "" H 4550 5300 50  0001 C CNN
-	1    4550 5300
+F 0 "#PWR04" H 4550 5050 50  0001 C CNN
+F 1 "+5V" H 4600 5400 50  0000 C CNN
+F 2 "" H 4550 5200 50  0001 C CNN
+F 3 "" H 4550 5200 50  0001 C CNN
+	1    4550 5200
 	1    0    0    1
 $EndComp
 Wire Wire Line
-	4550 5300 4550 5200
+	4550 5200 4550 5100
 Wire Wire Line
-	4550 5200 4200 5200
+	4550 5100 4200 5100
 $Comp
 L power:GND #PWR?
@@
 Wire Wire Line
 	4550 4800 4550 4650
-Wire Wire Line
-	4200 5100 4550 5100
 $Comp
 L taobao-r:R220,0603 R?
 U 1 1 5CE4404D
-P 4550 4900
+P 4800 4900
 AR Path="/5CC29851/5CC2A1CB/5CE4404D" Ref="R?"  Part="1"
 AR Path="/5CC0166A/5CE4404D" Ref="R4"  Part="1"
 AR Path="/5CE4404D" Ref="R4"  Part="1"
-F 0 "R4" V 4300 4900 50  0000 C CNN
-F 1 "R220,0603" V 4400 4900 50  0000 C CNN
-F 2 "Resistor_SMD:R_0603_1608Metric_Pad1.05x0.95mm_HandSolder" H 4550 4900 50  0001 C CNN
-F 3 "~" H 4550 4900 50  0001 C CNN
-	1    4550 4900
+F 0 "R4" V 4550 4900 50  0000 C CNN
+F 1 "R220,0603" V 4650 4900 50  0000 C CNN
+F 2 "Resistor_SMD:R_0603_1608Metric_Pad1.05x0.95mm_HandSolder" H 4800 4900 50  0001 C CNN
+F 3 "~" H 4800 4900 50  0001 C CNN
+	1    4800 4900
 	0    1    1    0
 $EndComp
@@
 L taobao-r:R220,0603 R?
 U 1 1 5CE44054
-P 4550 5000
+P 4800 5000
 AR Path="/5CC29851/5CC2A1CB/5CE44054" Ref="R?"  Part="1"
 AR Path="/5CC0166A/5CE44054" Ref="R5"  Part="1"
 AR Path="/5CE44054" Ref="R5"  Part="1"
-F 0 "R5" V 4300 5000 50  0000 C CNN
-F 1 "R220,0603" V 4400 5000 50  0000 C CNN
-F 2 "Resistor_SMD:R_0603_1608Metric_Pad1.05x0.95mm_HandSolder" H 4550 5000 50  0001 C CNN
-F 3 "~" H 4550 5000 50  0001 C CNN
-	1    4550 5000
+F 0 "R5" V 4550 5000 50  0000 C CNN
+F 1 "R220,0603" V 4650 5000 50  0000 C CNN
+F 2 "Resistor_SMD:R_0603_1608Metric_Pad1.05x0.95mm_HandSolder" H 4800 5000 50  0001 C CNN
+F 3 "~" H 4800 5000 50  0001 C CNN
+	1    4800 5000
 	0    1    1    0
 $EndComp
 Wire Wire Line
-	4200 4900 4450 4900
+	4200 4900 4700 4900
 Wire Wire Line
-	4200 5000 4450 5000
+	4200 5000 4700 5000
 $Comp
 L taobao-r:R152,0603 R?
@@
 USB-DP2
 Wire Wire Line
-	4650 4900 5700 4900
+	4900 4900 5700 4900
 Wire Wire Line
 	1100 700  2600 700
 Wire Wire Line
 	1100 800  2600 800
-Wire Wire Line
-	1100 1150 2600 1150
-Wire Wire Line
-	1100 1250 2600 1250
 $Comp
 L taobao-cp:CP100uf,10V C1
@@
 $EndComp
 Wire Wire Line
-	4650 5000 5100 5000
+	4900 5000 5100 5000
 Wire Wire Line
 	5100 5000 5100 5150
@@
 Text Notes 5250 5450 0    50   ~ 0
 THIS IS OPTIONAL\nREFER TO STM32 SIDE
+Text Label 4300 4900 0    50   ~ 0
+OPI_USB-DM2
+Text Label 4300 5000 0    50   ~ 0
+OPI_USB-DP2
 $EndSCHEMATC
