File: hardware/printer-board/FAN2.sch (KiCad schematic (older format))
At the start: 8 parts, among them J1 TO FAN2, Q6 D882

Commit message: update,
Parts:
- Q6: footprint Package_TO_SOT_SMD:SOT-89-3 -> footprint-lib:SOT-89-3,thermal_vias
Changed lines of the file:
@@
 $Descr A4 11693 8268
 encoding utf-8
-Sheet 26 29
+Sheet 24 29
 Title ""
 Date ""
@@
 F 0 "Q6" H 3350 3700 50  0000 L CNN
 F 1 "D882" H 3350 3650 50  0000 L CNN
-F 2 "Package_TO_SOT_SMD:SOT-89-3" H 3350 3750 50  0001 C CNN
+F 2 "footprint-lib:SOT-89-3,thermal_vias" H 3350 3750 50  0001 C CNN
 F 3 "" H 3150 3650 50  0001 C CNN
 	1    3150 3650

Commit message: update to re-annotation,
Parts:
- renumbered C1 to C38, D1 to D22, J1 to J35, R3 to R64, R4 to R65, R49 to R66, R1 to R67
Changed lines of the file:
@@
 AR Path="/5CC2401E/5CC242A1/5CC8A034" Ref="J?"  Part="1"
 AR Path="/5CC2401E/5CC24321/5CC8A034" Ref="J?"  Part="1"
-AR Path="/5CC8A034" Ref="J1"  Part="1"
-AR Path="/5CC2401E/5CC24398/5CC8A034" Ref="J1"  Part="1"
-F 0 "J1" H 4300 2550 50  0000 C CNN
+AR Path="/5CC8A034" Ref="J?"  Part="1"
+AR Path="/5CC2401E/5CC24398/5CC8A034" Ref="J35"  Part="1"
+F 0 "J35" H 4300 2550 50  0000 C CNN
 F 1 "TO FAN2" H 4300 2650 50  0000 C CNN
 F 2 "footprint-lib:b2b-ph-kl,fan_pwm_out" H 4350 2900 50  0001 C CNN
@@
 AR Path="/5CC2401E/5CC242A1/5CC8A043" Ref="R?"  Part="1"
 AR Path="/5CC2401E/5CC24321/5CC8A043" Ref="R?"  Part="1"
-AR Path="/5CC8A043" Ref="R3"  Part="1"
-AR Path="/5CC2401E/5CC24398/5CC8A043" Ref="R3"  Part="1"
-F 0 "R3" V 2304 3650 50  0000 C CNN
+AR Path="/5CC8A043" Ref="R?"  Part="1"
+AR Path="/5CC2401E/5CC24398/5CC8A043" Ref="R64"  Part="1"
+F 0 "R64" V 2304 3650 50  0000 C CNN
 F 1 "R100,0805" V 2395 3650 50  0000 C CNN
 F 2 "Resistor_SMD:R_0603_1608Metric_Pad1.05x0.95mm_HandSolder" H 2500 3650 50  0001 C CNN
@@
 AR Path="/5CC2401E/5CC242A1/5CC04D61" Ref="R?"  Part="1"
 AR Path="/5CC2401E/5CC24321/5CC04D61" Ref="R?"  Part="1"
-AR Path="/5CC04D61" Ref="R4"  Part="1"
-AR Path="/5CC2401E/5CC24398/5CC04D61" Ref="R86"  Part="1"
-F 0 "R86" V 2304 4050 50  0000 C CNN
+AR Path="/5CC04D61" Ref="R?"  Part="1"
+AR Path="/5CC2401E/5CC24398/5CC04D61" Ref="R65"  Part="1"
+F 0 "R65" V 2304 4050 50  0000 C CNN
 F 1 "R104,0805" V 2395 4050 50  0000 C CNN
 F 2 "Resistor_SMD:R_0805_2012Metric_Pad1.15x1.40mm_HandSolder" H 2500 4050 50  0001 C CNN
@@
 AR Path="/5CC2401E/5CC242A1/5CC8A039" Ref="#PWR?"  Part="1"
 AR Path="/5CC2401E/5CC24321/5CC8A039" Ref="#PWR?"  Part="1"
-AR Path="/5CC8A039" Ref="#PWR0101"  Part="1"
-AR Path="/5CC2401E/5CC24398/5CC8A039" Ref="#PWR0158"  Part="1"
-F 0 "#PWR0158" H 3250 4000 50  0001 C CNN
+AR Path="/5CC8A039" Ref="#PWR?"  Part="1"
+AR Path="/5CC2401E/5CC24398/5CC8A039" Ref="#PWR0170"  Part="1"
+F 0 "#PWR0170" H 3250 4000 50  0001 C CNN
 F 1 "GND" H 3255 4077 50  0000 C CNN
 F 2 "" H 3250 4250 50  0001 C CNN
@@
 AR Path="/5CC2401E/5CC242A1/5CC8A036" Ref="R?"  Part="1"
 AR Path="/5CC2401E/5CC24321/5CC8A036" Ref="R?"  Part="1"
-AR Path="/5CC8A036" Ref="R1"  Part="1"
-AR Path="/5CC2401E/5CC24398/5CC8A036" Ref="R48"  Part="1"
-F 0 "R48" H 3809 2546 50  0000 L CNN
+AR Path="/5CC8A036" Ref="R?"  Part="1"
+AR Path="/5CC2401E/5CC24398/5CC8A036" Ref="R67"  Part="1"
+F 0 "R67" H 3809 2546 50  0000 L CNN
 F 1 "R182,0603" H 3809 2455 50  0000 L CNN
 F 2 "Resistor_SMD:R_0603_1608Metric_Pad1.05x0.95mm_HandSolder" H 3750 2500 50  0001 C CNN
@@
 AR Path="/5CC2401E/5CC242A1/5CC8A03A" Ref="#PWR?"  Part="1"
 AR Path="/5CC2401E/5CC24321/5CC8A03A" Ref="#PWR?"  Part="1"
-AR Path="/5CC8A03A" Ref="#PWR0102"  Part="1"
-AR Path="/5CC2401E/5CC24398/5CC8A03A" Ref="#PWR0163"  Part="1"
-F 0 "#PWR0163" H 4000 2050 50  0001 C CNN
+AR Path="/5CC8A03A" Ref="#PWR?"  Part="1"
+AR Path="/5CC2401E/5CC24398/5CC8A03A" Ref="#PWR0171"  Part="1"
+F 0 "#PWR0171" H 4000 2050 50  0001 C CNN
 F 1 "+12V" H 4015 2373 50  0000 C CNN
 F 2 "" H 4000 2200 50  0001 C CNN
@@
 AR Path="/5CC2401E/5CC242A1/5CC24377" Ref="D?"  Part="1"
 AR Path="/5CC2401E/5CC24321/5CC24377" Ref="D?"  Part="1"
-AR Path="/5CC24377" Ref="D1"  Part="1"
-AR Path="/5CC2401E/5CC24398/5CC24377" Ref="D1"  Part="1"
-F 0 "D1" V 3704 2898 50  0000 L CNN
+AR Path="/5CC24377" Ref="D?"  Part="1"
+AR Path="/5CC2401E/5CC24398/5CC24377" Ref="D22"  Part="1"
+F 0 "D22" V 3704 2898 50  0000 L CNN
 F 1 "LED_BLUE,0603" V 3795 2898 50  0000 L CNN
 F 2 "LED_SMD:LED_0603_1608Metric_Pad1.05x0.95mm_HandSolder" V 3750 2800 50  0001 C CNN
@@
 AR Path="/5CC2401E/5CC242A1/5CC8A03C" Ref="#PWR?"  Part="1"
 AR Path="/5CC2401E/5CC24321/5CC8A03C" Ref="#PWR?"  Part="1"
-AR Path="/5CC8A03C" Ref="#PWR0103"  Part="1"
-AR Path="/5CC2401E/5CC24398/5CC8A03C" Ref="#PWR0164"  Part="1"
-F 0 "#PWR0164" H 2600 4600 50  0001 C CNN
+AR Path="/5CC8A03C" Ref="#PWR?"  Part="1"
+AR Path="/5CC2401E/5CC24398/5CC8A03C" Ref="#PWR0168"  Part="1"
+F 0 "#PWR0168" H 2600 4600 50  0001 C CNN
 F 1 "+12V" V 2615 4878 50  0000 L CNN
 F 2 "" H 2600 4750 50  0001 C CNN
@@
 AR Path="/5CC2401E/5CC242A1/5CC8A03E" Ref="#PWR?"  Part="1"
 AR Path="/5CC2401E/5CC24321/5CC8A03E" Ref="#PWR?"  Part="1"
-AR Path="/5CC8A03E" Ref="#PWR0104"  Part="1"
-AR Path="/5CC2401E/5CC24398/5CC8A03E" Ref="#PWR0165"  Part="1"
-F 0 "#PWR0165" H 3100 4500 50  0001 C CNN
+AR Path="/5CC8A03E" Ref="#PWR?"  Part="1"
+AR Path="/5CC2401E/5CC24398/5CC8A03E" Ref="#PWR0169"  Part="1"
+F 0 "#PWR0169" H 3100 4500 50  0001 C CNN
 F 1 "GND" H 3105 4577 50  0000 C CNN
 F 2 "" H 3100 4750 50  0001 C CNN
@@
 AR Path="/5CC2401E/5CC242A1/5CC24303" Ref="C?"  Part="1"
 AR Path="/5CC2401E/5CC24321/5CC24303" Ref="C?"  Part="1"
-AR Path="/5CC24303" Ref="C1"  Part="1"
-AR Path="/5CC2401E/5CC24398/5CC24303" Ref="C55"  Part="1"
-F 0 "C55" V 3075 4750 50  0000 C CNN
+AR Path="/5CC24303" Ref="C?"  Part="1"
+AR Path="/5CC2401E/5CC24398/5CC24303" Ref="C38"  Part="1"
+F 0 "C38" V 3075 4750 50  0000 C CNN
 F 1 "CP100uf,16V" V 2984 4750 50  0000 C CNN
 F 2 "Capacitor_SMD:CP_Elec_6.3x5.3" H 2850 4750 50  0001 C CNN
@@
 $EndComp
 $Comp
-L taobao-r:R100,0603 R49
+L taobao-r:R100,0603 R66
 U 1 1 5CC88B15
 P 3250 3150
-F 0 "R49" H 3350 3200 50  0000 L CNN
+F 0 "R66" H 3350 3200 50  0000 L CNN
 F 1 "R100,0603" H 3350 3150 50  0000 L CNN
 F 2 "Resistor_SMD:R_0603_1608Metric_Pad1.05x0.95mm_HandSolder" H 3250 3150 50  0001 C CNN

Commit message: update step motor terminal orientation,
Parts:
- removed C38: CP100uf,16V, Capacitor_SMD:CP_Elec_6.3x5.3, symbol taobao-cp:CP100uf,16V
- added C38: CP1uf,50V, Capacitor_SMD:CP_Elec_4x5.3, symbol taobao-cp:CP1uf,50V
Connections:
- net +12V: now also C38.1
- net at D22.1 (K), J35.2 (Pin_2), R66.1: now also C38.2

Commit message: update ROUTING,
Connections:
- net FAN_EN renamed FAN2_EN
Changed lines of the file:
@@
 $Descr A4 11693 8268
 encoding utf-8
-Sheet 24 27
+Sheet 22 28
 Title ""
 Date ""
@@
 AR Path="/5CC8A034" Ref="J35"  Part="1"
 AR Path="/5CC2401E/5CC24398/5CC8A034" Ref="J35"  Part="1"
-F 0 "J35" H 4300 2550 50  0000 C CNN
+AR Path="/5CC2401E/5CE3779D/5CC8A034" Ref="J?"  Part="1"
+F 0 "J?" H 4300 2550 50  0000 C CNN
 F 1 "TO FAN2" H 4300 2650 50  0000 C CNN
 F 2 "footprint-lib:b2b-ph-kl,fan_pwm_out" H 4350 2900 50  0001 C CNN
@@
 AR Path="/5CC8A043" Ref="R64"  Part="1"
 AR Path="/5CC2401E/5CC24398/5CC8A043" Ref="R64"  Part="1"
-F 0 "R64" V 2304 3650 50  0000 C CNN
+AR Path="/5CC2401E/5CE3779D/5CC8A043" Ref="R?"  Part="1"
+F 0 "R?" V 2304 3650 50  0000 C CNN
 F 1 "R100,0805" V 2395 3650 50  0000 C CNN
 F 2 "Resistor_SMD:R_0603_1608Metric_Pad1.05x0.95mm_HandSolder" H 2500 3650 50  0001 C CNN
@@
 AR Path="/5CC04D61" Ref="R65"  Part="1"
 AR Path="/5CC2401E/5CC24398/5CC04D61" Ref="R65"  Part="1"
-F 0 "R65" V 2304 4050 50  0000 C CNN
+AR Path="/5CC2401E/5CE3779D/5CC04D61" Ref="R?"  Part="1"
+F 0 "R?" V 2304 4050 50  0000 C CNN
 F 1 "R104,0805" V 2395 4050 50  0000 C CNN
 F 2 "Resistor_SMD:R_0805_2012Metric_Pad1.15x1.40mm_HandSolder" H 2500 4050 50  0001 C CNN
@@
 AR Path="/5CC8A039" Ref="#PWR0170"  Part="1"
 AR Path="/5CC2401E/5CC24398/5CC8A039" Ref="#PWR0170"  Part="1"
-F 0 "#PWR0170" H 3250 4000 50  0001 C CNN
+AR Path="/5CC2401E/5CE3779D/5CC8A039" Ref="#PWR?"  Part="1"
+F 0 "#PWR?" H 3250 4000 50  0001 C CNN
 F 1 "GND" H 3255 4077 50  0000 C CNN
 F 2 "" H 3250 4250 50  0001 C CNN
@@
 AR Path="/5CC8A036" Ref="R67"  Part="1"
 AR Path="/5CC2401E/5CC24398/5CC8A036" Ref="R67"  Part="1"
-F 0 "R67" H 3809 2546 50  0000 L CNN
+AR Path="/5CC2401E/5CE3779D/5CC8A036" Ref="R?"  Part="1"
+F 0 "R?" H 3809 2546 50  0000 L CNN
 F 1 "R182,0603" H 3809 2455 50  0000 L CNN
 F 2 "Resistor_SMD:R_0603_1608Metric_Pad1.05x0.95mm_HandSolder" H 3750 2500 50  0001 C CNN
@@
 	4150 2900 4000 2900
 Text HLabel 1250 900  0    50   Input ~ 0
-FAN_EN
+FAN2_EN
 Text Label 2050 900  2    50   ~ 0
-FAN_EN
+FAN2_EN
 Wire Wire Line
 	1250 900  2050 900
 Text Label 1350 3650 0    50   ~ 0
-FAN_EN
+FAN2_EN
 Wire Wire Line
 	1350 3650 2000 3650
@@
 AR Path="/5CC8A03A" Ref="#PWR0171"  Part="1"
 AR Path="/5CC2401E/5CC24398/5CC8A03A" Ref="#PWR0171"  Part="1"
-F 0 "#PWR0171" H 4000 2050 50  0001 C CNN
+AR Path="/5CC2401E/5CE3779D/5CC8A03A" Ref="#PWR?"  Part="1"
+F 0 "#PWR?" H 4000 2050 50  0001 C CNN
 F 1 "+12V" H 4015 2373 50  0000 C CNN
 F 2 "" H 4000 2200 50  0001 C CNN
@@
 AR Path="/5CC24377" Ref="D22"  Part="1"
 AR Path="/5CC2401E/5CC24398/5CC24377" Ref="D22"  Part="1"
-F 0 "D22" V 3704 2898 50  0000 L CNN
+AR Path="/5CC2401E/5CE3779D/5CC24377" Ref="D?"  Part="1"
+F 0 "D?" V 3704 2898 50  0000 L CNN
 F 1 "LED_BLUE,0603" V 3795 2898 50  0000 L CNN
 F 2 "LED_SMD:LED_0603_1608Metric_Pad1.05x0.95mm_HandSolder" V 3750 2800 50  0001 C CNN
@@
 U 1 1 5CC8A046
 P 3150 3650
-F 0 "Q6" H 3350 3700 50  0000 L CNN
+AR Path="/5CC2401E/5CC24398/5CC8A046" Ref="Q6"  Part="1"
+AR Path="/5CC2401E/5CE3779D/5CC8A046" Ref="Q?"  Part="1"
+F 0 "Q?" H 3350 3700 50  0000 L CNN
 F 1 "D882" H 3350 3650 50  0000 L CNN
 F 2 "footprint-lib:SOT-89-3,thermal_vias" H 3350 3750 50  0001 C CNN
@@
 U 1 1 5CC88B15
 P 3250 3150
-F 0 "R66" H 3350 3200 50  0000 L CNN
+AR Path="/5CC2401E/5CC24398/5CC88B15" Ref="R66"  Part="1"
+AR Path="/5CC2401E/5CE3779D/5CC88B15" Ref="R?"  Part="1"
+F 0 "R?" H 3350 3200 50  0000 L CNN
 F 1 "R100,0603" H 3350 3150 50  0000 L CNN
 F 2 "Resistor_SMD:R_0603_1608Metric_Pad1.05x0.95mm_HandSolder" H 3250 3150 50  0001 C CNN
@@
 U 1 1 5CCBFCA7
 P 3450 2700
-F 0 "C38" H 3363 2746 50  0000 R CNN
+AR Path="/5CC2401E/5CC24398/5CCBFCA7" Ref="C38"  Part="1"
+AR Path="/5CC2401E/5CE3779D/5CCBFCA7" Ref="C?"  Part="1"
+F 0 "C?" H 3363 2746 50  0000 R CNN
 F 1 "CP1uf,50V" H 3363 2655 50  0000 R CNN
 F 2 "Capacitor_SMD:CP_Elec_4x5.3" H 3450 2700 50  0001 C CNN
