File: hardware/printer-board/MP2303A_power_supply_5V.sch (KiCad schematic (older format))
At the start: 10 parts, among them U12 MP2303A_ALT

Commit message: update to re-annotation,
Parts:
- U11: renamed from U12; footprint Package_SO:SOIC-8_3.9x4.9mm_P1.27mm -> footprint-lib:SOIC-8_3.9x4.9mm_P1.27mm,thermal_via
- renumbered C50 to C45, C51 to C46, C54 to C47, C49 to C48, C53 to C49, L4 to L2, R91 to R74, R90 to R75, R89 to R76
Changed lines of the file:
@@
 $Descr A4 11693 8268
 encoding utf-8
-Sheet 33 29
+Sheet 28 29
 Title ""
 Date ""
@@
 $EndBitmap
 $Comp
-L taobao-components:MP2303A_ALT U12
+L taobao-components:MP2303A_ALT U?
 U 1 1 5CC8BB6B
 P 5000 3500
-AR Path="/5CC86276/5CC8BB6B" Ref="U12"  Part="1"
-AR Path="/5CCA7EF8/5CC8BB6B" Ref="U2"  Part="1"
-F 0 "U2" H 5600 3550 50  0000 L CNN
+AR Path="/5CC86276/5CC8BB6B" Ref="U?"  Part="1"
+AR Path="/5CCA7EF8/5CC8BB6B" Ref="U11"  Part="1"
+F 0 "U11" H 5600 3550 50  0000 L CNN
 F 1 "MP2303A_ALT" H 5600 3450 50  0000 L CNN
-F 2 "Package_SO:SOIC-8_3.9x4.9mm_P1.27mm" H 5000 3500 50  0001 C CNN
+F 2 "footprint-lib:SOIC-8_3.9x4.9mm_P1.27mm,thermal_via" H 5000 3500 50  0001 C CNN
 F 3 "" H 5000 3500 50  0001 C CNN
 	1    5000 3500
@@
 $EndComp
 $Comp
-L power:+12V #PWR0131
+L power:+12V #PWR?
 U 1 1 5CC8BD49
 P 3100 2700
-AR Path="/5CC86276/5CC8BD49" Ref="#PWR0131"  Part="1"
-AR Path="/5CCA7EF8/5CC8BD49" Ref="#PWR0110"  Part="1"
-F 0 "#PWR0110" H 3100 2550 50  0001 C CNN
+AR Path="/5CC86276/5CC8BD49" Ref="#PWR?"  Part="1"
+AR Path="/5CCA7EF8/5CC8BD49" Ref="#PWR0203"  Part="1"
+F 0 "#PWR0203" H 3100 2550 50  0001 C CNN
 F 1 "+12V" H 3150 2900 50  0000 C CNN
 F 2 "" H 3100 2700 50  0001 C CNN
@@
 	3100 2700 3100 2850
 $Comp
-L power:GND #PWR0136
+L power:GND #PWR?
 U 1 1 5CC8BDB4
 P 3100 3900
-AR Path="/5CC86276/5CC8BDB4" Ref="#PWR0136"  Part="1"
-AR Path="/5CCA7EF8/5CC8BDB4" Ref="#PWR0114"  Part="1"
-F 0 "#PWR0114" H 3100 3650 50  0001 C CNN
+AR Path="/5CC86276/5CC8BDB4" Ref="#PWR?"  Part="1"
+AR Path="/5CCA7EF8/5CC8BDB4" Ref="#PWR0204"  Part="1"
+F 0 "#PWR0204" H 3100 3650 50  0001 C CNN
 F 1 "GND" H 3150 3700 50  0000 C CNN
 F 2 "" H 3100 3900 50  0001 C CNN
@@
 	3100 2850 3100 3250
 $Comp
-L taobao-c:C104,0603 C51
+L taobao-c:C104,0603 C?
 U 1 1 5CCACF45
 P 4250 3900
-AR Path="/5CC86276/5CCACF45" Ref="C51"  Part="1"
-AR Path="/5CCA7EF8/5CCACF45" Ref="C47"  Part="1"
-F 0 "C47" H 4350 3950 50  0000 L CNN
+AR Path="/5CC86276/5CCACF45" Ref="C?"  Part="1"
+AR Path="/5CCA7EF8/5CCACF45" Ref="C46"  Part="1"
+F 0 "C46" H 4350 3950 50  0000 L CNN
 F 1 "C104,0603" H 4350 3900 50  0000 L CNN
 F 2 "Capacitor_SMD:C_0603_1608Metric_Pad1.05x0.95mm_HandSolder" H 4250 3900 50  0001 C CNN
@@
 	4250 3650 4450 3650
 $Comp
-L power:GND #PWR0141
+L power:GND #PWR?
 U 1 1 5CC8C048
 P 4250 4200
-AR Path="/5CC86276/5CC8C048" Ref="#PWR0141"  Part="1"
-AR Path="/5CCA7EF8/5CC8C048" Ref="#PWR0119"  Part="1"
-F 0 "#PWR0119" H 4250 3950 50  0001 C CNN
+AR Path="/5CC86276/5CC8C048" Ref="#PWR?"  Part="1"
+AR Path="/5CCA7EF8/5CC8C048" Ref="#PWR0205"  Part="1"
+F 0 "#PWR0205" H 4250 3950 50  0001 C CNN
 F 1 "GND" H 4300 4000 50  0000 C CNN
 F 2 "" H 4250 4200 50  0001 C CNN
@@
 	4250 4200 4250 4000
 $Comp
-L power:GND #PWR0142
+L power:GND #PWR?
 U 1 1 5CC8C171
 P 4850 4200
-AR Path="/5CC86276/5CC8C171" Ref="#PWR0142"  Part="1"
-AR Path="/5CCA7EF8/5CC8C171" Ref="#PWR0120"  Part="1"
-F 0 "#PWR0120" H 4850 3950 50  0001 C CNN
+AR Path="/5CC86276/5CC8C171" Ref="#PWR?"  Part="1"
+AR Path="/5CCA7EF8/5CC8C171" Ref="#PWR0206"  Part="1"
+F 0 "#PWR0206" H 4850 3950 50  0001 C CNN
 F 1 "GND" H 4900 4000 50  0000 C CNN
 F 2 "" H 4850 4200 50  0001 C CNN
@@
 	4850 4200 4850 3950
 $Comp
-L taobao-c:C103,0603 C49
+L taobao-c:C103,0603 C?
 U 1 1 5CC8C369
 P 5650 2850
-AR Path="/5CC86276/5CC8C369" Ref="C49"  Part="1"
-AR Path="/5CCA7EF8/5CC8C369" Ref="C5"  Part="1"
-F 0 "C5" V 5400 2850 50  0000 C CNN
+AR Path="/5CC86276/5CC8C369" Ref="C?"  Part="1"
+AR Path="/5CCA7EF8/5CC8C369" Ref="C48"  Part="1"
+F 0 "C48" V 5400 2850 50  0000 C CNN
 F 1 "C103,0603" V 5500 2850 50  0000 C CNN
 F 2 "Capacitor_SMD:C_0603_1608Metric_Pad1.05x0.95mm_HandSolder" H 5650 2850 50  0001 C CNN
@@
 	5150 2850 5150 3100
 $Comp
-L taobao-l:L_15uH L4
+L taobao-l:L_15uH L?
 U 1 1 5CC8C4E9
 P 6450 3450
-AR Path="/5CC86276/5CC8C4E9" Ref="L4"  Part="1"
-AR Path="/5CCA7EF8/5CC8C4E9" Ref="L1"  Part="1"
-F 0 "L1" V 6650 3450 50  0000 C CNN
+AR Path="/5CC86276/5CC8C4E9" Ref="L?"  Part="1"
+AR Path="/5CCA7EF8/5CC8C4E9" Ref="L2"  Part="1"
+F 0 "L2" V 6650 3450 50  0000 C CNN
 F 1 "L_15uH" V 6550 3450 50  0000 C CNN
 F 2 "w_smd_inductors:inductor_smd_4.8x2.8mm" H 6450 3450 50  0001 C CNN
@@
 	6100 3450 6350 3450
 $Comp
-L taobao-r:R562,0603 R91
+L taobao-r:R562,0603 R?
 U 1 1 5CC8C6EB
 P 5150 4550
-AR Path="/5CC86276/5CC8C6EB" Ref="R91"  Part="1"
-AR Path="/5CCA7EF8/5CC8C6EB" Ref="R50"  Part="1"
-F 0 "R50" H 5250 4600 50  0000 L CNN
+AR Path="/5CC86276/5CC8C6EB" Ref="R?"  Part="1"
+AR Path="/5CCA7EF8/5CC8C6EB" Ref="R74"  Part="1"
+F 0 "R74" H 5250 4600 50  0000 L CNN
 F 1 "R562,0603" H 5250 4550 50  0000 L CNN
 F 2 "Resistor_SMD:R_0603_1608Metric_Pad1.05x0.95mm_HandSolder" H 5150 4550 50  0001 C CNN
@@
 $EndComp
 $Comp
-L power:GND #PWR0143
+L power:GND #PWR?
 U 1 1 5CC8C737
 P 5150 5000
-AR Path="/5CC86276/5CC8C737" Ref="#PWR0143"  Part="1"
-AR Path="/5CCA7EF8/5CC8C737" Ref="#PWR0121"  Part="1"
-F 0 "#PWR0121" H 5150 4750 50  0001 C CNN
+AR Path="/5CC86276/5CC8C737" Ref="#PWR?"  Part="1"
+AR Path="/5CCA7EF8/5CC8C737" Ref="#PWR0207"  Part="1"
+F 0 "#PWR0207" H 5150 4750 50  0001 C CNN
 F 1 "GND" H 5200 4800 50  0000 C CNN
 F 2 "" H 5150 5000 50  0001 C CNN
@@
 $EndComp
 $Comp
-L taobao-c:C332,0603 C54
+L taobao-c:C332,0603 C?
 U 1 1 5CC8C910
 P 5150 4250
-AR Path="/5CC86276/5CC8C910" Ref="C54"  Part="1"
-AR Path="/5CCA7EF8/5CC8C910" Ref="C49"  Part="1"
-F 0 "C49" H 5250 4300 50  0000 L CNN
+AR Path="/5CC86276/5CC8C910" Ref="C?"  Part="1"
+AR Path="/5CCA7EF8/5CC8C910" Ref="C47"  Part="1"
+F 0 "C47" H 5250 4300 50  0000 L CNN
 F 1 "C332,0603" H 5250 4250 50  0000 L CNN
 F 2 "Capacitor_SMD:C_0603_1608Metric_Pad1.05x0.95mm_HandSolder" H 5150 4250 50  0001 C CNN
@@
 	5150 4650 5150 4850
 $Comp
-L taobao-r:R103,0603 R90
+L taobao-r:R103,0603 R?
 U 1 1 5CCACF4D
 P 6200 4400
-AR Path="/5CC86276/5CCACF4D" Ref="R90"  Part="1"
-AR Path="/5CCA7EF8/5CCACF4D" Ref="R2"  Part="1"
-F 0 "R2" H 6300 4450 50  0000 L CNN
+AR Path="/5CC86276/5CCACF4D" Ref="R?"  Part="1"
+AR Path="/5CCA7EF8/5CCACF4D" Ref="R75"  Part="1"
+F 0 "R75" H 6300 4450 50  0000 L CNN
 F 1 "R103,0603" H 6300 4400 50  0000 L CNN
 F 2 "Resistor_SMD:R_0603_1608Metric_Pad1.05x0.95mm_HandSolder" H 6200 4400 50  0001 C CNN
@@
 $EndComp
 $Comp
-L taobao-r:R333,0603 R89
+L taobao-r:R333,0603 R?
 U 1 1 5CCACF4E
 P 6400 3750
-AR Path="/5CC86276/5CCACF4E" Ref="R89"  Part="1"
-AR Path="/5CCA7EF8/5CCACF4E" Ref="R1"  Part="1"
-F 0 "R1" V 6150 3750 50  0000 C CNN
+AR Path="/5CC86276/5CCACF4E" Ref="R?"  Part="1"
+AR Path="/5CCA7EF8/5CCACF4E" Ref="R76"  Part="1"
+F 0 "R76" V 6150 3750 50  0000 C CNN
 F 1 "R333,0603" V 6250 3750 50  0000 C CNN
 F 2 "Resistor_SMD:R_0603_1608Metric_Pad1.05x0.95mm_HandSolder" H 6400 3750 50  0001 C CNN
@@
 	6200 4850 7050 4850
 $Comp
-L taobao-c:C226,6.3v,0603 C53
+L taobao-c:C226,6.3v,0603 C?
 U 1 1 5CC95BA7
 P 7050 4150
-AR Path="/5CC86276/5CC95BA7" Ref="C53"  Part="1"
-AR Path="/5CCA7EF8/5CC95BA7" Ref="C48"  Part="1"
-F 0 "C48" H 7150 4200 50  0000 L CNN
+AR Path="/5CC86276/5CC95BA7" Ref="C?"  Part="1"
+AR Path="/5CCA7EF8/5CC95BA7" Ref="C49"  Part="1"
+F 0 "C49" H 7150 4200 50  0000 L CNN
 F 1 "C226,6.3v,0603" H 7150 4150 50  0000 L CNN
 F 2 "Capacitor_SMD:C_0603_1608Metric_Pad1.05x0.95mm_HandSolder" H 7050 4150 50  0001 C CNN
@@
 $EndComp
 $Comp
-L taobao-c:C106,0603 C50
+L taobao-c:C106,0603 C?
 U 1 1 5CCACF50
 P 3100 3350
-AR Path="/5CC86276/5CCACF50" Ref="C50"  Part="1"
-AR Path="/5CCA7EF8/5CCACF50" Ref="C46"  Part="1"
-F 0 "C46" H 3200 3400 50  0000 L CNN
+AR Path="/5CC86276/5CCACF50" Ref="C?"  Part="1"
+AR Path="/5CCA7EF8/5CCACF50" Ref="C45"  Part="1"
+F 0 "C45" H 3200 3400 50  0000 L CNN
 F 1 "C106,0603" H 3200 3350 50  0000 L CNN
 F 2 "Capacitor_SMD:C_0603_1608Metric_Pad1.05x0.95mm_HandSolder" H 3100 3350 50  0001 C CNN
@@
 $EndComp
 $Comp
-L power:+5V #PWR0111
+L power:+5V #PWR0208
 U 1 1 5CCA8721
 P 7050 3250
-F 0 "#PWR0111" H 7050 3100 50  0001 C CNN
+F 0 "#PWR0208" H 7050 3100 50  0001 C CNN
 F 1 "+5V" H 7100 3450 50  0000 C CNN
 F 2 "" H 7050 3250 50  0001 C CNN
