File: hardware/printer-board/MP2303A_power_supply_5V (copy).kicad_pcb (KiCad board)
At the start: 2 copper layers, 100 x 100 mm, 207 parts, among them J1 USB_DEBUG, J10 MS_SELECT, J11 E0, J12 MS_SELECT, J13 E1, J14 HEATBED, J15 X_MIN, J16 X_MAX, J17 Y_MIN, J18 Y_MAX, J19 Z_MIN, J2 MS_SELECT, J20 Z_MAX, J21 HEATBED_TEMP, J22 HOTEND_TEMP0, J23 HOTEND_TEMP1, J24 AUX_TEMP, J25 12V_INPUT_2, J26 12V_INPUT, J27 12V_OUT, J28 SWD, J29 STM32_USB_DEBUG, J3 X, J30 PWR_DEBUG, J31 HOT_END, J32 HOT_END, J33 FAN0, J34 FAN1, J35 FAN2, J36 MS_SELECT, J37 Z2, J38 MS_SELECT, J39 Y, J4 MS_SELECT, J41 EXP1, J42 EXP2, J45 END_SWITCH_DEBUG, J46 HOTEND_DEBUG, J47 TEMP_DEBUG, J5 Z, J6 MS_SELECT, J7 Z1, J8 MS_SELECT, J9 Z3, Q1 WSK220N04, Q2 STP55NF06, Q3 STP55NF06, Q4 D882, Q5 D882, Q6 D882, SW1 SW_Push, U1 orange_pi_zero, U10 A4988_MODULE, U2 A4988_MODULE, U3 A4988_MODULE, U4 A4988_MODULE, U5 A4988_MODULE, U6 A4988_MODULE, U7 A4988_MODULE, U8 STM32F407VET6, U9 A4988_MODULE, Y1 O_8M

Commit message: update,
Parts:
- removed J45: END_SWITCH_DEBUG, Connector_PinHeader_1.27mm:PinHeader_1x06_P1.27mm_Vertical
- removed J46: HOTEND_DEBUG, Connector_PinHeader_1.27mm:PinHeader_1x03_P1.27mm_Vertical
- removed J47: TEMP_DEBUG, Connector_PinHeader_1.27mm:PinHeader_1x05_P1.27mm_Vertical
- added C1: CP100uf,10V, Capacitor_SMD:CP_Elec_6.3x5.3, F.Cu at (76.3, 33.4)
- added C33: C104,0603, Capacitor_SMD:C_0603_1608Metric_Pad1.05x0.95mm_HandSolder, F.Cu at (120.1, 83.5)
- added C45: C106,0603, Capacitor_SMD:C_0603_1608Metric_Pad1.05x0.95mm_HandSolder, F.Cu at (67.5, 33.5)
- added C46: C104,0603, Capacitor_SMD:C_0603_1608Metric_Pad1.05x0.95mm_HandSolder, F.Cu at (71.5, 40.0)
- added C47: C332,0603, Capacitor_SMD:C_0603_1608Metric_Pad1.05x0.95mm_HandSolder, F.Cu at (63.0, 41.0)
- added C48: C103,0603, Capacitor_SMD:C_0603_1608Metric_Pad1.05x0.95mm_HandSolder, F.Cu at (70.0, 32.5)
- added C49: C226,6.3v,0603, Capacitor_SMD:C_0603_1608Metric_Pad1.05x0.95mm_HandSolder, F.Cu at (63.0, 37.5)
- added C50: C106,0603, Capacitor_SMD:C_0603_1608Metric_Pad1.05x0.95mm_HandSolder, F.Cu at (48.2, 40.2)
- added C51: C104,0603, Capacitor_SMD:C_0603_1608Metric_Pad1.05x0.95mm_HandSolder, F.Cu at (43.5, 33.2)
- added C52: C332,0603, Capacitor_SMD:C_0603_1608Metric_Pad1.05x0.95mm_HandSolder, F.Cu at (49.2, 30.0)
- added C53: C103,0603, Capacitor_SMD:C_0603_1608Metric_Pad1.05x0.95mm_HandSolder, F.Cu at (45.5, 40.8)
- added C54: C226,6.3v,0603, Capacitor_SMD:C_0603_1608Metric_Pad1.05x0.95mm_HandSolder, F.Cu at (52.3, 35.5)
- added D15: SD_M4, Diode_SMD:D_SOD-323_HandSoldering, F.Cu at (11.2, 3.75)
- added D16: SD_M4, Diode_SMD:D_SOD-323_HandSoldering, F.Cu at (21.4, 21.4)
- added J40: SPI_DEBUG, Connector_PinHeader_1.27mm:PinHeader_1x07_P1.27mm_Vertical, F.Cu at (116.8, 83.9)
- added L2: L_15uH, w_smd_inductors:inductor_smd_4.8x2.8mm, F.Cu at (61.8, 33.8)
- added L3: L_15uH, w_smd_inductors:inductor_smd_4.8x2.8mm, F.Cu at (53.5, 39.2)
- added R74: R562,0603, Resistor_SMD:R_0603_1608Metric_Pad1.05x0.95mm_HandSolder, F.Cu at (59.5, 41.0)
- added R75: R103,0603, Resistor_SMD:R_0603_1608Metric_Pad1.05x0.95mm_HandSolder, F.Cu at (59.5, 37.5)
- added R76: R333,0603, Resistor_SMD:R_0603_1608Metric_Pad1.05x0.95mm_HandSolder, F.Cu at (59.5, 39.2)
- added R77: R562,0603, Resistor_SMD:R_0603_1608Metric_Pad1.05x0.95mm_HandSolder, F.Cu at (52.8, 30.0)
- added R78: R103,0603, Resistor_SMD:R_0603_1608Metric_Pad1.05x0.95mm_HandSolder, F.Cu at (52.2, 32.0)
- added R79: R333,0603, Resistor_SMD:R_0603_1608Metric_Pad1.05x0.95mm_HandSolder, F.Cu at (52.2, 33.8)
- added U11: MP2303A_ALT, footprint-lib:SOIC-8_3.9x4.9mm_P1.27mm,thermal_via, F.Cu at (68.0, 38.1)
- added U12: MP2303A_ALT, footprint-lib:SOIC-8_3.9x4.9mm_P1.27mm,thermal_via, F.Cu at (47.5, 35.1)
- C19, R3, R47, R48: moved to F.Cu
- D20: value FAN0_EN -> LED_BLUE,0603
- D21: value FAN1_EN -> LED_BLUE,0603
- D22: value FAN2_EN -> LED_BLUE,0603
- J29: value STM32_USB_DEBUG -> USB_DEBUG
- J33: value FAN0 -> TO FAN0
- J34: value FAN1 -> TO FAN1
- J35: value FAN2 -> TO FAN2
- JP6: value BOOT0 -> Jumper_NO_Small
- JP7: value BOOT1 -> Jumper_NO_Small
- moved R3 100.4 mm to (139.0, 83.5), turned to 0 degrees
- moved J29 21.7 mm to (33.4, 47.6), turned to 180 degrees
- moved R73 10.8 mm to (74.5, 85.5), turned to 180 degrees
- moved R10 10.8 mm to (90.8, 85.5), turned to 180 degrees
- moved R1 10.7 mm to (76.2, 61.5), turned to 90 degrees
- moved R46 9.71 mm to (39.1, 55.0), turned to 225 degrees
- moved C42 9.35 mm to (74.5, 73.2), turned to 0 degrees
- moved C3 9.07 mm to (90.8, 73.5), turned to 0 degrees
- moved R2 7.81 mm to (78.2, 61.5), turned to 90 degrees
- moved R70 7.71 mm to (29.8, 82.5)
- moved R45 7.69 mm to (40.2, 56.0), turned to 225 degrees
- moved R16 7.65 mm to (45.8, 82.5)
- moved R22 7.62 mm to (16.8, 67.2)
- moved C19 7.56 mm to (11.0, 1.75)
- moved R47 7.01 mm to (51.5, 50.2), turned to 0 degrees
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Connections:
- net /FANS/FAN0/FAN0_N renamed Net-(C36-Pad2)
- net /FANS/FAN1/FAN1_N renamed Net-(C37-Pad2)
- net /FANS/FAN2/FAN2_N renamed Net-(C38-Pad2)
- C15 pad 1: PA1 -> /Thermistors/HOTEND_TEMP0
- C16 pad 1: PA2 -> PA1
- D10 pad 1: PD9 -> PB3
- D11 pad 1: PD10 -> PB4
- D12 pad 1: PD11 -> PB5
- D13 pad 1: PD12 -> PB6
- D14 pad 1: PD13 -> PB7
- D2 pad 1: PE15 -> PD3
- D23 pad 1: PC13 -> PC12
- D24 pad 1: PE12 -> PD6
- D3 pad 1: PE7 -> PC6
- D4 pad 1: PC2 -> PC9
- D5 pad 1: PE2 -> PD0
- D6 pad 1: PD6 -> PC0
- D7 pad 1: PD3 -> PC3
- D9 pad 1: PD8 -> PB2
- J1 pad 1: +5V -> GND
- J1 pad 4: GND -> +5V
- J15 pad 1: PD8 -> PB2
- J16 pad 1: PD9 -> PB3
- J17 pad 1: PD10 -> PB4
- J18 pad 1: PD11 -> PB5
- J19 pad 1: PD12 -> PB6
- J20 pad 1: PD13 -> PB7
- J22 pad 1: PA1 -> /Thermistors/HOTEND_TEMP0
- J23 pad 1: PA2 -> PA1
- J30 pad 5: (no net) -> Net-(J30-Pad5)
- J41 pad 1: (no net) -> /st7920 type lcd/BEEPER
- J41 pad 2: PD1 -> PB7
- J41 pad 3: PC11 -> PB10
- J41 pad 4: PA15 -> PB8
- J41 pad 5: PC10 -> PB9
- J41 pad 6: (no net) -> Net-(J41-Pad6)
- J41 pad 7: (no net) -> Net-(J41-Pad7)
- J41 pad 8: (no net) -> Net-(J41-Pad8)
- J42 pad 1: (no net) -> Net-(J42-Pad1)
- J42 pad 10: PD2 -> PA8
- J42 pad 2: (no net) -> Net-(J42-Pad2)
- J42 pad 3: PD0 -> PB6
- J42 pad 4: (no net) -> Net-(J42-Pad4)
- J42 pad 5: PC12 -> PB5
- J42 pad 6: (no net) -> Net-(J42-Pad6)
- J42 pad 7: (no net) -> Net-(J42-Pad7)
- J42 pad 8: (no net) -> /st7920 type lcd/RESET
- R10 pad 2: PE15 -> PD3
- R13 pad 2: PE7 -> PC6
- R16 pad 2: PC2 -> PC9
- R19 pad 2: PE2 -> PD0
- R22 pad 2: PD6 -> PC0
- R25 pad 2: PD3 -> PC3
- R26 pad 2: PC6 -> PA8
- R27 pad 2: PC6 -> PA8
- R36 pad 2: PA1 -> /Thermistors/HOTEND_TEMP0
- R37 pad 2: PA2 -> PA1
- R50 pad 2: PD15 -> PA9
- R51 pad 2: PD15 -> PA9
- R53 pad 2: PD14 -> PA10
- R54 pad 2: PD14 -> PA10
- R70 pad 2: PC13 -> PC12
- R73 pad 2: PE12 -> PD6
- U1 pad 10: (no net) -> Net-(U1-Pad10)
- U1 pad 101: (no net) -> Net-(U1-Pad101)
- U1 pad 102: (no net) -> Net-(U1-Pad102)
- U1 pad 103: (no net) -> Net-(U1-Pad103)
- U1 pad 104: (no net) -> Net-(U1-Pad104)
- U1 pad 105: (no net) -> Net-(U1-Pad105)
- U1 pad 106: (no net) -> Net-(U1-Pad106)
- U1 pad 107: (no net) -> Net-(U1-Pad107)
- U1 pad 108: (no net) -> Net-(U1-Pad108)
- U1 pad 109: (no net) -> Net-(U1-Pad109)
- U1 pad 11: (no net) -> Net-(U1-Pad11)
- U1 pad 110: (no net) -> Net-(U1-Pad110)
- U1 pad 111: (no net) -> Net-(U1-Pad111)
- U1 pad 112: (no net) -> Net-(U1-Pad112)
- U1 pad 113: (no net) -> Net-(U1-Pad113)
- U1 pad 114: (no net) -> Net-(U1-Pad114)
- U1 pad 115: (no net) -> Net-(U1-Pad115)
- U1 pad 116: (no net) -> Net-(U1-Pad116)
- U1 pad 117: (no net) -> Net-(U1-Pad117)
- U1 pad 118: (no net) -> Net-(U1-Pad118)
- U1 pad 119: (no net) -> Net-(U1-Pad119)
- U1 pad 12: (no net) -> Net-(U1-Pad12)
- U1 pad 120: (no net) -> Net-(U1-Pad120)
- U1 pad 121: (no net) -> Net-(U1-Pad121)
- U1 pad 122: (no net) -> Net-(U1-Pad122)
- U1 pad 123: (no net) -> Net-(U1-Pad123)
- U1 pad 124: (no net) -> Net-(U1-Pad124)
- U1 pad 125: (no net) -> Net-(U1-Pad125)
- U1 pad 126: (no net) -> Net-(U1-Pad126)
- U1 pad 13: (no net) -> Net-(U1-Pad13)
- U1 pad 201: (no net) -> Net-(U1-Pad201)
- U1 pad 202: (no net) -> Net-(U1-Pad202)
- U1 pad 203: (no net) -> Net-(U1-Pad203)
- U1 pad 5: (no net) -> /orange_pi/USB-DM3
- U1 pad 6: (no net) -> /orange_pi/USB-DP3
- U1 pad 7: (no net) -> Net-(U1-Pad7)
- U1 pad 8: (no net) -> Net-(U1-Pad8)
- U1 pad 9: (no net) -> Net-(U1-Pad9)
- U10 pad 1: PE12 -> PD6
- U10 pad 7: PE11 -> PD7
- U10 pad 8: PE10 -> PD8
- U2 pad 1: PE15 -> PD3
- U2 pad 7: PE14 -> PD4
- U2 pad 8: PE13 -> PD5
- U3 pad 1: PE7 -> PC6
- U3 pad 7: PE9 -> PC7
- U3 pad 8: PE8 -> PC8
- U4 pad 1: PC2 -> PC9
- U4 pad 7: PC1 -> PC10
- U4 pad 8: PC0 -> PC11
- U5 pad 1: PE2 -> PD0
- U5 pad 7: PE3 -> PD1
- U5 pad 8: PE4 -> PD2
- U6 pad 1: PD6 -> PC0
- U6 pad 7: PD7 -> PC1
- U6 pad 8: PB3 -> PC2
- U7 pad 1: PD3 -> PC3
- U7 pad 7: PD4 -> /E1_~E1_STEP~PER_DRIVER/E1_STEP
- U7 pad 8: PD5 -> /E1_~E1_STEP~PER_DRIVER/E1_DIR
- U8 pad 18: (no net) -> PC3
- U8 pad 30: (no net) -> PA5
- U8 pad 31: (no net) -> PA6
- U8 pad 32: (no net) -> PA7
- U8 pad 33: (no net) -> PC4
- U8 pad 34: (no net) -> PC5
- U8 pad 35: (no net) -> PB0
- U8 pad 36: (no net) -> PB1
- U8 pad 4: (no net) -> PE5
- U8 pad 47: (no net) -> PB10
- U8 pad 48: (no net) -> PB11
- U8 pad 5: (no net) -> PE6
- U8 pad 51: (no net) -> PB12
- U8 pad 52: (no net) -> /STM32_CORE/STM32_CORE_MCU/SCK
- U8 pad 53: (no net) -> /STM32_CORE/STM32_CORE_MCU/MISO2
- U8 pad 54: (no net) -> /STM32_CORE/STM32_CORE_MCU/MOSI2
- U8 pad 64: (no net) -> PC7
- U8 pad 65: (no net) -> PC8
- U8 pad 66: (no net) -> PC9
- U8 pad 67: (no net) -> PA8
- U8 pad 68: (no net) -> Net-(J43-Pad2)
- U8 pad 69: (no net) -> Net-(J43-Pad1)
- U8 pad 90: (no net) -> PB4
- U8 pad 91: (no net) -> PB5
- U8 pad 92: (no net) -> /STM32_CORE/STM32_SCL1
- U8 pad 93: (no net) -> /STM32_CORE/STM32_SDA1
- U8 pad 95: (no net) -> PB8
- U8 pad 97: (no net) -> PE0
- U8 pad 98: (no net) -> PE1
- U9 pad 1: PC13 -> PC12
- U9 pad 7: PC14 -> PC13
- U9 pad 8: PC15 -> PC14
Routing:
- net +3V3: track 640.8 -> 33.8 mm, vias 13 -> 1
- net +12V: track 569.4 -> 57.5 mm, vias 9 -> 1
- net PA0: track 88.8 -> 0.00 mm, vias 2 -> 0
- net PE15: track 80.2 -> 0.00 mm
- net PA1: track 77.9 -> 0.00 mm, vias 2 -> 0
- net PE2: track 75.5 -> 0.00 mm, vias 4 -> 0
- net /HOTENDS/HOTEND_1/-12V: track 74.1 -> 0.00 mm
- net /HOTENDS/HOTEND_0/-12V: track 74.0 -> 0.00 mm
- net /HEATBED/-12V2: track 72.4 -> 0.00 mm
- net PA2: track 63.3 -> 0.00 mm, vias 2 -> 0
- net PE13: track 60.9 -> 0.00 mm
- net PD8: track 60.9 -> 0.00 mm, vias 2 -> 0
- net PD14: track 60.3 -> 0.00 mm
- net PE14: track 58.8 -> 0.00 mm
- net +5V: track 55.4 -> 0.00 mm, vias 1 -> 0
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Other:
- outline, holes or cut-outs redrawn
