File: hardware/printer-board/_autosave-END_STOP.sch (KiCad schematic (older format))
At the start: 19 parts, among them J15 X_MIN, J16 X_MAX, J17 Y_MIN, J18 Y_MAX, J19 Z_MIN, J20 Z_MAX, J45 END_SWITCH_DEBUG

Commit message: update,
Parts:
- D10: value LED_BLUE,0603 -> XMAX
- D9: value LED_BLUE,0603 -> XMIN
Changed lines of the file:
@@
 P 4250 2100
 F 0 "D9" V 4296 2032 50  0000 R CNN
-F 1 "LED_BLUE,0603" V 4205 2032 50  0000 R CNN
+F 1 "XMIN" V 4205 2032 50  0000 R CNN
 F 2 "LED_SMD:LED_0603_1608Metric_Pad1.05x0.95mm_HandSolder" V 4250 2100 50  0001 C CNN
 F 3 "" V 4250 2100 50  0001 C CNN
@@
 P 4250 3000
 F 0 "D10" V 4296 2932 50  0000 R CNN
-F 1 "LED_BLUE,0603" V 4205 2932 50  0000 R CNN
+F 1 "XMAX" V 4205 2932 50  0000 R CNN
 F 2 "LED_SMD:LED_0603_1608Metric_Pad1.05x0.95mm_HandSolder" V 4250 3000 50  0001 C CNN
 F 3 "" V 4250 3000 50  0001 C CNN
