File: hardware/printer-board/END_STOP.kicad_pcb (KiCad board)
At the start: 2 copper layers, 100 x 100 mm, 22 parts, among them J15 X_MIN, J16 X_MAX, J17 Y_MIN, J18 Y_MAX, J19 Z_MIN, J20 Z_MAX

Commit message: update ROUTING,
Parts:
- added C1: CP100uf,10V, Capacitor_SMD:CP_Elec_6.3x5.3, F.Cu at (76.3, 33.4)
- added C10: CP100uf,25V, Capacitor_SMD:CP_Elec_6.3x7.7, F.Cu at (9.23, 64.2)
- added C11: C104,0603, Capacitor_SMD:C_0603_1608Metric_Pad1.05x0.95mm_HandSolder, F.Cu at (20.6, 67.2)
- added C12: CP100uf,25V, Capacitor_SMD:CP_Elec_6.3x7.7, F.Cu at (9.23, 48.3)
- added C13: C104,0603, Capacitor_SMD:C_0603_1608Metric_Pad1.05x0.95mm_HandSolder, F.Cu at (16.8, 51.3)
- added C14: C106,0603, Capacitor_SMD:C_0603_1608Metric_Pad1.05x0.95mm_HandSolder, B.Cu at (2.75, 31.8)
- added C15: C106,0603, Capacitor_SMD:C_0603_1608Metric_Pad1.05x0.95mm_HandSolder, B.Cu at (10.0, 31.8)
- added C16: C106,0603, Capacitor_SMD:C_0603_1608Metric_Pad1.05x0.95mm_HandSolder, B.Cu at (16.8, 31.8)
- added C17: C106,0603, Capacitor_SMD:C_0603_1608Metric_Pad1.05x0.95mm_HandSolder, B.Cu at (23.5, 31.8)
- added C18: C106,0603, Capacitor_SMD:C_0603_1608Metric_Pad1.05x0.95mm_HandSolder, B.Cu at (27.4, 20.1)
- added C19: C104,0603, Capacitor_SMD:C_0603_1608Metric_Pad1.05x0.95mm_HandSolder, F.Cu at (11.0, 1.75)
- added C2: CP100uf,25V, Capacitor_SMD:CP_Elec_6.3x7.7, F.Cu at (90.5, 90.2)
- added C20: CP100uf,35V, Capacitor_SMD:CP_Elec_6.3x7.7, F.Cu at (11.8, 9.35)
- added C21: C104,0603, Capacitor_SMD:C_0603_1608Metric_Pad1.05x0.95mm_HandSolder, B.Cu at (40.2, 69.8)
- added C22: C10pf,0603, Capacitor_SMD:C_0603_1608Metric_Pad1.05x0.95mm_HandSolder, B.Cu at (28.5, 62.2)
- added C23: C104,0603, Capacitor_SMD:C_0603_1608Metric_Pad1.05x0.95mm_HandSolder, B.Cu at (33.1, 60.3)
- added C24: C10pf,0603, Capacitor_SMD:C_0603_1608Metric_Pad1.05x0.95mm_HandSolder, B.Cu at (35.8, 69.2)
- added C25: C104,0603, Capacitor_SMD:C_0603_1608Metric_Pad1.05x0.95mm_HandSolder, B.Cu at (31.4, 56.1)
- added C26: C104,0603, Capacitor_SMD:C_0603_1608Metric_Pad1.05x0.95mm_HandSolder, B.Cu at (42.3, 47.9)
- added C27: C104,0603, Capacitor_SMD:C_0603_1608Metric_Pad1.05x0.95mm_HandSolder, B.Cu at (50.8, 58.5)
- added C28: C104,0603, Capacitor_SMD:C_0603_1608Metric_Pad1.05x0.95mm_HandSolder, B.Cu at (42.6, 66.6)
- added C29: C105,0603, Capacitor_SMD:C_0603_1608Metric_Pad1.05x0.95mm_HandSolder, B.Cu at (34.7, 61.9)
- added C3: C104,0603, Capacitor_SMD:C_0603_1608Metric_Pad1.05x0.95mm_HandSolder, F.Cu at (90.8, 73.5)
- added C30: C104,0603, Capacitor_SMD:C_0603_1608Metric_Pad1.05x0.95mm_HandSolder, B.Cu at (49.7, 59.6)
- added C31: C104,0603, Capacitor_SMD:C_0603_1608Metric_Pad1.05x0.95mm_HandSolder, B.Cu at (43.3, 49.0)
- added C32: C104,0603, Capacitor_SMD:C_0603_1608Metric_Pad1.05x0.95mm_HandSolder, B.Cu at (47.6, 68.0)
- added C33: C104,0603, Capacitor_SMD:C_0603_1608Metric_Pad1.05x0.95mm_HandSolder, F.Cu at (120.1, 83.5)
- added C36: CP1uf,50V, Capacitor_SMD:CP_Elec_4x5.3, F.Cu at (21.5, 13.8)
- added C37: CP1uf,50V, Capacitor_SMD:CP_Elec_4x5.3, F.Cu at (29.5, 13.8)
- added C38: CP1uf,50V, Capacitor_SMD:CP_Elec_4x5.3, F.Cu at (38.0, 13.8)
- added C39: CP100uf,25V, Capacitor_SMD:CP_Elec_6.3x7.7, F.Cu at (25.7, 90.2)
- added C4: CP100uf,25V, Capacitor_SMD:CP_Elec_6.3x7.7, F.Cu at (58.1, 90.2)
- added C40: C104,0603, Capacitor_SMD:C_0603_1608Metric_Pad1.05x0.95mm_HandSolder, F.Cu at (29.8, 78.6)
- added C41: CP100uf,25V, Capacitor_SMD:CP_Elec_6.3x7.7, F.Cu at (74.3, 90.2)
- added C42: C104,0603, Capacitor_SMD:C_0603_1608Metric_Pad1.05x0.95mm_HandSolder, F.Cu at (74.5, 73.2)
- added C44: CP100uf,16V, Capacitor_SMD:CP_Elec_6.3x5.3, F.Cu at (36.3, 21.1)
- added C45: C106,0603, Capacitor_SMD:C_0603_1608Metric_Pad1.05x0.95mm_HandSolder, F.Cu at (67.5, 33.5)
- added C46: C104,0603, Capacitor_SMD:C_0603_1608Metric_Pad1.05x0.95mm_HandSolder, F.Cu at (71.5, 40.0)
- added C47: C332,0603, Capacitor_SMD:C_0603_1608Metric_Pad1.05x0.95mm_HandSolder, F.Cu at (63.0, 41.0)
- added C48: C103,0603, Capacitor_SMD:C_0603_1608Metric_Pad1.05x0.95mm_HandSolder, F.Cu at (70.0, 32.5)
- added C49: C226,6.3v,0603, Capacitor_SMD:C_0603_1608Metric_Pad1.05x0.95mm_HandSolder, F.Cu at (63.0, 37.5)
- added C5: C104,0603, Capacitor_SMD:C_0603_1608Metric_Pad1.05x0.95mm_HandSolder, F.Cu at (61.5, 82.5)
- added C50: C106,0603, Capacitor_SMD:C_0603_1608Metric_Pad1.05x0.95mm_HandSolder, F.Cu at (48.2, 40.2)
- added C51: C104,0603, Capacitor_SMD:C_0603_1608Metric_Pad1.05x0.95mm_HandSolder, F.Cu at (43.5, 33.2)
- added C52: C332,0603, Capacitor_SMD:C_0603_1608Metric_Pad1.05x0.95mm_HandSolder, F.Cu at (49.2, 30.0)
- added C53: C103,0603, Capacitor_SMD:C_0603_1608Metric_Pad1.05x0.95mm_HandSolder, F.Cu at (45.5, 40.8)
- added C54: C226,6.3v,0603, Capacitor_SMD:C_0603_1608Metric_Pad1.05x0.95mm_HandSolder, F.Cu at (52.3, 35.5)
- added C55: C105,0603, Capacitor_SMD:C_0603_1608Metric_Pad1.05x0.95mm_HandSolder, B.Cu at (38.7, 65.9)
- added C6: CP100uf,25V, Capacitor_SMD:CP_Elec_6.3x7.7, F.Cu at (41.9, 90.2)
- added C7: C104,0603, Capacitor_SMD:C_0603_1608Metric_Pad1.05x0.95mm_HandSolder, F.Cu at (45.8, 78.6)
- added C8: CP100uf,25V, Capacitor_SMD:CP_Elec_6.3x7.7, F.Cu at (9.50, 90.2)
- added C9: C104,0603, Capacitor_SMD:C_0603_1608Metric_Pad1.05x0.95mm_HandSolder, F.Cu at (12.5, 82.5)
- added D1: 5V HEALTHY, LED_SMD:LED_0603_1608Metric_Pad1.05x0.95mm_HandSolder, F.Cu at (50.8, 70.8)
- added D15: SD_M4, Diode_SMD:D_SOD-323_HandSoldering, F.Cu at (11.2, 3.75)
- added D16: SD_M4, Diode_SMD:D_SOD-323_HandSoldering, F.Cu at (21.4, 21.4)
- added D17: PB9, LED_SMD:LED_0603_1608Metric_Pad1.05x0.95mm_HandSolder, F.Cu at (30.3, 52.5)
- added D18: LED_RED,0603, LED_SMD:LED_0603_1608Metric_Pad1.05x0.95mm_HandSolder, F.Cu at (63.9, 5.50)
- added D19: LED_RED,0603, LED_SMD:LED_0603_1608Metric_Pad1.05x0.95mm_HandSolder, F.Cu at (75.8, 5.50)
- added D2: LED_BLUE,0603, LED_SMD:LED_0603_1608Metric_Pad1.05x0.95mm_HandSolder, F.Cu at (92.2, 97.7)
- added D20: LED_BLUE,0603, LED_SMD:LED_0603_1608Metric_Pad1.05x0.95mm_HandSolder, F.Cu at (25.1, 2.52)
- added D21: LED_BLUE,0603, LED_SMD:LED_0603_1608Metric_Pad1.05x0.95mm_HandSolder, F.Cu at (33.4, 2.52)
- added D22: LED_BLUE,0603, LED_SMD:LED_0603_1608Metric_Pad1.05x0.95mm_HandSolder, F.Cu at (41.8, 2.50)
- added D23: LED_BLUE,0603, LED_SMD:LED_0603_1608Metric_Pad1.05x0.95mm_HandSolder, F.Cu at (33.0, 97.7)
- added D24: LED_BLUE,0603, LED_SMD:LED_0603_1608Metric_Pad1.05x0.95mm_HandSolder, F.Cu at (78.2, 97.7)
- added D3: LED_BLUE,0603, LED_SMD:LED_0603_1608Metric_Pad1.05x0.95mm_HandSolder, F.Cu at (63.1, 97.7)
- added D4: LED_BLUE,0603, LED_SMD:LED_0603_1608Metric_Pad1.05x0.95mm_HandSolder, F.Cu at (48.1, 97.7)
- added D5: LED_BLUE,0603, LED_SMD:LED_0603_1608Metric_Pad1.05x0.95mm_HandSolder, F.Cu at (17.8, 97.7)
- added D6: LED_BLUE,0603, LED_SMD:LED_0603_1608Metric_Pad1.05x0.95mm_HandSolder, F.Cu at (3.00, 70.5)
- added D7: LED_BLUE,0603, LED_SMD:LED_0603_1608Metric_Pad1.05x0.95mm_HandSolder, F.Cu at (3.00, 54.7)
- added D8: LED_RED,0603, LED_SMD:LED_0603_1608Metric_Pad1.05x0.95mm_HandSolder, F.Cu at (51.8, 5.50)
- added F1: 16V/30A, w_misc_comp:fuse_smf, F.Cu at (11.8, 17.9)
- added F2: 30V/5A, w_misc_comp:fuse_smf, F.Cu at (11.8, 26.4)
- added J1: USB_DEBUG, Connector_PinHeader_1.27mm:PinHeader_1x04_P1.27mm_Vertical, F.Cu at (91.4, 65.4)
- added J10: MS_SELECT, Connector_PinHeader_2.54mm:PinHeader_2x03_P2.54mm_Vertical, F.Cu at (22.5, 61.2)
- added J11: E0, footprint-lib:b4b-ph-kl,stepper_terminal, F.Cu at (2.40, 64.2)
- added J12: MS_SELECT, Connector_PinHeader_2.54mm:PinHeader_2x03_P2.54mm_Vertical, F.Cu at (22.4, 45.3)
- added J13: E1, footprint-lib:b4b-ph-kl,stepper_terminal, F.Cu at (2.40, 48.2)
- added J14: HEATBED, footprint-lib:mpt_0,5%2f2-2,54,heatbed, F.Cu at (46.8, 3.00)
- added J2: MS_SELECT, Connector_PinHeader_2.54mm:PinHeader_2x03_P2.54mm_Vertical, F.Cu at (89.5, 78.0)
- added J21: HEATBED_TEMP, w_conn_jst-ph:b2b-ph-kl, F.Cu at (2.39, 36.2)
- added J22: HOTEND_TEMP0, w_conn_jst-ph:b2b-ph-kl, F.Cu at (9.26, 36.2)
- added J23: HOTEND_TEMP1, w_conn_jst-ph:b2b-ph-kl, F.Cu at (16.1, 36.2)
- added J24: AUX_TEMP, w_conn_jst-ph:b2b-ph-kl, F.Cu at (23.0, 36.2)
- added J25: 12V_INPUT_2, footprint-lib:mpt_0,5%2f2-2,54,12V_SRC, F.Cu at (3.25, 18.2)
- added J26: 12V_INPUT, footprint-lib:mpt_0,5%2f2-2,54,12V_SRC, F.Cu at (3.15, 26.4)
- added J27: 12V_OUT, footprint-lib:mpt_0,5%2f2-2,54,12V_SRC, F.Cu at (3.15, 10.2)
- added J28: SWD, Connector_PinHeader_1.27mm:PinHeader_1x04_P1.27mm_Vertical, F.Cu at (37.4, 42.6)
- added J29: USB_DEBUG, Connector_PinHeader_1.27mm:PinHeader_1x05_P1.27mm_Vertical, F.Cu at (33.4, 47.6)
- added J3: X, footprint-lib:b4b-ph-kl,stepper_terminal, F.Cu at (86.0, 97.3)
- added J30: PWR_DEBUG, Connector_PinHeader_1.27mm:PinHeader_1x05_P1.27mm_Vertical, F.Cu at (29.4, 42.8)
- added J31: HOT_END, footprint-lib:mpt_0,5%2f2-2,54,heatbed, F.Cu at (58.8, 3.00)
- added J32: HOT_END, footprint-lib:mpt_0,5%2f2-2,54,heatbed, F.Cu at (70.8, 3.00)
- added J33: TO FAN0, footprint-lib:b2b-ph-kl,fan_pwm_out, F.Cu at (21.0, 2.00)
- added J34: TO FAN1, footprint-lib:b2b-ph-kl,fan_pwm_out, F.Cu at (29.2, 2.00)
- added J35: TO FAN2, footprint-lib:b2b-ph-kl,fan_pwm_out, F.Cu at (37.5, 2.00)
- added J36: MS_SELECT, Connector_PinHeader_2.54mm:PinHeader_2x03_P2.54mm_Vertical, F.Cu at (22.7, 77.0)
- added J37: Z2, footprint-lib:b4b-ph-kl,stepper_terminal, F.Cu at (26.7, 97.3)
- added J38: MS_SELECT, Connector_PinHeader_2.54mm:PinHeader_2x03_P2.54mm_Vertical, F.Cu at (73.3, 77.8)
- added J39: Y, footprint-lib:b4b-ph-kl,stepper_terminal, F.Cu at (71.9, 97.3)
- added J4: MS_SELECT, Connector_PinHeader_2.54mm:PinHeader_2x03_P2.54mm_Vertical, F.Cu at (55.1, 77.0)
- added J40: SPI_DEBUG, Connector_PinHeader_1.27mm:PinHeader_1x07_P1.27mm_Vertical, F.Cu at (116.8, 83.9)
- added J41: EXP1, Connector_PinHeader_2.54mm:PinHeader_2x05_P2.54mm_Vertical, F.Cu at (39.0, 38.4)
- added J42: EXP2, Connector_PinHeader_2.54mm:PinHeader_2x05_P2.54mm_Vertical, F.Cu at (31.8, 38.4)
- added J5: Z, footprint-lib:b4b-ph-kl,stepper_terminal, F.Cu at (56.8, 97.3)
- added J6: MS_SELECT, Connector_PinHeader_2.54mm:PinHeader_2x03_P2.54mm_Vertical, F.Cu at (38.9, 77.0)
- added J7: Z1, footprint-lib:b4b-ph-kl,stepper_terminal, F.Cu at (41.8, 97.3)
- added J8: MS_SELECT, Connector_PinHeader_2.54mm:PinHeader_2x03_P2.54mm_Vertical, F.Cu at (6.50, 77.0)
- added J9: Z3, footprint-lib:b4b-ph-kl,stepper_terminal, F.Cu at (11.6, 97.3)
- added JP5: Jumper_NO_Small, SolderJumper-2_P1.3mm_Open_TrianglePad1.0x1.5mm, B.Cu at (8.55, 22.2)
- added JP6: Jumper_NO_Small, SolderJumper-2_P1.3mm_Open_TrianglePad1.0x1.5mm, B.Cu at (42.3, 58.2)
- added JP7: Jumper_NO_Small, SolderJumper-2_P1.3mm_Open_TrianglePad1.0x1.5mm, B.Cu at (44.2, 60.1)
- added L1: L_Small, w_smd_inductors:inductor_smd_0603, F.Cu at (40.2, 69.8)
- added L2: L_15uH, w_smd_inductors:inductor_smd_4.8x2.8mm, F.Cu at (61.8, 33.8)
- added L3: L_15uH, w_smd_inductors:inductor_smd_4.8x2.8mm, F.Cu at (53.5, 39.2)
- added Q1: WSK220N04, footprint-lib:TO-263-2,thermal_vias, F.Cu at (49.2, 15.0)
- added Q2: STP55NF06, footprint-lib:TO-263-2,thermal_vias, F.Cu at (61.2, 15.0)
- added Q3: STP55NF06, footprint-lib:TO-263-2,thermal_vias, F.Cu at (73.2, 15.0)
- added Q4: D882, footprint-lib:SOT-89-3,thermal_vias, F.Cu at (21.1, 8.00)
- added Q5: D882, footprint-lib:SOT-89-3,thermal_vias, F.Cu at (29.2, 8.00)
- added Q6: D882, footprint-lib:SOT-89-3,thermal_vias, F.Cu at (37.8, 8.00)
- added R1: R153,0603, Resistor_SMD:R_0603_1608Metric_Pad1.05x0.95mm_HandSolder, F.Cu at (76.2, 61.5)
- added R10: R103,0603, Resistor_SMD:R_0603_1608Metric_Pad1.05x0.95mm_HandSolder, F.Cu at (90.8, 85.5)
- added R11: R104,0603, Resistor_SMD:R_0603_1608Metric_Pad1.05x0.95mm_HandSolder, F.Cu at (61.5, 78.6)
- added R12: R102,0603, Resistor_SMD:R_0603_1608Metric_Pad1.05x0.95mm_HandSolder, B.Cu at (63.1, 97.7)
- added R13: R103,0603, Resistor_SMD:R_0603_1608Metric_Pad1.05x0.95mm_HandSolder, F.Cu at (61.5, 74.8)
- added R14: R104,0603, Resistor_SMD:R_0603_1608Metric_Pad1.05x0.95mm_HandSolder, F.Cu at (45.8, 74.8)
- added R15: R102,0603, Resistor_SMD:R_0603_1608Metric_Pad1.05x0.95mm_HandSolder, B.Cu at (48.0, 97.7)
- added R16: R103,0603, Resistor_SMD:R_0603_1608Metric_Pad1.05x0.95mm_HandSolder, F.Cu at (45.8, 82.5)
- added R17: R104,0603, Resistor_SMD:R_0603_1608Metric_Pad1.05x0.95mm_HandSolder, F.Cu at (12.5, 78.6)
- added R18: R102,0603, Resistor_SMD:R_0603_1608Metric_Pad1.05x0.95mm_HandSolder, B.Cu at (17.8, 97.7)
- added R19: R103,0603, Resistor_SMD:R_0603_1608Metric_Pad1.05x0.95mm_HandSolder, F.Cu at (12.5, 74.8)
- added R2: R153,0603, Resistor_SMD:R_0603_1608Metric_Pad1.05x0.95mm_HandSolder, F.Cu at (78.2, 61.5)
- added R20: R104,0603, Resistor_SMD:R_0603_1608Metric_Pad1.05x0.95mm_HandSolder, F.Cu at (24.4, 67.2)
- added R21: R102,0603, Resistor_SMD:R_0603_1608Metric_Pad1.05x0.95mm_HandSolder, B.Cu at (3.00, 70.5)
- added R22: R103,0603, Resistor_SMD:R_0603_1608Metric_Pad1.05x0.95mm_HandSolder, F.Cu at (16.8, 67.2)
- added R23: R104,0603, Resistor_SMD:R_0603_1608Metric_Pad1.05x0.95mm_HandSolder, F.Cu at (20.6, 51.3)
- added R24: R102,0603, Resistor_SMD:R_0603_1608Metric_Pad1.05x0.95mm_HandSolder, F.Cu at (24.4, 51.3)
- added R25: R103,0603, Resistor_SMD:R_0603_1608Metric_Pad1.05x0.95mm_HandSolder, B.Cu at (3.00, 54.7)
- added R26: R100,0805, Resistor_SMD:R_0805_2012Metric_Pad1.15x1.40mm_HandSolder, B.Cu at (46.8, 19.5)
- added R27: R104,0805, Resistor_SMD:R_0805_2012Metric_Pad1.15x1.40mm_HandSolder, B.Cu at (51.8, 19.5)
- added R28: R182,0603, Resistor_SMD:R_0603_1608Metric_Pad1.05x0.95mm_HandSolder, B.Cu at (51.8, 5.50)
- added R3: R220,0603, Resistor_SMD:R_0603_1608Metric_Pad1.05x0.95mm_HandSolder, F.Cu at (139.0, 83.5)
- added R35: R472,0603, Resistor_SMD:R_0603_1608Metric_Pad1.05x0.95mm_HandSolder, F.Cu at (2.75, 31.8)
- added R36: R472,0603, Resistor_SMD:R_0603_1608Metric_Pad1.05x0.95mm_HandSolder, F.Cu at (10.0, 31.8)
- added R37: R472,0603, Resistor_SMD:R_0603_1608Metric_Pad1.05x0.95mm_HandSolder, F.Cu at (16.8, 31.8)
- added R38: R472,0603, Resistor_SMD:R_0603_1608Metric_Pad1.05x0.95mm_HandSolder, F.Cu at (23.5, 31.8)
- added R39: R472,0603, Resistor_SMD:R_0603_1608Metric_Pad1.05x0.95mm_HandSolder, F.Cu at (27.4, 20.1)
- added R4: R220,0603, Resistor_SMD:R_0603_1608Metric_Pad1.05x0.95mm_HandSolder, B.Cu at (86.1, 70.8)
- added R40: R472,0603, Resistor_SMD:R_0603_1608Metric_Pad1.05x0.95mm_HandSolder, B.Cu at (44.6, 55.9)
- added R41: R472,0603, Resistor_SMD:R_0603_1608Metric_Pad1.05x0.95mm_HandSolder, B.Cu at (46.5, 57.8)
- added R42: R0,0603, Resistor_SMD:R_0603_1608Metric_Pad1.05x0.95mm_HandSolder, B.Cu at (37.7, 64.9)
- added R43: R0,0603, Resistor_SMD:R_0603_1608Metric_Pad1.05x0.95mm_HandSolder, B.Cu at (36.6, 63.8)
- added R44: R102,0603, Resistor_SMD:R_0603_1608Metric_Pad1.05x0.95mm_HandSolder, B.Cu at (30.3, 52.5)
- added R45: R103,0603, Resistor_SMD:R_0603_1608Metric_Pad1.05x0.95mm_HandSolder, B.Cu at (40.2, 56.0)
- added R46: R103,0603, Resistor_SMD:R_0603_1608Metric_Pad1.05x0.95mm_HandSolder, B.Cu at (39.1, 55.0)
- added R47: R220,0603, Resistor_SMD:R_0603_1608Metric_Pad1.05x0.95mm_HandSolder, F.Cu at (51.5, 50.2)
- added R48: R152,0603, Resistor_SMD:R_0603_1608Metric_Pad1.05x0.95mm_HandSolder, F.Cu at (51.5, 51.8)
- added R5: R220,0603, Resistor_SMD:R_0603_1608Metric_Pad1.05x0.95mm_HandSolder, B.Cu at (84.5, 70.8)
- added R50: R100,0805, Resistor_SMD:R_0805_2012Metric_Pad1.15x1.40mm_HandSolder, B.Cu at (58.8, 19.5)
- added R51: R104,0805, Resistor_SMD:R_0805_2012Metric_Pad1.15x1.40mm_HandSolder, B.Cu at (63.8, 19.5)
- added R52: R182,0603, Resistor_SMD:R_0603_1608Metric_Pad1.05x0.95mm_HandSolder, B.Cu at (63.8, 5.50)
- added R53: R100,0805, Resistor_SMD:R_0805_2012Metric_Pad1.15x1.40mm_HandSolder, B.Cu at (70.8, 20.0)
- added R54: R104,0805, Resistor_SMD:R_0805_2012Metric_Pad1.15x1.40mm_HandSolder, B.Cu at (75.8, 20.0)
- added R55: R182,0603, Resistor_SMD:R_0603_1608Metric_Pad1.05x0.95mm_HandSolder, B.Cu at (75.8, 5.50)
- added R56: R100,0805, Resistor_SMD:R_0805_2012Metric_Pad1.15x1.40mm_HandSolder, B.Cu at (22.9, 5.10)
- added R57: R104,0805, Resistor_SMD:R_0805_2012Metric_Pad1.15x1.40mm_HandSolder, B.Cu at (19.4, 5.10)
- added R58: R100,0603, Resistor_SMD:R_0603_1608Metric_Pad1.05x0.95mm_HandSolder, B.Cu at (25.1, 2.50)
- added R59: R182,0603, Resistor_SMD:R_0603_1608Metric_Pad1.05x0.95mm_HandSolder, B.Cu at (21.1, 5.10)
- added R6: R152,0603, Resistor_SMD:R_0603_1608Metric_Pad1.05x0.95mm_HandSolder, B.Cu at (82.9, 70.8)
- added R60: R100,0805, Resistor_SMD:R_0805_2012Metric_Pad1.15x1.40mm_HandSolder, B.Cu at (31.0, 5.25)
- added R61: R104,0805, Resistor_SMD:R_0805_2012Metric_Pad1.15x1.40mm_HandSolder, B.Cu at (27.5, 5.25)
- added R62: R100,0603, Resistor_SMD:R_0603_1608Metric_Pad1.05x0.95mm_HandSolder, B.Cu at (29.2, 5.38)
- added R63: R182,0603, Resistor_SMD:R_0603_1608Metric_Pad1.05x0.95mm_HandSolder, B.Cu at (33.4, 2.50)
- added R64: R100,0805, Resistor_SMD:R_0603_1608Metric_Pad1.05x0.95mm_HandSolder, B.Cu at (39.2, 5.25)
- added R65: R104,0805, Resistor_SMD:R_0805_2012Metric_Pad1.15x1.40mm_HandSolder, B.Cu at (36.0, 5.25)
- added R66: R100,0603, Resistor_SMD:R_0603_1608Metric_Pad1.05x0.95mm_HandSolder, B.Cu at (37.8, 5.25)
- added R67: R182,0603, Resistor_SMD:R_0603_1608Metric_Pad1.05x0.95mm_HandSolder, B.Cu at (41.8, 2.50)
- added R68: R104,0603, Resistor_SMD:R_0603_1608Metric_Pad1.05x0.95mm_HandSolder, F.Cu at (29.8, 74.8)
- added R69: R102,0603, Resistor_SMD:R_0603_1608Metric_Pad1.05x0.95mm_HandSolder, B.Cu at (33.0, 97.7)
- added R7: R102,0603, Resistor_SMD:R_0603_1608Metric_Pad1.05x0.95mm_HandSolder, B.Cu at (50.8, 70.8)
- added R70: R103,0603, Resistor_SMD:R_0603_1608Metric_Pad1.05x0.95mm_HandSolder, F.Cu at (29.8, 82.5)
- added R71: R104,0603, Resistor_SMD:R_0603_1608Metric_Pad1.05x0.95mm_HandSolder, F.Cu at (74.5, 75.0)
- added R72: R102,0603, Resistor_SMD:R_0603_1608Metric_Pad1.05x0.95mm_HandSolder, B.Cu at (78.2, 97.7)
- added R73: R103,0603, Resistor_SMD:R_0603_1608Metric_Pad1.05x0.95mm_HandSolder, F.Cu at (74.5, 85.5)
- added R74: R562,0603, Resistor_SMD:R_0603_1608Metric_Pad1.05x0.95mm_HandSolder, F.Cu at (59.5, 41.0)
- added R75: R103,0603, Resistor_SMD:R_0603_1608Metric_Pad1.05x0.95mm_HandSolder, F.Cu at (59.5, 37.5)
- added R76: R333,0603, Resistor_SMD:R_0603_1608Metric_Pad1.05x0.95mm_HandSolder, F.Cu at (59.5, 39.2)
- added R77: R562,0603, Resistor_SMD:R_0603_1608Metric_Pad1.05x0.95mm_HandSolder, F.Cu at (52.8, 30.0)
- added R78: R103,0603, Resistor_SMD:R_0603_1608Metric_Pad1.05x0.95mm_HandSolder, F.Cu at (52.2, 32.0)
- added R79: R333,0603, Resistor_SMD:R_0603_1608Metric_Pad1.05x0.95mm_HandSolder, F.Cu at (52.2, 33.8)
- added R8: R104,0603, Resistor_SMD:R_0603_1608Metric_Pad1.05x0.95mm_HandSolder, F.Cu at (90.8, 75.2)
- added R9: R102,0603, Resistor_SMD:R_0603_1608Metric_Pad1.05x0.95mm_HandSolder, B.Cu at (92.2, 97.7)
- added SW1: SW_Push, Button_Switch_SMD:SW_SPST_CK_RS282G05A3, F.Cu at (47.6, 68.0)
- added TH1: Thermistor_NTC, Resistor_SMD:R_0603_1608Metric_Pad1.05x0.95mm_HandSolder, F.Cu at (27.4, 21.6)
- added U1: orange_pi_zero, footprint-lib:orangepi-zero, B.Cu at (52.0, 69.5)
- added U10: A4988_MODULE, footprint-lib:Pololu_Breakout-16_15.2x20.3mm, F.Cu at (68.1, 74.4)
- added U11: MP2303A_ALT, footprint-lib:SOIC-8_3.9x4.9mm_P1.27mm,thermal_via, F.Cu at (68.0, 38.1)
- added U12: MP2303A_ALT, footprint-lib:SOIC-8_3.9x4.9mm_P1.27mm,thermal_via, F.Cu at (47.5, 35.1)
- added U2: A4988_MODULE, footprint-lib:Pololu_Breakout-16_15.2x20.3mm, F.Cu at (84.3, 74.4)
- added U3: A4988_MODULE, footprint-lib:Pololu_Breakout-16_15.2x20.3mm, F.Cu at (51.9, 74.4)
- added U4: A4988_MODULE, footprint-lib:Pololu_Breakout-16_15.2x20.3mm, F.Cu at (35.6, 74.4)
- added U5: A4988_MODULE, footprint-lib:Pololu_Breakout-16_15.2x20.3mm, F.Cu at (3.18, 74.4)
- added U6: A4988_MODULE, footprint-lib:Pololu_Breakout-16_15.2x20.3mm, F.Cu at (25.0, 57.9)
- added U7: A4988_MODULE, footprint-lib:Pololu_Breakout-16_15.2x20.3mm, F.Cu at (25.0, 41.9)
- added U8: STM32F407VET6, w_smd_lqfp:TQFP-100, F.Cu at (40.9, 57.5)
- added U9: A4988_MODULE, footprint-lib:Pololu_Breakout-16_15.2x20.3mm, F.Cu at (19.4, 74.4)
- added Y1: O_8M, Crystal:Crystal_HC49-4H_Vertical, F.Cu at (30.6, 64.0)
Connections:
- net +3V3_STM32 renamed +3V3
- net /X_MAX renamed PB3
- net /X_MIN renamed PB2
- net /Y_MAX renamed PB5
- net /Y_MIN renamed PB4
- net /Z_MAX renamed PB7
- net /Z_MIN renamed PB6
Routing:
- net +12V: track 0.00 -> 57.5 mm, vias 0 -> 1
- net +3V3: track 0.00 -> 33.8 mm, vias 0 -> 1
- net GND: track 0.00 -> 32.8 mm, vias 0 -> 2
- net PD3: track 0.00 -> 30.0 mm
- net Net-(J3-Pad4): track 0.00 -> 24.0 mm
- net Net-(C37-Pad2): track 0.00 -> 23.5 mm
- net Net-(J39-Pad4): track 0.00 -> 22.7 mm
- net Net-(J3-Pad3): track 0.00 -> 20.2 mm
- net Net-(J39-Pad3): track 0.00 -> 19.3 mm
- net Net-(J3-Pad2): track 0.00 -> 16.8 mm
- net Net-(J39-Pad2): track 0.00 -> 15.9 mm
- net Net-(J3-Pad1): track 0.00 -> 13.5 mm
- net Net-(J39-Pad1): track 0.00 -> 12.6 mm
- net Net-(Q5-Pad2): track 0.00 -> 10.1 mm
- net Net-(J2-Pad1): track 0.00 -> 8.54 mm
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Other:
- net class 12V added: clearance 0.2, trace_width 1.25, via_dia 0.8, via_drill 0.4
- net class 3V3 added: clearance 0.2, trace_width 0.25, via_dia 0.8, via_drill 0.4
- net class 5V added: clearance 0.2, trace_width 0.5, via_dia 0.8, via_drill 0.4
- net class GND added: clearance 0.2, trace_width 1.5, via_dia 0.8, via_drill 0.4

Commit message: update,
Parts:
- removed C1: CP100uf,10V, Capacitor_SMD:CP_Elec_6.3x5.3
- removed C10, C12, C2, C39, C4, C41, C6, C8: CP100uf,25V, Capacitor_SMD:CP_Elec_6.3x7.7
- removed C11, C13, C19, C21, C23, C25, C26, C27, C28, C3, C30, C31, C32, C33, C40, C42, C46, C5, C51, C7, C9: C104,0603, Capacitor_SMD:C_0603_1608Metric_Pad1.05x0.95mm_HandSolder
- removed C14, C15, C16, C17, C18, C45, C50: C106,0603, Capacitor_SMD:C_0603_1608Metric_Pad1.05x0.95mm_HandSolder
- removed C20: CP100uf,35V, Capacitor_SMD:CP_Elec_6.3x7.7
- removed C22, C24: C10pf,0603, Capacitor_SMD:C_0603_1608Metric_Pad1.05x0.95mm_HandSolder
- removed C29, C55: C105,0603, Capacitor_SMD:C_0603_1608Metric_Pad1.05x0.95mm_HandSolder
- removed C36, C37, C38: CP1uf,50V, Capacitor_SMD:CP_Elec_4x5.3
- removed C44: CP100uf,16V, Capacitor_SMD:CP_Elec_6.3x5.3
- removed C47, C52: C332,0603, Capacitor_SMD:C_0603_1608Metric_Pad1.05x0.95mm_HandSolder
- removed C48, C53: C103,0603, Capacitor_SMD:C_0603_1608Metric_Pad1.05x0.95mm_HandSolder
- removed C49, C54: C226,6.3v,0603, Capacitor_SMD:C_0603_1608Metric_Pad1.05x0.95mm_HandSolder
- removed D1: 5V HEALTHY, LED_SMD:LED_0603_1608Metric_Pad1.05x0.95mm_HandSolder
- removed D15, D16: SD_M4, Diode_SMD:D_SOD-323_HandSoldering
- removed D17: PB9, LED_SMD:LED_0603_1608Metric_Pad1.05x0.95mm_HandSolder
- removed D18, D19, D8: LED_RED,0603, LED_SMD:LED_0603_1608Metric_Pad1.05x0.95mm_HandSolder
- removed D2, D20, D21, D22, D23, D24, D3, D4, D5, D6, D7: LED_BLUE,0603, LED_SMD:LED_0603_1608Metric_Pad1.05x0.95mm_HandSolder
- removed F1: 16V/30A, w_misc_comp:fuse_smf
- removed F2: 30V/5A, w_misc_comp:fuse_smf
- removed H1, H2, H3, H4: MOUNT_M3, MountingHole:MountingHole_2.7mm_M2.5
- removed J1: USB_DEBUG, Connector_PinHeader_1.27mm:PinHeader_1x04_P1.27mm_Vertical
- removed J10, J12, J2, J36, J38, J4, J6, J8: MS_SELECT, Connector_PinHeader_2.54mm:PinHeader_2x03_P2.54mm_Vertical
- removed J11: E0, footprint-lib:b4b-ph-kl,stepper_terminal
- removed J13: E1, footprint-lib:b4b-ph-kl,stepper_terminal
- removed J14: HEATBED, footprint-lib:mpt_0,5%2f2-2,54,heatbed
- removed J21: HEATBED_TEMP, w_conn_jst-ph:b2b-ph-kl
- removed J22: HOTEND_TEMP0, w_conn_jst-ph:b2b-ph-kl
- removed J23: HOTEND_TEMP1, w_conn_jst-ph:b2b-ph-kl
- removed J24: AUX_TEMP, w_conn_jst-ph:b2b-ph-kl
- removed J25: 12V_INPUT_2, footprint-lib:mpt_0,5%2f2-2,54,12V_SRC
- removed J26: 12V_INPUT, footprint-lib:mpt_0,5%2f2-2,54,12V_SRC
- removed J27: 12V_OUT, footprint-lib:mpt_0,5%2f2-2,54,12V_SRC
- removed J28: SWD, Connector_PinHeader_1.27mm:PinHeader_1x04_P1.27mm_Vertical
- removed J29: USB_DEBUG, Connector_PinHeader_1.27mm:PinHeader_1x05_P1.27mm_Vertical
- removed J3: X, footprint-lib:b4b-ph-kl,stepper_terminal
- removed J30: PWR_DEBUG, Connector_PinHeader_1.27mm:PinHeader_1x05_P1.27mm_Vertical
- removed J31, J32: HOT_END, footprint-lib:mpt_0,5%2f2-2,54,heatbed
- removed J33: TO FAN0, footprint-lib:b2b-ph-kl,fan_pwm_out
- removed J34: TO FAN1, footprint-lib:b2b-ph-kl,fan_pwm_out
- removed J35: TO FAN2, footprint-lib:b2b-ph-kl,fan_pwm_out
- removed J37: Z2, footprint-lib:b4b-ph-kl,stepper_terminal
- removed J39: Y, footprint-lib:b4b-ph-kl,stepper_terminal
- removed J40: SPI_DEBUG, Connector_PinHeader_1.27mm:PinHeader_1x07_P1.27mm_Vertical
- removed J41: EXP1, Connector_PinHeader_2.54mm:PinHeader_2x05_P2.54mm_Vertical
- removed J42: EXP2, Connector_PinHeader_2.54mm:PinHeader_2x05_P2.54mm_Vertical
- removed J5: Z, footprint-lib:b4b-ph-kl,stepper_terminal
- removed J7: Z1, footprint-lib:b4b-ph-kl,stepper_terminal
- removed J9: Z3, footprint-lib:b4b-ph-kl,stepper_terminal
- removed JP5, JP6, JP7: Jumper_NO_Small, SolderJumper-2_P1.3mm_Open_TrianglePad1.0x1.5mm
- removed L1: L_Small, w_smd_inductors:inductor_smd_0603
- removed L2, L3: L_15uH, w_smd_inductors:inductor_smd_4.8x2.8mm
- removed Q1: WSK220N04, footprint-lib:TO-263-2,thermal_vias
- removed Q2, Q3: STP55NF06, footprint-lib:TO-263-2,thermal_vias
- removed Q4, Q5, Q6: D882, footprint-lib:SOT-89-3,thermal_vias
- removed R1, R2: R153,0603, Resistor_SMD:R_0603_1608Metric_Pad1.05x0.95mm_HandSolder
- removed R10, R13, R16, R19, R22, R25, R45, R46, R70, R73, R75, R78: R103,0603, Resistor_SMD:R_0603_1608Metric_Pad1.05x0.95mm_HandSolder
- removed R11, R14, R17, R20, R23, R68, R71, R8: R104,0603, Resistor_SMD:R_0603_1608Metric_Pad1.05x0.95mm_HandSolder
- removed R12, R15, R18, R21, R24, R44, R69, R7, R72, R9: R102,0603, Resistor_SMD:R_0603_1608Metric_Pad1.05x0.95mm_HandSolder
- removed R26, R50, R53, R56, R60: R100,0805, Resistor_SMD:R_0805_2012Metric_Pad1.15x1.40mm_HandSolder
- removed R27, R51, R54, R57, R61, R65: R104,0805, Resistor_SMD:R_0805_2012Metric_Pad1.15x1.40mm_HandSolder
- removed R28, R52, R55, R59, R63, R67: R182,0603, Resistor_SMD:R_0603_1608Metric_Pad1.05x0.95mm_HandSolder
- removed R3, R4, R47, R5: R220,0603, Resistor_SMD:R_0603_1608Metric_Pad1.05x0.95mm_HandSolder
- removed R35, R36, R37, R38, R39, R40, R41: R472,0603, Resistor_SMD:R_0603_1608Metric_Pad1.05x0.95mm_HandSolder
- removed R42, R43: R0,0603, Resistor_SMD:R_0603_1608Metric_Pad1.05x0.95mm_HandSolder
- removed R48, R6: R152,0603, Resistor_SMD:R_0603_1608Metric_Pad1.05x0.95mm_HandSolder
- removed R58, R62, R66: R100,0603, Resistor_SMD:R_0603_1608Metric_Pad1.05x0.95mm_HandSolder
- removed R64: R100,0805, Resistor_SMD:R_0603_1608Metric_Pad1.05x0.95mm_HandSolder
- removed R74, R77: R562,0603, Resistor_SMD:R_0603_1608Metric_Pad1.05x0.95mm_HandSolder
- removed R76, R79: R333,0603, Resistor_SMD:R_0603_1608Metric_Pad1.05x0.95mm_HandSolder
- removed SW1: SW_Push, Button_Switch_SMD:SW_SPST_CK_RS282G05A3
- removed TH1: Thermistor_NTC, Resistor_SMD:R_0603_1608Metric_Pad1.05x0.95mm_HandSolder
- removed U1: orange_pi_zero, footprint-lib:orangepi-zero
- removed U10, U2, U3, U4, U5, U6, U7, U9: A4988_MODULE, footprint-lib:Pololu_Breakout-16_15.2x20.3mm
- removed U11, U12: MP2303A_ALT, footprint-lib:SOIC-8_3.9x4.9mm_P1.27mm,thermal_via
- removed U8: STM32F407VET6, w_smd_lqfp:TQFP-100
- removed Y1: O_8M, Crystal:Crystal_HC49-4H_Vertical
- added J45: END_SWITCH_DEBUG, Connector_PinHeader_1.27mm:PinHeader_1x06_P1.27mm_Vertical, F.Cu at (64.8, 28.8)
- D10: value LED_BLUE,0603 -> XMAX
- D9: value LED_BLUE,0603 -> XMIN
- moved J19 29.7 mm to (71.8, 32.7)
- moved J15 23.3 mm to (71.8, 21.4)
- moved R33 22.9 mm to (76.9, 15.6)
- moved D13 22.8 mm to (76.9, 15.6)
- moved R29 21.8 mm to (69.3, 15.6)
- moved D9 21.8 mm to (69.3, 15.6)
- moved R30 21.6 mm to (71.2, 15.6)
- moved D10 21.6 mm to (71.2, 15.6)
- moved R31 21.5 mm to (73.1, 15.6)
- moved D11 21.5 mm to (73.1, 15.6)
- moved R32 21.3 mm to (75.0, 15.6)
- moved D12 21.3 mm to (75.0, 15.6)
- moved D14 19.3 mm to (78.8, 15.6)
- moved R34 19.3 mm to (78.9, 15.6)
- moved J17 18.7 mm to (71.8, 27.1)
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Connections:
- net +3V3 renamed +3V3_STM32
- net PB2 renamed /X_MIN
- net PB3 renamed /X_MAX
- net PB4 renamed /Y_MIN
- net PB5 renamed /Y_MAX
- net PB6 renamed /Z_MIN
- net PB7 renamed /Z_MAX
Routing:
- net +12V: track 57.5 -> 0.00 mm, vias 1 -> 0
- net /Z_MAX: track 0.00 -> 53.6 mm
- net /Z_MIN: track 0.00 -> 35.9 mm, vias 0 -> 1
- net /X_MAX: track 0.00 -> 32.8 mm, vias 0 -> 1
- net /Y_MAX: track 0.00 -> 30.3 mm, vias 0 -> 1
- net PD3: track 30.0 -> 0.00 mm
- net Net-(J3-Pad4): track 24.0 -> 0.00 mm
- net Net-(C37-Pad2): track 23.5 -> 0.00 mm
- net Net-(J39-Pad4): track 22.7 -> 0.00 mm
- net /Y_MIN: track 0.00 -> 21.9 mm
- net Net-(J3-Pad3): track 20.2 -> 0.00 mm
- net Net-(J39-Pad3): track 19.3 -> 0.00 mm
- net Net-(J3-Pad2): track 16.8 -> 0.00 mm
- net Net-(J39-Pad2): track 15.9 -> 0.00 mm
- net /X_MIN: track 0.00 -> 14.6 mm
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Other:
- board outline removed

Commit message: update,
Parts:
- added D15: LED_BLUE,0603, LED_SMD:LED_0603_1608Metric_Pad1.05x0.95mm_HandSolder, F.Cu at (39.6, 17.1)
- added D16: SD_1N5817_SS12, w_smd_diode:do214ac, B.Cu at (39.9, 19.1)
- added D25: SD_1N5817_SS12, w_smd_diode:do214ac, F.Cu at (67.5, 16.1)
- added D26: SD_1N5817_SS12, w_smd_diode:do214ac, F.Cu at (56.0, 34.0)
- added J1: HOTEND_PROBE, footprint-lib:b3b-ph-kl,end_stop, F.Cu at (34.6, 20.1)
- added JP1: SolderJumper_2_Open, Jumper:SolderJumper-2_P1.3mm_Open_RoundedPad1.0x1.5mm, F.Cu at (53.2, 23.2)
- added JP2: SolderJumper_2_Open, Jumper:SolderJumper-2_P1.3mm_Open_RoundedPad1.0x1.5mm, F.Cu at (39.4, 22.2)
- added R49: R102,0603, Resistor_SMD:R_0603_1608Metric_Pad1.05x0.95mm_HandSolder, F.Cu at (39.6, 18.9)
- D10: value XMAX -> LED_BLUE,0603
Connections:
- D13 pad 1: /Z_MIN -> Net-(D13-Pad1)
- D14 pad 1: /Z_MAX -> Net-(D14-Pad1)
- J15 pad 2: +3V3_STM32 -> Net-(J15-Pad2)
- J16 pad 2: +3V3_STM32 -> Net-(J15-Pad2)
- J17 pad 2: +3V3_STM32 -> Net-(J15-Pad2)
- J18 pad 2: +3V3_STM32 -> Net-(J15-Pad2)
- J19 pad 1: /Z_MIN -> Net-(D13-Pad1)
- J19 pad 2: +3V3_STM32 -> Net-(J15-Pad2)
- J20 pad 1: /Z_MAX -> Net-(D14-Pad1)
- J20 pad 2: +3V3_STM32 -> Net-(J15-Pad2)
