File: hardware/printer-board/POWER_SUPPLY.sch (KiCad schematic (older format))
At the start: 10 parts, among them J26 12V_INPUT_2, J34 12V_INPUT, J35 12V_OUT

Commit message: update to re-annotation,
Parts:
- renumbered C21 to C20, D6 to D15, D7 to D16, J26 to J25, J34 to J26, J35 to J27, JP12 to JP5
Changed lines of the file:
@@
 $EndDescr
 $Comp
-L Connector:Screw_Terminal_01x02 J34
+L Connector:Screw_Terminal_01x02 J26
 U 1 1 5CC1F612
 P 4950 2150
-AR Path="/5CC1F2C3/5CC1F612" Ref="J34"  Part="1"
+AR Path="/5CC1F2C3/5CC1F612" Ref="J26"  Part="1"
 AR Path="/5CC2225A/5CC1F612" Ref="J?"  Part="1"
-F 0 "J34" H 4870 2367 50  0000 C CNN
+F 0 "J26" H 4870 2367 50  0000 C CNN
 F 1 "12V_INPUT" H 4870 2276 50  0000 C CNN
 F 2 "footprint-lib:mpt_0,5%2f2-2,54,12V_SRC" H 4950 2150 50  0001 C CNN
@@
 $EndComp
 $Comp
-L power:GND #PWR0246
+L power:GND #PWR098
 U 1 1 5CC1F72C
 P 5250 2550
-AR Path="/5CC1F2C3/5CC1F72C" Ref="#PWR0246"  Part="1"
+AR Path="/5CC1F2C3/5CC1F72C" Ref="#PWR098"  Part="1"
 AR Path="/5CC2225A/5CC1F72C" Ref="#PWR?"  Part="1"
-F 0 "#PWR0246" H 5250 2300 50  0001 C CNN
+F 0 "#PWR098" H 5250 2300 50  0001 C CNN
 F 1 "GND" H 5255 2377 50  0000 C CNN
 F 2 "" H 5250 2550 50  0001 C CNN
@@
 AR Path="/5CC1F2C3/5CC1F828" Ref="F1"  Part="1"
 AR Path="/5CC2225A/5CC1F828" Ref="F?"  Part="1"
-AR Path="/5CC1F828" Ref="F1"  Part="1"
+AR Path="/5CC1F828" Ref="F?"  Part="1"
 F 0 "F1" H 5700 1535 50  0000 C CNN
 F 1 "16V/30A" H 5700 1444 50  0000 C CNN
@@
 AR Path="/5CC1F2C3/5CC1F89C" Ref="F2"  Part="1"
 AR Path="/5CC2225A/5CC1F89C" Ref="F?"  Part="1"
-AR Path="/5CC1F89C" Ref="F2"  Part="1"
+AR Path="/5CC1F89C" Ref="F?"  Part="1"
 F 0 "F2" H 5700 2335 50  0000 C CNN
 F 1 "30V/5A" H 5700 2244 50  0000 C CNN
@@
 $EndComp
 $Comp
-L taobao-components:+12V2 #PWR0247
+L taobao-components:+12V2 #PWR0101
 U 1 1 5CC1F959
 P 6100 1100
-AR Path="/5CC1F2C3/5CC1F959" Ref="#PWR0247"  Part="1"
+AR Path="/5CC1F2C3/5CC1F959" Ref="#PWR0101"  Part="1"
 AR Path="/5CC2225A/5CC1F959" Ref="#PWR?"  Part="1"
-F 0 "#PWR0247" H 6100 950 50  0001 C CNN
+F 0 "#PWR0101" H 6100 950 50  0001 C CNN
 F 1 "+12V2" H 6115 1273 50  0000 C CNN
 F 2 "" H 6100 1100 50  0001 C CNN
@@
 	6100 1350 5800 1350
 $Comp
-L Connector:Screw_Terminal_01x02 J35
+L Connector:Screw_Terminal_01x02 J27
 U 1 1 5CC1F9B4
 P 8250 2150
-AR Path="/5CC1F2C3/5CC1F9B4" Ref="J35"  Part="1"
+AR Path="/5CC1F2C3/5CC1F9B4" Ref="J27"  Part="1"
 AR Path="/5CC2225A/5CC1F9B4" Ref="J?"  Part="1"
-F 0 "J35" H 8329 2142 50  0000 L CNN
+F 0 "J27" H 8329 2142 50  0000 L CNN
 F 1 "12V_OUT" H 8329 2051 50  0000 L CNN
 F 2 "footprint-lib:mpt_0,5%2f2-2,54,12V_SRC" H 8250 2150 50  0001 C CNN
@@
 $EndComp
 $Comp
-L power:GND #PWR0248
+L power:GND #PWR0105
 U 1 1 5CC1FAAA
 P 7950 2400
-AR Path="/5CC1F2C3/5CC1FAAA" Ref="#PWR0248"  Part="1"
+AR Path="/5CC1F2C3/5CC1FAAA" Ref="#PWR0105"  Part="1"
 AR Path="/5CC2225A/5CC1FAAA" Ref="#PWR?"  Part="1"
-F 0 "#PWR0248" H 7950 2150 50  0001 C CNN
+F 0 "#PWR0105" H 7950 2150 50  0001 C CNN
 F 1 "GND" H 7955 2227 50  0000 C CNN
 F 2 "" H 7950 2400 50  0001 C CNN
@@
 	8050 2150 7950 2150
 $Comp
-L taobao-sd:SD_M4 D6
+L taobao-sd:SD_M4 D15
 U 1 1 5CC20016
 P 6000 3550
-AR Path="/5CC1F2C3/5CC20016" Ref="D6"  Part="1"
+AR Path="/5CC1F2C3/5CC20016" Ref="D15"  Part="1"
 AR Path="/5CC2225A/5CC20016" Ref="D?"  Part="1"
-F 0 "D6" V 5954 3618 50  0000 L CNN
+F 0 "D15" V 5954 3618 50  0000 L CNN
 F 1 "SD_M4" V 6045 3618 50  0000 L CNN
 F 2 "Diode_SMD:D_SOD-323_HandSoldering" V 6000 3550 50  0001 C CNN
@@
 $EndComp
 $Comp
-L taobao-sd:SD_M4 D7
+L taobao-sd:SD_M4 D16
 U 1 1 5CC200A7
 P 6450 3350
-AR Path="/5CC1F2C3/5CC200A7" Ref="D7"  Part="1"
+AR Path="/5CC1F2C3/5CC200A7" Ref="D16"  Part="1"
 AR Path="/5CC2225A/5CC200A7" Ref="D?"  Part="1"
-F 0 "D7" H 6450 3145 50  0000 C CNN
+F 0 "D16" H 6450 3145 50  0000 C CNN
 F 1 "SD_M4" H 6450 3236 50  0000 C CNN
 F 2 "Diode_SMD:D_SOD-323_HandSoldering" V 6450 3350 50  0001 C CNN
@@
 $EndComp
 $Comp
-L power:GND #PWR0249
+L power:GND #PWR0100
 U 1 1 5CC2014F
 P 6000 3850
-AR Path="/5CC1F2C3/5CC2014F" Ref="#PWR0249"  Part="1"
+AR Path="/5CC1F2C3/5CC2014F" Ref="#PWR0100"  Part="1"
 AR Path="/5CC2225A/5CC2014F" Ref="#PWR?"  Part="1"
-F 0 "#PWR0249" H 6000 3600 50  0001 C CNN
+F 0 "#PWR0100" H 6000 3600 50  0001 C CNN
 F 1 "GND" H 6005 3677 50  0000 C CNN
 F 2 "" H 6000 3850 50  0001 C CNN
@@
 $EndBitmap
 $Comp
-L power:+12V #PWR041
+L power:+12V #PWR0104
 U 1 1 5CC6A38A
 P 7950 2000
-F 0 "#PWR041" H 7950 1850 50  0001 C CNN
+F 0 "#PWR0104" H 7950 1850 50  0001 C CNN
 F 1 "+12V" H 7950 2200 50  0000 C CNN
 F 2 "" H 7950 2000 50  0001 C CNN
@@
 	6000 2150 6000 3350
 $Comp
-L power:GND #PWR042
+L power:GND #PWR0102
 U 1 1 5CC6F3BF
 P 6650 2550
-F 0 "#PWR042" H 6650 2300 50  0001 C CNN
+F 0 "#PWR0102" H 6650 2300 50  0001 C CNN
 F 1 "GND" H 6700 2350 50  0000 C CNN
 F 2 "" H 6650 2550 50  0001 C CNN
@@
 	6650 2400 6650 2550
 $Comp
-L power:GND #PWR043
+L power:GND #PWR0103
 U 1 1 5CC6F579
 P 7200 2550
-F 0 "#PWR043" H 7200 2300 50  0001 C CNN
+F 0 "#PWR0103" H 7200 2300 50  0001 C CNN
 F 1 "GND" H 7250 2350 50  0000 C CNN
 F 2 "" H 7200 2550 50  0001 C CNN
@@
 $EndComp
 $Comp
-L taobao-cp:CP100uf,35V C21
+L taobao-cp:CP100uf,35V C20
 U 1 1 5CC6F6C1
 P 7200 2350
-F 0 "C21" H 7300 2400 50  0000 L CNN
+F 0 "C20" H 7300 2400 50  0000 L CNN
 F 1 "CP100uf,35V" H 7300 2350 50  0000 L CNN
 F 2 "Capacitor_SMD:CP_Elec_6.3x7.7" H 7200 2350 50  0001 C CNN
@@
 	5150 2150 5500 2150
 $Comp
-L Connector:Screw_Terminal_01x02 J26
+L Connector:Screw_Terminal_01x02 J25
 U 1 1 5CCBA098
 P 4950 1350
-AR Path="/5CC1F2C3/5CCBA098" Ref="J26"  Part="1"
+AR Path="/5CC1F2C3/5CCBA098" Ref="J25"  Part="1"
 AR Path="/5CC2225A/5CCBA098" Ref="J?"  Part="1"
-F 0 "J26" H 4870 1567 50  0000 C CNN
+F 0 "J25" H 4870 1567 50  0000 C CNN
 F 1 "12V_INPUT_2" H 4870 1476 50  0000 C CNN
 F 2 "footprint-lib:mpt_0,5%2f2-2,54,12V_SRC" H 4950 1350 50  0001 C CNN
@@
 	5150 1350 5500 1350
 $Comp
-L power:GND #PWR040
+L power:GND #PWR099
 U 1 1 5CCBB25F
 P 5300 1550
-F 0 "#PWR040" H 5300 1300 50  0001 C CNN
+F 0 "#PWR099" H 5300 1300 50  0001 C CNN
 F 1 "GND" H 5350 1350 50  0000 C CNN
 F 2 "" H 5300 1550 50  0001 C CNN
@@
 	5300 1450 5300 1550
 $Comp
-L Device:Jumper_NO_Small JP12
+L Device:Jumper_NO_Small JP5
 U 1 1 5CCBB5DC
 P 5500 1750
-F 0 "JP12" V 5450 1800 50  0000 L CNN
+F 0 "JP5" V 5450 1800 50  0000 L CNN
 F 1 "Jumper_NO_Small" V 5500 1800 50  0000 L CNN
 F 2 "SolderJumper-2_P1.3mm_Open_TrianglePad1.0x1.5mm" H 5500 1750 50  0001 C CNN

Commit message: update ROUTING,
Parts:
- removed D15, D16: SD_M4, Diode_SMD:D_SOD-323_HandSoldering, symbol taobao-sd:SD_M4
Other:
- note added: "optional to get another source for +12v2\n"
Changed lines of the file:
@@
 EESchema Schematic File Version 4
 LIBS:printer-board-cache
-EELAYER 26 0
+EELAYER 29 0
 EELAYER END
 $Descr A4 11693 8268
@@
 Wire Wire Line
 	8050 2150 7950 2150
-$Comp
-L taobao-sd:SD_M4 D15
-U 1 1 5CC20016
-P 6000 3550
-AR Path="/5CC1F2C3/5CC20016" Ref="D15"  Part="1"
-AR Path="/5CC2225A/5CC20016" Ref="D?"  Part="1"
-AR Path="/5CC20016" Ref="D15"  Part="1"
-F 0 "D15" V 5954 3618 50  0000 L CNN
-F 1 "SD_M4" V 6045 3618 50  0000 L CNN
-F 2 "Diode_SMD:D_SOD-323_HandSoldering" V 6000 3550 50  0001 C CNN
-F 3 "~" V 6000 3550 50  0001 C CNN
-	1    6000 3550
-	0    1    1    0
-$EndComp
-$Comp
-L taobao-sd:SD_M4 D16
-U 1 1 5CC200A7
-P 6450 3350
-AR Path="/5CC1F2C3/5CC200A7" Ref="D16"  Part="1"
-AR Path="/5CC2225A/5CC200A7" Ref="D?"  Part="1"
-AR Path="/5CC200A7" Ref="D16"  Part="1"
-F 0 "D16" H 6450 3145 50  0000 C CNN
-F 1 "SD_M4" H 6450 3236 50  0000 C CNN
-F 2 "Diode_SMD:D_SOD-323_HandSoldering" V 6450 3350 50  0001 C CNN
-F 3 "~" V 6450 3350 50  0001 C CNN
-	1    6450 3350
-	-1   0    0    1
-$EndComp
-$Comp
-L power:GND #PWR0100
-U 1 1 5CC2014F
-P 6000 3850
-AR Path="/5CC1F2C3/5CC2014F" Ref="#PWR0100"  Part="1"
-AR Path="/5CC2225A/5CC2014F" Ref="#PWR?"  Part="1"
-AR Path="/5CC2014F" Ref="#PWR0100"  Part="1"
-F 0 "#PWR0100" H 6000 3600 50  0001 C CNN
-F 1 "GND" H 6005 3677 50  0000 C CNN
-F 2 "" H 6000 3850 50  0001 C CNN
-F 3 "" H 6000 3850 50  0001 C CNN
-	1    6000 3850
-	1    0    0    -1
-$EndComp
-Wire Wire Line
-	6000 3850 6000 3650
-Wire Wire Line
-	6000 3450 6000 3350
-Wire Wire Line
-	6350 3350 6000 3350
-Text Label 7150 3350 2    50   ~ 0
-AM-VIN
-Wire Wire Line
-	6550 3350 7150 3350
 $Bitmap
 Pos 9000 5750
@@
 Wire Wire Line
 	5250 2250 5250 2550
-Connection ~ 6000 3350
-Wire Wire Line
-	5800 2150 6000 2150
-Wire Wire Line
-	6000 2150 6000 3350
 $Comp
 L power:GND #PWR0102
@@
 Wire Wire Line
 	7200 2150 7950 2150
-Wire Wire Line
-	6650 2150 6000 2150
 Connection ~ 6650 2150
-Connection ~ 6000 2150
 Wire Wire Line
 	5150 2150 5500 2150
@@
 Wire Wire Line
 	5500 2150 5600 2150
+Wire Wire Line
+	5800 2150 6650 2150
+Wire Notes Line
+	3550 750  5400 750
+Wire Notes Line
+	5400 750  5400 1700
+Wire Notes Line
+	5400 1700 3550 1700
+Wire Notes Line
+	3550 1700 3550 750
+Text Notes 3550 850  0    50   ~ 0
+optional to get another source for +12v2\n
 $EndSCHEMATC

Commit message: update ROUTING,
Parts:
- J25: value 12V_INPUT_2 -> 12V_IN2
- J26: value 12V_INPUT -> 12V_IN
- J27: value 12V_OUT -> 12V/OUT
Changed lines of the file:
@@
 AR Path="/5CC1F612" Ref="J26"  Part="1"
 F 0 "J26" H 4870 2367 50  0000 C CNN
-F 1 "12V_INPUT" H 4870 2276 50  0000 C CNN
+F 1 "12V_IN" H 4870 2276 50  0000 C CNN
 F 2 "footprint-lib:mpt_0,5%2f2-2,54,12V_SRC" H 4950 2150 50  0001 C CNN
 F 3 "~" H 4950 2150 50  0001 C CNN
@@
 AR Path="/5CC1F9B4" Ref="J27"  Part="1"
 F 0 "J27" H 8329 2142 50  0000 L CNN
-F 1 "12V_OUT" H 8329 2051 50  0000 L CNN
+F 1 "12V/OUT" H 8329 2051 50  0000 L CNN
 F 2 "footprint-lib:mpt_0,5%2f2-2,54,12V_SRC" H 8250 2150 50  0001 C CNN
 F 3 "~" H 8250 2150 50  0001 C CNN
@@
 AR Path="/5CCBA098" Ref="J25"  Part="1"
 F 0 "J25" H 4870 1567 50  0000 C CNN
-F 1 "12V_INPUT_2" H 4870 1476 50  0000 C CNN
+F 1 "12V_IN2" H 4870 1476 50  0000 C CNN
 F 2 "footprint-lib:mpt_0,5%2f2-2,54,12V_SRC" H 4950 1350 50  0001 C CNN
 F 3 "~" H 4950 1350 50  0001 C CNN
