File: hardware/printer-board/Thermistors.sch (KiCad schematic (older format))
At the start: 15 parts, among them J32 Screw_Terminal_01x02, J33 Screw_Terminal_01x02, J43 Screw_Terminal_01x02, J44 Screw_Terminal_01x02

Commit message: remove jumper in display FPC,
Parts:
- removed C29, C30, C31, C35, C36: CP10uf,50V, Capacitor_SMD:CP_Elec_5x5.3, symbol taobao-cp:CP10uf,50V
- added C29, C30, C31, C35, C36: C106,0603, Capacitor_SMD:C_0603_1608Metric_Pad1.05x0.95mm_HandSolder, symbol taobao-c:C106,0603
Connections:
- net AUX_TEMP: now also C35.1
- net GND: now also C29.2, C30.2, C31.2, C35.2, C36.2
- net HEATBED_TEMP: now also C29.1
- net HOTEND_TEMP1: now also C31.1
- net HOTEND_TEMP2: now also C30.1
- net PCB_TEMP: now also C36.1
Changed lines of the file:
@@
-$EndComp
-$Comp
-L taobao-cp:CP10uf,50V C31
-U 1 1 5CC409ED
-P 950 3300
-F 0 "C31" H 1038 3346 50  0000 L CNN
-F 1 "CP10uf,50V" H 1038 3255 50  0000 L CNN
-F 2 "Capacitor_SMD:CP_Elec_5x5.3" H 950 3300 50  0001 C CNN
-F 3 "~" H 950 3300 50  0001 C CNN
-	1    950  3300
-	1    0    0    -1
 $EndComp
 $Comp
@@
 $EndComp
 $Comp
-L taobao-cp:CP10uf,50V C35
-U 1 1 5CC40ECB
-P 950 4950
-F 0 "C35" H 1038 4996 50  0000 L CNN
-F 1 "CP10uf,50V" H 1038 4905 50  0000 L CNN
-F 2 "Capacitor_SMD:CP_Elec_5x5.3" H 950 4950 50  0001 C CNN
-F 3 "~" H 950 4950 50  0001 C CNN
-	1    950  4950
-	1    0    0    -1
-$EndComp
-$Comp
 L power:GND #PWR0275
 U 1 1 5CC40ED1
@@
 $EndComp
 $Comp
-L taobao-cp:CP10uf,50V C30
-U 1 1 5CC416F9
-P 3500 1750
-F 0 "C30" H 3588 1796 50  0000 L CNN
-F 1 "CP10uf,50V" H 3588 1705 50  0000 L CNN
-F 2 "Capacitor_SMD:CP_Elec_5x5.3" H 3500 1750 50  0001 C CNN
-F 3 "~" H 3500 1750 50  0001 C CNN
-	1    3500 1750
-	1    0    0    -1
-$EndComp
-$Comp
 L power:GND #PWR0281
 U 1 1 5CC416FF
@@
 $EndComp
 $Comp
-L taobao-cp:CP10uf,50V C36
-U 1 1 5CC40EFD
-P 3500 3650
-F 0 "C36" H 3588 3696 50  0000 L CNN
-F 1 "CP10uf,50V" H 3588 3605 50  0000 L CNN
-F 2 "Capacitor_SMD:CP_Elec_5x5.3" H 3500 3650 50  0001 C CNN
-F 3 "~" H 3500 3650 50  0001 C CNN
-	1    3500 3650
-	1    0    0    -1
-$EndComp
-$Comp
 L taobao-r:R472,0603 R58
 U 1 1 5CC40EF7
@@
 	4150 3450 4350 3450
 $Comp
-L taobao-cp:CP10uf,50V C29
-U 1 1 5CC3DD4B
+L taobao-c:C106,0603 C31
+U 1 1 5CCAA148
+P 950 3300
+F 0 "C31" H 1042 3346 50  0000 L CNN
+F 1 "C106,0603" H 1042 3255 50  0000 L CNN
+F 2 "Capacitor_SMD:C_0603_1608Metric_Pad1.05x0.95mm_HandSolder" H 950 3300 50  0001 C CNN
+F 3 "~" H 950 3300 50  0001 C CNN
+	1    950  3300
+	1    0    0    -1
+$EndComp
+$Comp
+L taobao-c:C106,0603 C29
+U 1 1 5CCAA34C
 P 950 1750
-F 0 "C29" H 1038 1796 50  0000 L CNN
-F 1 "CP10uf,50V" H 1038 1705 50  0000 L CNN
-F 2 "Capacitor_SMD:CP_Elec_5x5.3" H 950 1750 50  0001 C CNN
+F 0 "C29" H 1042 1796 50  0000 L CNN
+F 1 "C106,0603" H 1042 1705 50  0000 L CNN
+F 2 "Capacitor_SMD:C_0603_1608Metric_Pad1.05x0.95mm_HandSolder" H 950 1750 50  0001 C CNN
 F 3 "~" H 950 1750 50  0001 C CNN
 	1    950  1750
 	1    0    0    -1
 $EndComp
+$Comp
+L taobao-c:C106,0603 C35
+U 1 1 5CCAA3BA
+P 3500 1750
+F 0 "C35" H 3592 1796 50  0000 L CNN
+F 1 "C106,0603" H 3592 1705 50  0000 L CNN
+F 2 "Capacitor_SMD:C_0603_1608Metric_Pad1.05x0.95mm_HandSolder" H 3500 1750 50  0001 C CNN
+F 3 "~" H 3500 1750 50  0001 C CNN
+	1    3500 1750
+	1    0    0    -1
+$EndComp
+$Comp
+L taobao-c:C106,0603 C36
+U 1 1 5CCAA42C
+P 3500 3650
+F 0 "C36" H 3592 3696 50  0000 L CNN
+F 1 "C106,0603" H 3592 3605 50  0000 L CNN
+F 2 "Capacitor_SMD:C_0603_1608Metric_Pad1.05x0.95mm_HandSolder" H 3500 3650 50  0001 C CNN
+F 3 "~" H 3500 3650 50  0001 C CNN
+	1    3500 3650
+	1    0    0    -1
+$EndComp
+$Comp
+L taobao-c:C106,0603 C30
+U 1 1 5CCAA49C
+P 950 4950
+F 0 "C30" H 1042 4996 50  0000 L CNN
+F 1 "C106,0603" H 1042 4905 50  0000 L CNN
+F 2 "Capacitor_SMD:C_0603_1608Metric_Pad1.05x0.95mm_HandSolder" H 950 4950 50  0001 C CNN
+F 3 "~" H 950 4950 50  0001 C CNN
+	1    950  4950
+	1    0    0    -1
+$EndComp

Commit message: update to re-annotation,
Parts:
- J21: renamed from J32; value Screw_Terminal_01x02 -> HEATBED_TEMP
- J22: renamed from J43; value Screw_Terminal_01x02 -> HOTEND_TEMP0
- J23: renamed from J44; value Screw_Terminal_01x02 -> HOTEND_TEMP1
- J24: renamed from J33; value Screw_Terminal_01x02 -> AUX_TEMP
- renumbered C29 to C14, C31 to C15, C30 to C16, C35 to C17, C36 to C18, R33 to R35, R35 to R36, R57 to R37, R34 to R38, R58 to R39
Connections:
- net HOTEND_TEMP2 is gone; now on net HOTEND_TEMP1: C16.1, J23.1 (Pin_1), R37.2
- net HOTEND_TEMP1: no longer C15.1, J22.1 (Pin_1), R36.2
- new net HOTEND_TEMP0: C15.1, J22.1 (Pin_1), R36.2
Changed lines of the file:
@@
 $EndBitmap
 $Comp
-L taobao-r:R472,0603 R33
+L taobao-r:R472,0603 R35
 U 1 1 5CC3DD45
 P 950 1300
-F 0 "R33" H 1009 1346 50  0000 L CNN
+F 0 "R35" H 1009 1346 50  0000 L CNN
 F 1 "R472,0603" H 1009 1255 50  0000 L CNN
 F 2 "Resistor_SMD:R_0603_1608Metric_Pad1.05x0.95mm_HandSolder" H 950 1300 50  0001 C CNN
@@
 $EndComp
 $Comp
-L power:GND #PWR0240
+L power:GND #PWR084
 U 1 1 5CC3DD51
 P 950 2100
-F 0 "#PWR0240" H 950 1850 50  0001 C CNN
+F 0 "#PWR084" H 950 1850 50  0001 C CNN
 F 1 "GND" H 955 1927 50  0000 C CNN
 F 2 "" H 950 2100 50  0001 C CNN
@@
 	950  1550 950  1650
 $Comp
-L Connector:Screw_Terminal_01x02 J32
+L Connector:Screw_Terminal_01x02 J21
 U 1 1 5CC3E589
 P 1950 1550
-F 0 "J32" H 2050 1550 50  0000 L CNN
-F 1 "Screw_Terminal_01x02" H 2050 1450 50  0000 L CNN
+F 0 "J21" H 2050 1550 50  0000 L CNN
+F 1 "HEATBED_TEMP" H 2050 1450 50  0000 L CNN
 F 2 "w_conn_jst-ph:b2b-ph-kl" H 1950 1550 50  0001 C CNN
 F 3 "~" H 1950 1550 50  0001 C CNN
@@
 	950  1550 1600 1550
 $Comp
-L power:GND #PWR0241
+L power:GND #PWR089
 U 1 1 5CC3F185
 P 1650 2100
-F 0 "#PWR0241" H 1650 1850 50  0001 C CNN
+F 0 "#PWR089" H 1650 1850 50  0001 C CNN
 F 1 "GND" H 1655 1927 50  0000 C CNN
 F 2 "" H 1650 2100 50  0001 C CNN
@@
 HEATBED_TEMP
 $Comp
-L taobao-r:R472,0603 R35
+L taobao-r:R472,0603 R36
 U 1 1 5CC409E7
 P 950 2850
-F 0 "R35" H 1009 2896 50  0000 L CNN
+F 0 "R36" H 1009 2896 50  0000 L CNN
 F 1 "R472,0603" H 1009 2805 50  0000 L CNN
 F 2 "Resistor_SMD:R_0603_1608Metric_Pad1.05x0.95mm_HandSolder" H 950 2850 50  0001 C CNN
@@
 $EndComp
 $Comp
-L power:GND #PWR0243
+L power:GND #PWR086
 U 1 1 5CC409F3
 P 950 3650
-F 0 "#PWR0243" H 950 3400 50  0001 C CNN
+F 0 "#PWR086" H 950 3400 50  0001 C CNN
 F 1 "GND" H 955 3477 50  0000 C CNN
 F 2 "" H 950 3650 50  0001 C CNN
@@
 	950  3100 950  3200
 $Comp
-L Connector:Screw_Terminal_01x02 J43
+L Connector:Screw_Terminal_01x02 J22
 U 1 1 5CC409FE
 P 1950 3100
-F 0 "J43" H 2050 3100 50  0000 L CNN
-F 1 "Screw_Terminal_01x02" H 2050 3000 50  0000 L CNN
+F 0 "J22" H 2050 3100 50  0000 L CNN
+F 1 "HOTEND_TEMP0" H 2050 3000 50  0000 L CNN
 F 2 "w_conn_jst-ph:b2b-ph-kl" H 1950 3100 50  0001 C CNN
 F 3 "~" H 1950 3100 50  0001 C CNN
@@
 	950  3100 1600 3100
 $Comp
-L power:GND #PWR0244
+L power:GND #PWR090
 U 1 1 5CC40A05
 P 1650 3650
-F 0 "#PWR0244" H 1650 3400 50  0001 C CNN
+F 0 "#PWR090" H 1650 3400 50  0001 C CNN
 F 1 "GND" H 1655 3477 50  0000 C CNN
 F 2 "" H 1650 3650 50  0001 C CNN
@@
 	1650 3200 1750 3200
 Text Label 2200 2850 2    50   ~ 0
-HOTEND_TEMP1
+HOTEND_TEMP0
 Wire Wire Line
 	2250 2850 1600 2850
@@
 	1600 3100 1750 3100
 Text HLabel 2250 2850 2    50   Input ~ 0
-HOTEND_TEMP1
-$Comp
-L taobao-r:R472,0603 R57
+HOTEND_TEMP0
+$Comp
+L taobao-r:R472,0603 R37
 U 1 1 5CC40EC5
 P 950 4500
-F 0 "R57" H 1009 4546 50  0000 L CNN
+F 0 "R37" H 1009 4546 50  0000 L CNN
 F 1 "R472,0603" H 1009 4455 50  0000 L CNN
 F 2 "Resistor_SMD:R_0603_1608Metric_Pad1.05x0.95mm_HandSolder" H 950 4500 50  0001 C CNN
@@
 $EndComp
 $Comp
-L power:GND #PWR0275
+L power:GND #PWR088
 U 1 1 5CC40ED1
 P 950 5300
-F 0 "#PWR0275" H 950 5050 50  0001 C CNN
+F 0 "#PWR088" H 950 5050 50  0001 C CNN
 F 1 "GND" H 955 5127 50  0000 C CNN
 F 2 "" H 950 5300 50  0001 C CNN
@@
 	950  4750 950  4850
 $Comp
-L Connector:Screw_Terminal_01x02 J44
+L Connector:Screw_Terminal_01x02 J23
 U 1 1 5CC40EDC
 P 1950 4750
-F 0 "J44" H 2050 4750 50  0000 L CNN
-F 1 "Screw_Terminal_01x02" H 2050 4650 50  0000 L CNN
+F 0 "J23" H 2050 4750 50  0000 L CNN
+F 1 "HOTEND_TEMP1" H 2050 4650 50  0000 L CNN
 F 2 "w_conn_jst-ph:b2b-ph-kl" H 1950 4750 50  0001 C CNN
 F 3 "~" H 1950 4750 50  0001 C CNN
@@
 	950  4750 1600 4750
 $Comp
-L power:GND #PWR0276
+L power:GND #PWR091
 U 1 1 5CC40EE3
 P 1650 5300
-F 0 "#PWR0276" H 1650 5050 50  0001 C CNN
+F 0 "#PWR091" H 1650 5050 50  0001 C CNN
 F 1 "GND" H 1655 5127 50  0000 C CNN
 F 2 "" H 1650 5300 50  0001 C CNN
@@
 	1650 4850 1750 4850
 Text Label 2200 4500 2    50   ~ 0
-HOTEND_TEMP2
+HOTEND_TEMP1
 Wire Wire Line
 	2250 4500 1600 4500
@@
 	1600 4750 1750 4750
 Text HLabel 2250 4500 2    50   Input ~ 0
-HOTEND_TEMP2
-$Comp
-L taobao-r:R472,0603 R34
+HOTEND_TEMP1
+$Comp
+L taobao-r:R472,0603 R38
 U 1 1 5CC416F3
 P 3500 1300
-F 0 "R34" H 3559 1346 50  0000 L CNN
+F 0 "R38" H 3559 1346 50  0000 L CNN
 F 1 "R472,0603" H 3559 1255 50  0000 L CNN
 F 2 "Resistor_SMD:R_0603_1608Metric_Pad1.05x0.95mm_HandSolder" H 3500 1300 50  0001 C CNN
@@
 $EndComp
 $Comp
-L power:GND #PWR0281
+L power:GND #PWR093
 U 1 1 5CC416FF
 P 3500 2100
-F 0 "#PWR0281" H 3500 1850 50  0001 C CNN
+F 0 "#PWR093" H 3500 1850 50  0001 C CNN
 F 1 "GND" H 3505 1927 50  0000 C CNN
 F 2 "" H 3500 2100 50  0001 C CNN
@@
 	3500 1550 3500 1650
 $Comp
-L Connector:Screw_Terminal_01x02 J33
+L Connector:Screw_Terminal_01x02 J24
 U 1 1 5CC4170A
 P 4500 1550
-F 0 "J33" H 4600 1550 50  0000 L CNN
-F 1 "Screw_Terminal_01x02" H 4600 1450 50  0000 L CNN
+F 0 "J24" H 4600 1550 50  0000 L CNN
+F 1 "AUX_TEMP" H 4600 1450 50  0000 L CNN
 F 2 "w_conn_jst-ph:b2b-ph-kl" H 4500 1550 50  0001 C CNN
 F 3 "~" H 4500 1550 50  0001 C CNN
@@
 	3500 1550 4150 1550
 $Comp
-L power:GND #PWR0282
+L power:GND #PWR096
 U 1 1 5CC41711
 P 4200 2100
-F 0 "#PWR0282" H 4200 1850 50  0001 C CNN
+F 0 "#PWR096" H 4200 1850 50  0001 C CNN
 F 1 "GND" H 4205 1927 50  0000 C CNN
 F 2 "" H 4200 2100 50  0001 C CNN
@@
 AUX_TEMP
 $Comp
-L taobao-components:+3V3_STM32 #PWR035
+L taobao-components:+3V3_STM32 #PWR083
 U 1 1 5CC462ED
 P 950 1000
-F 0 "#PWR035" H 950 850 50  0001 C CNN
+F 0 "#PWR083" H 950 850 50  0001 C CNN
 F 1 "+3V3_STM32" H 965 1173 50  0000 C CNN
 F 2 "" H 950 1000 50  0001 C CNN
@@
 $EndComp
 $Comp
-L taobao-components:+3V3_STM32 #PWR036
+L taobao-components:+3V3_STM32 #PWR092
 U 1 1 5CC46405
 P 3500 1000
-F 0 "#PWR036" H 3500 850 50  0001 C CNN
+F 0 "#PWR092" H 3500 850 50  0001 C CNN
 F 1 "+3V3_STM32" H 3515 1173 50  0000 C CNN
 F 2 "" H 3500 1000 50  0001 C CNN
@@
 $EndComp
 $Comp
-L taobao-components:+3V3_STM32 #PWR037
+L taobao-components:+3V3_STM32 #PWR085
 U 1 1 5CC4653D
 P 950 2550
-F 0 "#PWR037" H 950 2400 50  0001 C CNN
+F 0 "#PWR085" H 950 2400 50  0001 C CNN
 F 1 "+3V3_STM32" H 965 2723 50  0000 C CNN
 F 2 "" H 950 2550 50  0001 C CNN
@@
 $EndComp
 $Comp
-L taobao-components:+3V3_STM32 #PWR039
+L taobao-components:+3V3_STM32 #PWR087
 U 1 1 5CC465DE
 P 950 4200
-F 0 "#PWR039" H 950 4050 50  0001 C CNN
+F 0 "#PWR087" H 950 4050 50  0001 C CNN
 F 1 "+3V3_STM32" H 965 4373 50  0000 C CNN
 F 2 "" H 950 4200 50  0001 C CNN
@@
 $EndComp
 $Comp
-L taobao-components:+3V3_STM32 #PWR038
+L taobao-components:+3V3_STM32 #PWR094
 U 1 1 5CE5E7CF
 P 3500 2900
-F 0 "#PWR038" H 3500 2750 50  0001 C CNN
+F 0 "#PWR094" H 3500 2750 50  0001 C CNN
 F 1 "+3V3_STM32" H 3515 3073 50  0000 C CNN
 F 2 "" H 3500 2900 50  0001 C CNN
@@
 	4350 4000 4350 3850
 $Comp
-L power:GND #PWR0279
+L power:GND #PWR097
 U 1 1 5CC40F15
 P 4350 4000
-F 0 "#PWR0279" H 4350 3750 50  0001 C CNN
+F 0 "#PWR097" H 4350 3750 50  0001 C CNN
 F 1 "GND" H 4355 3827 50  0000 C CNN
 F 2 "" H 4350 4000 50  0001 C CNN
@@
 	3500 2900 3500 3100
 $Comp
-L power:GND #PWR0278
+L power:GND #PWR095
 U 1 1 5CC40F03
 P 3500 4000
-F 0 "#PWR0278" H 3500 3750 50  0001 C CNN
+F 0 "#PWR095" H 3500 3750 50  0001 C CNN
 F 1 "GND" H 3505 3827 50  0000 C CNN
 F 2 "" H 3500 4000 50  0001 C CNN
@@
 $EndComp
 $Comp
-L taobao-r:R472,0603 R58
+L taobao-r:R472,0603 R39
 U 1 1 5CC40EF7
 P 3500 3200
-F 0 "R58" H 3559 3246 50  0000 L CNN
+F 0 "R39" H 3559 3246 50  0000 L CNN
 F 1 "R472,0603" H 3559 3155 50  0000 L CNN
 F 2 "Resistor_SMD:R_0603_1608Metric_Pad1.05x0.95mm_HandSolder" H 3500 3200 50  0001 C CNN
@@
 	4150 3450 4350 3450
 $Comp
-L taobao-c:C106,0603 C31
+L taobao-c:C106,0603 C15
 U 1 1 5CCAA148
 P 950 3300
-F 0 "C31" H 1042 3346 50  0000 L CNN
+F 0 "C15" H 1042 3346 50  0000 L CNN
 F 1 "C106,0603" H 1042 3255 50  0000 L CNN
 F 2 "Capacitor_SMD:C_0603_1608Metric_Pad1.05x0.95mm_HandSolder" H 950 3300 50  0001 C CNN
@@
 $EndComp
 $Comp
-L taobao-c:C106,0603 C29
+L taobao-c:C106,0603 C14
 U 1 1 5CCAA34C
 P 950 1750
-F 0 "C29" H 1042 1796 50  0000 L CNN
+F 0 "C14" H 1042 1796 50  0000 L CNN
 F 1 "C106,0603" H 1042 1705 50  0000 L CNN
 F 2 "Capacitor_SMD:C_0603_1608Metric_Pad1.05x0.95mm_HandSolder" H 950 1750 50  0001 C CNN
@@
 $EndComp
 $Comp
-L taobao-c:C106,0603 C35
+L taobao-c:C106,0603 C17
 U 1 1 5CCAA3BA
 P 3500 1750
-F 0 "C35" H 3592 1796 50  0000 L CNN
+F 0 "C17" H 3592 1796 50  0000 L CNN
 F 1 "C106,0603" H 3592 1705 50  0000 L CNN
 F 2 "Capacitor_SMD:C_0603_1608Metric_Pad1.05x0.95mm_HandSolder" H 3500 1750 50  0001 C CNN
@@
 $EndComp
 $Comp
-L taobao-c:C106,0603 C36
+L taobao-c:C106,0603 C18
 U 1 1 5CCAA42C
 P 3500 3650
-F 0 "C36" H 3592 3696 50  0000 L CNN
+F 0 "C18" H 3592 3696 50  0000 L CNN
 F 1 "C106,0603" H 3592 3605 50  0000 L CNN
 F 2 "Capacitor_SMD:C_0603_1608Metric_Pad1.05x0.95mm_HandSolder" H 3500 3650 50  0001 C CNN
@@
 $EndComp
 $Comp
-L taobao-c:C106,0603 C30
+L taobao-c:C106,0603 C16
 U 1 1 5CCAA49C
 P 950 4950
-F 0 "C30" H 1042 4996 50  0000 L CNN
+F 0 "C16" H 1042 4996 50  0000 L CNN
 F 1 "C106,0603" H 1042 4905 50  0000 L CNN
 F 2 "Capacitor_SMD:C_0603_1608Metric_Pad1.05x0.95mm_HandSolder" H 950 4950 50  0001 C CNN

Commit message: update,
Parts:
- added J47: TEMP_DEBUG, Connector_PinHeader_1.27mm:PinHeader_1x05_P1.27mm_Vertical, symbol Connector_Generic:Conn_01x05
Connections:
- net AUX_TEMP: now also J47.5 (Pin_5)
- net HEATBED_TEMP: now also J47.2 (Pin_2)
- net HOTEND_TEMP0: now also J47.3 (Pin_3)
- net HOTEND_TEMP1: now also J47.4 (Pin_4)
- net PCB_TEMP: now also J47.1 (Pin_1)
Changed lines of the file:
@@
 	1    0    0    -1
 $EndComp
+$Comp
+L Connector_Generic:Conn_01x05 J47
+U 1 1 5CD2F161
+P 6450 2800
+F 0 "J47" H 6350 3250 50  0000 C CNN
+F 1 "TEMP_DEBUG" H 6350 3150 50  0000 C CNN
+F 2 "Connector_PinHeader_1.27mm:PinHeader_1x05_P1.27mm_Vertical" H 6450 2800 50  0001 C CNN
+F 3 "~" H 6450 2800 50  0001 C CNN
+	1    6450 2800
+	-1   0    0    -1
+$EndComp
+Text Label 7400 2700 2    50   ~ 0
+HEATBED_TEMP
+Text Label 7400 2800 2    50   ~ 0
+HOTEND_TEMP0
+Text Label 7400 2900 2    50   ~ 0
+HOTEND_TEMP1
+Text Label 7400 3000 2    50   ~ 0
+AUX_TEMP
+Wire Wire Line
+	6650 2700 7400 2700
+Wire Wire Line
+	6650 2800 7400 2800
+Wire Wire Line
+	6650 2900 7400 2900
+Wire Wire Line
+	6650 3000 7400 3000
+Text Label 7400 2600 2    50   ~ 0
+PCB_TEMP
+Wire Wire Line
+	7400 2600 6650 2600
 $EndSCHEMATC

Commit message: update ROUTING,
Parts:
- J21: value HEATBED_TEMP -> HEATBED_T
- J22: value HOTEND_TEMP0 -> HOTEND_T0
- J23: value HOTEND_TEMP1 -> HOTEND_T1
- J24: value AUX_TEMP -> AUX_T
Changed lines of the file:
@@
 P 1950 1550
 F 0 "J21" H 2050 1550 50  0000 L CNN
-F 1 "HEATBED_TEMP" H 2050 1450 50  0000 L CNN
+F 1 "HEATBED_T" H 2050 1450 50  0000 L CNN
 F 2 "w_conn_jst-ph:b2b-ph-kl" H 1950 1550 50  0001 C CNN
 F 3 "~" H 1950 1550 50  0001 C CNN
@@
 P 1950 3100
 F 0 "J22" H 2050 3100 50  0000 L CNN
-F 1 "HOTEND_TEMP0" H 2050 3000 50  0000 L CNN
+F 1 "HOTEND_T0" H 2050 3000 50  0000 L CNN
 F 2 "w_conn_jst-ph:b2b-ph-kl" H 1950 3100 50  0001 C CNN
 F 3 "~" H 1950 3100 50  0001 C CNN
@@
 P 1950 4750
 F 0 "J23" H 2050 4750 50  0000 L CNN
-F 1 "HOTEND_TEMP1" H 2050 4650 50  0000 L CNN
+F 1 "HOTEND_T1" H 2050 4650 50  0000 L CNN
 F 2 "w_conn_jst-ph:b2b-ph-kl" H 1950 4750 50  0001 C CNN
 F 3 "~" H 1950 4750 50  0001 C CNN
@@
 P 4500 1550
 F 0 "J24" H 4600 1550 50  0000 L CNN
-F 1 "AUX_TEMP" H 4600 1450 50  0000 L CNN
+F 1 "AUX_T" H 4600 1450 50  0000 L CNN
 F 2 "w_conn_jst-ph:b2b-ph-kl" H 4500 1550 50  0001 C CNN
 F 3 "~" H 4500 1550 50  0001 C CNN

Commit message: update ROUTING,
Changed lines of the file:
@@
 F 0 "R36" H 1009 2896 50  0000 L CNN
 F 1 "R472,0603" H 1009 2805 50  0000 L CNN
-F 2 "Resistor_SMD:R_0603_1608Metric_Pad1.05x0.95mm_HandSolder" H 950 2850 50  0001 C CNN
+F 2 "Resistor_SMD:R_0603_1608Metric_Pad1.05x0.95mm_HandSolder" H 950 2850 50  0000 C CNN
 F 3 "~" H 950 2850 50  0001 C CNN
 	1    950  2850
