File: hardware/printer-board/END_STOP.sch (KiCad schematic (older format))
At the start: 18 parts, among them J15 X_MIN, J16 X_MAX, J17 Y_MIN, J18 Y_MAX, J19 Z_MIN, J20 Z_MAX

Commit message: update,
Parts:
- added J45: END_SWITCH_DEBUG, Connector_PinHeader_1.27mm:PinHeader_1x06_P1.27mm_Vertical, symbol Connector_Generic:Conn_01x06
Connections:
- net X_MAX: now also J45.2 (Pin_2)
- net X_MIN: now also J45.1 (Pin_1)
- net Y_MAX: now also J45.4 (Pin_4)
- net Y_MIN: now also J45.3 (Pin_3)
- net Z_MAX: now also J45.6 (Pin_6)
- net Z_MIN: now also J45.5 (Pin_5)
Changed lines of the file:
@@
 Wire Wire Line
 	3800 6600 3800 7250
+$Comp
+L Connector_Generic:Conn_01x06 J45
+U 1 1 5CD1988B
+P 6400 5650
+F 0 "J45" H 6500 5650 50  0000 L CNN
+F 1 "END_SWITCH_DEBUG" H 6500 5550 50  0000 L CNN
+F 2 "Connector_PinHeader_1.27mm:PinHeader_1x06_P1.27mm_Vertical" H 6400 5650 50  0001 C CNN
+F 3 "~" H 6400 5650 50  0001 C CNN
+	1    6400 5650
+	1    0    0    -1
+$EndComp
+Text Label 5850 5450 0    50   ~ 0
+X_MIN
+Text Label 5850 5550 0    50   ~ 0
+X_MAX
+Text Label 5850 5650 0    50   ~ 0
+Y_MIN
+Text Label 5850 5750 0    50   ~ 0
+Y_MAX
+Text Label 5850 5850 0    50   ~ 0
+Z_MIN
+Text Label 5850 5950 0    50   ~ 0
+Z_MAX
+Wire Wire Line
+	5850 5450 6200 5450
+Wire Wire Line
+	5850 5550 6200 5550
+Wire Wire Line
+	5850 5650 6200 5650
+Wire Wire Line
+	5850 5750 6200 5750
+Wire Wire Line
+	5850 5850 6200 5850
+Wire Wire Line
+	5850 5950 6200 5950
 $EndSCHEMATC

Commit message: update,
Other:
- note added: "COM ? SENSOR\nNO ? POWER\nNC ? GND"
Changed lines of the file:
@@
 EESchema Schematic File Version 4
-LIBS:printer-board-cache
+LIBS:END_STOP-cache
 EELAYER 29 0
 EELAYER END
 $Descr A4 11693 8268
 encoding utf-8
-Sheet 10 28
+Sheet 1 1
 Title ""
 Date ""
@@
 Wire Wire Line
 	5850 5950 6200 5950
+Text Notes 2550 2100 0    50   ~ 0
+COM ? SENSOR\nNO ? POWER\nNC ? GND
 $EndSCHEMATC

Commit message: update,
Parts:
- D9: value LED_BLUE,0603 -> XMIN
Changed lines of the file:
@@
 P 4250 2100
 F 0 "D9" V 4296 2032 50  0000 R CNN
-F 1 "LED_BLUE,0603" V 4205 2032 50  0000 R CNN
+F 1 "XMIN" V 4205 2032 50  0000 R CNN
 F 2 "LED_SMD:LED_0603_1608Metric_Pad1.05x0.95mm_HandSolder" V 4250 2100 50  0001 C CNN
 F 3 "" V 4250 2100 50  0001 C CNN

Commit message: update,
Parts:
- added D15: LED_BLUE,0603, LED_SMD:LED_0603_1608Metric_Pad1.05x0.95mm_HandSolder, symbol taobao-led:LED_BLUE,0603
- added D16, D25, D26: SD_1N5817_SS12, symbol taobao-sd:SD_1N5817_SS12
- added J48: HOTEND_PROBE, footprint-lib:b3b-ph-kl,end_stop, symbol Connector_Generic:Conn_01x03
- added JP1, JP2: SolderJumper_2_Open, symbol Jumper:SolderJumper_2_Open
- added R49: R102,0603, Resistor_SMD:R_0603_1608Metric_Pad1.05x0.95mm_HandSolder, symbol taobao-r:R102,0603
Connections:
- net +3V3_STM32: now also R49.1; no longer J15.2 (Pin_2), J16.2 (Pin_2), J17.2 (Pin_2), J18.2 (Pin_2), J19.2 (Pin_2), J20.2 (Pin_2)
- net GND: now also J48.3 (Pin_3)
- net Z_MAX: now also D26.2 (A); no longer D14.1 (K), J20.1 (Pin_1)
- net Z_MIN: now also D25.2 (A); no longer D13.1 (K), J19.1 (Pin_1)
- new net: J15.2 (Pin_2), J16.2 (Pin_2), J17.2 (Pin_2), J18.2 (Pin_2), J19.2 (Pin_2), J20.2 (Pin_2), JP1.2 (B)
- new net: D13.1 (K), D25.1 (K), J19.1 (Pin_1)
- new net: D14.1 (K), D26.1 (K), J20.1 (Pin_1)
- new net: D15.1 (K), D16.1 (K), J48.1 (Pin_1)
- new net: J48.2 (Pin_2), JP2.2 (B)
- new net: D15.2 (A), R49.2
- new net +12V: JP1.1 (A), JP2.1 (A)
- new net HOTEND_PROBE: D16.2 (A)
Other:
- note added: "assume dry contact here"
- note added: "protection against active sensor"
- moved on the sheet: D10, D11, D12, D13, D14, D9, R29, R30, R31, R32, R33, R34

Commit message: update,
Parts:
- D16, D25, D26: footprint (none) -> w_smd_diode:do214ac
- JP1, JP2: footprint (none) -> Jumper:SolderJumper-2_P1.3mm_Open_RoundedPad1.0x1.5mm
Changed lines of the file:
@@
 F 0 "D16" H 7750 2250 50  0000 C CNN
 F 1 "SD_1N5817_SS12" H 7750 2150 50  0000 C CNN
-F 2 "" V 7750 2000 50  0001 C CNN
+F 2 "w_smd_diode:do214ac" V 7750 2000 50  0001 C CNN
 F 3 "~" V 7750 2000 50  0001 C CNN
 	1    7750 2000
@@
 F 0 "JP1" V 3600 1450 50  0000 L CNN
 F 1 "SolderJumper_2_Open" V 3650 1450 50  0000 L CNN
-F 2 "" H 3650 1350 50  0001 C CNN
+F 2 "Jumper:SolderJumper-2_P1.3mm_Open_RoundedPad1.0x1.5mm" H 3650 1350 50  0001 C CNN
 F 3 "~" H 3650 1350 50  0001 C CNN
 	1    3650 1350
@@
 F 0 "JP2" V 6700 1550 50  0000 L CNN
 F 1 "SolderJumper_2_Open" V 6750 1550 50  0000 L CNN
-F 2 "" H 6750 1450 50  0001 C CNN
+F 2 "Jumper:SolderJumper-2_P1.3mm_Open_RoundedPad1.0x1.5mm" H 6750 1450 50  0001 C CNN
 F 3 "~" H 6750 1450 50  0001 C CNN
 	1    6750 1450
@@
 F 0 "D25" H 4750 5750 50  0000 C CNN
 F 1 "SD_1N5817_SS12" H 4750 5650 50  0000 C CNN
-F 2 "" V 4750 5500 50  0001 C CNN
+F 2 "w_smd_diode:do214ac" V 4750 5500 50  0001 C CNN
 F 3 "~" V 4750 5500 50  0001 C CNN
 	1    4750 5500
@@
 F 0 "D26" H 4750 6650 50  0000 C CNN
 F 1 "SD_1N5817_SS12" H 4750 6550 50  0000 C CNN
-F 2 "" V 4750 6400 50  0001 C CNN
+F 2 "w_smd_diode:do214ac" V 4750 6400 50  0001 C CNN
 F 3 "~" V 4750 6400 50  0001 C CNN
 	1    4750 6400
@@
 Wire Wire Line
 	4850 6400 5400 6400
+Text HLabel 1100 1600 0    50   Input ~ 0
+HOTEND_PROBE
+Text Label 1650 1600 2    50   ~ 0
+HOTEND_PROBE
+Wire Wire Line
+	1100 1600 1650 1600
 $EndSCHEMATC

Commit message: update ROUTING,
Parts:
- D10, D12, D14: value LED_BLUE,0603 -> ↑
- D11: value LED_BLUE,0603 -> Y↓
- D13: value LED_BLUE,0603 -> Z↓
- D9: value XMIN -> X↓
Changed lines of the file:
@@
 U 1 1 5CC31819
 P 4250 1450
-F 0 "R29" H 4309 1496 50  0000 L CNN
-F 1 "R102,0603" H 4309 1405 50  0000 L CNN
+F 0 "R29" H 4150 1500 50  0000 R CNN
+F 1 "R102,0603" H 4150 1450 50  0000 R CNN
 F 2 "Resistor_SMD:R_0603_1608Metric_Pad1.05x0.95mm_HandSolder" H 4250 1450 50  0001 C CNN
 F 3 "~" H 4250 1450 50  0001 C CNN
@@
 U 1 1 5CC31941
 P 4250 1700
-F 0 "D9" V 4296 1632 50  0000 R CNN
-F 1 "XMIN" V 4205 1632 50  0000 R CNN
+F 0 "D9" V 4300 1800 50  0000 L CNN
+F 1 "X↓" V 4250 1800 50  0000 L CNN
 F 2 "LED_SMD:LED_0603_1608Metric_Pad1.05x0.95mm_HandSolder" V 4250 1700 50  0001 C CNN
 F 3 "" V 4250 1700 50  0001 C CNN
@@
 U 1 1 5CC33066
 P 4250 2400
-F 0 "R30" H 4309 2446 50  0000 L CNN
-F 1 "R102,0603" H 4309 2355 50  0000 L CNN
+F 0 "R30" H 4150 2450 50  0000 R CNN
+F 1 "R102,0603" H 4150 2400 50  0000 R CNN
 F 2 "Resistor_SMD:R_0603_1608Metric_Pad1.05x0.95mm_HandSolder" H 4250 2400 50  0001 C CNN
 F 3 "~" H 4250 2400 50  0001 C CNN
@@
 U 1 1 5CC3306C
 P 4250 2650
-F 0 "D10" V 4296 2582 50  0000 R CNN
-F 1 "LED_BLUE,0603" V 4205 2582 50  0000 R CNN
+F 0 "D10" V 4300 2750 50  0000 L CNN
+F 1 "↑" V 4250 2750 50  0000 L CNN
 F 2 "LED_SMD:LED_0603_1608Metric_Pad1.05x0.95mm_HandSolder" V 4250 2650 50  0001 C CNN
 F 3 "" V 4250 2650 50  0001 C CNN
@@
 U 1 1 5CC3434E
 P 4250 3250
-F 0 "R31" H 4309 3296 50  0000 L CNN
-F 1 "R102,0603" H 4309 3205 50  0000 L CNN
+F 0 "R31" H 4150 3300 50  0000 R CNN
+F 1 "R102,0603" H 4150 3250 50  0000 R CNN
 F 2 "Resistor_SMD:R_0603_1608Metric_Pad1.05x0.95mm_HandSolder" H 4250 3250 50  0001 C CNN
 F 3 "~" H 4250 3250 50  0001 C CNN
@@
 U 1 1 5CC34354
 P 4250 3500
-F 0 "D11" V 4296 3432 50  0000 R CNN
-F 1 "LED_BLUE,0603" V 4205 3432 50  0000 R CNN
+F 0 "D11" V 4300 3600 50  0000 L CNN
+F 1 "Y↓" V 4250 3600 50  0000 L CNN
 F 2 "LED_SMD:LED_0603_1608Metric_Pad1.05x0.95mm_HandSolder" V 4250 3500 50  0001 C CNN
 F 3 "" V 4250 3500 50  0001 C CNN
@@
 U 1 1 5CC34FAC
 P 4250 4150
-F 0 "R32" H 4309 4196 50  0000 L CNN
-F 1 "R102,0603" H 4309 4105 50  0000 L CNN
+F 0 "R32" H 4150 4200 50  0000 R CNN
+F 1 "R102,0603" H 4150 4150 50  0000 R CNN
 F 2 "Resistor_SMD:R_0603_1608Metric_Pad1.05x0.95mm_HandSolder" H 4250 4150 50  0001 C CNN
 F 3 "~" H 4250 4150 50  0001 C CNN
@@
 U 1 1 5CC34FB2
 P 4250 4400
-F 0 "D12" V 4296 4332 50  0000 R CNN
-F 1 "LED_BLUE,0603" V 4205 4332 50  0000 R CNN
+F 0 "D12" V 4300 4500 50  0000 L CNN
+F 1 "↑" V 4250 4500 50  0000 L CNN
 F 2 "LED_SMD:LED_0603_1608Metric_Pad1.05x0.95mm_HandSolder" V 4250 4400 50  0001 C CNN
 F 3 "" V 4250 4400 50  0001 C CNN
@@
 U 1 1 5CC35E90
 P 4250 5000
-F 0 "R33" H 4309 5046 50  0000 L CNN
-F 1 "R102,0603" H 4309 4955 50  0000 L CNN
+F 0 "R33" H 4150 5050 50  0000 R CNN
+F 1 "R102,0603" H 4150 5000 50  0000 R CNN
 F 2 "Resistor_SMD:R_0603_1608Metric_Pad1.05x0.95mm_HandSolder" H 4250 5000 50  0001 C CNN
 F 3 "~" H 4250 5000 50  0001 C CNN
@@
 U 1 1 5CC35E96
 P 4250 5250
-F 0 "D13" V 4296 5182 50  0000 R CNN
-F 1 "LED_BLUE,0603" V 4205 5182 50  0000 R CNN
+F 0 "D13" V 4300 5350 50  0000 L CNN
+F 1 "Z↓" V 4250 5350 50  0000 L CNN
 F 2 "LED_SMD:LED_0603_1608Metric_Pad1.05x0.95mm_HandSolder" V 4250 5250 50  0001 C CNN
 F 3 "" V 4250 5250 50  0001 C CNN
@@
 U 1 1 5CC36FE8
 P 4250 5900
-F 0 "R34" H 4309 5946 50  0000 L CNN
-F 1 "R102,0603" H 4309 5855 50  0000 L CNN
+F 0 "R34" H 4150 5950 50  0000 R CNN
+F 1 "R102,0603" H 4150 5900 50  0000 R CNN
 F 2 "Resistor_SMD:R_0603_1608Metric_Pad1.05x0.95mm_HandSolder" H 4250 5900 50  0001 C CNN
 F 3 "~" H 4250 5900 50  0001 C CNN
@@
 U 1 1 5CC36FEE
 P 4250 6150
-F 0 "D14" V 4296 6082 50  0000 R CNN
-F 1 "LED_BLUE,0603" V 4205 6082 50  0000 R CNN
+F 0 "D14" V 4300 6050 50  0000 R CNN
+F 1 "↑" V 4250 6050 50  0000 R CNN
 F 2 "LED_SMD:LED_0603_1608Metric_Pad1.05x0.95mm_HandSolder" V 4250 6150 50  0001 C CNN
 F 3 "" V 4250 6150 50  0001 C CNN
@@
 U 1 1 5CD6EA2D
 P 3650 1350
-F 0 "JP1" V 3600 1450 50  0000 L CNN
-F 1 "SolderJumper_2_Open" V 3650 1450 50  0000 L CNN
+F 0 "JP1" V 3600 1250 50  0000 R CNN
+F 1 "SolderJumper_2_Open" V 3650 1250 50  0000 R CNN
 F 2 "Jumper:SolderJumper-2_P1.3mm_Open_RoundedPad1.0x1.5mm" H 3650 1350 50  0001 C CNN
 F 3 "~" H 3650 1350 50  0001 C CNN
@@
 Wire Wire Line
 	6750 1250 6750 1300
-Text Notes 2450 1300 0    50   ~ 0
+Text Notes 2450 1150 0    50   ~ 0
 assume dry contact here
 Wire Notes Line
@@
 U 1 1 5CD8DF8F
 P 4750 5500
-F 0 "D25" H 4750 5750 50  0000 C CNN
-F 1 "SD_1N5817_SS12" H 4750 5650 50  0000 C CNN
+F 0 "D25" H 4750 5350 50  0000 C CNN
+F 1 "SD_1N5817_SS12" H 4750 5250 50  0000 C CNN
 F 2 "w_smd_diode:do214ac" V 4750 5500 50  0001 C CNN
 F 3 "~" V 4750 5500 50  0001 C CNN

Commit message: update ROUTING,
Changed lines of the file:
@@
 F 0 "D10" V 4300 2750 50  0000 L CNN
 F 1 "↑" V 4250 2750 50  0000 L CNN
-F 2 "LED_SMD:LED_0603_1608Metric_Pad1.05x0.95mm_HandSolder" V 4250 2650 50  0001 C CNN
+F 2 "LED_SMD:LED_0603_1608Metric_Pad1.05x0.95mm_HandSolder" V 4250 2650 50  0000 C CNN
 F 3 "" V 4250 2650 50  0001 C CNN
 	1    4250 2650

Commit message: update,
Parts:
- added JP3, JP4: SolderJumper_2_Open, Jumper:SolderJumper-2_P1.3mm_Open_RoundedPad1.0x1.5mm, symbol Jumper:SolderJumper_2_Open
Connections:
- net +12V: now also JP3.1 (A), JP4.1 (A)
- new net: J15.2 (Pin_2), J16.2 (Pin_2), JP1.2 (B)
- new net: J17.2 (Pin_2), J18.2 (Pin_2), JP3.2 (B)
- new net: J19.2 (Pin_2), J20.2 (Pin_2), JP4.2 (B)
Changed lines of the file:
@@
 Wire Wire Line
 	4250 5350 4250 5500
-Wire Wire Line
-	4250 5500 3450 5500
 $Comp
 L taobao-r:R102,0603 R34
@@
 Wire Wire Line
 	3450 2900 3650 2900
-Connection ~ 3650 2900
 Wire Wire Line
 	3450 3000 3800 3000
@@
 Wire Wire Line
 	3450 3850 3650 3850
-Connection ~ 3650 3850
 Wire Wire Line
 	3450 3950 3800 3950
@@
 Wire Wire Line
 	3450 4750 3650 4750
-Connection ~ 3650 4750
 Wire Wire Line
 	3450 4850 3800 4850
@@
 Wire Wire Line
 	3450 5600 3650 5600
-Connection ~ 3650 5600
 Wire Wire Line
 	3450 5700 3800 5700
@@
 	4250 2800 4650 2800
 Wire Wire Line
-	3650 2900 3650 3850
-Wire Wire Line
 	3650 3850 3650 4750
-Wire Wire Line
-	3650 4750 3650 5600
 Wire Wire Line
 	3650 5600 3650 6500
@@
 Wire Wire Line
 	1100 1600 1650 1600
+$Comp
+L power:+12V #PWR0195
+U 1 1 5CD07A9A
+P 3250 3450
+F 0 "#PWR0195" H 3250 3300 50  0001 C CNN
+F 1 "+12V" H 3300 3650 50  0000 C CNN
+F 2 "" H 3250 3450 50  0001 C CNN
+F 3 "" H 3250 3450 50  0001 C CNN
+	1    3250 3450
+	0    -1   -1   0
+$EndComp
+$Comp
+L Jumper:SolderJumper_2_Open JP3
+U 1 1 5CD07AA4
+P 3450 3450
+F 0 "JP3" V 3400 3350 50  0000 R CNN
+F 1 "SolderJumper_2_Open" V 3450 3350 50  0000 R CNN
+F 2 "Jumper:SolderJumper-2_P1.3mm_Open_RoundedPad1.0x1.5mm" H 3450 3450 50  0001 C CNN
+F 3 "~" H 3450 3450 50  0001 C CNN
+	1    3450 3450
+	1    0    0    -1
+$EndComp
+Wire Wire Line
+	3250 3450 3300 3450
+Text Notes 1400 3050 0    50   ~ 0
+assume dry contact here
+Connection ~ 3650 3850
+Wire Wire Line
+	4250 5500 3450 5500
+Wire Wire Line
+	3550 5150 3650 5150
+Wire Wire Line
+	3200 5150 3250 5150
+$Comp
+L Jumper:SolderJumper_2_Open JP4
+U 1 1 5CD18A57
+P 3400 5150
+F 0 "JP4" V 3350 5050 50  0000 R CNN
+F 1 "SolderJumper_2_Open" V 3400 5050 50  0000 R CNN
+F 2 "Jumper:SolderJumper-2_P1.3mm_Open_RoundedPad1.0x1.5mm" H 3400 5150 50  0001 C CNN
+F 3 "~" H 3400 5150 50  0001 C CNN
+	1    3400 5150
+	1    0    0    -1
+$EndComp
+$Comp
+L power:+12V #PWR0196
+U 1 1 5CD18A4D
+P 3200 5150
+F 0 "#PWR0196" H 3200 5000 50  0001 C CNN
+F 1 "+12V" H 3250 5350 50  0000 C CNN
+F 2 "" H 3200 5150 50  0001 C CNN
+F 3 "" H 3200 5150 50  0001 C CNN
+	1    3200 5150
+	0    -1   -1   0
+$EndComp
+Wire Wire Line
+	3650 5150 3650 5600
+Connection ~ 3650 5600
+Wire Wire Line
+	3600 3450 3650 3450
+Wire Wire Line
+	3650 3450 3650 3850
 $EndSCHEMATC
