File: hardware/printer-board/MP1584_3V3.sch (KiCad schematic (older format))
At the start: 15 parts, among them J49 Conn_01x03_Female, U13 MP1584

Commit message: update footprint,
Parts:
- U13: footprint footprint-lib:MP2303,SOIC-8_3.9x4.9mm_P1.27mm,thermal_via -> footprint-lib:MP1584,SOIC-8_3.9x4.9mm_P1.27mm,thermal_via
Changed lines of the file:
@@
 $Descr A4 11693 8268
 encoding utf-8
-Sheet 29 30
+Sheet 27 28
 Title ""
 Date ""
@@
 F 0 "U13" H 5800 4050 50  0000 C CNN
 F 1 "MP1584" H 5800 3950 50  0000 C CNN
-F 2 "footprint-lib:MP2303,SOIC-8_3.9x4.9mm_P1.27mm,thermal_via" H 5800 2500 50  0001 C CNN
+F 2 "footprint-lib:MP1584,SOIC-8_3.9x4.9mm_P1.27mm,thermal_via" H 5800 2500 50  0001 C CNN
 F 3 "" H 5800 3350 50  0001 C CNN
 	1    5800 3350

Commit message: update footprint,
Parts:
- L4: footprint footprint-lib:L_SMD_ALL -> w_smd_inductors:inductor_smd_6.8x3.8mm
Changed lines of the file:
@@
 F 0 "L4" V 7750 3200 50  0000 C CNN
 F 1 "L_15uH" V 7650 3200 50  0000 C CNN
-F 2 "footprint-lib:L_SMD_ALL" H 7550 3200 50  0001 C CNN
+F 2 "w_smd_inductors:inductor_smd_6.8x3.8mm" H 7550 3200 50  0001 C CNN
 F 3 "test_datasheet" H 7550 3200 50  0001 C CNN
 	1    7550 3200

Commit message: update,
Connections:
- net +12V: now reaches C35.1, J49.2 (Pin_2), R80.1, U13.7 (VIN)
Changed lines of the file:
@@
 	3150 3200 3150 3400
 Wire Wire Line
-	3150 3200 3750 3200
+	3150 3200 3400 3200
 Connection ~ 3150 3200
 Wire Wire Line
@@
 	1    0    0    -1
 $EndComp
+$Comp
+L power:+12V #PWR0203
+U 1 1 5CE69FC8
+P 3400 2950
+F 0 "#PWR0203" H 3400 2800 50  0001 C CNN
+F 1 "+12V" H 3450 3150 50  0000 C CNN
+F 2 "" H 3400 2950 50  0001 C CNN
+F 3 "" H 3400 2950 50  0001 C CNN
+	1    3400 2950
+	1    0    0    -1
+$EndComp
+Wire Wire Line
+	3400 2950 3400 3200
+Connection ~ 3400 3200
+Wire Wire Line
+	3400 3200 3750 3200
 $EndSCHEMATC
